File: Kicad/front-gp2y/gp2y.kicad_pcb (KiCad board)
At the start: 2 copper layers, 48 x 35 mm, 14 parts, among them IC1 MCP1755-50, K1 GP2Y, K2 MCU

Commit message: Update GP2Y
Connections:
- K2 pad 1: VIN -> GND
- K2 pad 2: GP2Y_OUT -> MCU_ENABLE
- K2 pad 3: MCU_ENABLE -> GP2Y_OUT
- K2 pad 4: GND -> VIN
Routing:
- net VIN: track 15.6 -> 10.2 mm
- net GP2Y_OUT: track 19.5 -> 17.5 mm
- net MCU_ENABLE: track 13.4 -> 14.3 mm
Changed lines of the file:
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@@
       ) (layer "B.Fab") (width 0.1) (fill solid))
     (pad "1" thru_hole oval locked (at 0 0 180) (size 1.2 1.75) (drill 0.8) (layers *.Cu *.Mask)
-      (net 3 "VIN") (pinfunction "1") (pintype "passive"))
+      (net 1 "GND") (pinfunction "1") (pintype "passive"))
     (pad "2" thru_hole oval locked (at 2 0 180) (size 1.2 1.75) (drill 0.8) (layers *.Cu *.Mask)
-      (net 7 "GP2Y_OUT") (pinfunction "2") (pintype "passive"))
+      (net 5 "MCU_ENABLE") (pinfunction "2") (pintype "passive"))
     (pad "3" thru_hole oval locked (at 4 0 180) (size 1.2 1.75) (drill 0.8) (layers *.Cu *.Mask)
-      (net 5 "MCU_ENABLE") (pinfunction "3") (pintype "passive"))
+      (net 7 "GP2Y_OUT") (pinfunction "3") (pintype "passive"))
     (pad "4" thru_hole oval locked (at 6 0 180) (size 1.2 1.75) (drill 0.8) (layers *.Cu *.Mask)
-      (net 1 "GND") (pinfunction "4") (pintype "passive"))
+      (net 3 "VIN") (pinfunction "4") (pintype "passive"))
     (model "${KICAD6_USER_3DMODEL_DIR}/Connector/MOLEX-532540470.step"
       (offset (xyz 3 2.35 2.1))
@@
     (effects (font (size 1.3 1.3) (thickness 0.2)) (justify mirror))
   )
-  (gr_text "GND" (at 126 69.5 90) (layer "F.SilkS")
+  (gr_text "VIN" (at 126 69.5 90) (layer "F.SilkS")
     (effects (font (size 0.8 0.8) (thickness 0.1)) (justify left))
   )
@@
     (effects (font (size 0.8 0.8) (thickness 0.1)) (justify left))
   )
-  (gr_text "GP2Y" (at 130 69.5 90) (layer "F.SilkS")
+  (gr_text "EN" (at 130 69.5 90) (layer "F.SilkS")
     (effects (font (size 0.8 0.8) (thickness 0.1)) (justify left))
   )
@@
     (effects (font (size 1.3 1.3) (thickness 0.2)))
   )
-  (gr_text "EN" (at 128 69.5 90) (layer "F.SilkS")
+  (gr_text "GP2Y" (at 128 69.5 90) (layer "F.SilkS")
     (effects (font (size 0.8 0.8) (thickness 0.1)) (justify left))
   )
@@
     (effects (font (size 1.3 1.3) (thickness 0.2)))
   )
-  (gr_text "VIN" (at 132 69.5 90) (layer "F.SilkS")
+  (gr_text "GND" (at 132 69.5 90) (layer "F.SilkS")
     (effects (font (size 0.8 0.8) (thickness 0.1)) (justify left))
   )
@@
   (segment (start 120.5 79.5) (end 121 79) (width 0.5) (layer "B.Cu") (net 2))
   (segment (start 121 79) (end 130 79) (width 0.5) (layer "B.Cu") (net 2))
-  (segment (start 132 72.5) (end 132 71) (width 0.8) (layer "B.Cu") (net 3))
-  (segment (start 131 73.5) (end 132 72.5) (width 0.8) (layer "B.Cu") (net 3))
+  (segment (start 126 71) (end 126 73.5) (width 0.8) (layer "B.Cu") (net 3))
   (segment (start 125 77.5) (end 123.5 77.5) (width 0.5) (layer "B.Cu") (net 3))
   (segment (start 125.2 77.7) (end 125 77.5) (width 0.5) (layer "B.Cu") (net 3))
   (segment (start 123.5 76) (end 126 73.5) (width 0.8) (layer "B.Cu") (net 3))
-  (segment (start 126 73.5) (end 131 73.5) (width 0.8) (layer "B.Cu") (net 3))
   (segment (start 126.05 77.7) (end 125.2 77.7) (width 0.5) (layer "B.Cu") (net 3))
   (segment (start 123.5 77.5) (end 123.5 76) (width 0.8) (layer "B.Cu") (net 3))
   (segment (start 114.5 77.5) (end 117.5 77.5) (width 0.5) (layer "B.Cu") (net 4))
-  (segment (start 128 71) (end 128 76) (width 0.5) (layer "F.Cu") (net 5))
-  (via (at 128 76) (size 0.8) (drill 0.4) (layers "F.Cu" "B.Cu") (net 5))
+  (segment (start 130 73.95) (end 130 71) (width 0.5) (layer "F.Cu") (net 5))
+  (segment (start 127.95 76) (end 130 73.95) (width 0.5) (layer "F.Cu") (net 5))
+  (via (at 127.95 76) (size 0.8) (drill 0.4) (layers "F.Cu" "B.Cu") (net 5))
   (segment (start 133 76) (end 133.5 76.5) (width 0.5) (layer "B.Cu") (net 5))
   (segment (start 127.95 77.7) (end 127.95 76.05) (width 0.5) (layer "B.Cu") (net 5))
   (segment (start 127.95 76.05) (end 128 76) (width 0.5) (layer "B.Cu") (net 5))
-  (segment (start 128 76) (end 133 76) (width 0.5) (layer "B.Cu") (net 5))
+  (segment (start 133 76) (end 127.95 76) (width 0.5) (layer "B.Cu") (net 5))
   (segment (start 133.5 76.5) (end 133.5 77.5) (width 0.5) (layer "B.Cu") (net 5))
-  (segment (start 130 70) (end 130 71) (width 0.5) (layer "B.Cu") (net 7))
+  (segment (start 128 70) (end 128 71) (width 0.5) (layer "B.Cu") (net 7))
+  (segment (start 120 71) (end 120 70) (width 0.5) (layer "B.Cu") (net 7))
   (segment (start 120 70) (end 121 69) (width 0.5) (layer "B.Cu") (net 7))
-  (segment (start 121 69) (end 129 69) (width 0.5) (layer "B.Cu") (net 7))
-  (segment (start 129 69) (end 130 70) (width 0.5) (layer "B.Cu") (net 7))
   (segment (start 120.5 77.5) (end 120.5 76.5) (width 0.5) (layer "B.Cu") (net 7))
-  (segment (start 120 71) (end 120 70) (width 0.5) (layer "B.Cu") (net 7))
+  (segment (start 121 69) (end 127 69) (width 0.5) (layer "B.Cu") (net 7))
   (segment (start 120 76) (end 120 71) (width 0.5) (layer "B.Cu") (net 7))
   (segment (start 120.5 76.5) (end 120 76) (width 0.5) (layer "B.Cu") (net 7))
+  (segment (start 127 69) (end 128 70) (width 0.5) (layer "B.Cu") (net 7))
   (zone (net 1) (net_name "GND") (layers F&B.Cu) (hatch edge 0.508)
     (connect_pads (clearance 0.508))
