File: Kicad/front-gp2y/gp2y.kicad_pcb (KiCad board)
At the start: 2 copper layers, 48 x 35 mm, 14 parts, among them IC1 MCP1755-50, K1 GP2Y, K2 MCU

Commit message: Update GP2Y
Routing:
- net GP2Y_OUT: track 17.5 -> 18.1 mm
Changed lines of the file:
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@@
       (net 2 "+5V") (pintype "passive") (zone_connect 2))
     (pad "2" smd roundrect (at 1.5 0 270) (size 1.3 1.75) (layers "B.Cu" "B.Paste" "B.Mask") (roundrect_rratio 0.15)
-      (net 1 "GND") (pintype "passive") (zone_connect 2))
+      (net 1 "GND") (pintype "passive") (zone_connect 1))
     (model "${KICAD6_USER_3DMODEL_DIR}/SMD/CAPACITOR-1206.wrl"
       (offset (xyz 0 0 0))
@@
     (fp_rect (start -1.2 -0.8) (end 1.2 0.8) (layer "B.Fab") (width 0.1) (fill none))
     (pad "1" smd roundrect (at -1.5 0 90) (size 1.3 1.75) (layers "B.Cu" "B.Paste" "B.Mask") (roundrect_rratio 0.15)
-      (net 1 "GND") (pinfunction "K") (pintype "passive") (zone_connect 2))
+      (net 1 "GND") (pinfunction "K") (pintype "passive") (zone_connect 1))
     (pad "2" smd roundrect (at 1.5 0 90) (size 1.3 1.75) (layers "B.Cu" "B.Paste" "B.Mask") (roundrect_rratio 0.15)
       (net 4 "Net-(LED1-Pad2)") (pinfunction "A") (pintype "passive") (zone_connect 2))
@@
       (net 3 "VIN") (pintype "passive") (zone_connect 2))
     (pad "2" smd roundrect (at 1.5 0 270) (size 1.3 1.75) (layers "B.Cu" "B.Paste" "B.Mask") (roundrect_rratio 0.15)
-      (net 1 "GND") (pintype "passive") (zone_connect 2))
+      (net 1 "GND") (pintype "passive") (zone_connect 1))
     (model "${KICAD6_USER_3DMODEL_DIR}/SMD/CAPACITOR-1206.wrl"
       (offset (xyz 0 0 0))
@@
       (net 5 "MCU_ENABLE") (pintype "passive") (zone_connect 2))
     (pad "2" smd roundrect (at 1.5 0 270) (size 1.3 1.75) (layers "B.Cu" "B.Paste" "B.Mask") (roundrect_rratio 0.15)
-      (net 1 "GND") (pintype "passive") (zone_connect 2))
+      (net 1 "GND") (pintype "passive") (zone_connect 1))
     (model "${KICAD6_USER_3DMODEL_DIR}/SMD/RESISTOR-1206.wrl"
       (offset (xyz 0 0 0))
@@
   (segment (start 133 76) (end 127.95 76) (width 0.5) (layer "B.Cu") (net 5))
   (segment (start 133.5 76.5) (end 133.5 77.5) (width 0.5) (layer "B.Cu") (net 5))
-  (segment (start 128 70) (end 128 71) (width 0.5) (layer "B.Cu") (net 7))
-  (segment (start 120 71) (end 120 70) (width 0.5) (layer "B.Cu") (net 7))
-  (segment (start 120 70) (end 121 69) (width 0.5) (layer "B.Cu") (net 7))
+  (segment (start 128 69.5) (end 128 71) (width 0.5) (layer "B.Cu") (net 7))
+  (segment (start 120.5 69) (end 127.5 69) (width 0.5) (layer "B.Cu") (net 7))
+  (segment (start 127.5 69) (end 128 69.5) (width 0.5) (layer "B.Cu") (net 7))
+  (segment (start 120 71) (end 120 69.5) (width 0.5) (layer "B.Cu") (net 7))
   (segment (start 120.5 77.5) (end 120.5 76.5) (width 0.5) (layer "B.Cu") (net 7))
-  (segment (start 121 69) (end 127 69) (width 0.5) (layer "B.Cu") (net 7))
+  (segment (start 120 69.5) (end 120.5 69) (width 0.5) (layer "B.Cu") (net 7))
   (segment (start 120 76) (end 120 71) (width 0.5) (layer "B.Cu") (net 7))
   (segment (start 120.5 76.5) (end 120 76) (width 0.5) (layer "B.Cu") (net 7))
-  (segment (start 127 69) (end 128 70) (width 0.5) (layer "B.Cu") (net 7))
   (zone (net 1) (net_name "GND") (layers F&B.Cu) (hatch edge 0.508)
     (connect_pads (clearance 0.5))

Commit message: Update
Parts:
- added kibuzzard-6277EDE4: G002, kibuzzard-6277EDE4, F.Cu at (118.0, 68.0)
- added kibuzzard-6277EDE4: G004, kibuzzard-6277EDE4, F.Cu at (132.0, 68.0)
- added kibuzzard-6277EE2E: G003, kibuzzard-6277EE2E, F.Cu at (126.0, 68.0)
- added kibuzzard-6277EE50: G001, kibuzzard-6277EE50, F.Cu at (116.0, 68.0)
Other:
- board text removed: "+5V"
- board text removed: "GND"
- board text removed: "VIN"
