File: Kicad/front-gp2y/gp2y.kicad_sch (KiCad schematic)
At the start: 12 parts, among them IC1 MCP1755-50, K1 GP2Y, K2 MCU

Commit message: Update GP2Y
Parts:
- IR1: footprint tronixio:zzzSHARP-GP2Y0A -> tronixio:SHARP-GP2Y0A
Changed lines of the file:
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@@
     )
   )
-  (global_label "MCU_ENABLE" (shape output) (at 213.36 83.82 0)
+  (global_label "MCU_ENABLE" (shape input) (at 213.36 83.82 0)
     (effects (font (size 1.27 1.27)) (justify left))
     (property "Intersheet References" "${INTERSHEET_REFS}" (id 0) (at 222.9214 83.7406 0)
@@
     )
   )
-  (global_label "GP2Y_OUT" (shape input) (at 213.36 81.28 0)
+  (global_label "GP2Y_OUT" (shape output) (at 213.36 81.28 0)
     (effects (font (size 1.27 1.27)) (justify left))
     (property "Intersheet References" "${INTERSHEET_REFS}" (id 0) (at 222.9214 81.2006 0)
@@
       (effects (font (size 1.15 1.15)))
     )
-    (property "Footprint" "tronixio:zzzSHARP-GP2Y0A" (id 2) (at 261.62 180.34 0)
+    (property "Footprint" "tronixio:SHARP-GP2Y0A" (id 2) (at 261.62 180.34 0)
       (effects (font (size 1 1)) hide)
     )
@@
     )
     (path "/61de8734-825b-4a6f-8a19-c68b9be180d1"
-      (reference "IR1") (unit 1) (value "SHARP-GP2Y0xx1") (footprint "tronixio:zzzSHARP-GP2Y0A")
+      (reference "IR1") (unit 1) (value "SHARP-GP2Y0xx1") (footprint "tronixio:SHARP-GP2Y0A")
     )
     (path "/ed89b481-faca-420e-bee6-8599929a6bcc"

Commit message: Update GP2Y
Connections:
- net GND: now also K2.1; no longer K2.4
- net GP2Y_OUT: now also K2.3; no longer K2.2
- net MCU_ENABLE: now also K2.2; no longer K2.3
- net VIN: now also K2.4; no longer K2.1
Other:
- moved on the sheet: K2
Changed lines of the file:
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@@
     )
   )
-  (global_label "GP2Y_OUT" (shape output) (at 177.8 83.82 0)
+  (global_label "GP2Y_OUT" (shape input) (at 177.8 83.82 0)
     (effects (font (size 1.27 1.27)) (justify left))
     (property "Intersheet References" "${INTERSHEET_REFS}" (id 0) (at 187.3614 83.7406 0)
@@
     (pin "1")
   )
-  (symbol (lib_id "tronixio:MOLEX-MICRO-LATCH-04-RIGHT-ANGLE") (at 203.2 78.74 0) (mirror y) (unit 1)
+  (symbol (lib_id "tronixio:MOLEX-MICRO-LATCH-04-RIGHT-ANGLE") (at 203.2 86.36 180) (unit 1)
     (in_bom yes) (on_board yes)
-    (property "Reference" "K2" (id 0) (at 203.2 88.9 0)
+    (property "Reference" "K2" (id 0) (at 203.2 76.2 0)
       (effects (font (size 1.15 1.15)))
     )
-    (property "Value" "MCU" (id 1) (at 203.2 76.2 0)
+    (property "Value" "MCU" (id 1) (at 203.2 88.9 0)
       (effects (font (size 1.15 1.15)))
     )
-    (property "Footprint" "tronixio:MOLEX-532540470" (id 2) (at 203.2 91.44 0)
+    (property "Footprint" "tronixio:MOLEX-532540470" (id 2) (at 203.2 73.66 0)
       (effects (font (size 1 1)) hide)
     )
-    (property "Datasheet" "https://www.molex.com/pdm_docs/sd/532540470_sd.pdf" (id 3) (at 203.2 93.98 0)
+    (property "Datasheet" "https://www.molex.com/pdm_docs/sd/532540470_sd.pdf" (id 3) (at 203.2 71.12 0)
       (effects (font (size 1 1)) hide)
     )
-    (property "MOUSER" "538-53254-0470" (id 4) (at 203.2 96.52 0)
+    (property "MOUSER" "538-53254-0470" (id 4) (at 203.2 68.58 0)
       (effects (font (size 1 1)) hide)
     )
