File: Kicad/front-gp2y/gp2y.kicad_sch (KiCad schematic)
At the start: 12 parts, among them IC1 MCP1755-50, K1 GP2Y, K2 MCU

Commit message: Update GP2Y
Parts:
- IC1: value MCP1755-50 -> (none)
- IR1: value SHARP-GP2Y0xx1 -> (none); Name GP2Y0x21 -> GP2Y0A21
- K1: value GP2Y -> (none); MOUSER 538-53254-0370 -> (none); Mouser (none) -> 538-53254-0370
- K2: value MCU -> (none); MOUSER 538-53254-0470 -> (none); Mouser (none) -> 538-53254-0470
- LED1: value Power -> (none); MOUSER 604-APT3216LSECKJ4RV -> (none); Mouser (none) -> 604-APT3216LSECKJ4RV
Other:
- note added: "*R3: For GP2Y0D21 or MCU Pull-Up Resistor"
- note removed: "*R3: For GP2Y0D21"
Changed lines of the file:
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@@
     (effects (font (size 1.27 1.27)) (justify left bottom))
   )
-  (text "*R3: For GP2Y0D21" (at 185.42 179.07 0)
+  (text "*R3: For GP2Y0D21 or MCU Pull-Up Resistor" (at 185.42 179.07 0)
     (effects (font (size 1.27 1.27)) (justify left bottom))
   )
@@
       (effects (font (size 1.15 1.15)))
     )
-    (property "Value" "MCU" (id 1) (at 208.28 88.9 0)
+    (property "Value" "" (id 1) (at 208.28 88.9 0)
       (effects (font (size 1.15 1.15)))
     )
@@
       (effects (font (size 1 1)) hide)
     )
-    (property "MOUSER" "538-53254-0470" (id 4) (at 208.28 68.58 0)
+    (property "Mouser" "538-53254-0470" (id 4) (at 208.28 68.58 0)
       (effects (font (size 1 1)) hide)
     )
@@
       (effects (font (size 1.15 1.15)))
     )
-    (property "Value" "SHARP-GP2Y0xx1" (id 1) (at 261.62 171.45 0)
-      (effects (font (size 1 1)) hide)
-    )
-    (property "Footprint" "tronixio:SHARP-GP2Y0A" (id 2) (at 261.62 180.34 0)
-      (effects (font (size 1 1)) hide)
-    )
-    (property "Datasheet" "http://global.sharp/products/device/lineup/selection/opto/haca/diagram.html" (id 3) (at 261.62 182.88 0)
-      (effects (font (size 1 1)) hide)
-    )
-    (property "Name" "GP2Y0x21" (id 4) (at 261.62 171.45 0)
+    (property "Value" "" (id 1) (at 261.62 171.45 0)
+      (effects (font (size 1 1)) hide)
+    )
+    (property "Footprint" "tronixio:SHARP-GP2Y0A" (id 2) (at 261.62 182.88 0)
+      (effects (font (size 1 1)) hide)
+    )
+    (property "Datasheet" "http://global.sharp/products/device/lineup/selection/opto/haca/diagram.html" (id 3) (at 261.62 185.42 0)
+      (effects (font (size 1 1)) hide)
+    )
+    (property "Name" "GP2Y0A21" (id 4) (at 261.62 171.45 0)
       (effects (font (size 1.15 1.15)))
     )
@@
       (effects (font (size 1 1)) hide)
     )
-    (property "Footprint" "tronixio:M3-MASK" (id 2) (at 274.32 180.34 0)
+    (property "Footprint" "tronixio:M3-MASK" (id 2) (at 274.32 182.88 0)
       (effects (font (size 1 1)) hide)
     )
@@
       (effects (font (size 1 1)) hide)
     )
-    (property "Footprint" "tronixio:M3-MASK" (id 2) (at 279.4 180.34 0)
+    (property "Footprint" "tronixio:M3-MASK" (id 2) (at 279.4 182.88 0)
       (effects (font (size 1 1)) hide)
     )
@@
       (effects (font (size 1.15 1.15)))
     )
-    (property "Value" "MCP1755-50" (id 1) (at 114.3 87.63 0)
-      (effects (font (size 1.15 1.15)))
-    )
-    (property "Footprint" "tronixio:SOT-23-5" (id 2) (at 114.3 91.44 0)
-      (effects (font (size 1 1)) hide)
-    )
-    (property "Datasheet" "https://www.microchip.com/wwwproducts/en/MCP1755" (id 3) (at 114.3 93.98 0)
+    (property "Value" "" (id 1) (at 114.3 87.63 0)
+      (effects (font (size 1.15 1.15)))
+    )
+    (property "Footprint" "tronixio:SOT-23-5" (id 2) (at 114.3 93.98 0)
+      (effects (font (size 1 1)) hide)
+    )
+    (property "Datasheet" "https://www.microchip.com/en-us/product/MCP1755" (id 3) (at 114.3 93.98 0)
       (effects (font (size 1 1)) hide)
     )
@@
       (effects (font (size 1.15 1.15)))
     )
-    (property "Value" "Power" (id 1) (at 150.495 91.44 90)
+    (property "Value" "" (id 1) (at 150.495 91.44 90)
       (effects (font (size 1.15 1.15)) (justify left))
     )
@@
       (effects (font (size 1 1)) hide)
     )
-    (property "MOUSER" "604-APT3216LSECKJ4RV" (id 4) (at 137.16 88.9 0)
+    (property "Mouser" "604-APT3216LSECKJ4RV" (id 4) (at 137.16 88.9 0)
       (effects (font (size 1 1)) hide)
     )
@@
       (effects (font (size 1.15 1.15)))
     )
-    (property "Value" "GP2Y" (id 1) (at 167.64 86.36 0)
+    (property "Value" "" (id 1) (at 167.64 86.36 0)
       (effects (font (size 1.15 1.15)))
     )
@@
       (effects (font (size 1 1)) hide)
     )
-    (property "MOUSER" "538-53254-0370" (id 4) (at 167.64 68.58 0)
-      (effects (font (size 1 1)) hide)
-    )
+    (property "Mouser" "538-53254-0370" (id 4) (at 167.64 68.58 0)
+      (effects (font (size 1 1)) hide)
+    )
