File: Kicad/front-hc/hc-sr04.kicad_pcb (KiCad board)
At the start: 2 copper layers, 48 x 35 mm, 15 parts, among them IC1 MCP1755-50, K1 HC-SR04, K2 MCU

Commit message: Update HC-SR04
Connections:
- K2 pad 1: VIN -> GND
- K2 pad 2: MCU_TRIGGER -> MCU_ENABLE
- K2 pad 3: MCU_ECHO -> MCU_TRIGGER
- K2 pad 4: MCU_ENABLE -> MCU_ECHO
- K2 pad 5: GND -> VIN
Routing:
- net VIN: track 16.8 -> 11.7 mm
- net MCU_ECHO: track 18.9 -> 20.1 mm, vias 1 -> 0
- net MCU_TRIGGER: track 26.3 -> 27.3 mm
Changed lines of the file:
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@@
       ) (layer "B.Fab") (width 0.1) (fill solid))
     (pad "1" thru_hole oval locked (at 0 0 180) (size 1.2 1.75) (drill 0.8) (layers *.Cu *.Mask)
-      (net 4 "VIN") (pinfunction "1") (pintype "passive"))
+      (net 1 "GND") (pinfunction "1") (pintype "passive"))
     (pad "2" thru_hole oval locked (at 2 0 180) (size 1.2 1.75) (drill 0.8) (layers *.Cu *.Mask)
-      (net 8 "MCU_TRIGGER") (pinfunction "2") (pintype "passive"))
+      (net 7 "MCU_ENABLE") (pinfunction "2") (pintype "passive"))
     (pad "3" thru_hole oval locked (at 4 0 180) (size 1.2 1.75) (drill 0.8) (layers *.Cu *.Mask)
-      (net 6 "MCU_ECHO") (pinfunction "3") (pintype "passive"))
+      (net 8 "MCU_TRIGGER") (pinfunction "3") (pintype "passive"))
     (pad "4" thru_hole oval locked (at 6 0 180) (size 1.2 1.75) (drill 0.8) (layers *.Cu *.Mask)
-      (net 7 "MCU_ENABLE") (pinfunction "4") (pintype "passive"))
+      (net 6 "MCU_ECHO") (pinfunction "4") (pintype "passive"))
     (pad "5" thru_hole oval locked (at 8 0 180) (size 1.2 1.75) (drill 0.8) (layers *.Cu *.Mask)
-      (net 1 "GND") (pinfunction "5") (pintype "passive"))
+      (net 4 "VIN") (pinfunction "5") (pintype "passive"))
     (model "${KICAD6_USER_3DMODEL_DIR}/Connector/MOLEX-532540570.step"
       (offset (xyz 4 2.35 2.1))
@@
     (effects (font (size 1 1) (thickness 0.15)) (justify left mirror))
   )
-  (gr_text "GND" (at 120 69.75 90) (layer "F.SilkS")
+  (gr_text "VIN" (at 120 69.75 90) (layer "F.SilkS")
     (effects (font (size 0.8 0.8) (thickness 0.1)) (justify left))
   )
-  (gr_text "ECHO" (at 124 69.75 90) (layer "F.SilkS")
+  (gr_text "TRIG" (at 124 69.75 90) (layer "F.SilkS")
     (effects (font (size 0.8 0.8) (thickness 0.1)) (justify left))
   )
@@
     (effects (font (size 1.3 1.3) (thickness 0.2)))
   )
-  (gr_text "EN" (at 122 69.75 90) (layer "F.SilkS")
+  (gr_text "ECHO" (at 122 69.75 90) (layer "F.SilkS")
     (effects (font (size 0.8 0.8) (thickness 0.1)) (justify left))
   )
@@
     (effects (font (size 1.3 1.3) (thickness 0.2)))
   )
-  (gr_text "VIN" (at 128 69.75 90) (layer "F.SilkS")
+  (gr_text "GND" (at 128 69.75 90) (layer "F.SilkS")
     (effects (font (size 0.8 0.8) (thickness 0.1)) (justify left))
   )
@@
     (effects (font (size 1.3 1.3) (thickness 0.2)) (justify left))
   )
-  (gr_text "TRIG" (at 126 69.75 90) (layer "F.SilkS")
+  (gr_text "EN" (at 126 69.75 90) (layer "F.SilkS")
     (effects (font (size 0.8 0.8) (thickness 0.1)) (justify left))
   )
@@
     (style (thickness 0.1) (arrow_length 1) (text_position_mode 1) (extension_height 0.58642) (extension_offset 0.5) keep_text_aligned)
   )
-  (via (at 122 78) (size 0.8) (drill 0.4) (layers "F.Cu" "B.Cu") (free) (net 1))
+  (via (at 123 78.5) (size 0.8) (drill 0.4) (layers "F.Cu" "B.Cu") (free) (net 1))
   (segment (start 126.5 81) (end 126.5 80) (width 0.5) (layer "B.Cu") (net 2))
   (segment (start 117 81.5) (end 122 81.5) (width 0.5) (layer "B.Cu") (net 2))
@@
   (segment (start 132.5 88.78) (end 132.5 83) (width 0.5) (layer "B.Cu") (net 3))
   (segment (start 125.28 96) (end 132.5 88.78) (width 0.5) (layer "B.Cu") (net 3))
-  (segment (start 128 72.5) (end 128 71.1) (width 0.5) (layer "B.Cu") (net 4))
+  (segment (start 120 78) (end 120 71.1) (width 0.5) (layer "B.Cu") (net 4))
   (segment (start 121.2 80.2) (end 121 80) (width 0.5) (layer "B.Cu") (net 4))
   (segment (start 121 80) (end 119.5 80) (width 0.5) (layer "B.Cu") (net 4))
-  (segment (start 119.5 80) (end 119.5 78) (width 0.5) (layer "B.Cu") (net 4))
-  (segment (start 119.5 78) (end 123.5 74) (width 0.5) (layer "B.Cu") (net 4))
-  (segment (start 123.5 74) (end 126.5 74) (width 0.5) (layer "B.Cu") (net 4))
+  (segment (start 119.5 78.5) (end 120 78) (width 0.5) (layer "B.Cu") (net 4))
   (segment (start 122.05 80.2) (end 121.2 80.2) (width 0.5) (layer "B.Cu") (net 4))
-  (segment (start 126.5 74) (end 128 72.5) (width 0.5) (layer "B.Cu") (net 4))
+  (segment (start 119.5 80) (end 119.5 78.5) (width 0.5) (layer "B.Cu") (net 4))
   (segment (start 113.5 80) (end 116.5 80) (width 0.5) (layer "B.Cu") (net 5))
-  (segment (start 124 76) (end 124 71.1) (width 0.5) (layer "F.Cu") (net 6))
-  (via (at 124 76) (size 0.8) (drill 0.4) (layers "F.Cu" "B.Cu") (net 6))
+  (segment (start 130 76) (end 123.5 76) (width 0.5) (layer "B.Cu") (net 6))
+  (segment (start 122 74.5) (end 122 71.1) (width 0.5) (layer "B.Cu") (net 6))
+  (segment (start 132.5 78.5) (end 130 76) (width 0.5) (layer "B.Cu") (net 6))
   (segment (start 135.5 80) (end 132.5 80) (width 0.5) (layer "B.Cu") (net 6))
   (segment (start 132.5 80) (end 132.5 78.5) (width 0.5) (layer "B.Cu") (net 6))
-  (segment (start 132.5 78.5) (end 130 76) (width 0.5) (layer "B.Cu") (net 6))
-  (segment (start 130 76) (end 124 76) (width 0.5) (layer "B.Cu") (net 6))
-  (segment (start 124 78) (end 122 76) (width 0.5) (layer "F.Cu") (net 7))
-  (segment (start 122 76) (end 122 71.1) (width 0.5) (layer "F.Cu") (net 7))
-  (via (at 124 78) (size 0.8) (drill 0.4) (layers "F.Cu" "B.Cu") (net 7))
+  (segment (start 123.5 76) (end 122 74.5) (width 0.5) (layer "B.Cu") (net 6))
+  (segment (start 126 75.95) (end 126 71.1) (width 0.5) (layer "F.Cu") (net 7))
+  (segment (start 123.95 78) (end 126 75.95) (width 0.5) (layer "F.Cu") (net 7))
+  (via (at 123.95 78) (size 0.8) (drill 0.4) (layers "F.Cu" "B.Cu") (net 7))
   (segment (start 129.5 80) (end 129.5 78.5) (width 0.5) (layer "B.Cu") (net 7))
+  (segment (start 129 78) (end 123.95 78) (width 0.5) (layer "B.Cu") (net 7))
   (segment (start 123.95 78.05) (end 124 78) (width 0.5) (layer "B.Cu") (net 7))
   (segment (start 129.5 78.5) (end 129 78) (width 0.5) (layer "B.Cu") (net 7))
-  (segment (start 129 78) (end 124 78) (width 0.5) (layer "B.Cu") (net 7))
   (segment (start 123.95 80.2) (end 123.95 78.05) (width 0.5) (layer "B.Cu") (net 7))
-  (segment (start 126 92.74) (end 122.74 96) (width 0.5) (layer "F.Cu") (net 8))
-  (segment (start 126 71.1) (end 126 92.74) (width 0.5) (layer "F.Cu") (net 8))
+  (segment (start 124 74) (end 124 71.1) (width 0.5) (layer "F.Cu") (net 8))
+  (segment (start 120.5 93.76) (end 120.5 77.5) (width 0.5) (layer "F.Cu") (net 8))
+  (segment (start 120.5 77.5) (end 124 74) (width 0.5) (layer "F.Cu") (net 8))
+  (segment (start 122.74 96) (end 120.5 93.76) (width 0.5) (layer "F.Cu") (net 8))
   (zone (net 1) (net_name "GND") (layers F&B.Cu) (hatch edge 0.508)
     (connect_pads (clearance 0.508))
