File: Kicad/front-hc/hc-sr04.kicad_pcb (KiCad board)
At the start: 2 copper layers, 48 x 35 mm, 15 parts, among them IC1 MCP1755-50, K1 HC-SR04, K2 MCU

Commit message: Update HC-SR04
Parts:
- IC1: value MCP1755-50 -> MCP1755
Connections:
- net +5V renamed VCC

Commit message: Update hc-sr04.kicad_pcb
Parts:
- moved K1 0.50 mm to (120.2, 95.5)
Routing:
- net MCU_TRIGGER: track 27.3 -> 25.9 mm
- net MCU_ECHO: track 20.1 -> 18.9 mm
- net HC_ECHO: track 16.0 -> 15.5 mm
Changed lines of the file:
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@@
   )
   (footprint "tronixio:zzSAMTEC-SSW-104-02-T-S-RA" (layer "F.Cu")
-    (at 120.2 96)
+    (at 120.2 95.5)
     (property "MOUSER" "200-SSW10402TSRA")
     (property "Sheetfile" "hc-sr04.kicad_sch")
@@
   (segment (start 126.5 81) (end 126.5 80) (width 0.5) (layer "B.Cu") (net 2))
   (segment (start 117 81.5) (end 122 81.5) (width 0.5) (layer "B.Cu") (net 2))
-  (segment (start 120.2 96) (end 116.5 92.3) (width 0.5) (layer "B.Cu") (net 2))
   (segment (start 117 81.5) (end 116.5 82) (width 0.5) (layer "B.Cu") (net 2))
+  (segment (start 116.5 84.5) (end 116.5 83) (width 0.5) (layer "B.Cu") (net 2))
+  (segment (start 120.2 88.2) (end 116.5 84.5) (width 0.5) (layer "B.Cu") (net 2))
   (segment (start 116.5 82) (end 116.5 83) (width 0.5) (layer "B.Cu") (net 2))
   (segment (start 122.05 82.8) (end 122.05 81.55) (width 0.5) (layer "B.Cu") (net 2))
   (segment (start 122 81.5) (end 126 81.5) (width 0.5) (layer "B.Cu") (net 2))
-  (segment (start 116.5 92.3) (end 116.5 83) (width 0.5) (layer "B.Cu") (net 2))
   (segment (start 122.05 81.55) (end 122 81.5) (width 0.4) (layer "B.Cu") (net 2))
+  (segment (start 120.2 95.5) (end 120.2 88.2) (width 0.5) (layer "B.Cu") (net 2))
   (segment (start 126 81.5) (end 126.5 81) (width 0.5) (layer "B.Cu") (net 2))
-  (segment (start 132.5 88.78) (end 132.5 83) (width 0.5) (layer "B.Cu") (net 3))
-  (segment (start 125.28 96) (end 132.5 88.78) (width 0.5) (layer "B.Cu") (net 3))
+  (segment (start 125.28 91.72) (end 132.5 84.5) (width 0.5) (layer "B.Cu") (net 3))
+  (segment (start 125.28 95.5) (end 125.28 91.72) (width 0.5) (layer "B.Cu") (net 3))
+  (segment (start 132.5 84.5) (end 132.5 83) (width 0.5) (layer "B.Cu") (net 3))
   (segment (start 120 78) (end 120 71.1) (width 0.5) (layer "B.Cu") (net 4))
   (segment (start 121.2 80.2) (end 121 80) (width 0.5) (layer "B.Cu") (net 4))
@@
   (segment (start 119.5 80) (end 119.5 78.5) (width 0.5) (layer "B.Cu") (net 4))
   (segment (start 113.5 80) (end 116.5 80) (width 0.5) (layer "B.Cu") (net 5))
-  (segment (start 130 76) (end 123.5 76) (width 0.5) (layer "B.Cu") (net 6))
-  (segment (start 122 74.5) (end 122 71.1) (width 0.5) (layer "B.Cu") (net 6))
-  (segment (start 132.5 78.5) (end 130 76) (width 0.5) (layer "B.Cu") (net 6))
+  (segment (start 125.5 76) (end 122 72.5) (width 0.5) (layer "B.Cu") (net 6))
+  (segment (start 130 76) (end 125.5 76) (width 0.5) (layer "B.Cu") (net 6))
+  (segment (start 122 72.5) (end 122 71.1) (width 0.5) (layer "B.Cu") (net 6))
   (segment (start 135.5 80) (end 132.5 80) (width 0.5) (layer "B.Cu") (net 6))
   (segment (start 132.5 80) (end 132.5 78.5) (width 0.5) (layer "B.Cu") (net 6))
-  (segment (start 123.5 76) (end 122 74.5) (width 0.5) (layer "B.Cu") (net 6))
+  (segment (start 132.5 78.5) (end 130 76) (width 0.5) (layer "B.Cu") (net 6))
   (segment (start 126 75.95) (end 126 71.1) (width 0.5) (layer "F.Cu") (net 7))
   (segment (start 123.95 78) (end 126 75.95) (width 0.5) (layer "F.Cu") (net 7))
@@
   (segment (start 129.5 78.5) (end 129 78) (width 0.5) (layer "B.Cu") (net 7))
   (segment (start 123.95 80.2) (end 123.95 78.05) (width 0.5) (layer "B.Cu") (net 7))
-  (segment (start 124 74) (end 124 71.1) (width 0.5) (layer "F.Cu") (net 8))
-  (segment (start 120.5 93.76) (end 120.5 77.5) (width 0.5) (layer "F.Cu") (net 8))
-  (segment (start 120.5 77.5) (end 124 74) (width 0.5) (layer "F.Cu") (net 8))
-  (segment (start 122.74 96) (end 120.5 93.76) (width 0.5) (layer "F.Cu") (net 8))
+  (segment (start 121.5 75) (end 124 72.5) (width 0.5) (layer "F.Cu") (net 8))
+  (segment (start 121.5 94.26) (end 121.5 75) (width 0.5) (layer "F.Cu") (net 8))
+  (segment (start 122.74 95.5) (end 121.5 94.26) (width 0.5) (layer "F.Cu") (net 8))
+  (segment (start 124 72.5) (end 124 71.1) (width 0.5) (layer "F.Cu") (net 8))
   (zone (net 1) (net_name "GND") (layers F&B.Cu) (hatch edge 0.508)
     (connect_pads (clearance 0.5))

Commit message: Update HC-SR04
Connections:
- net VCC renamed +5V
Changed lines of the file:
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@@
   (net 0 "")
   (net 1 "GND")
-  (net 2 "VCC")
+  (net 2 "+5V")
   (net 3 "HC_ECHO")
   (net 4 "VIN")
@@
     (fp_rect (start 7.3 0) (end 7.95 -1.9) (layer "F.Fab") (width 0.1) (fill solid))
     (pad "1" thru_hole circle locked (at 0 0) (size 1.8 1.8) (drill 0.8) (layers *.Cu *.Mask)
-      (net 2 "VCC") (pinfunction "1") (pintype "passive"))
+      (net 2 "+5V") (pinfunction "1") (pintype "passive"))
     (pad "2" thru_hole circle locked (at 2.54 0) (size 1.8 1.8) (drill 0.8) (layers *.Cu *.Mask)
       (net 8 "MCU_TRIGGER") (pinfunction "2") (pintype "passive"))
@@
     (fp_rect (start 1.2 -0.8) (end 1.5 0.8) (layer "B.Fab") (width 0.1) (fill solid))
     (pad "1" smd roundrect (at -1.5 0 270) (size 1.3 1.75) (layers "B.Cu" "B.Paste" "B.Mask") (roundrect_rratio 0.15)
-      (net 2 "VCC") (pintype "passive") (zone_connect 2))
+      (net 2 "+5V") (pintype "passive") (zone_connect 2))
     (pad "2" smd roundrect (at 1.5 0 270) (size 1.3 1.75) (layers "B.Cu" "B.Paste" "B.Mask") (roundrect_rratio 0.15)
       (net 1 "GND") (pintype "passive") (zone_connect 2))
@@
   (footprint "tronixio:SOT-23-5" (layer "B.Cu")
     (at 123 81.5 -90)
-    (property "MOUSER" "579-MCP1755T-5002EOT")
+    (property "Mouser" "579-MCP1755T-5002EOT")
+    (property "Name" "MCP1755-50")
     (property "Sheetfile" "hc-sr04.kicad_sch")
     (property "Sheetname" "")
@@
       (net 9 "unconnected-(IC1-Pad4)") (pinfunction "PWRGD") (pintype "open_collector+no_connect"))
     (pad "5" smd roundrect locked (at 1.3 0.95 270) (size 1.2 0.6) (layers "B.Cu" "B.Paste" "B.Mask") (roundrect_rratio 0.15)
-      (net 2 "VCC") (pinfunction "VOUT") (pintype "power_out"))
+      (net 2 "+5V") (pinfunction "VOUT") (pintype "power_out"))
     (model "${KICAD6_USER_3DMODEL_DIR}/SMD/SOT-23-5.wrl"
       (offset (xyz 0 0 0))
@@
     (fp_rect (start -1.5 -0.8) (end -1.2 0.8) (layer "B.Fab") (width 0.1) (fill solid))
     (pad "1" smd roundrect (at -1.5 0 90) (size 1.3 1.75) (layers "B.Cu" "B.Paste" "B.Mask") (roundrect_rratio 0.15)
-      (net 2 "VCC") (pintype "passive") (zone_connect 2))
+      (net 2 "+5V") (pintype "passive") (zone_connect 2))
     (pad "2" smd roundrect (at 1.5 0 90) (size 1.3 1.75) (layers "B.Cu" "B.Paste" "B.Mask") (roundrect_rratio 0.15)
       (net 5 "Net-(LED1-Pad2)") (pintype "passive") (zone_connect 2))
