File: Kicad/front-hc/hc-sr04.kicad_pcb (KiCad board)
At the start: 2 copper layers, 48 x 35 mm, 15 parts, among them IC1 MCP1755, K1 HC-SR04, K2 MCU

Commit message: Update HC-SR04
Parts:
- removed R3: 0Ω, tronixio:RESISTOR-1206
- removed R4: NP, tronixio:RESISTOR-1206
- moved C1 2.50 mm to (122.0, 81.5)
- moved C2 2.50 mm to (129.0, 81.5)
- moved IC1 2.50 mm to (125.5, 81.5)
- moved LED1 2.50 mm to (116.0, 81.5)
- moved R1 2.50 mm to (132.0, 81.5)
- moved R2 2.50 mm to (119.0, 81.5)
- moved GB 1.00 mm to (133.0, 76.0)
Connections:
- K1 pad 3: HC_ECHO -> MCU_ECHO
Routing:
- net HC_ECHO: track 15.5 -> 0.00 mm
- net MCU_ECHO: track 18.9 -> 26.6 mm, vias 0 -> 1
- net MCU_ENABLE: track 17.2 -> 16.0 mm
- net +5V: track 27.8 -> 26.7 mm
- net MCU_TRIGGER: track 25.9 -> 24.9 mm
- net VIN: track 11.7 -> 12.4 mm
- net GND: vias 1 -> 0
Other:
- board text removed: "*"
- board text removed: "Output 3V3"
- board text removed: "Output 5V"
