File: Kicad/front-hc/hc-sr04.kicad_sch (KiCad schematic)
At the start: 13 parts, among them IC1 MCP1755-50, K1 HC-SR04, K2 MCU

Commit message: Update HC-SR04
Connections:
- net GND: now also K2.1; no longer K2.5
- net MCU_ECHO: now also K2.4; no longer K2.3
- net MCU_ENABLE: now also K2.2; no longer K2.4
- net MCU_TRIGGER: now also K2.3; no longer K2.2
- net VIN: now also K2.5; no longer K2.1
Other:
- moved on the sheet: K2
Changed lines of the file:
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@@
     )
   )
-  (global_label "MCU_ENABLE" (shape output) (at 231.14 86.36 0)
+  (global_label "MCU_ENABLE" (shape input) (at 231.14 86.36 0)
     (effects (font (size 1.27 1.27)) (justify left))
     (property "Intersheet References" "${INTERSHEET_REFS}" (id 0) (at 240.7014 86.2806 0)
@@
     )
   )
-  (global_label "HC_ECHO" (shape input) (at 195.58 83.82 0)
+  (global_label "HC_ECHO" (shape output) (at 195.58 83.82 0)
     (effects (font (size 1.27 1.27)) (justify left))
     (property "Intersheet References" "${INTERSHEET_REFS}" (id 0) (at 205.1414 83.7406 0)
@@
     )
   )
-  (global_label "MCU_TRIGGER" (shape output) (at 231.14 81.28 0)
+  (global_label "MCU_TRIGGER" (shape input) (at 231.14 83.82 0)
     (effects (font (size 1.27 1.27)) (justify left))
-    (property "Intersheet References" "${INTERSHEET_REFS}" (id 0) (at 240.7014 81.2006 0)
+    (property "Intersheet References" "${INTERSHEET_REFS}" (id 0) (at 240.7014 83.7406 0)
       (effects (font (size 1.27 1.27)) (justify left) hide)
     )
   )
-  (global_label "MCU_ECHO" (shape input) (at 231.14 83.82 0)
+  (global_label "MCU_ECHO" (shape output) (at 231.14 81.28 0)
     (effects (font (size 1.27 1.27)) (justify left))
-    (property "Intersheet References" "${INTERSHEET_REFS}" (id 0) (at 240.7014 83.7406 0)
+    (property "Intersheet References" "${INTERSHEET_REFS}" (id 0) (at 240.7014 81.2006 0)
       (effects (font (size 1.27 1.27)) (justify left) hide)
     )
@@
     (pin "1")
   )
-  (symbol (lib_id "tronixio:MOLEX-MICRO-LATCH-05-RIGHT-ANGLE") (at 220.98 78.74 0) (mirror y) (unit 1)
+  (symbol (lib_id "tronixio:MOLEX-MICRO-LATCH-05-RIGHT-ANGLE") (at 220.98 88.9 180) (unit 1)
     (in_bom yes) (on_board yes)
-    (property "Reference" "K2" (id 0) (at 220.98 76.2 0)
+    (property "Reference" "K2" (id 0) (at 220.98 91.44 0)
       (effects (font (size 1.15 1.15)))
     )
-    (property "Value" "MCU" (id 1) (at 220.98 91.44 0)
+    (property "Value" "MCU" (id 1) (at 220.98 76.2 0)
       (effects (font (size 1.15 1.15)))
     )
-    (property "Footprint" "tronixio:MOLEX-532540570" (id 2) (at 220.98 93.98 0)
+    (property "Footprint" "tronixio:MOLEX-532540570" (id 2) (at 220.98 73.66 0)
       (effects (font (size 1 1)) hide)
     )
-    (property "Datasheet" "https://www.molex.com/pdm_docs/sd/532540570_sd.pdf" (id 3) (at 220.98 96.52 0)
+    (property "Datasheet" "https://www.molex.com/pdm_docs/sd/532540570_sd.pdf" (id 3) (at 220.98 71.12 0)
       (effects (font (size 1 1)) hide)
     )
-    (property "MOUSER" "538-53254-0570" (id 4) (at 220.98 99.06 0)
+    (property "MOUSER" "538-53254-0570" (id 4) (at 220.98 68.58 0)
       (effects (font (size 1 1)) hide)
     )

Commit message: Update HC-SR04
Parts:
- IC1: value MCP1755-50 -> MCP1755
Connections:
- net +5V renamed VCC
Other:
- note added: "*IC1: +3V3 or +5V Depend MCU Voltage."
Changed lines of the file:
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@@
     (effects (font (size 1.27 1.27)) (justify left bottom))
   )
+  (text "*" (at 96.52 76.2 0)
+    (effects (font (size 1.27 1.27)) (justify left bottom))
+  )
   (text "*" (at 147.32 86.36 0)
+    (effects (font (size 1.27 1.27)) (justify left bottom))
+  )
+  (text "*IC1: +3V3 or +5V Depend MCU Voltage." (at 185.42 173.99 0)
     (effects (font (size 1.27 1.27)) (justify left bottom))
   )
@@
     (pin "2")
   )
-  (symbol (lib_id "tronixio:POWER-+5V") (at 132.08 71.12 0) (unit 1)
+  (symbol (lib_id "tronixio:POWER-VCC") (at 132.08 71.12 0) (unit 1)
     (in_bom yes) (on_board yes)
     (property "Reference" "#PWR07" (id 0) (at 132.08 81.28 0)
@@
       (effects (font (size 1 1)) hide)
     )
-    (property "Name" "+5V" (id 4) (at 132.08 66.04 0)
+    (property "Name" "VCC" (id 4) (at 132.08 66.04 0)
       (effects (font (size 1.15 1.15)))
     )
@@
     (pin "1")
   )
-  (symbol (lib_id "tronixio:POWER-+5V") (at 190.5 71.12 0) (unit 1)
+  (symbol (lib_id "tronixio:POWER-VCC") (at 190.5 71.12 0) (unit 1)
     (in_bom yes) (on_board yes)
     (property "Reference" "#PWR013" (id 0) (at 190.5 81.28 0)
@@
       (effects (font (size 1 1)) hide)
     )
-    (property "Name" "+5V" (id 4) (at 190.5 66.04 0)
+    (property "Name" "VCC" (id 4) (at 190.5 66.04 0)
       (effects (font (size 1.15 1.15)))
     )
@@
     (pin "1")
   )
-  (symbol (lib_id "tronixio:POWER-+5V") (at 111.76 71.12 0) (unit 1)
+  (symbol (lib_id "tronixio:POWER-VCC") (at 111.76 71.12 0) (unit 1)
     (in_bom yes) (on_board yes)
     (property "Reference" "#PWR05" (id 0) (at 111.76 81.28 0)
@@
       (effects (font (size 1 1)) hide)
     )
-    (property "Name" "+5V" (id 4) (at 111.76 66.04 0)
+    (property "Name" "VCC" (id 4) (at 111.76 66.04 0)
       (effects (font (size 1.15 1.15)))
     )
@@
       (effects (font (size 1.15 1.15)))
     )
-    (property "Value" "MCP1755-50" (id 1) (at 99.06 87.63 0)
+    (property "Value" "MCP1755" (id 1) (at 99.06 87.63 0)
       (effects (font (size 1.15 1.15)))
     )
@@
     )
     (path "/b0f807f7-df5c-4c93-8b4c-5933ccbdfd3a"
-      (reference "IC1") (unit 1) (value "MCP1755-50") (footprint "tronixio:SOT-23-5")
+      (reference "IC1") (unit 1) (value "MCP1755") (footprint "tronixio:SOT-23-5")
     )
     (path "/ed89b481-faca-420e-bee6-8599929a6bcc"

Commit message: Update HC-SR04
Connections:
- net VCC renamed +5V
Other:
- note added: "*R3 & *R4: 1K & 1K8 For 3V3 Output."
- note removed: "*IC1: +3V3 or +5V Depend MCU Voltage."
- note removed: "*R3 & *R4: 1K & 1K8 For 3V3 Level Shifting Output"
Changed lines of the file:
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@@
-    (effects (font (size 1.27 1.27)) (justify left bottom))
-  )
-  (text "*" (at 96.52 76.2 0)
     (effects (font (size 1.27 1.27)) (justify left bottom))
   )
@@
     (effects (font (size 1.27 1.27)) (justify left bottom))
   )
-  (text "*IC1: +3V3 or +5V Depend MCU Voltage." (at 185.42 173.99 0)
-    (effects (font (size 1.27 1.27)) (justify left bottom))
-  )
   (text "*R3 & *R4: 0Ω & NP For 5V Output." (at 185.42 176.53 0)
     (effects (font (size 1.27 1.27)) (justify left bottom))
   )
-  (text "*R3 & *R4: 1K & 1K8 For 3V3 Level Shifting Output" (at 185.42 179.07 0)
+  (text "*R3 & *R4: 1K & 1K8 For 3V3 Output." (at 185.42 179.07 0)
     (effects (font (size 1.27 1.27)) (justify left bottom))
   )
@@
     )
   )
-  (global_label "MCU_ENABLE" (shape input) (at 231.14 86.36 0)
+  (global_label "MCU_ENABLE" (shape output) (at 231.14 86.36 0)
     (effects (font (size 1.27 1.27)) (justify left))
     (property "Intersheet References" "${INTERSHEET_REFS}" (id 0) (at 240.7014 86.2806 0)
@@
     )
   )
-  (global_label "MCU_TRIGGER" (shape input) (at 231.14 83.82 0)
+  (global_label "MCU_TRIGGER" (shape output) (at 231.14 83.82 0)
     (effects (font (size 1.27 1.27)) (justify left))
     (property "Intersheet References" "${INTERSHEET_REFS}" (id 0) (at 240.7014 83.7406 0)
@@
     )
   )
-  (global_label "MCU_ECHO" (shape output) (at 231.14 81.28 0)
+  (global_label "MCU_ECHO" (shape input) (at 231.14 81.28 0)
     (effects (font (size 1.27 1.27)) (justify left))
     (property "Intersheet References" "${INTERSHEET_REFS}" (id 0) (at 240.7014 81.2006 0)
@@
     (pin "2")
   )
-  (symbol (lib_id "tronixio:POWER-VCC") (at 132.08 71.12 0) (unit 1)
+  (symbol (lib_id "tronixio:POWER-+5V") (at 132.08 71.12 0) (unit 1)
     (in_bom yes) (on_board yes)
     (property "Reference" "#PWR07" (id 0) (at 132.08 81.28 0)
@@
       (effects (font (size 1 1)) hide)
     )
-    (property "Name" "VCC" (id 4) (at 132.08 66.04 0)
+    (property "Name" "+5V" (id 4) (at 132.08 66.04 0)
       (effects (font (size 1.15 1.15)))
     )
@@
     (pin "1")
   )
-  (symbol (lib_id "tronixio:POWER-VCC") (at 190.5 71.12 0) (unit 1)
+  (symbol (lib_id "tronixio:POWER-+5V") (at 190.5 71.12 0) (unit 1)
     (in_bom yes) (on_board yes)
     (property "Reference" "#PWR013" (id 0) (at 190.5 81.28 0)
@@
       (effects (font (size 1 1)) hide)
     )
-    (property "Name" "VCC" (id 4) (at 190.5 66.04 0)
+    (property "Name" "+5V" (id 4) (at 190.5 66.04 0)
       (effects (font (size 1.15 1.15)))
     )
@@
     (pin "1")
   )
-  (symbol (lib_id "tronixio:POWER-VCC") (at 111.76 71.12 0) (unit 1)
+  (symbol (lib_id "tronixio:POWER-+5V") (at 111.76 71.12 0) (unit 1)
     (in_bom yes) (on_board yes)
     (property "Reference" "#PWR05" (id 0) (at 111.76 81.28 0)
       (effects (font (size 1 1)) hide)
     )
-    (property "Value" "POWER-+5V" (id 1) (at 111.76 83.82 0)
+    (property "Value" "POWER-VCC" (id 1) (at 111.76 83.82 0)
       (effects (font (size 1 1)) hide)
     )
@@
       (effects (font (size 1 1)) hide)
     )
-    (property "Name" "VCC" (id 4) (at 111.76 66.04 0)
+    (property "Name" "+5V" (id 4) (at 111.76 66.04 0)
       (effects (font (size 1.15 1.15)))
     )
@@
     )
     (path "/5fa73fb5-2d5a-4dc9-8bc9-d707e448c51f"
-      (reference "#PWR05") (unit 1) (value "POWER-+5V") (footprint "")
+      (reference "#PWR05") (unit 1) (value "POWER-VCC") (footprint "")
     )
     (path "/b9b9ed69-122a-4a3b-ad44-5ae3baedfe97"
