File: Kicad/front-hc/hc-sr04.kicad_sch (KiCad schematic)
At the start: 13 parts, among them IC1 MCP1755, K1 HC-SR04, K2 MCU

Commit message: Draft
Other:
- note added: "DRAFT"
Changed lines of the file:
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@@
     (effects (font (size 1.27 1.27)) (justify left bottom))
+  )
+  (text "DRAFT" (at 208.28 190.5 0)
+    (effects (font (size 5 5)) (justify left bottom))
   )
   (text "*R3 & *R4: 1K & 1K8 For 3V3 Output." (at 185.42 179.07 0)

Commit message: Update HC-SR04
Parts:
- IC1: symbol tronixio:MCP1755-50-SOT23 -> tronixio:MICROCHIP-MCP1755-50-SOT23; MOUSER 579-MCP1755T-5002EOT -> (none); Mouser (none) -> 579-MCP1755T-5002EOT; Name (none) -> MCP1755-50
Changed lines of the file:
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@@
     )
   )
-  (symbol (lib_id "tronixio:MCP1755-50-SOT23") (at 99.06 81.28 0) (unit 1)
+  (symbol (lib_id "tronixio:MICROCHIP-MCP1755-50-SOT23") (at 99.06 81.28 0) (unit 1)
     (in_bom yes) (on_board yes)
     (property "Reference" "IC1" (id 0) (at 99.06 74.93 0)
@@
     )
     (property "Value" "MCP1755" (id 1) (at 99.06 87.63 0)
-      (effects (font (size 1.15 1.15)))
+      (effects (font (size 1 1)) hide)
     )
     (property "Footprint" "tronixio:SOT-23-5" (id 2) (at 99.06 91.44 0)
@@
       (effects (font (size 1 1)) hide)
     )
-    (property "MOUSER" "579-MCP1755T-5002EOT" (id 4) (at 99.06 93.98 0)
+    (property "Name" "MCP1755-50" (id 4) (at 99.06 87.63 0)
+      (effects (font (size 1.15 1.15)))
+    )
+    (property "Mouser" "579-MCP1755T-5002EOT" (id 5) (at 99.06 96.52 0)
       (effects (font (size 1 1)) hide)
     )

Commit message: Update HC-SR04
Parts:
- removed R3: 0Ω, tronixio:RESISTOR-1206, symbol tronixio:R-1206
- removed R4: NP, tronixio:RESISTOR-1206, symbol tronixio:R-1206
- HC1: value HC-SR04 -> (none); footprint tronixio:zzHC-SR04 -> tronixio:HC-SR04
- IC1: value MCP1755 -> (none)
- K1: footprint tronixio:zzSAMTEC-SSW-104-02-T-S-RA -> tronixio:SAMTEC-SSW-104-02-T-S-RA; MOUSER 200-SSW10402TSRA -> (none); Mouser (none) -> 200-SSW10402TSRA
- LED1: value Power -> (none); MOUSER 604-APTR3216-VFX -> (none); Mouser (none) -> 604-APTR3216-VFX
Connections:
- net HC_ECHO is gone; now on net MCU_ECHO: K1.3
Other:
- note removed: "*"
- note removed: "*R3 & *R4: 0Ω & NP For 5V Output."
- note removed: "*R3 & *R4: 1K & 1K8 For 3V3 Output."
- moved on the sheet: C1, C2, IC1, K1, K2, LED1, R1, R2
