File: Kicad/charger/tbot-charger.kicad_sch (KiCad schematic)
At the start: 19 parts, among them IC1 BQ2057W, K1 Charger, K2 Battery, T1 STN790A

Commit message: Update Charger
Other:
- title: Charger 2x18650 -> TBOT - Charger 2x18650
- moved on the sheet: BT1A, BT1B, C1, C2, D1, IC1, K1, K2, LED1, R1, R2, R3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
