File: Kicad/charger/tbot-charger.kicad_pcb (KiCad board)
At the start: 2 copper layers, 78 x 57 mm, 21 parts, among them IC1 BQ2057W, K1 Charger, K2 Battery, T1 STN790A

Commit message: Update Charger
Other:
- board text added: "Charging"
Changed lines of the file:
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@@
     (effects (font (size 1.5 1.5) (thickness 0.2)) (justify right))
+  )
+  (gr_text "Charging" (at 154 79.5 90) (layer "F.SilkS")
+    (effects (font (size 0.8 0.8) (thickness 0.15)))
   )
   (gr_text "*" (at 149.5 73.4) (layer "F.SilkS")
