File: Kicad/charger/charger.kicad_sch (KiCad schematic)
At the start: 19 parts, among them IC1 BQ2057W, K1 Charger, K2 Battery, T1 STN790A

Commit message: Update Charger
Parts:
- BT1: MOUSER 534-1049 -> (none); Mouser (none) -> 534-1049
- D1: MOUSER 771-PMEG3030EP115 -> (none); Mouser (none) -> 771-PMEG3030EP115
- IC1: symbol tronixio:BQ2057W -> tronixio:TI-BQ2057W; MOUSER 595-BQ2057WSN -> (none); Mouser (none) -> 595-BQ2057WSN; Name (none) -> BQ2057W
- K1: MOUSER 490-PJ-102AH -> (none); Mouser (none) -> 490-PJ-102AH
- K2: MOUSER 538-22-05-7025 -> (none); Mouser (none) -> 538-22-05-7025
- LED1: MOUSER 604-APTR3216-VFX -> (none); Mouser (none) -> 604-APTR3216-VFX
- T1: symbol tronixio:STN790A -> tronixio:ST-STN790A; MOUSER 511-STN790A -> (none); Mouser (none) -> 511-STN790A; Name (none) -> STN90
- TH1: MOUSER 594-NTCLE213E3103FL -> (none); Mouser (none) -> 594-NTCLE213E3103FL; Name (none) -> 10K

Commit message: Update Charger
Parts:
- D1: symbol tronixio:PMEG3030 -> tronixio:NEXPERIA-PMEG3030; Name (none) -> PMEG3030
- K1: value Charger -> (none)
- LED1: value Charging -> (none)

Commit message: Update Charger
Parts:
- K1: value (none) -> Charger
- LED1: value (none) -> Charging
Changed lines of the file:
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@@
       (effects (font (size 1.15 1.15)))
     )
-    (property "Value" "" (id 1) (at 81.28 91.44 0)
+    (property "Value" "Charger" (id 1) (at 81.28 91.44 0)
       (effects (font (size 1.15 1.15)))
     )
@@
   (symbol (lib_id "tronixio:LED-1206-PURPLE") (at 109.22 101.6 90) (unit 1)
     (in_bom yes) (on_board yes)
-    (property "Reference" "LED1" (id 0) (at 109.22 99.06 90)
+    (property "Reference" "LED1" (id 0) (at 108.585 99.06 90)
       (effects (font (size 1.15 1.15)) (justify left))
     )
-    (property "Value" "" (id 1) (at 109.22 104.14 90)
+    (property "Value" "Charging" (id 1) (at 108.585 104.14 90)
       (effects (font (size 1.15 1.15)) (justify left))
     )
