File: Kicad/charger/charger.kicad_sch (KiCad schematic)
At the start: 19 parts, among them IC1 BQ2057W, K1 Charger, K2 Battery, T1 STN790A

Commit message: Update
Parts:
- U1: renamed from IC1; value BQ2057W -> TI-BQ2057W
- renumbered T1 to Q1
Other:
- moved on the sheet: BT1A, BT1B, C1, C2, K1, K2, LED1, Q1, R1, R2, R3, R4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

Commit message: Update
Parts:
- BT1: Name (none) -> KEYSTONE-1049
- C1: symbol tronixio:C-1206 -> tronixio:CAPACITOR-1206-100N; Mouser (none) -> 80-C1206C104M5R; Name (none) -> CAPACITOR-1206-100N; Tolerance (none) -> 20%; Voltage (none) -> 50V
- C2: symbol tronixio:C-1206 -> tronixio:CAPACITOR-1206-1U; Mouser (none) -> C1206C105M5RACTU; Name (none) -> CAPACITOR-1206-1U; Tolerance (none) -> 20%; Voltage (none) -> 50V
- D1: Name PMEG3030 -> NEXPERIA-PMEG3030
- K1: Name (none) -> CUI-PJ-102AH-TH
- K2: Name (none) -> MOLEX-MINI-SPOX-02-RIGHT-ANGLE
- LED1: symbol tronixio:LED-1206-PURPLE -> tronixio:KINGBRIGHT-LED-1206-PURPLE; Name (none) -> KINGBRIGHT-LED-1206-PURPLE
- Q1: symbol tronixio:ST-STN790A -> tronixio:ST-STN790A-SOT-223; Name STN90 -> ST-STN790A-SOT-223
- R1: symbol tronixio:R-1206 -> tronixio:RESISTOR-1206-4K7; Mouser (none) -> 660-RK73B2BTTDD472J; Name (none) -> RESISTOR-1206-4K7; Tolerance (none) -> 5%
- R2, R3: symbol tronixio:R-1210 -> tronixio:RESISTOR-1210-0R1; Mouser (none) -> 660-SR732ETTER100F; Name (none) -> RESISTOR-1210-0R1; Tolerance (none) -> 1%
- R4: symbol tronixio:R-1206 -> tronixio:RESISTOR-1206-1K; Mouser (none) -> 660-RK73B2BTTDD102J; Name (none) -> RESISTOR-1206-1K; Tolerance (none) -> 5%
- R5: symbol tronixio:R-1206 -> tronixio:RESISTOR-1206-10K; Mouser (none) -> 660-RK73B2BTTDD103J; Name (none) -> RESISTOR-1206-10K; Tolerance (none) -> 5%
- R6: symbol tronixio:R-1206 -> tronixio:RESISTOR-1206-36K; Mouser (none) -> 660-RK73B2BTTD363J; Name (none) -> RESISTOR-1206-36K; Tolerance (none) -> 5%
- TH1: footprint tronixio:THERMISTOR -> tronixio:THERMISTOR-SMD; Name 10K -> THERMISTOR-NTC-10K
- U1: value TI-BQ2057W -> BQ2057W; symbol tronixio:TI-BQ2057W -> tronixio:TI-BQ2057W-SOIC-08; Name BQ2057W -> TI-BQ2057W-SOIC

Commit message: Update
Parts:
- C1, C2: footprint tronixio:CAPACITOR-1206 -> tronixio:CAPACITOR-SMD-1206
- H1, H2, H3: footprint tronixio:M3-MASK -> tronixio:MOUNTING-HOLE-3MM-MASK; symbol tronixio:MOUNTING-HOLE-MASK-3MM -> tronixio:MOUNTING-HOLE-3MM-MASK
- LED1: footprint tronixio:LED-1206 -> tronixio:LED-SMD-1206
- R1, R4, R5, R6: footprint tronixio:RESISTOR-1206 -> tronixio:RESISTOR-SMD-1206
- R2, R3: footprint tronixio:RESISTOR-1210 -> tronixio:RESISTOR-SMD-1210

Commit message: Update
Parts:
- K1: value Charger -> 9V - 1A
- LED1: value Charging -> Charge
Other:
- note removed: "9V - 1A"
Changed lines of the file:
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@@
     (effects (font (size 1.27 1.27)) (justify left bottom))
-  )
-  (text "9V - 1A" (at 73.66 87.63 180)
-    (effects (font (size 1.27 1.27)) (justify right bottom))
   )
   (text "*" (at 160.02 99.06 0)
@@
       (effects (font (size 1.15 1.15)))
     )
-    (property "Value" "Charger" (id 1) (at 78.74 91.44 0)
+    (property "Value" "9V - 1A" (id 1) (at 78.74 91.44 0)
       (effects (font (size 1.15 1.15)))
     )
@@
       (effects (font (size 1.15 1.15)) (justify left))
     )
-    (property "Value" "Charging" (id 1) (at 100.965 104.14 90)
+    (property "Value" "Charge" (id 1) (at 100.965 104.14 90)
       (effects (font (size 1.15 1.15)) (justify left))
     )
@@
       (effects (font (size 1.27 1.27)) hide)
     )
-    (property "Value" "PWR_FLAG" (id 1) (at 162.56 189.23 0)
+    (property "Value" "POWER-FLAG" (id 1) (at 162.56 189.23 0)
       (effects (font (size 1.27 1.27)) hide)
     )
@@
     )
     (path "/fc217884-314f-464c-b6f5-43d868b35e41"
-      (reference "#FLG02") (unit 1) (value "PWR_FLAG") (footprint "")
+      (reference "#FLG02") (unit 1) (value "POWER-FLAG") (footprint "")
     )
     (path "/9702bc62-2308-42c6-8752-e186afd16157"
@@
     )
     (path "/44227ce2-fa9a-44dd-a461-f169f8e4bd8d"
-      (reference "K1") (unit 1) (value "Charger") (footprint "tronixio:CUI-PJ-102AH")
+      (reference "K1") (unit 1) (value "9V - 1A") (footprint "tronixio:CUI-PJ-102AH")
     )
     (path "/9c9a6027-25dc-4df4-b3ca-f6ee7d6946d5"
@@
     )
     (path "/539d6d6a-97ce-45d4-a3ca-21493b6ed8a8"
-      (reference "LED1") (unit 1) (value "Charging") (footprint "tronixio:LED-SMD-1206")
+      (reference "LED1") (unit 1) (value "Charge") (footprint "tronixio:LED-SMD-1206")
     )
     (path "/75ab6d8e-2241-4f8a-a9db-1a91d88bfede"

Commit message: Update
Parts:
- BT1: Name KEYSTONE-1049 -> (none)
- C1: symbol tronixio:CAPACITOR-1206-100N -> tronixio:CAPACITOR-1206-100N-5P-X7R; Mouser 80-C1206C104M5R -> 80-C1206C104J5R; Name CAPACITOR-1206-100N -> (none); Tolerance 20% -> 5%
- C2: symbol tronixio:CAPACITOR-1206-1U -> tronixio:CAPACITOR-1206-1U-10P-X7R; Mouser C1206C105M5RACTU -> 80-C1206C105K4R; Name CAPACITOR-1206-1U -> (none); Tolerance 20% -> 10%; Voltage 50V -> 16V
- D1: Name NEXPERIA-PMEG3030 -> (none)
- H1, H2, H3: value MOUNTING-HOLE-MASK-3MM -> MOUNTING-HOLE-3MM-MASK
- K1: value 9V - 1A -> 9V / 1A; Name CUI-PJ-102AH-TH -> (none)
- K2: Name MOLEX-MINI-SPOX-02-RIGHT-ANGLE -> (none)
- LED1: value Charge -> PURPLE; Name KINGBRIGHT-LED-1206-PURPLE -> (none)
- Q1: Name ST-STN790A-SOT-223 -> (none)
- R1: value 4K7 -> 4k7; symbol tronixio:RESISTOR-1206-4K7 -> tronixio:RESISTOR-1206-4K7-5P; Name RESISTOR-1206-4K7 -> (none)
- R2, R3: symbol tronixio:RESISTOR-1210-0R1 -> tronixio:RESISTOR-1210-0R1-1P; Name RESISTOR-1210-0R1 -> (none)
- R4: value 1K -> 1k; symbol tronixio:RESISTOR-1206-1K -> tronixio:RESISTOR-1206-1K-5P; Name RESISTOR-1206-1K -> (none)
- R5: value 10K -> 10k; symbol tronixio:RESISTOR-1206-10K -> tronixio:RESISTOR-1206-10K-5P; Name RESISTOR-1206-10K -> (none)
- R6: value 36K -> 36k; symbol tronixio:RESISTOR-1206-36K -> tronixio:RESISTOR-1206-36K-5P; Mouser 660-RK73B2BTTD363J -> 660-RK73B2BTTDD363J; Name RESISTOR-1206-36K -> (none)
- TH1: value 10K -> 10k; Name THERMISTOR-NTC-10K -> (none)
- U1: symbol tronixio:TI-BQ2057W-SOIC-08 -> tronixio:TI-BQ2057W-SOIC; Name TI-BQ2057W-SOIC -> (none)

Commit message: Update
Other:
- note added: "*R6: 10k if NTC TH1 Not Populate."
- note removed: "*R6: 10K if NTC TH1 Not Populate."
Changed lines of the file:
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@@
     (effects (font (size 1.27 1.27)) (justify left bottom))
   )
-  (text "*R6: 10K if NTC TH1 Not Populate." (at 181.61 179.07 0)
+  (text "*R6: 10k if NTC TH1 Not Populate." (at 181.61 179.07 0)
     (effects (font (size 1.27 1.27)) (justify left bottom))
   )

Commit message: Update
Parts:
- LED1: value PURPLE -> Charging
Other:
- moved on the sheet: R1
Changed lines of the file:
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@@
     (stroke (width 0) (type solid))
-  )
-  (wire (pts (xy 101.6 97.79) (xy 101.6 99.06))
-    (stroke (width 0) (type default))
   )
   (wire (pts (xy 213.36 86.36) (xy 218.44 86.36))
@@
     (stroke (width 0) (type solid))
   )
-  (wire (pts (xy 101.6 86.36) (xy 101.6 87.63))
+  (wire (pts (xy 101.6 86.36) (xy 101.6 88.9))
     (stroke (width 0) (type default))
   )
@@
   (symbol (lib_id "tronixio:RESISTOR-1206-1K-5P") (at 144.78 78.74 180) (unit 1)
     (in_bom yes) (on_board yes) (dnp no)
-    (property "Reference" "R4" (at 147.32 74.93 0)
-      (effects (font (size 1.15 1.15)) (justify left))
+    (property "Reference" "R4" (at 145.415 74.93 0) (do_not_autoplace)
+      (effects (font (size 1.15 1.15)) (justify right))
     )
     (property "Value" "1k" (at 144.78 78.74 90)
@@
       (effects (font (size 1 1)) hide)
     )
-    (property "Datasheet" "https://www.ti.com/product/BQ2057W" (at 127 101.6 0)
+    (property "Datasheet" "https://www.ti.com/product/BQ2057W/part-details/BQ2057WSN" (at 127 101.6 0)
       (effects (font (size 1 1)) hide)
     )
@@
       (effects (font (size 1 1)) hide)
     )
-    (property "Tolerance" "1%" (at 130.175 64.77 90) (do_not_autoplace)
+    (property "Tolerance" "1%" (at 130.175 67.31 90) (do_not_autoplace)
       (effects (font (size 1.15 1.15)) (justify right))
     )
@@
       (effects (font (size 1.15 1.15)) (justify left))
     )
-    (property "Value" "PURPLE" (at 100.965 104.14 90)
+    (property "Value" "Charging" (at 100.965 104.14 90)
       (effects (font (size 1.15 1.15)) (justify left))
     )
@@
     )
   )
-  (symbol (lib_id "tronixio:RESISTOR-1206-4K7-5P") (at 101.6 92.71 180) (unit 1)
-    (in_bom yes) (on_board yes) (dnp no)
-    (property "Reference" "R1" (at 98.425 88.9 0)
+  (symbol (lib_id "tronixio:RESISTOR-1206-4K7-5P") (at 101.6 93.98 180) (unit 1)
+    (in_bom yes) (on_board yes) (dnp no)
+    (property "Reference" "R1" (at 98.425 90.17 0)
       (effects (font (size 1.15 1.15)) (justify right))
     )
-    (property "Value" "4k7" (at 101.6 92.71 90)
-      (effects (font (size 1.15 1.15)))
-    )
-    (property "Footprint" "tronixio:RESISTOR-SMD-1206" (at 101.6 80.01 0) (do_not_autoplace)
-      (effects (font (size 1 1)) hide)
-    )
-    (property "Datasheet" "" (at 101.6 77.47 0)
-      (effects (font (size 1 1)) hide)
-    )
-    (property "Tolerance" "5%" (at 99.06 91.44 0) (do_not_autoplace)
+    (property "Value" "4k7" (at 101.6 93.98 90)
+      (effects (font (size 1.15 1.15)))
+    )
+    (property "Footprint" "tronixio:RESISTOR-SMD-1206" (at 101.6 81.28 0) (do_not_autoplace)
+      (effects (font (size 1 1)) hide)
+    )
+    (property "Datasheet" "" (at 101.6 78.74 0)
+      (effects (font (size 1 1)) hide)
+    )
+    (property "Tolerance" "5%" (at 99.06 92.71 0) (do_not_autoplace)
       (effects (font (size 1.15 1.15)) (justify left) hide)
     )
-    (property "Mouser" "660-RK73B2BTTDD472J" (at 101.6 77.47 0) (do_not_autoplace)
+    (property "Mouser" "660-RK73B2BTTDD472J" (at 101.6 78.74 0) (do_not_autoplace)
       (effects (font (size 1 1)) hide)
     )
@@
   (symbol (lib_id "tronixio:RESISTOR-1206-10K-5P") (at 160.02 78.74 180) (unit 1)
     (in_bom yes) (on_board yes) (dnp no)
-    (property "Reference" "R5" (at 162.56 74.93 0)
-      (effects (font (size 1.15 1.15)) (justify left))
+    (property "Reference" "R5" (at 160.655 74.93 0) (do_not_autoplace)
+      (effects (font (size 1.15 1.15)) (justify right))
     )
     (property "Value" "10k" (at 160.02 78.74 90)
@@
       (effects (font (size 1 1)) hide)
     )
-    (property "Tolerance" "1%" (at 130.175 69.85 90) (do_not_autoplace)
+    (property "Tolerance" "1%" (at 130.175 72.39 90) (do_not_autoplace)
       (effects (font (size 1.15 1.15)) (justify right))
     )

Commit message: UP
Parts:
- C1: symbol tronixio:CAPACITOR-1206-100N-5P-X7R -> tronixio:CAPACITOR-1206-100N-50V-5P-X7R
- C2: symbol tronixio:CAPACITOR-1206-1U-10P-X7R -> tronixio:CAPACITOR-1206-1U-16V-10P-X7R
- K1: value 9V / 1A -> PJ-102H
- K2: value Battery -> MOLEX-MINI-SPOX-02-RIGHT-ANGLE
- LED1: value Charging -> PURPLE
Connections:
- net VBAT renamed +VBAT
- net VIN renamed +VIN
