File: Kicad/charger/charger.kicad_sch (KiCad schematic)
At the start: 19 parts, among them K1 PJ-102H, K2 MOLEX-MINI-SPOX-02-RIGHT-ANGLE, Q1 STN790A, U1 BQ2057W

Commit message: Up
Parts:
- K1: value PJ-102H -> Charger
- K2: value MOLEX-MINI-SPOX-02-RIGHT-ANGLE -> Battery
- LED1: value PURPLE -> Charging
Other:
- note added: "9V/1A"
Changed lines of the file:
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@@
     (effects (font (size 1.27 1.27)) (justify left bottom))
+  )
+  (text "9V/1A" (at 73.66 86.995 0)
+    (effects (font (size 1.27 1.27)) (justify right bottom))
   )
   (symbol (lib_id "tronixio:RESISTOR-1206-1K-5P") (at 144.78 78.74 180) (unit 1)
@@
     )
     (property "Value" "18650" (at 191.135 78.74 0) (do_not_autoplace)
-      (effects (font (size 1.15 1.15)) (justify right))
+      (effects (font (size 1.15 1.15)) (justify left))
     )
     (property "Footprint" "tronixio:KEYSTONE-1049" (at 190.5 88.9 0) (do_not_autoplace)
@@
       (effects (font (size 1 1)) hide)
     )
-    (property "Tolerance" "1%" (at 130.175 67.31 0) (do_not_autoplace)
-      (effects (font (size 1.15 1.15)) (justify left))
+    (property "Tolerance" "1%" (at 130.175 64.77 90) (do_not_autoplace)
+      (effects (font (size 1.15 1.15)) (justify right))
     )
     (property "Mouser" "660-SR732ETTER100F" (at 147.32 66.04 0) (do_not_autoplace)
@@
       (effects (font (size 1.15 1.15)))
     )
-    (property "Value" "PJ-102H" (at 78.74 91.44 0) (do_not_autoplace)
+    (property "Value" "Charger" (at 78.74 91.44 0) (do_not_autoplace)
       (effects (font (size 1.15 1.15)))
     )
@@
     )
     (property "Value" "18650" (at 191.135 93.98 0) (do_not_autoplace)
-      (effects (font (size 1.15 1.15)) (justify right))
+      (effects (font (size 1.15 1.15)) (justify left))
     )
     (property "Footprint" "tronixio:KEYSTONE-1049" (at 190.5 104.14 0) (do_not_autoplace)
@@
       (effects (font (size 1.15 1.15)) (justify left))
     )
-    (property "Value" "PURPLE" (at 100.965 104.14 0) (do_not_autoplace)
-      (effects (font (size 1.15 1.15)))
+    (property "Value" "Charging" (at 100.965 104.14 90) (do_not_autoplace)
+      (effects (font (size 1.15 1.15)) (justify left))
     )
     (property "Footprint" "tronixio:LED-SMD-1206" (at 111.76 101.6 0) (do_not_autoplace)
@@
       (effects (font (size 1.15 1.15)))
     )
-    (property "Value" "STN790A" (at 144.78 62.23 0) (do_not_autoplace)
-      (effects (font (size 1.15 1.15)) (justify left))
+    (property "Value" "STN790A" (at 144.78 62.23 90) (do_not_autoplace)
+      (effects (font (size 1.15 1.15)))
     )
     (property "Footprint" "tronixio:SOT-223-3" (at 132.08 68.58 0) (do_not_autoplace)
@@
       (effects (font (size 1.15 1.15)))
     )
-    (property "Value" "MOLEX-MINI-SPOX-02-RIGHT-ANGLE" (at 220.98 88.9 0) (do_not_autoplace)
+    (property "Value" "Battery" (at 220.98 88.9 0) (do_not_autoplace)
       (effects (font (size 1.15 1.15)))
     )
@@
     )
     (property "Value" "100n" (at 108.585 104.14 0) (do_not_autoplace)
-      (effects (font (size 1.15 1.15)) (justify left))
+      (effects (font (size 1.15 1.15)) (justify right))
     )
     (property "Footprint" "tronixio:CAPACITOR-SMD-1206" (at 109.22 114.3 0) (do_not_autoplace)
@@
       (effects (font (size 1 1)) hide)
     )
-    (property "Tolerance" "1%" (at 130.175 72.39 0) (do_not_autoplace)
-      (effects (font (size 1.15 1.15)) (justify left))
+    (property "Tolerance" "1%" (at 130.175 69.85 90) (do_not_autoplace)
+      (effects (font (size 1.15 1.15)) (justify right))
     )
     (property "Mouser" "660-SR732ETTER100F" (at 147.32 71.12 0) (do_not_autoplace)
