File: Kicad/charger/charger.kicad_pcb (KiCad board)
At the start: 2 copper layers, 78 x 57 mm, 21 parts, among them IC1 BQ2057W, K1 Charger, K2 Battery, T1 STN790A

Commit message: Update
Parts:
- U1: renamed from IC1; value BQ2057W -> TI-BQ2057W
- renumbered T1 to Q1
Changed lines of the file:
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@@
   (net 0 "")
   (net 1 "GND")
-  (net 2 "Net-(IC1-Pad7)")
-  (net 3 "Net-(IC1-Pad5)")
+  (net 2 "Net-(R2-Pad2)")
+  (net 3 "Net-(R1-Pad2)")
   (net 4 "VBAT")
   (net 5 "VIN")
   (net 6 "Net-(LED1-Pad2)")
   (net 7 "Net-(R4-Pad2)")
-  (net 8 "Net-(IC1-Pad1)")
-  (net 9 "Net-(IC1-Pad4)")
+  (net 8 "Net-(R4-Pad1)")
+  (net 9 "Net-(R5-Pad1)")
   (net 10 "Net-(D1-Pad2)")
   (net 11 "Net-(BT1-Pad1)")
@@
       (net 1 "GND") (pintype "passive") (zone_connect 2))
     (pad "2" smd roundrect (at 1.5 0 270) (size 1.3 1.75) (layers "F.Cu" "F.Paste" "F.Mask") (roundrect_rratio 0.15)
-      (net 9 "Net-(IC1-Pad4)") (pintype "passive") (zone_connect 2))
+      (net 9 "Net-(R5-Pad1)") (pintype "passive") (zone_connect 2))
     (model "${KICAD6_USER_3DMODEL_DIR}/SMD/RESISTOR-1206.wrl"
       (offset (xyz 0 0 0))
@@
     (fp_rect (start 1.2 0.8) (end 1.5 -0.8) (layer "F.Fab") (width 0.1) (fill solid))
     (pad "1" smd roundrect (at -1.5 0 90) (size 1.3 1.75) (layers "F.Cu" "F.Paste" "F.Mask") (roundrect_rratio 0.15)
-      (net 9 "Net-(IC1-Pad4)") (pintype "passive") (zone_connect 2))
+      (net 9 "Net-(R5-Pad1)") (pintype "passive") (zone_connect 2))
     (pad "2" smd roundrect (at 1.5 0 90) (size 1.3 1.75) (layers "F.Cu" "F.Paste" "F.Mask") (roundrect_rratio 0.15)
       (net 5 "VIN") (pintype "passive") (zone_connect 2))
@@
       (net 6 "Net-(LED1-Pad2)") (pintype "passive") (zone_connect 2))
     (pad "2" smd roundrect (at 1.5 0 270) (size 1.3 1.75) (layers "F.Cu" "F.Paste" "F.Mask") (roundrect_rratio 0.15)
-      (net 3 "Net-(IC1-Pad5)") (pintype "passive") (zone_connect 2))
+      (net 3 "Net-(R1-Pad2)") (pintype "passive") (zone_connect 2))
     (model "${KICAD6_USER_3DMODEL_DIR}/SMD/RESISTOR-1206.wrl"
       (offset (xyz 0 0 0))
@@
     (property "Sheetname" "")
     (attr smd)
-    (fp_text reference "T1" (at 0 0 180) (layer "F.Fab")
+    (fp_text reference "Q1" (at 0 0 180) (layer "F.Fab")
       (effects (font (size 1 1) (thickness 0.15)))
     )
@@
       (net 4 "VBAT") (pinfunction "C") (pintype "passive"))
     (pad "3" smd roundrect (at -3.15 2.3 90) (size 2 1.5) (layers "F.Cu" "F.Paste" "F.Mask") (roundrect_rratio 0.15)
-      (net 8 "Net-(IC1-Pad1)") (pinfunction "E") (pintype "passive"))
+      (net 2 "Net-(R2-Pad2)") (pinfunction "E") (pintype "passive"))
     (model "${KICAD6_USER_3DMODEL_DIR}/SMD/SOT-223.wrl"
       (offset (xyz 0 0 0))
@@
       (net 5 "VIN") (pintype "passive") (zone_connect 1))
     (pad "2" smd roundrect (at 1.5 0 90) (size 1.3 2.65) (layers "F.Cu" "F.Paste" "F.Mask") (roundrect_rratio 0.15)
-      (net 8 "Net-(IC1-Pad1)") (pintype "passive") (zone_connect 1))
+      (net 2 "Net-(R2-Pad2)") (pintype "passive") (zone_connect 1))
     (model "${KICAD6_USER_3DMODEL_DIR}/SMD/RESISTOR-1210.wrl"
       (offset (xyz 0 0 0))
@@
     (fp_circle (center 0 0) (end 1.3 0) (layer "F.Fab") (width 0.1) (fill none))
     (pad "1" smd roundrect locked (at -4 0 270) (size 1.2 2) (layers "F.Cu" "F.Paste" "F.Mask") (roundrect_rratio 0.15)
-      (net 9 "Net-(IC1-Pad4)") (pintype "passive") (zone_connect 2))
+      (net 9 "Net-(R5-Pad1)") (pintype "passive") (zone_connect 2))
     (pad "2" smd roundrect locked (at 4 0 270) (size 1.2 2) (layers "F.Cu" "F.Paste" "F.Mask") (roundrect_rratio 0.15)
       (net 1 "GND") (pintype "passive") (zone_connect 1))
@@
       (net 5 "VIN") (pintype "passive") (zone_connect 1))
     (pad "2" smd roundrect (at 1.5 0 90) (size 1.3 2.65) (layers "F.Cu" "F.Paste" "F.Mask") (roundrect_rratio 0.15)
-      (net 8 "Net-(IC1-Pad1)") (pintype "passive") (zone_connect 1))
+      (net 2 "Net-(R2-Pad2)") (pintype "passive") (zone_connect 1))
     (model "${KICAD6_USER_3DMODEL_DIR}/SMD/RESISTOR-1210.wrl"
       (offset (xyz 0 0 0))
@@
     (property "Sheetname" "")
     (attr smd)
-    (fp_text reference "IC1" (at 0 -3.4) (layer "F.Fab")
-      (effects (font (size 1 1) (thickness 0.15)))
-    )
-    (fp_text value "BQ2057W" (at 0 3.4) (layer "F.Fab")
+    (fp_text reference "U1" (at 0 -3.4) (layer "F.Fab")
+      (effects (font (size 1 1) (thickness 0.15)))
+    )
+    (fp_text value "TI-BQ2057W" (at 0 3.4) (layer "F.Fab")
       (effects (font (size 1 1) (thickness 0.15)))
     )
@@
     (fp_arc (start 0.5 -2.2) (mid 0 -1.7) (end -0.5 -2.2) (layer "F.Fab") (width 0.1))
     (pad "1" smd roundrect locked (at -2.7 -1.905) (size 1.8 0.7) (layers "F.Cu" "F.Paste" "F.Mask") (roundrect_rratio 0.15)
-      (net 8 "Net-(IC1-Pad1)") (pinfunction "SNS") (pintype "input"))
+      (net 2 "Net-(R2-Pad2)") (pinfunction "SNS") (pintype "input"))
     (pad "2" smd roundrect locked (at -2.7 -0.635) (size 1.8 0.7) (layers "F.Cu" "F.Paste" "F.Mask") (roundrect_rratio 0.15)
       (net 4 "VBAT") (pinfunction "BAT") (pintype "input"))
@@
       (net 5 "VIN") (pinfunction "VCC") (pintype "power_in"))
     (pad "4" smd roundrect locked (at -2.7 1.905) (size 1.8 0.7) (layers "F.Cu" "F.Paste" "F.Mask") (roundrect_rratio 0.15)
-      (net 9 "Net-(IC1-Pad4)") (pinfunction "TS") (pintype "input"))
+      (net 9 "Net-(R5-Pad1)") (pinfunction "TS") (pintype "input"))
     (pad "5" smd roundrect locked (at 2.7 1.905) (size 1.8 0.7) (layers "F.Cu" "F.Paste" "F.Mask") (roundrect_rratio 0.15)
-      (net 3 "Net-(IC1-Pad5)") (pinfunction "STAT") (pintype "open_collector"))
+      (net 3 "Net-(R1-Pad2)") (pinfunction "STAT") (pintype "open_collector"))
     (pad "6" smd roundrect locked (at 2.7 0.635) (size 1.8 0.7) (layers "F.Cu" "F.Paste" "F.Mask") (roundrect_rratio 0.15)
       (net 1 "GND") (pinfunction "VSS") (pintype "power_in"))
     (pad "7" smd roundrect locked (at 2.7 -0.635) (size 1.8 0.7) (layers "F.Cu" "F.Paste" "F.Mask") (roundrect_rratio 0.15)
-      (net 2 "Net-(IC1-Pad7)") (pinfunction "CC") (pintype "output"))
+      (net 8 "Net-(R4-Pad1)") (pinfunction "CC") (pintype "output"))
     (pad "8" smd roundrect locked (at 2.7 -1.905) (size 1.8 0.7) (layers "F.Cu" "F.Paste" "F.Mask") (roundrect_rratio 0.15)
       (net 5 "VIN") (pinfunction "COMP") (pintype "input"))
@@
     (fp_rect (start -1.5 0.8) (end -1.2 -0.8) (layer "F.Fab") (width 0.1) (fill solid))
     (pad "1" smd roundrect (at -1.5 0 90) (size 1.3 1.75) (layers "F.Cu" "F.Paste" "F.Mask") (roundrect_rratio 0.15)
-      (net 2 "Net-(IC1-Pad7)") (pintype "passive") (zone_connect 2))
+      (net 8 "Net-(R4-Pad1)") (pintype "passive") (zone_connect 2))
     (pad "2" smd roundrect (at 1.5 0 90) (size 1.3 1.75) (layers "F.Cu" "F.Paste" "F.Mask") (roundrect_rratio 0.15)
       (net 7 "Net-(R4-Pad2)") (pintype "passive") (zone_connect 2))
@@
   )
   (gr_text "TBOT Charger" (at 135 96.5) (layer "B.SilkS")
-    (effects (font (size 1.5 1.5) (thickness 0.25)) (justify left mirror))
+    (effects (font (size 1.5 1.5) (thickness 0.3)) (justify left mirror))
   )
   (gr_text "(CC) - BY-SA" (at 162 50.25) (layer "B.SilkS")
@@
   )
   (gr_text "TBOT Charger" (at 143 87) (layer "F.SilkS")
-    (effects (font (size 1.5 1.5) (thickness 0.25)) (justify left))
+    (effects (font (size 1.5 1.5) (thickness 0.3)) (justify left))
   )
   (gr_text "www.tronix.io" (at 135 87) (layer "F.SilkS")
@@
     (style (thickness 0.1) (arrow_length 1) (text_position_mode 0) (extension_height 0.58642) (extension_offset 0.5) keep_text_aligned)
   )
-  (segment (start 132.5 76) (end 132.5 74.5) (width 0.5) (layer "F.Cu") (net 2))
-  (segment (start 141.7 78.865) (end 139.635 78.865) (width 0.5) (layer "F.Cu") (net 2))
-  (via (at 139.5 78.865) (size 0.6) (drill 0.3) (layers "F.Cu" "B.Cu") (net 2))
-  (via (at 132.5 76) (size 0.6) (drill 0.3) (layers "F.Cu" "B.Cu") (net 2))
-  (segment (start 132.5 76) (end 135.365 78.865) (width 0.5) (layer "B.Cu") (net 2))
-  (segment (start 139.5 78.865) (end 135.365 78.865) (width 0.5) (layer "B.Cu") (net 2))
+  (segment (start 136.3 77.595) (end 136.3 74.5) (width 0.5) (layer "F.Cu") (net 2))
+  (segment (start 141.3 71.5) (end 145.5 71.5) (width 1) (layer "F.Cu") (net 2))
+  (segment (start 145.5 71.5) (end 149.5 71.5) (width 1) (layer "F.Cu") (net 2))
+  (segment (start 141.3 74.5) (end 141.3 71.65) (width 0.5) (layer "F.Cu") (net 2))
+  (via (at 141.3 74.5) (size 0.6) (drill 0.3) (layers "F.Cu" "B.Cu") (net 2))
+  (via (at 136.3 74.5) (size 0.6) (drill 0.3) (layers "F.Cu" "B.Cu") (net 2))
+  (segment (start 136.3 74.5) (end 141.3 74.5) (width 0.5) (layer "B.Cu") (net 2))
   (segment (start 147.75 82.75) (end 148.5 82) (width 0.5) (layer "F.Cu") (net 3))
   (segment (start 144.25 82.75) (end 147.75 82.75) (width 0.5) (layer "F.Cu") (net 3))
@@
   (segment (start 148.5 78) (end 151.5 78) (width 0.5) (layer "F.Cu") (net 6))
   (segment (start 132.5 71.5) (end 136.7 71.5) (width 0.5) (layer "F.Cu") (net 7))
-  (segment (start 136.3 77.595) (end 136.3 74.5) (width 0.5) (layer "F.Cu") (net 8))
-  (segment (start 141.3 71.5) (end 145.5 71.5) (width 1) (layer "F.Cu") (net 8))
-  (segment (start 145.5 71.5) (end 149.5 71.5) (width 1) (layer "F.Cu") (net 8))
-  (segment (start 141.3 74.5) (end 141.3 71.65) (width 0.5) (layer "F.Cu") (net 8))
-  (via (at 141.3 74.5) (size 0.6) (drill 0.3) (layers "F.Cu" "B.Cu") (net 8))
-  (via (at 136.3 74.5) (size 0.6) (drill 0.3) (layers "F.Cu" "B.Cu") (net 8))
-  (segment (start 136.3 74.5) (end 141.3 74.5) (width 0.5) (layer "B.Cu") (net 8))
+  (segment (start 132.5 76) (end 132.5 74.5) (width 0.5) (layer "F.Cu") (net 8))
+  (segment (start 141.7 78.865) (end 139.635 78.865) (width 0.5) (layer "F.Cu") (net 8))
+  (via (at 139.5 78.865) (size 0.6) (drill 0.3) (layers "F.Cu" "B.Cu") (net 8))
+  (via (at 132.5 76) (size 0.6) (drill 0.3) (layers "F.Cu" "B.Cu") (net 8))
+  (segment (start 132.5 76) (end 135.365 78.865) (width 0.5) (layer "B.Cu") (net 8))
+  (segment (start 139.5 78.865) (end 135.365 78.865) (width 0.5) (layer "B.Cu") (net 8))
   (segment (start 133.75 82.75) (end 130.25 82.75) (width 0.5) (layer "F.Cu") (net 9))
   (segment (start 136.3 81.405) (end 135.095 81.405) (width 0.5) (layer "F.Cu") (net 9))

Commit message: Update
Parts:
- TH1: footprint tronixio:THERMISTOR -> tronixio:THERMISTOR-SMD
- U1: value TI-BQ2057W -> BQ2057W

Commit message: Update
Parts:
- C1, C2: footprint tronixio:CAPACITOR-1206 -> tronixio:CAPACITOR-SMD-1206
- H1, H2, H3: footprint tronixio:M3-MASK -> tronixio:MOUNTING-HOLE-3MM-MASK
- LED1: footprint tronixio:LED-1206 -> tronixio:LED-SMD-1206
- R1, R4, R5, R6: footprint tronixio:RESISTOR-1206 -> tronixio:RESISTOR-SMD-1206
- R2, R3: footprint tronixio:RESISTOR-1210 -> tronixio:RESISTOR-SMD-1210

Commit message: Update
Parts:
- K1: value Charger -> 9V - 1A

Commit message: Update
Parts:
- H1, H2, H3: value MOUNTING-HOLE-MASK-3MM -> MOUNTING-HOLE-3MM-MASK
- K1: value 9V - 1A -> 9V / 1A
- LED1: value Charging -> PURPLE
- R1: value 4K7 -> 4k7
- R4: value 1K -> 1k
- R5, TH1: value 10K -> 10k
- R6: value 36K -> 36k
Routing:
- net VBAT: track 46.4 -> 40.1 mm

Commit message: Update
Parts:
- LED1: value PURPLE -> Charging
Changed lines of the file:
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@@
     (zone_connect 2)
     (attr smd)
-    (fp_text reference "D1" (at 4 0 90) (layer "F.Fab")
-        (effects (font (size 1 1) (thickness 0.15)))
-    )
-    (fp_text value "PMEG3030" (at 0 -2.5 90) (layer "F.Fab")
+    (fp_text reference "D1" (at 0 0 90) (layer "F.SilkS") hide
+        (effects (font (size 1 1) (thickness 0.15)))
+    )
+    (fp_text value "PMEG3030" (at 0 2.5 90) (layer "F.Fab")
         (effects (font (size 1 1) (thickness 0.15)))
     )
@@
     (zone_connect 2)
     (attr smd)
-    (fp_text reference "R6" (at 0 -2 -90) (layer "F.Fab")
+    (fp_text reference "R6" (at 0 -2 -90) (layer "F.SilkS") hide
         (effects (font (size 1 1) (thickness 0.15)))
     )
@@
     (zone_connect 2)
     (attr smd)
-    (fp_text reference "R5" (at 0 -2 90) (layer "F.Fab")
+    (fp_text reference "R5" (at 0 -2 90) (layer "F.SilkS") hide
         (effects (font (size 1 1) (thickness 0.15)))
     )
@@
     (property "ki_description" "Unpolarized Capacitor")
     (attr smd)
-    (fp_text reference "C1" (at 0 -2 -90) (layer "F.Fab")
+    (fp_text reference "C1" (at 0 -2 -90) (layer "F.SilkS") hide
         (effects (font (size 1 1) (thickness 0.15)))
     )
@@
     (zone_connect 2)
     (attr smd)
-    (fp_text reference "R1" (at 0 -2 -90) (layer "F.Fab")
+    (fp_text reference "R1" (at 0 -2 -90) (layer "F.SilkS") hide
         (effects (font (size 1 1) (thickness 0.15)))
     )
@@
     (property "ki_description" "DC Barrel Jack with an Internal Switch")
     (attr through_hole)
-    (fp_text reference "K1" (at 1 5.4625 180) (layer "F.Fab")
-        (effects (font (size 1 1) (thickness 0.15)))
-    )
-    (fp_text value "9V / 1A" (at -1 5.4625 180) (layer "F.Fab")
+    (fp_text reference "K1" (at 0 -2.5 90) (layer "F.SilkS") hide
+        (effects (font (size 1 1) (thickness 0.15)))
+    )
+    (fp_text value "9V / 1A" (at 0 15 90) (layer "F.Fab")
         (effects (font (size 1 1) (thickness 0.15)))
     )
@@
     (property "ki_description" "Unpolarized Capacitor")
     (attr smd)
-    (fp_text reference "C2" (at 0 -2 -90) (layer "F.Fab")
+    (fp_text reference "C2" (at 0 -2 -90) (layer "F.SilkS") hide
         (effects (font (size 1 1) (thickness 0.15)))
     )
@@
     (property "ki_description" "Medium current, high performance, low voltage PNP transistor")
     (attr smd)
-    (fp_text reference "Q1" (at 0 0 180) (layer "F.Fab")
-        (effects (font (size 1 1) (thickness 0.15)))
-    )
-    (fp_text value "STN790A" (at -4 0 180) (layer "F.Fab")
+    (fp_text reference "Q1" (at 0 -4.5 90) (layer "F.SilkS") hide
+        (effects (font (size 1 1) (thickness 0.15)))
+    )
+    (fp_text value "STN790A" (at 0 4.5 90) (layer "F.Fab")
         (effects (font (size 1 1) (thickness 0.15)))
     )
@@
     (property "ki_description" "Resistor")
     (attr smd)
-    (fp_text reference "R2" (at 0 -2.5 90) (layer "F.Fab")
+    (fp_text reference "R2" (at 0 -2.5 90) (layer "F.SilkS") hide
         (effects (font (size 1 1) (thickness 0.15)))
     )
@@
     (zone_connect 2)
     (attr smd)
-    (fp_text reference "TH1" (at 0 -3.81 180) (layer "F.Fab")
-        (effects (font (size 1 1) (thickness 0.15)))
-    )
-    (fp_text value "10k" (at 0 3.81 180) (layer "F.Fab")
+    (fp_text reference "TH1" (at 0 -3 180) (layer "F.SilkS") hide
+        (effects (font (size 1 1) (thickness 0.15)))
+    )
+    (fp_text value "10k" (at 0 3 180) (layer "F.Fab")
         (effects (font (size 1 1) (thickness 0.15)))
     )
@@
     (zone_connect 2)
     (attr smd)
-    (fp_text reference "LED1" (at 0 -2 90) (layer "F.Fab")
-        (effects (font (size 1 1) (thickness 0.15)))
-    )
-    (fp_text value "PURPLE" (at 0 2 90) (layer "F.Fab")
+    (fp_text reference "LED1" (at 0 -2 90) (layer "F.SilkS") hide
+        (effects (font (size 1 1) (thickness 0.15)))
+    )
+    (fp_text value "Charging" (at 0 2 90) (layer "F.Fab")
         (effects (font (size 1 1) (thickness 0.15)))
     )
@@
     (property "ki_keywords" "538-22-05-7025 / 538-50-37-5023 / 538-08-70-1039-CT")
     (attr through_hole)
-    (fp_text reference "K2" (at -0.5 -4.5) (layer "F.Fab")
-        (effects (font (size 1 1) (thickness 0.15)))
-    )
-    (fp_text value "Battery" (at -0.5 -3) (layer "F.Fab")
+    (fp_text reference "K2" (at -1.5 -8) (layer "F.SilkS") hide
+        (effects (font (size 1 1) (thickness 0.15)))
+    )
+    (fp_text value "Battery" (at -1.5 3) (layer "F.Fab")
+        (effects (font (size 1 1) (thickness 0.15)))
+    )
+    (fp_text user "1" (at 2 0.2) (layer "F.Fab")
         (effects (font (size 1 1) (thickness 0.15)))
     )
     (fp_text user "${REFERENCE}" (at -1.25 -8) (layer "F.Fab")
-        (effects (font (size 1 1) (thickness 0.15)))
-    )
-    (fp_text user "1" (at 1.9 0.1 unlocked) (layer "F.Fab")
         (effects (font (size 1 1) (thickness 0.15)))
     )
@@
     (property "ki_description" "Resistor")
     (attr smd)
-    (fp_text reference "R3" (at 0 -2.5 90) (layer "F.Fab")
+    (fp_text reference "R3" (at 0 -2.5 90) (layer "F.SilkS") hide
         (effects (font (size 1 1) (thickness 0.15)))
     )
@@
     (property "ki_description" "Low Dropout linear 2-cell Li-ion charge controller with AutoCompTM, 8.4V")
     (attr smd)
-    (fp_text reference "U1" (at 0 -3.4) (layer "F.Fab")
-        (effects (font (size 1 1) (thickness 0.15)))
-    )
-    (fp_text value "BQ2057W" (at 0 3.4) (layer "F.Fab")
+    (fp_text reference "U1" (at 0 -3.5) (layer "F.SilkS") hide
+        (effects (font (size 1 1) (thickness 0.15)))
+    )
+    (fp_text value "BQ2057W" (at 0 3.5) (layer "F.Fab")
         (effects (font (size 1 1) (thickness 0.15)))
     )
@@
     (zone_connect 2)
     (attr smd)
-    (fp_text reference "R4" (at 0 -2 90) (layer "F.Fab")
+    (fp_text reference "R4" (at 0 -2 90) (layer "F.SilkS") hide
         (effects (font (size 1 1) (thickness 0.15)))
     )
@@
     (property "Sheetfile" "charger.kicad_sch")
     (property "Sheetname" "")
-    (attr exclude_from_pos_files)
-    (fp_text reference "H3" (at 0 4.2) (layer "B.Fab") hide
+    (attr exclude_from_pos_files exclude_from_bom)
+    (fp_text reference "H3" (at 0 4.5) (layer "B.Fab") hide
         (effects (font (size 1 1) (thickness 0.15)) (justify mirror))
     )
-    (fp_text value "MOUNTING-HOLE-3MM-MASK" (at 0 -4.2) (layer "B.Fab") hide
+    (fp_text value "MOUNTING-HOLE-3MM-MASK" (at 0 -4.5) (layer "B.Fab") hide
         (effects (font (size 1 1) (thickness 0.15)) (justify mirror))
     )
     (fp_circle (center 0 0) (end 3.2 0)
-      (stroke (width 0.15) (type solid)) (fill none) (layer "B.SilkS"))
+      (stroke (width 0.2) (type solid)) (fill none) (layer "B.SilkS"))
     (fp_circle (center 0 0) (end 3.2 0)
-      (stroke (width 0.15) (type solid)) (fill none) (layer "F.SilkS"))
+      (stroke (width 0.2) (type solid)) (fill none) (layer "F.SilkS"))
     (fp_circle (center 0 0) (end 3.2 0)
       (stroke (width 0.05) (type solid)) (fill none) (layer "B.CrtYd"))
@@
     (property "Sheetfile" "charger.kicad_sch")
     (property "Sheetname" "")
-    (attr exclude_from_pos_files)
-    (fp_text reference "H1" (at 0 4.2 270) (layer "B.Fab") hide
+    (attr exclude_from_pos_files exclude_from_bom)
+    (fp_text reference "H1" (at 0 4.5 270) (layer "B.Fab") hide
         (effects (font (size 1 1) (thickness 0.15)) (justify mirror))
     )
-    (fp_text value "MOUNTING-HOLE-3MM-MASK" (at 0 -4.2 270) (layer "B.Fab") hide
+    (fp_text value "MOUNTING-HOLE-3MM-MASK" (at 0 -4.5 270) (layer "B.Fab") hide
         (effects (font (size 1 1) (thickness 0.15)) (justify mirror))
     )
     (fp_circle (center 0 0) (end 3.2 0)
-      (stroke (width 0.15) (type solid)) (fill none) (layer "B.SilkS"))
+      (stroke (width 0.2) (type solid)) (fill none) (layer "B.SilkS"))
     (fp_circle (center 0 0) (end 3.2 0)
-      (stroke (width 0.15) (type solid)) (fill none) (layer "F.SilkS"))
+      (stroke (width 0.2) (type solid)) (fill none) (layer "F.SilkS"))
     (fp_circle (center 0 0) (end 3.2 0)
       (stroke (width 0.05) (type solid)) (fill none) (layer "B.CrtYd"))
@@
     (property "Sheetfile" "charger.kicad_sch")
     (property "Sheetname" "")
-    (attr exclude_from_pos_files)
-    (fp_text reference "H2" (at 0 4.2 270) (layer "B.Fab") hide
+    (attr exclude_from_pos_files exclude_from_bom)
+    (fp_text reference "H2" (at 0 4.5 270) (layer "B.Fab") hide
         (effects (font (size 1 1) (thickness 0.15)) (justify mirror))
     )
-    (fp_text value "MOUNTING-HOLE-3MM-MASK" (at 0 -4.2 270) (layer "B.Fab") hide
+    (fp_text value "MOUNTING-HOLE-3MM-MASK" (at 0 -4.5 270) (layer "B.Fab") hide
         (effects (font (size 1 1) (thickness 0.15)) (justify mirror))
     )
     (fp_circle (center 0 0) (end 3.2 0)
-      (stroke (width 0.15) (type solid)) (fill none) (layer "B.SilkS"))
+      (stroke (width 0.2) (type solid)) (fill none) (layer "B.SilkS"))
     (fp_circle (center 0 0) (end 3.2 0)
-      (stroke (width 0.15) (type solid)) (fill none) (layer "F.SilkS"))
+      (stroke (width 0.2) (type solid)) (fill none) (layer "F.SilkS"))
     (fp_circle (center 0 0) (end 3.2 0)
       (stroke (width 0.05) (type solid)) (fill none) (layer "B.CrtYd"))
@@
     (property "ki_description" "THM Holder for Dual 18650 Batteries")
     (attr through_hole)
-    (fp_text reference "BT1" (at 1 0 180) (layer "B.Fab")
+    (fp_text reference "BT1" (at 0 2 270) (layer "B.SilkS") hide
         (effects (font (size 1 1) (thickness 0.15)) (justify mirror))
     )
-    (fp_text value "18650" (at -1 0 180) (layer "B.Fab")
+    (fp_text value "18650" (at 0 -2 270) (layer "B.Fab")
         (effects (font (size 1 1) (thickness 0.15)) (justify mirror))
     )

Commit message: Update
Routing:
- net VBAT: vias 48 -> 46
Changed lines of the file:
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@@
   (via (at 156 67) (size 1) (drill 0.5) (layers "F.Cu" "B.Cu") (net 4))
   (via (at 128 61) (size 1) (drill 0.5) (layers "F.Cu" "B.Cu") (net 4))
-  (via (at 142 63) (size 1) (drill 0.5) (layers "F.Cu" "B.Cu") (net 4))
   (via (at 116 58) (size 1) (drill 0.5) (layers "F.Cu" "B.Cu") (net 4))
   (via (at 150 67) (size 1) (drill 0.5) (layers "F.Cu" "B.Cu") (net 4))
@@
   (via (at 128 63) (size 1) (drill 0.5) (layers "F.Cu" "B.Cu") (net 4))
   (via (at 133 63) (size 1) (drill 0.5) (layers "F.Cu" "B.Cu") (net 4))
-  (via (at 136 63) (size 1) (drill 0.5) (layers "F.Cu" "B.Cu") (net 4))
   (via (at 130.5 63) (size 1) (drill 0.5) (layers "F.Cu" "B.Cu") (net 4))
   (via (at 125 63) (size 1) (drill 0.5) (layers "F.Cu" "B.Cu") (net 4))
