File: Kicad/charger/charger.kicad_pcb (KiCad board)
At the start: 2 copper layers, 78 x 57 mm, 21 parts, among them K1 9V / 1A, K2 Battery, Q1 STN790A, U1 BQ2057W

Commit message: UP
Parts:
- K1: value 9V / 1A -> PJ-102H
- K2: value Battery -> MOLEX-MINI-SPOX-02-RIGHT-ANGLE
- LED1: value Charging -> PURPLE
Connections:
- net VBAT renamed +VBAT
- net VIN renamed +VIN

Commit message: Update charger.kicad_pcb
Parts:
- K1: value PJ-102H -> Charger
- K2: value MOLEX-MINI-SPOX-02-RIGHT-ANGLE -> Battery
- LED1: value PURPLE -> Charging
Other:
- board text removed: "Charging"
Changed lines of the file:
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@@
     (zone_connect 2)
     (attr smd)
-    (fp_text reference "D1" (at 0 2.5 90) (layer "F.SilkS") hide
-        (effects (font (size 1 1) (thickness 0.15)))
-    )
-    (fp_text value "PMEG3030" (at 0 2.5 90) (layer "F.Fab")
+    (fp_text reference "D1" (at 0 -2.5 90) (layer "F.SilkS") hide
+        (effects (font (size 1 1) (thickness 0.15)))
+    )
+    (fp_text value "PMEG3030" (at 0 -2.5 90) (layer "F.Fab")
         (effects (font (size 1 1) (thickness 0.15)))
     )
@@
     (zone_connect 2)
     (attr smd)
-    (fp_text reference "R6" (at 0 2 -90) (layer "F.SilkS") hide
-        (effects (font (size 1 1) (thickness 0.15)))
-    )
-    (fp_text value "36k" (at 0 2 -90) (layer "F.Fab")
+    (fp_text reference "R6" (at 3.5 0 -90) (layer "F.SilkS") hide
+        (effects (font (size 1 1) (thickness 0.15)))
+    )
+    (fp_text value "36k" (at 4 0 -90) (layer "F.Fab")
         (effects (font (size 1 1) (thickness 0.15)))
     )
@@
     (zone_connect 2)
     (attr smd)
-    (fp_text reference "R5" (at 0 2 90) (layer "F.SilkS") hide
-        (effects (font (size 1 1) (thickness 0.15)))
-    )
-    (fp_text value "10k" (at 0 2 90) (layer "F.Fab")
+    (fp_text reference "R5" (at 0 0 90) (layer "F.SilkS") hide
+        (effects (font (size 1 1) (thickness 0.15)))
+    )
+    (fp_text value "10k" (at 0 0 90) (layer "F.Fab")
         (effects (font (size 1 1) (thickness 0.15)))
     )
@@
     (property "ki_description" "Unpolarized Capacitor")
     (attr smd)
-    (fp_text reference "C1" (at 0 2 -90) (layer "F.SilkS") hide
-        (effects (font (size 1 1) (thickness 0.15)))
-    )
-    (fp_text value "100n" (at 0 2 -90) (layer "F.Fab")
+    (fp_text reference "C1" (at 0 0 -90) (layer "F.SilkS") hide
+        (effects (font (size 1 1) (thickness 0.15)))
+    )
+    (fp_text value "100n" (at 0 0 -90) (layer "F.Fab")
         (effects (font (size 1 1) (thickness 0.15)))
     )
@@
     (zone_connect 2)
     (attr smd)
-    (fp_text reference "R1" (at 0 2 -90) (layer "F.SilkS") hide
-        (effects (font (size 1 1) (thickness 0.15)))
-    )
-    (fp_text value "4k7" (at 0 2 -90) (layer "F.Fab")
+    (fp_text reference "R1" (at 0 0 -90) (layer "F.SilkS") hide
+        (effects (font (size 1 1) (thickness 0.15)))
+    )
+    (fp_text value "4k7" (at 0 0 -90) (layer "F.Fab")
         (effects (font (size 1 1) (thickness 0.15)))
     )
@@
     (property "Sheetname" "")
     (attr through_hole)
-    (fp_text reference "K1" (at 0 15 90) (layer "F.SilkS") hide
-        (effects (font (size 1 1) (thickness 0.15)))
-    )
-    (fp_text value "PJ-102H" (at 0 15 90) (layer "F.Fab")
+    (fp_text reference "K1" (at 5.5 8.4625 180) (layer "F.SilkS") hide
+        (effects (font (size 1 1) (thickness 0.15)))
+    )
+    (fp_text value "Charger" (at 5.5 8.9625 180) (layer "F.Fab")
         (effects (font (size 1 1) (thickness 0.15)))
     )
@@
     (property "ki_description" "Unpolarized Capacitor")
     (attr smd)
-    (fp_text reference "C2" (at 0 2 -90) (layer "F.SilkS") hide
-        (effects (font (size 1 1) (thickness 0.15)))
-    )
-    (fp_text value "1µ" (at 0 2 -90) (layer "F.Fab")
+    (fp_text reference "C2" (at 0 0 -90) (layer "F.SilkS") hide
+        (effects (font (size 1 1) (thickness 0.15)))
+    )
+    (fp_text value "1µ" (at 0 0 -90) (layer "F.Fab")
         (effects (font (size 1 1) (thickness 0.15)))
     )
@@
     (property "ki_description" "Medium current, high performance, low voltage PNP transistor")
     (attr smd)
-    (fp_text reference "Q1" (at 0 4.5 90) (layer "F.SilkS") hide
-        (effects (font (size 1 1) (thickness 0.15)))
-    )
-    (fp_text value "STN790A" (at 0 4.5 90) (layer "F.Fab")
+    (fp_text reference "Q1" (at -5.65 0 180) (layer "F.SilkS") hide
+        (effects (font (size 1 1) (thickness 0.15)))
+    )
+    (fp_text value "STN790A" (at -5.65 0 180) (layer "F.Fab")
         (effects (font (size 1 1) (thickness 0.15)))
     )
@@
     (property "ki_description" "Resistor")
     (attr smd)
-    (fp_text reference "R2" (at 0 2.5 90) (layer "F.SilkS") hide
-        (effects (font (size 1 1) (thickness 0.15)))
-    )
-    (fp_text value "0Ω1" (at 0 2.5 90) (layer "F.Fab")
+    (fp_text reference "R2" (at 0 0 90) (layer "F.SilkS") hide
+        (effects (font (size 1 1) (thickness 0.15)))
+    )
+    (fp_text value "0Ω1" (at 0 0 90) (layer "F.Fab")
         (effects (font (size 1 1) (thickness 0.15)))
     )
@@
         (effects (font (size 1 1) (thickness 0.15)))
     )
-    (fp_text value "PURPLE" (at 0 2 90) (layer "F.Fab")
-        (effects (font (size 1 1) (thickness 0.15)))
+    (fp_text value "Charging" (at 0 2 90) (layer "F.SilkS")
+        (effects (font (size 0.8 0.8) (thickness 0.15)))
     )
     (fp_line (start -0.6 -0.9) (end 0.6 -0.9)
@@
     (property "ki_keywords" "538-22-05-7025 / 538-50-37-5023 / 538-08-70-1039-CT")
     (attr through_hole)
-    (fp_text reference "K2" (at 0 3) (layer "F.SilkS") hide
-        (effects (font (size 1 1) (thickness 0.15)))
-    )
-    (fp_text value "MOLEX-MINI-SPOX-02-RIGHT-ANGLE" (at 0 3) (layer "F.Fab")
+    (fp_text reference "K2" (at -1 -4) (layer "F.SilkS") hide
+        (effects (font (size 1 1) (thickness 0.15)))
+    )
+    (fp_text value "Battery" (at -0.5 -4.5) (layer "F.Fab")
         (effects (font (size 1 1) (thickness 0.15)))
     )
@@
     (property "ki_description" "Low Dropout linear 2-cell Li-ion charge controller with AutoCompTM, 8.4V")
     (attr smd)
-    (fp_text reference "U1" (at 0 3.5) (layer "F.SilkS") hide
+    (fp_text reference "U1" (at 0 0) (layer "F.SilkS") hide
         (effects (font (size 1 1) (thickness 0.15)))
     )
@@
     (zone_connect 2)
     (attr smd)
-    (fp_text reference "R4" (at 0 2 90) (layer "F.SilkS") hide
-        (effects (font (size 1 1) (thickness 0.15)))
-    )
-    (fp_text value "1k" (at 0 2 90) (layer "F.Fab")
+    (fp_text reference "R4" (at 0 0 90) (layer "F.SilkS") hide
+        (effects (font (size 1 1) (thickness 0.15)))
+    )
+    (fp_text value "1k" (at 0 0 90) (layer "F.Fab")
         (effects (font (size 1 1) (thickness 0.15)))
     )
@@
     (property "Sheetfile" "charger.kicad_sch")
     (property "Sheetname" "")
-    (attr exclude_from_pos_files)
+    (attr exclude_from_pos_files exclude_from_bom)
     (fp_text reference "H3" (at 0 -4.5 unlocked) (layer "B.Fab") hide
         (effects (font (size 1 1) (thickness 0.15)) (justify mirror))
@@
     (property "Sheetfile" "charger.kicad_sch")
     (property "Sheetname" "")
-    (attr exclude_from_pos_files)
+    (attr exclude_from_pos_files exclude_from_bom)
     (fp_text reference "H1" (at 0 -4.5 270 unlocked) (layer "B.Fab") hide
         (effects (font (size 1 1) (thickness 0.15)) (justify mirror))
@@
     (property "Sheetfile" "charger.kicad_sch")
     (property "Sheetname" "")
-    (attr exclude_from_pos_files)
+    (attr exclude_from_pos_files exclude_from_bom)
     (fp_text reference "H2" (at 0 -4.5 270 unlocked) (layer "B.Fab") hide
         (effects (font (size 1 1) (thickness 0.15)) (justify mirror))
@@
     (property "ki_description" "THM Holder for Dual 18650 Batteries")
     (attr through_hole)
-    (fp_text reference "BT1" (at 0 0 270) (layer "B.SilkS") hide
+    (fp_text reference "BT1" (at 0 0) (layer "B.SilkS") hide
         (effects (font (size 1 1) (thickness 0.15)) (justify mirror))
     )
-    (fp_text value "18650" (at 0 0 270) (layer "B.Fab")
+    (fp_text value "18650" (at 0 0) (layer "B.Fab")
         (effects (font (size 1 1) (thickness 0.15)) (justify mirror))
     )
@@
     (effects (font (size 1.5 1.5) (thickness 0.2)) (justify right))
   )
-  (gr_text "Charging" (at 154 79.5 90) (layer "F.SilkS")
-    (effects (font (size 0.8 0.8) (thickness 0.15)))
-  )
   (gr_text "*" (at 149.5 73.4) (layer "F.SilkS")
     (effects (font (size 1.3 1.3) (thickness 0.15)))
@@
     (pts (xy 100 101) (xy 100 96.5))
     (height -1)
-    (gr_text "4.50 mm" (at 97 98.75 90) (layer "Dwgs.User")
+    (gr_text "4.50 mm" (at 97.5 98.75 90) (layer "Dwgs.User")
       (effects (font (size 1 1) (thickness 0.15)))
     )
