File: Kicad/charger/main.kicad_sch (KiCad schematic)
At the start: 19 parts, among them K1 Charger, K2 Battery, Q1 STN790A, U1 BQ2057W

Commit message: Up charger
Other:
- note added: "R2 (0Ω1): ICharge ~1.25A."
- note removed: "R2 (0Ω1): ICharge ~1A."
Changed lines of the file:
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@@
     (stroke (width 0) (type solid))
   )
-  (text "R2 (0Ω1): ICharge ~1A." (at 181.61 173.99 0)
+  (text "R2 (0Ω1): ICharge ~1.25A." (at 181.61 173.99 0)
     (effects (font (size 1.27 1.27)) (justify left bottom))
   )

Commit message: Update
Parts:
- D1: symbol tronixio:NEXPERIA-PMEG3030 -> tronixio:NEXPERIA-PMEG3030-SOD
Changed lines of the file:
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@@
     )
   )
-  (symbol (lib_id "tronixio:NEXPERIA-PMEG3030") (at 99.06 66.04 180) (unit 1)
+  (symbol (lib_id "tronixio:NEXPERIA-PMEG3030-SOD") (at 99.06 66.04 180) (unit 1)
     (in_bom yes) (on_board yes) (dnp no)
     (property "Reference" "D1" (at 99.06 63.5 0) (do_not_autoplace)
