File: Kicad/ir-line/ir-line.kicad_sch (KiCad schematic)
At the start: 28 parts, among them IC1 VISHAY-CNY70, IC2 VISHAY-CNY70, IC3 VISHAY-CNY70, IC4 VISHAY-CNY70, IC5 VISHAY-CNY70, IC6 TPS92612, IC7 TPS92612, K1 FRONT #1, K2 FRONT #2

Commit message: Update IR-LINE
Parts:
- K1, K2: footprint tronixio:zzMOLEX-532530570 -> tronixio:MOLEX-532530570
Other:
- note added: "(10n)"
Changed lines of the file:
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@@
     (stroke (width 0) (type default) (color 0 0 0 0))
+  )
+  (text "(10n)" (at 71.12 45.72 0)
+    (effects (font (size 1.27 1.27)) (justify left bottom))
   )
   (text "Iled = 0.098 / 4.7 = 20mA" (at 213.36 179.07 180)
     (effects (font (size 1.27 1.27)) (justify right bottom))
+  )
+  (text "(10n)" (at 154.94 43.18 0)
+    (effects (font (size 1.27 1.27)) (justify left bottom))
+  )
+  (text "(10n)" (at 154.94 78.74 0)
+    (effects (font (size 1.27 1.27)) (justify left bottom))
+  )
+  (text "(10n)" (at 154.94 109.22 0)
+    (effects (font (size 1.27 1.27)) (justify left bottom))
+  )
+  (text "(10n)" (at 68.58 78.74 0)
+    (effects (font (size 1.27 1.27)) (justify left bottom))
   )
   (global_label "LED 234" (shape input) (at 165.1 48.26 0)
@@
       (effects (font (size 1.15 1.15)))
     )
-    (property "Footprint" "tronixio:zzMOLEX-532530570" (id 2) (at 48.26 167.64 0)
+    (property "Footprint" "tronixio:MOLEX-532530570" (id 2) (at 48.26 167.64 0)
       (effects (font (size 1 1)) hide)
     )
@@
       (effects (font (size 1.15 1.15)))
     )
-    (property "Footprint" "tronixio:zzMOLEX-532530570" (id 2) (at 86.36 167.64 0)
+    (property "Footprint" "tronixio:MOLEX-532530570" (id 2) (at 86.36 167.64 0)
       (effects (font (size 1 1)) hide)
     )
@@
     )
     (path "/3759919d-bb2c-496b-a4ee-88cd6f0e1c67"
-      (reference "K1") (unit 1) (value "FRONT #1") (footprint "tronixio:zzMOLEX-532530570")
+      (reference "K1") (unit 1) (value "FRONT #1") (footprint "tronixio:MOLEX-532530570")
     )
     (path "/a5acb729-f959-4924-b1b7-57693519c813"
-      (reference "K2") (unit 1) (value "FRONT #2") (footprint "tronixio:zzMOLEX-532530570")
+      (reference "K2") (unit 1) (value "FRONT #2") (footprint "tronixio:MOLEX-532530570")
     )
     (path "/c7c884dd-0f5e-46e2-a90a-dcd0218e54b8"

Commit message: Update IR-LINE
Parts:
- IC1, IC2, IC3, IC4, IC5: footprint tronixio:zzVISHAY-CNY70 -> tronixio:VISHAY-CNY70
Changed lines of the file:
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@@
     (stroke (width 0) (type solid) (color 0 0 0 0))
   )
-  (wire (pts (xy 96.52 157.48) (xy 99.06 157.48))
+  (wire (pts (xy 96.52 157.48) (xy 101.6 157.48))
     (stroke (width 0) (type solid) (color 0 0 0 0))
   )
@@
     (stroke (width 0) (type solid) (color 0 0 0 0))
   )
-  (wire (pts (xy 88.9 160.02) (xy 99.06 160.02))
+  (wire (pts (xy 88.9 160.02) (xy 101.6 160.02))
     (stroke (width 0) (type default) (color 0 0 0 0))
   )
@@
   (wire (pts (xy 220.98 53.34) (xy 220.98 60.96))
     (stroke (width 0) (type solid) (color 0 0 0 0))
+  )
+  (wire (pts (xy 81.28 83.82) (xy 78.74 83.82))
+    (stroke (width 0) (type default) (color 0 0 0 0))
   )
   (wire (pts (xy 137.16 55.88) (xy 144.78 55.88))
@@
     (stroke (width 0) (type solid) (color 0 0 0 0))
   )
-  (wire (pts (xy 88.9 154.94) (xy 99.06 154.94))
+  (wire (pts (xy 88.9 154.94) (xy 101.6 154.94))
     (stroke (width 0) (type default) (color 0 0 0 0))
   )
@@
     )
   )
-  (global_label "IR 3" (shape input) (at 58.42 154.94 0)
+  (global_label "IR 3" (shape output) (at 58.42 154.94 0)
     (effects (font (size 1.27 1.27)) (justify left))
     (property "Intersheet References" "${INTERSHEET_REFS}" (id 0) (at 66.409 154.8606 0)
@@
     )
   )
-  (global_label "IR 4" (shape input) (at 165.1 53.34 0)
+  (global_label "IR 4" (shape output) (at 165.1 53.34 0)
     (effects (font (size 1.27 1.27)) (justify left))
     (property "Intersheet References" "${INTERSHEET_REFS}" (id 0) (at 173.089 53.2606 0)
@@
     )
   )
-  (global_label "LED 234" (shape input) (at 251.46 114.3 0)
+  (global_label "LED 234" (shape output) (at 251.46 114.3 0)
     (effects (font (size 1.27 1.27)) (justify left))
     (property "Intersheet References" "${INTERSHEET_REFS}" (id 0) (at 261.0214 114.2206 0)
@@
     )
   )
-  (global_label "IR 4" (shape input) (at 99.06 160.02 0)
+  (global_label "IR 4" (shape output) (at 101.6 160.02 0)
     (effects (font (size 1.27 1.27)) (justify left))
-    (property "Intersheet References" "${INTERSHEET_REFS}" (id 0) (at 107.049 159.9406 0)
+    (property "Intersheet References" "${INTERSHEET_REFS}" (id 0) (at 109.589 159.9406 0)
       (effects (font (size 1.27 1.27)) (justify left) hide)
     )
@@
     )
   )
-  (global_label "IR 1" (shape input) (at 58.42 160.02 0)
+  (global_label "IR 1" (shape output) (at 58.42 160.02 0)
     (effects (font (size 1.27 1.27)) (justify left))
     (property "Intersheet References" "${INTERSHEET_REFS}" (id 0) (at 66.409 159.9406 0)
@@
     )
   )
-  (global_label "LED 15" (shape input) (at 251.46 58.42 0)
+  (global_label "LED 15" (shape output) (at 251.46 58.42 0)
     (effects (font (size 1.27 1.27)) (justify left))
     (property "Intersheet References" "${INTERSHEET_REFS}" (id 0) (at 261.0214 58.3406 0)
@@
     )
   )
-  (global_label "IR 2" (shape input) (at 58.42 157.48 0)
+  (global_label "IR 2" (shape output) (at 58.42 157.48 0)
     (effects (font (size 1.27 1.27)) (justify left))
     (property "Intersheet References" "${INTERSHEET_REFS}" (id 0) (at 66.409 157.4006 0)
@@
     )
   )
-  (global_label "IR 3" (shape input) (at 165.1 83.82 0)
+  (global_label "IR 3" (shape output) (at 165.1 83.82 0)
     (effects (font (size 1.27 1.27)) (justify left))
     (property "Intersheet References" "${INTERSHEET_REFS}" (id 0) (at 173.089 83.7406 0)
@@
     )
   )
-  (global_label "IR 2" (shape input) (at 165.1 114.3 0)
+  (global_label "IR 2" (shape output) (at 165.1 114.3 0)
     (effects (font (size 1.27 1.27)) (justify left))
     (property "Intersheet References" "${INTERSHEET_REFS}" (id 0) (at 173.089 114.2206 0)
@@
     )
   )
-  (global_label "IR ENABLE" (shape input) (at 99.06 157.48 0)
+  (global_label "IR ENABLE" (shape input) (at 101.6 157.48 0)
     (effects (font (size 1.27 1.27)) (justify left))
-    (property "Intersheet References" "${INTERSHEET_REFS}" (id 0) (at 112.8547 157.4006 0)
+    (property "Intersheet References" "${INTERSHEET_REFS}" (id 0) (at 115.3947 157.4006 0)
       (effects (font (size 1.27 1.27)) (justify left) hide)
     )
   )
-  (global_label "IR 5" (shape input) (at 78.74 83.82 0)
+  (global_label "IR 5" (shape output) (at 81.28 83.82 0)
     (effects (font (size 1.27 1.27)) (justify left))
-    (property "Intersheet References" "${INTERSHEET_REFS}" (id 0) (at 86.729 83.7406 0)
+    (property "Intersheet References" "${INTERSHEET_REFS}" (id 0) (at 89.269 83.7406 0)
       (effects (font (size 1.27 1.27)) (justify left) hide)
     )
@@
     )
   )
-  (global_label "IR 5" (shape input) (at 99.06 154.94 0)
+  (global_label "IR 5" (shape output) (at 101.6 154.94 0)
     (effects (font (size 1.27 1.27)) (justify left))
-    (property "Intersheet References" "${INTERSHEET_REFS}" (id 0) (at 107.049 154.8606 0)
+    (property "Intersheet References" "${INTERSHEET_REFS}" (id 0) (at 109.589 154.8606 0)
       (effects (font (size 1.27 1.27)) (justify left) hide)
     )
   )
-  (global_label "IR 1" (shape input) (at 81.28 53.34 0)
+  (global_label "IR 1" (shape output) (at 81.28 53.34 0)
     (effects (font (size 1.27 1.27)) (justify left))
     (property "Intersheet References" "${INTERSHEET_REFS}" (id 0) (at 89.269 53.2606 0)
@@
       (effects (font (size 1 1)) hide)
     )
-    (property "Footprint" "tronixio:zzVISHAY-CNY70" (id 2) (at 132.08 62.23 0)
+    (property "Footprint" "tronixio:VISHAY-CNY70" (id 2) (at 132.08 62.23 0)
       (effects (font (size 1 1)) hide)
     )
@@
       (effects (font (size 1 1)) hide)
     )
-    (property "Footprint" "tronixio:zzVISHAY-CNY70" (id 2) (at 48.26 62.23 0)
+    (property "Footprint" "tronixio:VISHAY-CNY70" (id 2) (at 48.26 62.23 0)
       (effects (font (size 1 1)) hide)
     )
@@
       (effects (font (size 1 1)) hide)
     )
-    (property "Footprint" "tronixio:zzVISHAY-CNY70" (id 2) (at 48.26 92.71 0)
+    (property "Footprint" "tronixio:VISHAY-CNY70" (id 2) (at 48.26 92.71 0)
       (effects (font (size 1 1)) hide)
     )
@@
       (effects (font (size 1 1)) hide)
     )
-    (property "Footprint" "tronixio:zzVISHAY-CNY70" (id 2) (at 132.08 123.19 0)
+    (property "Footprint" "tronixio:VISHAY-CNY70" (id 2) (at 132.08 123.19 0)
       (effects (font (size 1 1)) hide)
     )
@@
       (effects (font (size 1 1)) hide)
     )
-    (property "Footprint" "tronixio:zzVISHAY-CNY70" (id 2) (at 132.08 92.71 0)
+    (property "Footprint" "tronixio:VISHAY-CNY70" (id 2) (at 132.08 92.71 0)
       (effects (font (size 1 1)) hide)
     )
@@
     )
     (path "/2d82a6ff-7772-4709-a5d5-5abcbcaa4446"
-      (reference "IC1") (unit 1) (value "VISHAY-CNY70") (footprint "tronixio:zzVISHAY-CNY70")
+      (reference "IC1") (unit 1) (value "VISHAY-CNY70") (footprint "tronixio:VISHAY-CNY70")
     )
     (path "/a3c8097b-7ea4-44ea-82e9-e441fec016e6"
-      (reference "IC2") (unit 1) (value "VISHAY-CNY70") (footprint "tronixio:zzVISHAY-CNY70")
+      (reference "IC2") (unit 1) (value "VISHAY-CNY70") (footprint "tronixio:VISHAY-CNY70")
     )
     (path "/102283fb-9aab-46c7-a9fe-32f441ce3701"
-      (reference "IC3") (unit 1) (value "VISHAY-CNY70") (footprint "tronixio:zzVISHAY-CNY70")
+      (reference "IC3") (unit 1) (value "VISHAY-CNY70") (footprint "tronixio:VISHAY-CNY70")
     )
     (path "/ac740f31-4df3-44e4-bb0f-eb8b4dfbff96"
-      (reference "IC4") (unit 1) (value "VISHAY-CNY70") (footprint "tronixio:zzVISHAY-CNY70")
+      (reference "IC4") (unit 1) (value "VISHAY-CNY70") (footprint "tronixio:VISHAY-CNY70")
     )
     (path "/ac07165f-6b52-487b-bb8f-23b4c5c03e34"
-      (reference "IC5") (unit 1) (value "VISHAY-CNY70") (footprint "tronixio:zzVISHAY-CNY70")
+      (reference "IC5") (unit 1) (value "VISHAY-CNY70") (footprint "tronixio:VISHAY-CNY70")
     )
     (path "/7c0bb4b7-5d89-4686-b03c-7c12bff2aab6"
