File: Kicad/ir-line/ir-line.kicad_pcb (KiCad board)
At the start: 2 copper layers, 74 x 20 mm, 30 parts, among them IC1 VISHAY-CNY70, IC2 VISHAY-CNY70, IC3 VISHAY-CNY70, IC4 VISHAY-CNY70, IC5 VISHAY-CNY70, IC6 TPS92612, IC7 TPS92612, K1 FRONT #1, K2 FRONT #2

Commit message: Update IR Line
Connections:
- IC1 pad 1: Net-(IC1-Pad1) -> LED 15
- IC1 pad 2: Net-(C1-Pad2) -> Net-(IC1-Pad2)
- IC1 pad 3: GND -> Net-(C1-Pad2)
- IC1 pad 4: LED 15 -> GND
- IC2 pad 1: GND -> Net-(IC1-Pad2)
- IC2 pad 2: Net-(C2-Pad2) -> GND
- IC2 pad 3: GND -> Net-(C2-Pad2)
- IC2 pad 4: Net-(IC1-Pad1) -> GND
- IC3 pad 1: Net-(IC3-Pad1) -> LED 234
- IC3 pad 2: Net-(C3-Pad2) -> Net-(IC3-Pad2)
- IC3 pad 3: GND -> Net-(C3-Pad2)
- IC3 pad 4: LED 234 -> GND
- IC4 pad 1: Net-(IC4-Pad1) -> Net-(IC3-Pad2)
- IC4 pad 2: Net-(C4-Pad2) -> Net-(IC4-Pad2)
- IC4 pad 3: GND -> Net-(C4-Pad2)
- IC4 pad 4: Net-(IC3-Pad1) -> GND
- IC5 pad 1: GND -> Net-(IC4-Pad2)
- IC5 pad 2: Net-(C5-Pad2) -> GND
- IC5 pad 3: GND -> Net-(C5-Pad2)
- IC5 pad 4: Net-(IC4-Pad1) -> GND
Routing:
- net Net-(IC1-Pad2): track 0.00 -> 63.6 mm
- net Net-(IC1-Pad1): track 63.6 -> 0.00 mm
- net Net-(IC3-Pad2): track 0.00 -> 14.7 mm
- net Net-(IC3-Pad1): track 14.7 -> 0.00 mm
- net Net-(IC4-Pad2): track 0.00 -> 13.9 mm
- net Net-(IC4-Pad1): track 13.9 -> 0.00 mm
