File: Kicad/ir-line/ir-line.kicad_pcb (KiCad board)
At the start: 2 copper layers, 74 x 20 mm, 30 parts, among them IC1 VISHAY-CNY70, IC2 VISHAY-CNY70, IC3 VISHAY-CNY70, IC4 VISHAY-CNY70, IC5 VISHAY-CNY70, IC6 TPS92612, IC7 TPS92612, K1 FRONT #1, K2 FRONT #2

Commit message: Update
Other:
- board text added: "VDD"
- board text removed: "+5V"
Changed lines of the file:
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@@
     (effects (font (size 1 1) (thickness 0.15)) (justify right mirror))
   )
-  (gr_text "IR3" (at 123 95.5 90) (layer "B.SilkS")
-    (effects (font (size 0.8 0.8) (thickness 0.15)) (justify right mirror))
+  (gr_text "IR3" (at 123 95.5 270) (layer "B.SilkS")
+    (effects (font (size 0.8 0.8) (thickness 0.15)) (justify left mirror))
   )
   (gr_text "IR5" (at 169 81.75) (layer "B.SilkS")
@@
     (effects (font (size 0.8 0.8) (thickness 0.1)) (justify mirror))
   )
-  (gr_text "+5V" (at 157 95.5 90) (layer "B.SilkS")
-    (effects (font (size 0.8 0.8) (thickness 0.15)) (justify right mirror))
+  (gr_text "VDD" (at 157 95.5 270) (layer "B.SilkS")
+    (effects (font (size 0.8 0.8) (thickness 0.15)) (justify left mirror))
   )
-  (gr_text "EN" (at 153 95.5 90) (layer "B.SilkS")
-    (effects (font (size 0.8 0.8) (thickness 0.15)) (justify right mirror))
+  (gr_text "EN" (at 153 95.5 270) (layer "B.SilkS")
+    (effects (font (size 0.8 0.8) (thickness 0.15)) (justify left mirror))
   )
   (gr_text "TBOT IR Line Follower" (at 172.5 91) (layer "B.SilkS")
     (effects (font (size 1 1) (thickness 0.15)) (justify left mirror))
   )
-  (gr_text "IR4" (at 155 95.5 90) (layer "B.SilkS")
-    (effects (font (size 0.8 0.8) (thickness 0.15)) (justify right mirror))
+  (gr_text "IR4" (at 155 95.5 270) (layer "B.SilkS")
+    (effects (font (size 0.8 0.8) (thickness 0.15)) (justify left mirror))
   )
-  (gr_text "IR2" (at 121 95.5 90) (layer "B.SilkS")
-    (effects (font (size 0.8 0.8) (thickness 0.15)) (justify right mirror))
+  (gr_text "IR2" (at 121 95.5 270) (layer "B.SilkS")
+    (effects (font (size 0.8 0.8) (thickness 0.15)) (justify left mirror))
   )
   (gr_text "IR4" (at 147 84.75) (layer "B.SilkS")
@@
     (effects (font (size 0.8 0.8) (thickness 0.1)) (justify mirror))
   )
-  (gr_text "VIN" (at 125 95.5 90) (layer "B.SilkS")
-    (effects (font (size 0.8 0.8) (thickness 0.15)) (justify right mirror))
+  (gr_text "VIN" (at 125 95.5 270) (layer "B.SilkS")
+    (effects (font (size 0.8 0.8) (thickness 0.15)) (justify left mirror))
   )
   (gr_text "#2" (at 158 97) (layer "B.SilkS")
     (effects (font (size 1 1) (thickness 0.15)) (justify right mirror))
   )
-  (gr_text "GND" (at 149 95.5 90) (layer "B.SilkS")
-    (effects (font (size 0.8 0.8) (thickness 0.15)) (justify right mirror))
+  (gr_text "GND" (at 149 95.5 270) (layer "B.SilkS")
+    (effects (font (size 0.8 0.8) (thickness 0.15)) (justify left mirror))
   )
-  (gr_text "IR1" (at 119 95.5 90) (layer "B.SilkS")
-    (effects (font (size 0.8 0.8) (thickness 0.15)) (justify right mirror))
+  (gr_text "IR1" (at 119 95.5 270) (layer "B.SilkS")
+    (effects (font (size 0.8 0.8) (thickness 0.15)) (justify left mirror))
   )
-  (gr_text "GND" (at 117 95.5 90) (layer "B.SilkS")
-    (effects (font (size 0.8 0.8) (thickness 0.15)) (justify right mirror))
+  (gr_text "GND" (at 117 95.5 270) (layer "B.SilkS")
+    (effects (font (size 0.8 0.8) (thickness 0.15)) (justify left mirror))
   )
-  (gr_text "IR5" (at 151 95.5 90) (layer "B.SilkS")
-    (effects (font (size 0.8 0.8) (thickness 0.15)) (justify right mirror))
+  (gr_text "IR5" (at 151 95.5 270) (layer "B.SilkS")
+    (effects (font (size 0.8 0.8) (thickness 0.15)) (justify left mirror))
   )
-  (gr_text "IR1" (at 119 94.5 270) (layer "F.SilkS")
-    (effects (font (size 0.8 0.8) (thickness 0.15)) (justify right))
+  (gr_text "IR1" (at 119 94.5 90) (layer "F.SilkS")
+    (effects (font (size 0.8 0.8) (thickness 0.15)) (justify left))
   )
-  (gr_text "GND" (at 149 94.5 270) (layer "F.SilkS")
-    (effects (font (size 0.8 0.8) (thickness 0.15)) (justify right))
+  (gr_text "GND" (at 149 94.5 90) (layer "F.SilkS")
+    (effects (font (size 0.8 0.8) (thickness 0.15)) (justify left))
   )
-  (gr_text "VIN" (at 124.9 94.5 270) (layer "F.SilkS")
-    (effects (font (size 0.8 0.8) (thickness 0.15)) (justify right))
+  (gr_text "VIN" (at 124.9 94.5 90) (layer "F.SilkS")
+    (effects (font (size 0.8 0.8) (thickness 0.15)) (justify left))
   )
   (gr_text "JLCJLCJLCJLC" (at 137 83) (layer "F.SilkS")
     (effects (font (size 0.8 0.8) (thickness 0.1)))
   )
-  (gr_text "GND" (at 117 94.5 270) (layer "F.SilkS")
-    (effects (font (size 0.8 0.8) (thickness 0.15)) (justify right))
+  (gr_text "GND" (at 117 94.5 90) (layer "F.SilkS")
+    (effects (font (size 0.8 0.8) (thickness 0.15)) (justify left))
   )
   (gr_text "www.tronix.io" (at 101 82) (layer "F.SilkS")
     (effects (font (size 1 1) (thickness 0.15)) (justify left))
   )
-  (gr_text "+5V" (at 157 94.5 270) (layer "F.SilkS")
-    (effects (font (size 0.8 0.8) (thickness 0.15)) (justify right))
+  (gr_text "VDD" (at 157 94.5 90) (layer "F.SilkS")
+    (effects (font (size 0.8 0.8) (thickness 0.15)) (justify left))
   )
-  (gr_text "IR3" (at 123 94.5 270) (layer "F.SilkS")
-    (effects (font (size 0.8 0.8) (thickness 0.15)) (justify right))
+  (gr_text "IR3" (at 123 94.5 90) (layer "F.SilkS")
+    (effects (font (size 0.8 0.8) (thickness 0.15)) (justify left))
   )
   (gr_text "IR4" (at 147 86) (layer "F.SilkS")
@@
     (effects (font (size 0.8 0.8) (thickness 0.15)))
   )
-  (gr_text "IR2" (at 121 94.5 270) (layer "F.SilkS")
-    (effects (font (size 0.8 0.8) (thickness 0.15)) (justify right))
+  (gr_text "IR2" (at 121 94.5 90) (layer "F.SilkS")
+    (effects (font (size 0.8 0.8) (thickness 0.15)) (justify left))
   )
-  (gr_text "IR1" (at 102 86 270) (layer "F.SilkS")
+  (gr_text "IR1" (at 105 89.25) (layer "F.SilkS")
     (effects (font (size 0.8 0.8) (thickness 0.15)))
   )
-  (gr_text "IR5" (at 155 94.5 270) (layer "F.SilkS")
-    (effects (font (size 0.8 0.8) (thickness 0.15)) (justify right))
+  (gr_text "IR5" (at 155 94.5 90) (layer "F.SilkS")
+    (effects (font (size 0.8 0.8) (thickness 0.15)) (justify left))
   )
-  (gr_text "EN" (at 153 94 270) (layer "F.SilkS")
-    (effects (font (size 0.8 0.8) (thickness 0.15)) (justify right))
+  (gr_text "EN" (at 153 94 90) (layer "F.SilkS")
+    (effects (font (size 0.8 0.8) (thickness 0.15)) (justify left))
   )
   (gr_text "#1" (at 127.5 97) (layer "F.SilkS")
@@
     (effects (font (size 1 1) (thickness 0.15)) (justify right))
   )
-  (gr_text "IR5" (at 172 86 270) (layer "F.SilkS")
+  (gr_text "IR5" (at 169 89.25) (layer "F.SilkS")
     (effects (font (size 0.8 0.8) (thickness 0.15)))
   )
@@
     (effects (font (size 0.8 0.8) (thickness 0.15)))
   )
-  (gr_text "IR4" (at 151 94.5 270) (layer "F.SilkS")
-    (effects (font (size 0.8 0.8) (thickness 0.15)) (justify right))
+  (gr_text "IR4" (at 151 94.5 90) (layer "F.SilkS")
+    (effects (font (size 0.8 0.8) (thickness 0.15)) (justify left))
   )
   (gr_text "TBOT IR Line Follower - Rev.A - (01/2022) - Scale 100%" (at 100 110) (layer "Dwgs.User")

Commit message: Update
Parts:
- C1, C2, C3, C4, C5, C6, C7, C8, C9: footprint tronixio:CAPACITOR-1206 -> tronixio:CAPACITOR-SMD-1206
- H1, H2: value MOUNTING-HOLE-MASK-3MM -> MOUNTING-HOLE-3MM-MASK; footprint tronixio:M3-MASK -> tronixio:MOUNTING-HOLE-3MM-MASK
- IC1, IC2, IC3, IC4, IC5: value VISHAY-CNY70 -> CNY70
- R1: value 100K -> 100k; footprint tronixio:RESISTOR-1206 -> tronixio:RESISTOR-SMD-1206
- R2, R3, R4, R5, R6: footprint tronixio:RESISTOR-1206 -> tronixio:RESISTOR-SMD-1206
- R7, R8: value 4Ω7 -> 220Ω; footprint tronixio:RESISTOR-1206 -> tronixio:RESISTOR-SMD-1206
