File: Kicad/mcu/mcu.kicad_sch (KiCad schematic)
At the start: 9 parts, among them IC301 PIC16F1778, K301 MCU 1, K302 ICSP, K303 MCU 2

Commit message: Update MCU 8Bit
Parts:
- IC301: footprint tronixio:DIP-28-W762 -> tronixio:DIP-28-W762-SOCKET
Other:
- note added: "GPIO"
- note removed: "Dans le label global laisser le nom de la broche trouver un moyne de representeer les CORE functions Faier une sorte de tableau pour les ASIDE Functions - HC-SR04 - or GPY - or IR LINE follower Donc il faut distribuer les broches des ASIDE Juste verifier que les broches diponible pourront bien remplir les besoins des ASIDE"
- note removed: "Dispo 7x RA 0x RB 6x RC sauf si i2c = 13 ou 11 + GND et VIN"

Commit message: Update MCU
Connections:
- net RB1/SWITCH_2 renamed RB1
- net RB2/SWITCH_1 renamed RB2
Other:
- note added: "GPI.PULL-UP"
- note added: "GPO"
- note removed: "GPIO"
- note removed: "GPIO.PULL-UP"
- moved on the sheet: C301, C302, IC301, K301, K302, K303, R301, R302, S301
