File: Kicad/mcu/power.kicad_sch (KiCad schematic)
At the start: 18 parts, among them IC201 TLV1117-50, K201 Battery, T201 DMP2305U, T202 DMP2305U

Commit message: Update MCU 8Bit
Parts:
- removed T201, T202: DMP2305U, tronixio:zzzSOT-23-3, symbol tronixio:DMP2305U
- removed TP203: GND, tronixio:KEYSTONE-5006, symbol tronixio:KEYSTONE-5006
- added T201, T202: DMP2305U, tronixio:SOT-23-3, symbol tronixio:DMP2305U-NEW
- R201: value 100K -> 1M
- S201: footprint tronixio:zzzE-SWITCH-200USPXT1A1M2RE -> tronixio:E-SWITCH-200USPXT1A1M2RE
- renumbered TP204 to TP203
Connections:
- net GND: now also S201.2, T201.1 (G); no longer S201.3
- net VBAT: now also T201.3 (D)
- net VIN: now also T202.3 (D)
- net at R201.1: now also S201.3, T202.1 (G); no longer S201.2
- net at R201.2: now also T201.2 (S), T202.2 (S)
Other:
- note added: "Max: Nom: Min:"
- note removed: "Ajouter des notes de tensions Max Nom Min"

Commit message: Update MCU
Parts:
- LED201: symbol tronixio:LED-1206-RED -> tronixio:LED-1206-PURPLE
