File: Kicad/mcu/tbot-8bit.kicad_pcb (KiCad board)
At the start: 2 copper layers, 80 x 100 mm, 61 parts, among them IC201 TLV1117-50, IC301 PIC16F1778, IC401 MCP2221A, K201 Battery, K301 MCU 1, K302 ICSP, K303 MCU 2, K401 FRONT #1, K402 FRONT #2, K403 VIN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

Commit message: Update MCU
Parts:
- added H107: MOUNTING-HOLE-3MM, tronixio:M3, F.Cu at (175.0, 86.0)
- added H108: MOUNTING-HOLE-3MM, tronixio:M3, F.Cu at (105.0, 86.0)
- moved TP203 62.8 mm to (125.0, 146.0), turned to 90 degrees
- moved TP201 21.0 mm to (176.0, 108.0)
- moved R405 0.40 mm to (105.1, 79.8)
- moved R408 0.40 mm to (174.9, 79.8)
Changed lines of the file:
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@@
   )
   (footprint "tronixio:KEYSTONE-5006" (layer "F.Cu")
-    (at 103.5 87)
+    (at 125 146 90)
     (property "MOUSER" "534-5006")
     (property "Sheetfile" "power.kicad_sch")
     (property "Sheetname" "Power")
     (attr through_hole)
-    (fp_text reference "TP203" (at 0 -2.54) (layer "F.Fab")
+    (fp_text reference "TP203" (at 0 -2.54 90) (layer "F.Fab")
       (effects (font (size 1 1) (thickness 0.15)))
     )
-    (fp_text value "GND" (at 0 2.54) (layer "F.Fab")
+    (fp_text value "GND" (at 3 0 180) (layer "F.Fab")
       (effects (font (size 1 1) (thickness 0.15)))
     )
@@
     (fp_circle (center 0 0) (end 1.6 0) (layer "F.CrtYd") (width 0.05) (fill none))
     (fp_circle (center 0 0) (end 1.6 0) (layer "F.Fab") (width 0.1) (fill none))
-    (pad "1" thru_hole circle locked (at 0 0) (size 2.5 2.5) (drill 1.5) (layers *.Cu *.Mask)
+    (pad "1" thru_hole circle locked (at 0 0 90) (size 2.5 2.5) (drill 1.5) (layers *.Cu *.Mask)
       (net 1 "GND") (pinfunction "1") (pintype "passive"))
     (model "${KICAD6_USER_3DMODEL_DIR}/Discret/KEYSTONE-5006.step"
@@
       (solder_mask_margin 1.5) (clearance 1.5))
   )
+  (footprint "tronixio:M3" (layer "F.Cu")
+    (at 175 86)
+    (property "Sheetfile" "tbot-8bit.kicad_sch")
+    (property "Sheetname" "")
+    (attr exclude_from_pos_files)
+    (fp_text reference "H107" (at 0 -4.2) (layer "F.Fab") hide
+      (effects (font (size 1 1) (thickness 0.15)))
+    )
+    (fp_text value "MOUNTING-HOLE-3MM" (at 0 4.2) (layer "F.Fab") hide
+      (effects (font (size 1 1) (thickness 0.15)))
+    )
+    (fp_circle (center 0 0) (end 3.4 0) (layer "B.SilkS") (width 0.15) (fill none))
+    (fp_circle (center 0 0) (end 3.4 0) (layer "F.SilkS") (width 0.15) (fill none))
+    (fp_circle (center 0 0) (end 3.4 0) (layer "F.CrtYd") (width 0.05) (fill none))
+    (pad "" np_thru_hole circle (at 0 0) (size 3 3) (drill 3) (layers F&B.Cu *.Mask))
+  )
   (footprint "tronixio:RESISTOR-1206" (layer "F.Cu")
     (at 163.25 104.28 -90)
@@
   )
   (footprint "tronixio:RESISTOR-1206" (layer "F.Cu")
-    (at 174.93 80.15 90)
+    (at 174.93 79.75 90)
     (property "Sheetfile" "hid.kicad_sch")
     (property "Sheetname" "HID")
@@
     )
   )
+  (footprint "tronixio:M3" (layer "F.Cu")
+    (at 105 86)
+    (property "Sheetfile" "tbot-8bit.kicad_sch")
+    (property "Sheetname" "")
+    (attr exclude_from_pos_files)
+    (fp_text reference "H108" (at 0 -4.2) (layer "F.Fab") hide
+      (effects (font (size 1 1) (thickness 0.15)))
+    )
+    (fp_text value "MOUNTING-HOLE-3MM" (at 0 4.2) (layer "F.Fab") hide
+      (effects (font (size 1 1) (thickness 0.15)))
+    )
+    (fp_circle (center 0 0) (end 3.4 0) (layer "B.SilkS") (width 0.15) (fill none))
+    (fp_circle (center 0 0) (end 3.4 0) (layer "F.SilkS") (width 0.15) (fill none))
+    (fp_circle (center 0 0) (end 3.4 0) (layer "F.CrtYd") (width 0.05) (fill none))
+    (pad "" np_thru_hole circle (at 0 0) (size 3 3) (drill 3) (layers F&B.Cu *.Mask))
+  )
   (footprint "tronixio:CAPACITOR-1206" (layer "F.Cu")
     (at 104 122 -90)
@@
   )
   (footprint "tronixio:KEYSTONE-5006" (layer "F.Cu")
-    (at 176.5 87)
+    (at 176 108)
     (property "MOUSER" "534-5006")
     (property "Sheetfile" "power.kicad_sch")
@@
   )
   (footprint "tronixio:RESISTOR-1206" (layer "F.Cu")
-    (at 105.08 80.15 90)
+    (at 105.08 79.75 90)
     (property "Sheetfile" "hid.kicad_sch")
     (property "Sheetname" "HID")
@@
     (effects (font (size 1 1) (thickness 0.15)))
   )
-  (gr_text "GND" (at 106.5 87 270) (layer "F.SilkS")
+  (gr_text "GND" (at 125 143) (layer "F.SilkS")
     (effects (font (size 1 1) (thickness 0.15)))
   )
@@
     (effects (font (size 1 1) (thickness 0.15)))
   )
-  (gr_text "GND" (at 173.5 87 90) (layer "F.SilkS")
+  (gr_text "GND" (at 173 108 90) (layer "F.SilkS")
     (effects (font (size 1 1) (thickness 0.15)))
   )
@@
   (segment (start 138.73 96.66) (end 138.73 100.47) (width 0.5) (layer "B.Cu") (net 22))
   (segment (start 148.89 100.47) (end 148.89 96.66) (width 0.5) (layer "B.Cu") (net 23))
-  (segment (start 166.445 81.65) (end 153.97 94.125) (width 0.5) (layer "F.Cu") (net 24))
-  (segment (start 174.93 81.65) (end 166.445 81.65) (width 0.5) (layer "F.Cu") (net 24))
   (segment (start 153.97 94.125) (end 153.97 96.66) (width 0.5) (layer "F.Cu") (net 24))
+  (segment (start 166.845 81.25) (end 153.97 94.125) (width 0.5) (layer "F.Cu") (net 24))
+  (segment (start 174.93 81.25) (end 166.845 81.25) (width 0.5) (layer "F.Cu") (net 24))
   (segment (start 153.97 100.47) (end 153.97 96.66) (width 0.5) (layer "B.Cu") (net 24))
-  (segment (start 165.405 80.15) (end 151.43 94.125) (width 0.5) (layer "F.Cu") (net 25))
-  (segment (start 177.47 73.8) (end 177.47 79) (width 0.5) (layer "F.Cu") (net 25))
   (segment (start 151.43 94.125) (end 151.43 96.66) (width 0.5) (layer "F.Cu") (net 25))
-  (segment (start 176.32 80.15) (end 165.405 80.15) (width 0.5) (layer "F.Cu") (net 25))
-  (segment (start 177.47 79) (end 176.32 80.15) (width 0.5) (layer "F.Cu") (net 25))
+  (segment (start 176.235 79.75) (end 165.805 79.75) (width 0.5) (layer "F.Cu") (net 25))
+  (segment (start 177.47 73.8) (end 177.47 78.515) (width 0.5) (layer "F.Cu") (net 25))
+  (segment (start 165.805 79.75) (end 151.43 94.125) (width 0.5) (layer "F.Cu") (net 25))
+  (segment (start 177.47 78.515) (end 176.235 79.75) (width 0.5) (layer "F.Cu") (net 25))
   (segment (start 151.43 96.66) (end 151.43 100.47) (width 0.5) (layer "B.Cu") (net 25))
   (segment (start 156.51 96.66) (end 156.51 100.47) (width 0.5) (layer "B.Cu") (net 26))
@@
   (segment (start 156.51 108.09) (end 156.51 111.9) (width 0.5) (layer "B.Cu") (net 28))
   (segment (start 143.81 111.9) (end 143.81 108.09) (width 0.5) (layer "B.Cu") (net 29))
-  (segment (start 103.69 80.15) (end 117.15 80.15) (width 0.5) (layer "F.Cu") (net 30))
-  (segment (start 117.15 80.15) (end 131.11 94.11) (width 0.5) (layer "F.Cu") (net 30))
-  (segment (start 102.54 79) (end 103.69 80.15) (width 0.5) (layer "F.Cu") (net 30))
+  (segment (start 102.54 78.54) (end 103.75 79.75) (width 0.5) (layer "F.Cu") (net 30))
   (segment (start 131.11 94.11) (end 131.11 96.66) (width 0.5) (layer "F.Cu") (net 30))
-  (segment (start 102.54 73.8) (end 102.54 79) (width 0.5) (layer "F.Cu") (net 30))
+  (segment (start 103.75 79.75) (end 116.75 79.75) (width 0.5) (layer "F.Cu") (net 30))
+  (segment (start 102.54 73.8) (end 102.54 78.54) (width 0.5) (layer "F.Cu") (net 30))
+  (segment (start 116.75 79.75) (end 131.11 94.11) (width 0.5) (layer "F.Cu") (net 30))
   (segment (start 131.11 100.47) (end 131.11 96.66) (width 0.5) (layer "B.Cu") (net 30))
+  (segment (start 115.75 81.25) (end 128.575 94.075) (width 0.5) (layer "F.Cu") (net 31))
+  (segment (start 105.08 81.25) (end 115.75 81.25) (width 0.5) (layer "F.Cu") (net 31))
   (segment (start 128.575 94.075) (end 128.575 96.655) (width 0.5) (layer "F.Cu") (net 31))
-  (segment (start 116.15 81.65) (end 128.575 94.075) (width 0.5) (layer "F.Cu") (net 31))
-  (segment (start 105.08 81.65) (end 116.15 81.65) (width 0.5) (layer "F.Cu") (net 31))
   (segment (start 128.57 96.66) (end 128.57 100.47) (width 0.5) (layer "B.Cu") (net 31))
   (segment (start 172 133.5) (end 172 134.5) (width 0.5) (layer "F.Cu") (net 32))
@@
   (segment (start 147.5 120) (end 148 119.5) (width 0.5) (layer "F.Cu") (net 46))
   (segment (start 136.75 122.25) (end 134.75 122.25) (width 0.5) (layer "F.Cu") (net 46))
-  (segment (start 105.08 78.65) (end 105.08 73.8) (width 0.5) (layer "F.Cu") (net 47))
+  (segment (start 105.08 78.25) (end 105.08 73.8) (width 0.5) (layer "F.Cu") (net 47))
   (segment (start 106.61 138.2) (end 108.025 138.2) (width 0.5) (layer "F.Cu") (net 48))
   (segment (start 112.5 139.5) (end 112.5 138.5) (width 0.5) (layer "F.Cu") (net 48))
@@
   (segment (start 115.05 135.8) (end 114.3 135.8) (width 0.5) (layer "F.Cu") (net 49))
   (segment (start 111 135.5) (end 112.5 135.5) (width 0.5) (layer "F.Cu") (net 49))
-  (segment (start 174.93 78.65) (end 174.93 73.8) (width 0.5) (layer "F.Cu") (net 50))
+  (segment (start 174.93 78.25) (end 174.93 73.8) (width 0.5) (layer "F.Cu") (net 50))
   (segment (start 104.25 114.3) (end 108.45 114.3) (width 0.5) (layer "F.Cu") (net 51))
   (segment (start 116 110.86) (end 113.5 110.86) (width 0.5) (layer "F.Cu") (net 51))
