File: Kicad/ir-wheel/ir-wheel.kicad_pcb (KiCad board)
At the start: 2 copper layers, 58 x 25 mm, 10 parts, among them IC1 TTE-OPB606, IC2 TTE-OPB606, K1 MOLEX-MICRO-LATCH-03-RIGHT-AN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, K2 MOLEX-MICRO-LATCH-03-RIGHT-AN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

Commit message: Update IR Wheel
Parts:
- moved R1 17.5 mm to (126.5, 80.5)
- moved R2 2.50 mm to (131.5, 80.5)
Connections:
- IC1 pad 1: +5V -> Net-(IC1-Pad1)
- IC1 pad 2: Net-(IC1-Pad2) -> GND
- IC1 pad 3: Net-(IC1-Pad3) -> +5V
- IC1 pad 4: GND -> Net-(IC1-Pad4)
- IC2 pad 1: +5V -> Net-(IC1-Pad1)
- IC2 pad 2: Net-(IC1-Pad2) -> GND
- IC2 pad 3: Net-(IC1-Pad3) -> +5V
- IC2 pad 4: GND -> Net-(IC1-Pad4)
- K1 pad 2: Net-(IC1-Pad2) -> Net-(IC1-Pad4)
- K2 pad 2: Net-(IC1-Pad2) -> Net-(IC1-Pad4)
- R1 pad 1: Net-(IC1-Pad3) -> Net-(IC1-Pad1)
- R2 pad 2: Net-(IC1-Pad2) -> Net-(IC1-Pad4)
Routing:
- net Net-(IC1-Pad2): track 50.4 -> 0.00 mm
- net Net-(IC1-Pad4): track 0.00 -> 50.0 mm
- net Net-(IC1-Pad3): track 27.2 -> 0.00 mm
- net Net-(IC1-Pad1): track 0.00 -> 23.5 mm
