File: Kicad/ir-wheel/ir-wheel.kicad_pcb (KiCad board)
At the start: 2 copper layers, 58 x 25 mm, 20 parts, among them IC1 TTE-OPB606, IC2 TTE-OPB606, K1 RIGHT, K2 LEFT, P1 BOURNS-TC33X-1K, U1 MICROCHIP-MCP6541-SOT-23

Commit message: Update
Parts:
- removed R4: 10K, tronixio:RESISTOR-1206
- P1: value BOURNS-TC33X-1K -> BOURNS-TC33X-200K
- R2: value 10K -> 100K
Routing:
- net Net-(U1-Pad1): track 5.92 -> 3.84 mm, vias 1 -> 0
- net Net-(K1-Pad2): track 58.2 -> 57.0 mm
- net +5V: track 58.4 -> 59.4 mm
Changed lines of the file:
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@@
   (net 4 "Net-(IC1-Pad4)")
   (net 5 "Net-(K1-Pad2)")
-  (net 6 "Net-(P1-Pad2)")
+  (net 6 "Net-(U1-Pad1)")
   (footprint "tronixio:zzzTC33X" (layer "F.Cu")
     (at 124.5 80.5 180)
-    (property "Mouser" "652-TC33X-1-102E")
-    (property "Name" "1K")
+    (property "Mouser" "652-TC33X-1-204E")
+    (property "Name" "200K")
     (property "Sheetfile" "ir-wheel.kicad_sch")
     (property "Sheetname" "")
@@
       (effects (font (size 1 1) (thickness 0.15)))
     )
-    (fp_text value "BOURNS-TC33X-1K" (at 0 3.81) (layer "F.Fab")
+    (fp_text value "BOURNS-TC33X-200K" (at 0 3.81) (layer "F.Fab")
       (effects (font (size 1 1) (thickness 0.15)))
     )
@@
       (net 2 "+5V") (pintype "passive") (zone_connect 2))
     (pad "2" smd roundrect (at 0 -2 180) (size 1.5 1.5) (layers "F.Cu" "F.Paste" "F.Mask") (roundrect_rratio 0.15)
-      (net 6 "Net-(P1-Pad2)") (pintype "passive") (zone_connect 2))
+      (net 6 "Net-(U1-Pad1)") (pintype "passive") (zone_connect 2))
     (pad "3" smd roundrect (at 1 2 180) (size 1.2 1.2) (layers "F.Cu" "F.Paste" "F.Mask") (roundrect_rratio 0.15)
       (net 1 "GND") (pintype "passive") (zone_connect 2))
@@
     (fp_circle (center -0.5 -1) (end -0.35 -1) (layer "F.Fab") (width 0.1) (fill solid))
     (pad "1" smd roundrect (at -1.3 -0.95 90) (size 1.2 0.6) (layers "F.Cu" "F.Paste" "F.Mask") (roundrect_rratio 0.15)
-      (net 6 "Net-(P1-Pad2)") (pinfunction "+") (pintype "input"))
+      (net 6 "Net-(U1-Pad1)") (pinfunction "+") (pintype "input"))
     (pad "2" smd roundrect (at -1.3 0 90) (size 1.2 0.6) (layers "F.Cu" "F.Paste" "F.Mask") (roundrect_rratio 0.15)
       (net 1 "GND") (pinfunction "GND") (pintype "power_in"))
@@
       (effects (font (size 1 1) (thickness 0.15)))
     )
-    (fp_text value "10K" (at 4 0 90) (layer "F.Fab")
+    (fp_text value "100K" (at 4 0 90) (layer "F.Fab")
       (effects (font (size 1 1) (thickness 0.15)))
     )
@@
     (pad "" np_thru_hole circle locked (at 0 0 180) (size 3 3) (drill 3) (layers F&B.Cu *.Mask)
       (solder_mask_margin 1.5) (clearance 1.5))
-  )
-  (footprint "tronixio:RESISTOR-1206" (layer "B.Cu")
-    (at 129 80.5 -90)
-    (property "Sheetfile" "ir-wheel.kicad_sch")
-    (property "Sheetname" "")
-    (zone_connect 2)
-    (attr smd)
-    (fp_text reference "R4" (at 0 2 90) (layer "B.Fab")
-      (effects (font (size 1 1) (thickness 0.15)) (justify mirror))
-    )
-    (fp_text value "10K" (at 0 -2 90) (layer "B.Fab")
-      (effects (font (size 1 1) (thickness 0.15)) (justify mirror))
-    )
-    (fp_line (start -0.6 -0.9) (end 0.6 -0.9) (layer "B.SilkS") (width 0.15))
-    (fp_line (start -0.6 0.9) (end 0.6 0.9) (layer "B.SilkS") (width 0.15))
-    (fp_rect (start -2.3 -1) (end 2.3 1) (layer "B.CrtYd") (width 0.05) (fill none))
-    (fp_rect (start 1.2 -0.8) (end 1.5 0.8) (layer "B.Fab") (width 0.1) (fill solid))
-    (fp_rect (start -1.5 -0.8) (end -1.2 0.8) (layer "B.Fab") (width 0.1) (fill solid))
-    (fp_rect (start -1.2 -0.8) (end 1.2 0.8) (layer "B.Fab") (width 0.1) (fill none))
-    (pad "1" smd roundrect (at -1.5 0 270) (size 1.3 1.75) (layers "B.Cu" "B.Paste" "B.Mask") (roundrect_rratio 0.15)
-      (net 5 "Net-(K1-Pad2)") (pintype "passive") (zone_connect 2))
-    (pad "2" smd roundrect (at 1.5 0 270) (size 1.3 1.75) (layers "B.Cu" "B.Paste" "B.Mask") (roundrect_rratio 0.15)
-      (net 6 "Net-(P1-Pad2)") (pintype "passive") (zone_connect 2))
-    (model "${KICAD6_USER_3DMODEL_DIR}/SMD/RESISTOR-1206.wrl"
-      (offset (xyz 0 0 0))
-      (scale (xyz 1 1 1))
-      (rotate (xyz 0 0 0))
-    )
   )
   (footprint "tronixio:MOLEX-532540370" locked (layer "B.Cu")
@@
   (via (at 135 83.5) (size 0.6) (drill 0.3) (layers "F.Cu" "B.Cu") (net 1))
   (segment (start 139.090489 80.470489) (end 137.75 79.13) (width 0.5) (layer "F.Cu") (net 2))
-  (segment (start 120.68 76.5) (end 135.12 76.5) (width 0.5) (layer "F.Cu") (net 2))
-  (segment (start 132.25 79) (end 132.25 77.5) (width 0.5) (layer "F.Cu") (net 2))
-  (segment (start 132.25 77.5) (end 132.25 76.5) (width 0.5) (layer "F.Cu") (net 2))
   (segment (start 142.429511 81.9) (end 144.5 81.9) (width 0.5) (layer "F.Cu") (net 2))
   (segment (start 151.5 82.5) (end 146.5 82.5) (width 0.5) (layer "F.Cu") (net 2))
@@
   (segment (start 126.5 78.5) (end 125.5 78.5) (width 0.5) (layer "F.Cu") (net 2))
   (segment (start 127.2 79.2) (end 126.5 78.5) (width 0.5) (layer "F.Cu") (net 2))
+  (segment (start 120.68 76.5) (end 132 76.5) (width 0.5) (layer "F.Cu") (net 2))
   (segment (start 141 80.470489) (end 142.429511 81.9) (width 0.5) (layer "F.Cu") (net 2))
   (segment (start 128.05 79.2) (end 127.2 79.2) (width 0.5) (layer "F.Cu") (net 2))
@@
   (segment (start 120.68 76.5) (end 118.05 79.13) (width 0.5) (layer "F.Cu") (net 2))
   (segment (start 111.6 78.5) (end 106.5 78.5) (width 0.5) (layer "F.Cu") (net 2))
+  (segment (start 132.25 79) (end 132.25 76.5) (width 0.5) (layer "F.Cu") (net 2))
   (segment (start 128.05 79.2) (end 128.05 76.5) (width 0.5) (layer "F.Cu") (net 2))
   (segment (start 137.75 79.13) (end 135.12 76.5) (width 0.5) (layer "F.Cu") (net 2))
@@
   (segment (start 118.05 79.13) (end 115 79.13) (width 0.5) (layer "F.Cu") (net 2))
   (segment (start 146.5 82.5) (end 145.9 81.9) (width 0.5) (layer "F.Cu") (net 2))
-  (via (at 132.25 77.5) (size 0.6) (drill 0.3) (layers "F.Cu" "B.Cu") (net 2))
-  (segment (start 132.25 79) (end 132.25 77.5) (width 0.5) (layer "B.Cu") (net 2))
+  (segment (start 132 76.5) (end 135.12 76.5) (width 0.5) (layer "F.Cu") (net 2))
+  (via (at 132.25 76.5) (size 0.6) (drill 0.3) (layers "F.Cu" "B.Cu") (net 2))
+  (segment (start 132.25 79) (end 132.25 76.5) (width 0.5) (layer "B.Cu") (net 2))
   (segment (start 120.25 81.67) (end 123.17952 84.59952) (width 0.5) (layer "F.Cu") (net 3))
   (segment (start 137.02048 84.59952) (end 139.95 81.67) (width 0.5) (layer "F.Cu") (net 3))
@@
   (segment (start 129.95 81.8) (end 129.95 80.5) (width 0.4) (layer "F.Cu") (net 4))
   (segment (start 144.5 80) (end 144.5 78.9) (width 0.5) (layer "F.Cu") (net 5))
-  (segment (start 129.95 78.2) (end 129.5 77.75) (width 0.5) (layer "F.Cu") (net 5))
-  (segment (start 129.95 79.2) (end 129.95 78.2) (width 0.5) (layer "F.Cu") (net 5))
-  (segment (start 129.5 77.75) (end 129 77.75) (width 0.5) (layer "F.Cu") (net 5))
   (segment (start 145 80.5) (end 144.5 80) (width 0.5) (layer "F.Cu") (net 5))
+  (segment (start 129.95 79.2) (end 129.95 78) (width 0.4) (layer "F.Cu") (net 5))
   (segment (start 151.5 80.5) (end 145 80.5) (width 0.5) (layer "F.Cu") (net 5))
-  (via (at 129 77.75) (size 0.6) (drill 0.3) (layers "F.Cu" "B.Cu") (net 5))
-  (segment (start 129 80.5) (end 151.5 80.5) (width 0.4) (layer "B.Cu") (net 5))
-  (segment (start 129 79) (end 129 77.75) (width 0.5) (layer "B.Cu") (net 5))
-  (segment (start 129 79) (end 129 80.5) (width 0.4) (layer "B.Cu") (net 5))
-  (segment (start 106.5 80.5) (end 129 80.5) (width 0.4) (layer "B.Cu") (net 5))
+  (via (at 129.95 78) (size 0.6) (drill 0.3) (layers "F.Cu" "B.Cu") (net 5))
+  (segment (start 129.95 80.5) (end 129.95 78) (width 0.4) (layer "B.Cu") (net 5))
+  (segment (start 106.5 80.5) (end 130 80.5) (width 0.4) (layer "B.Cu") (net 5))
+  (segment (start 130 80.5) (end 151.5 80.5) (width 0.4) (layer "B.Cu") (net 5))
   (segment (start 126.3 82.5) (end 127 81.8) (width 0.5) (layer "F.Cu") (net 6))
   (segment (start 124.5 82.5) (end 126.3 82.5) (width 0.5) (layer "F.Cu") (net 6))
   (segment (start 128.05 81.8) (end 127 81.8) (width 0.5) (layer "F.Cu") (net 6))
-  (via (at 127 81.8) (size 0.6) (drill 0.3) (layers "F.Cu" "B.Cu") (net 6))
-  (segment (start 127.2 82) (end 127 81.8) (width 0.5) (layer "B.Cu") (net 6))
-  (segment (start 129 82) (end 127.2 82) (width 0.5) (layer "B.Cu") (net 6))
   (zone (net 1) (net_name "GND") (layers F&B.Cu) (hatch edge 0.508)
     (connect_pads (clearance 0.5))

Commit message: Update ir-wheel.kicad_pcb
Parts:
- IC1, IC2: value TTE-OPB606 -> OPB606
- P1: value BOURNS-TC33X-200K -> 200K
- U1: value MICROCHIP-MCP6541-SOT-23 -> MCP6541
Changed lines of the file:
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@@
     (zone_connect 2)
     (attr smd)
-    (fp_text reference "P1" (at 0 -3.81) (layer "F.Fab")
-      (effects (font (size 1 1) (thickness 0.15)))
-    )
-    (fp_text value "BOURNS-TC33X-200K" (at 0 3.81) (layer "F.Fab")
+    (fp_text reference "P1" (at 0 -3) (layer "F.Fab")
+      (effects (font (size 1 1) (thickness 0.15)))
+    )
+    (fp_text value "200K" (at 0 3) (layer "F.Fab")
       (effects (font (size 1 1) (thickness 0.15)))
     )
@@
     (property "Sheetname" "")
     (attr smd)
-    (fp_text reference "U1" (at 0 -3 90) (layer "F.Fab")
-      (effects (font (size 1 1) (thickness 0.15)))
-    )
-    (fp_text value "MICROCHIP-MCP6541-SOT-23" (at 0 3 90) (layer "F.Fab")
+    (fp_text reference "U1" (at -2.5 0 180) (layer "F.Fab")
+      (effects (font (size 1 1) (thickness 0.15)))
+    )
+    (fp_text value "MCP6541" (at 3 1.5 180) (layer "F.Fab")
       (effects (font (size 1 1) (thickness 0.15)))
     )
@@
       (effects (font (size 1 1) (thickness 0.15)))
     )
-    (fp_text value "TTE-OPB606" (at 0 3.81) (layer "F.Fab")
+    (fp_text value "OPB606" (at 0 3.81) (layer "F.Fab")
       (effects (font (size 1 1) (thickness 0.15)))
     )
@@
     (zone_connect 2)
     (attr smd)
-    (fp_text reference "R2" (at -3 0 90) (layer "F.Fab")
-      (effects (font (size 1 1) (thickness 0.15)))
-    )
-    (fp_text value "100K" (at 4 0 90) (layer "F.Fab")
+    (fp_text reference "R2" (at 0 0 90) (layer "F.Fab")
+      (effects (font (size 1 1) (thickness 0.15)))
+    )
+    (fp_text value "100K" (at -4 0 90) (layer "F.Fab")
       (effects (font (size 1 1) (thickness 0.15)))
     )
@@
     (zone_connect 2)
     (attr smd)
-    (fp_text reference "R3" (at 0 -2 90) (layer "F.Fab")
-      (effects (font (size 1 1) (thickness 0.15)))
-    )
-    (fp_text value "10K" (at 0 2 90) (layer "F.Fab")
+    (fp_text reference "R3" (at 0 0 90) (layer "F.Fab")
+      (effects (font (size 1 1) (thickness 0.15)))
+    )
+    (fp_text value "10K" (at 3.1 0 90) (layer "F.Fab")
       (effects (font (size 1 1) (thickness 0.15)))
     )
@@
       (effects (font (size 1 1) (thickness 0.15)))
     )
-    (fp_text value "TTE-OPB606" (at 0 3.81) (layer "F.Fab")
+    (fp_text value "OPB606" (at 0 3.81) (layer "F.Fab")
       (effects (font (size 1 1) (thickness 0.15)))
     )
@@
     (zone_connect 2)
     (attr smd)
-    (fp_text reference "C1" (at 0 -2 90) (layer "F.Fab")
-      (effects (font (size 1 1) (thickness 0.15)))
-    )
-    (fp_text value "100n" (at 0 2 90) (layer "F.Fab")
+    (fp_text reference "C1" (at 0 0 90) (layer "F.Fab")
+      (effects (font (size 1 1) (thickness 0.15)))
+    )
+    (fp_text value "100n" (at 4 0 90) (layer "F.Fab")
       (effects (font (size 1 1) (thickness 0.15)))
     )
@@
     (zone_connect 2)
     (attr smd)
-    (fp_text reference "R1" (at 0 -2 90) (layer "F.Fab")
-      (effects (font (size 1 1) (thickness 0.15)))
-    )
-    (fp_text value "220Ω" (at 0 2 90) (layer "F.Fab")
+    (fp_text reference "R1" (at 0 0 90) (layer "F.Fab")
+      (effects (font (size 1 1) (thickness 0.15)))
+    )
+    (fp_text value "220Ω" (at -4.1 0 90) (layer "F.Fab")
       (effects (font (size 1 1) (thickness 0.15)))
     )
@@
     (zone_connect 2)
     (attr smd)
-    (fp_text reference "C2" (at 0 2 90) (layer "B.Fab")
+    (fp_text reference "C2" (at 0 0 90) (layer "B.Fab")
       (effects (font (size 1 1) (thickness 0.15)) (justify mirror))
     )
-    (fp_text value "1µ" (at 0 -2 90) (layer "B.Fab")
+    (fp_text value "1µ" (at 3 0 90) (layer "B.Fab")
       (effects (font (size 1 1) (thickness 0.15)) (justify mirror))
     )
@@
     (property "Sheetname" "")
     (attr through_hole)
-    (fp_text reference "K2" (at 2 7 90) (layer "B.Fab")
+    (fp_text reference "K2" (at 2 5 90) (layer "B.Fab")
       (effects (font (size 1 1) (thickness 0.15)) (justify mirror))
     )
-    (fp_text value "LEFT" (at 2 -3 90) (layer "B.Fab")
+    (fp_text value "LEFT" (at 2 0 90) (layer "B.Fab")
       (effects (font (size 1 1) (thickness 0.15)) (justify mirror))
     )
@@
     (property "Sheetname" "")
     (attr through_hole)
-    (fp_text reference "K1" (at 2 7 90) (layer "B.Fab")
+    (fp_text reference "K1" (at 2 5 90) (layer "B.Fab")
       (effects (font (size 1 1) (thickness 0.15)) (justify mirror))
     )
-    (fp_text value "RIGHT" (at 2 -3 90) (layer "B.Fab")
+    (fp_text value "RIGHT" (at 2 0 90) (layer "B.Fab")
       (effects (font (size 1 1) (thickness 0.15)) (justify mirror))
     )

Commit message: Update
Parts:
- removed kibuzzard-62813E44: G***, kibuzzard-62813E44
- removed kibuzzard-62813E52: G***, kibuzzard-62813E52
- removed kibuzzard-62813E5A: G***, kibuzzard-62813E5A
- removed kibuzzard-62813E63: G***, kibuzzard-62813E63
- added C3: 1n, tronixio:CAPACITOR-1206, B.Cu at (129.0, 80.0)
- added kibuzzard-629B8952: G***, kibuzzard-629B8952, F.Cu at (110.0, 78.5)
- added kibuzzard-629B895E: G***, kibuzzard-629B895E, F.Cu at (110.0, 82.5)
- added kibuzzard-629B8965: G***, kibuzzard-629B8965, F.Cu at (148.0, 78.5)
- added kibuzzard-629B896F: G***, kibuzzard-629B896F, F.Cu at (148.0, 82.5)
- IC1, IC2: value OPB606 -> TTE-OPB606
- K1, K2: moved to F.Cu
- P1: value 200K -> BOURNS-TC33X-200K
- U1: value MCP6541 -> MICROCHIP-MCP6541-SOT-23
- moved K1 4.00 mm to (106.5, 82.5), turned to 90 degrees
- moved K2 4.00 mm to (151.5, 78.5), turned to -90 degrees
- moved C1 0.50 mm to (132.2, 80.0)
- moved C2 0.50 mm to (132.2, 80.0)
- moved P1 0.50 mm to (124.5, 80.0)
- moved R2 0.50 mm to (135.0, 80.0), turned to -90 degrees
- moved U1 0.50 mm to (129.0, 80.0)
- moved IC1 0.41 mm to (119.2, 80.0)
- moved IC2 0.41 mm to (138.8, 80.0)
- moved R1 0.40 mm to (113.5, 80.0)
- moved R3 0.40 mm to (144.5, 80.0), turned to 90 degrees
Routing:
- net +5V: track 59.4 -> 80.2 mm
- net GND: track 9.46 -> 0.00 mm, vias 2 -> 1
- net Net-(IC1-Pad4): track 23.5 -> 30.0 mm, vias 0 -> 2
- net Net-(K1-Pad2): track 57.0 -> 51.1 mm
- net Net-(IC1-Pad1): track 30.9 -> 30.1 mm
Other:
- board text removed: "IC2: update y+1 19.5 -> 19.6"

Commit message: Up
Parts:
- added H3: MOUNTING-HOLE-3MM-MASK, tronixio:MOUNTING-HOLE-3MM-MASK, F.Cu at (169.4, 100.0)
- added H4: MOUNTING-HOLE-3MM-MASK, tronixio:MOUNTING-HOLE-3MM-MASK, F.Cu at (169.4, 90.0)
- C1, C2, C3: footprint tronixio:CAPACITOR-1206 -> tronixio:CAPACITOR-SMD-1206
- H1, H2: value MOUNTING-HOLE-MASK-3MM -> MOUNTING-HOLE-3MM-MASK; footprint tronixio:M3-MASK -> tronixio:MOUNTING-HOLE-3MM-MASK
- IC1, IC2: value TTE-OPB606 -> OPB606; footprint tronixio:zzOPB-606 -> tronixio:OPB-606
- K1: value RIGHT -> Right
- K2: value LEFT -> Left
- P1: value BOURNS-TC33X-200K -> 200k; footprint tronixio:zzzTC33X -> tronixio:TC33X
- R1: footprint tronixio:RESISTOR-1206 -> tronixio:RESISTOR-SMD-1206
- R2: value 100K -> 100k; footprint tronixio:RESISTOR-1206 -> tronixio:RESISTOR-SMD-1206
- R3: value 10K -> 10k; footprint tronixio:RESISTOR-1206 -> tronixio:RESISTOR-SMD-1206
- U1: value MICROCHIP-MCP6541-SOT-23 -> MCP6541
- moved H2 34.0 mm to (120.0, 100.0)
- moved K2 26.6 mm to (177.8, 82.5)
- moved kibuzzard-629B8965 26.3 mm to (174.0, 82.5)
- moved kibuzzard-629B896F 26.3 mm to (174.0, 86.5)
- moved GB 22.5 mm to (116.2, 69.0)
- moved GT 22.5 mm to (116.2, 69.0)
- moved H1 16.9 mm to (120.0, 90.0)
- moved C1 16.2 mm to (148.0, 84.0)
- moved C2 16.2 mm to (148.0, 84.0)
- moved C3 16.2 mm to (144.8, 84.0)
- moved IC1 16.2 mm to (135.0, 84.0)
- moved IC2 16.2 mm to (154.5, 84.0)
- moved P1 16.2 mm to (140.2, 84.0)
- moved R1 16.2 mm to (129.2, 84.0)
- moved R2 16.2 mm to (150.8, 84.0)
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Routing:
- net +5V: track 80.2 -> 0.00 mm, vias 1 -> 0
- net Net-(C3-Pad1): track 51.1 -> 0.00 mm, vias 1 -> 0
- net Net-(IC1-ANODE): track 30.1 -> 0.00 mm
- net Net-(IC1-EMITTER): track 30.0 -> 0.00 mm, vias 2 -> 0
- net Net-(U1A-+): track 3.84 -> 0.00 mm
- net GND: vias 1 -> 0
- removed copper zone on B.Cu, net GND
- removed copper zone on F.Cu, net GND
Other:
- board size 58 x 25 mm -> 127 x 31 mm
- board text added: "Bottom"
- board text removed: "1"
- board text removed: "2"
- board text removed: "Bot."
