File: Kicad/ir-wheel/ir-wheel.kicad_sch (KiCad schematic)
At the start: 8 parts, among them IC1 TTE-OPB606, IC2 TTE-OPB606, K1 MOLEX-MICRO-LATCH-03-RIGHT-AN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, K2 MOLEX-MICRO-LATCH-03-RIGHT-AN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

Commit message: Update IR Wheel
Parts:
- IC1, IC2: MOUSER 828-OPB606 -> (none); Mouser (none) -> 828-OPB606; Name (none) -> OPB606
Connections:
- net +5V: now also IC1.3 (COLLECTOR), IC2.3 (COLLECTOR); no longer IC1.1 (TRC), IC2.1 (TRC)
- net GND: now also IC1.2 (CATHODE), IC2.2 (CATHODE); no longer IC1.4 (LEDC), IC2.4 (LEDC)
- net at K1.2, K2.2, R2.2: now also IC1.4 (EMITTER), IC2.4 (EMITTER); no longer IC1.2 (TRE), IC2.2 (TRE)
- new net: IC1.1 (ANODE), IC2.1 (ANODE), R1.1
Other:
- moved on the sheet: K1, K2
