File: Kicad/ir-wheel/ir-wheel.kicad_sch (KiCad schematic)
At the start: 14 parts, among them IC1 TTE-OPB606, IC2 TTE-OPB606, K1 RIGHT, K2 LEFT, P1 BOURNS-TC33X-200K, U1 MICROCHIP-MCP6541-SOT-23

Commit message: Up
Parts:
- added H1, H2: MOUNTING-HOLE-3MM-MASK, tronixio:MOUNTING-HOLE-3MM-MASK, symbol tronixio:MOUNTING-HOLE-3MM-MASK
- C1: footprint tronixio:CAPACITOR-1206 -> tronixio:CAPACITOR-SMD-1206; symbol tronixio:C-1206 -> tronixio:CAPACITOR-1206-100N-10P-X7R; Mouser (none) -> 187-CL31B106KAHNFNE; Tolerance (none) -> 10%; Voltage (none) -> 50V
- C2: footprint tronixio:CAPACITOR-1206 -> tronixio:CAPACITOR-SMD-1206; symbol tronixio:C-1206 -> tronixio:CAPACITOR-1206-1U-10P-X7R; Mouser (none) -> 80-C1206C105K4R; Tolerance (none) -> 10%; Voltage (none) -> 16V
- C3: footprint tronixio:CAPACITOR-1206 -> tronixio:CAPACITOR-SMD-1206; symbol tronixio:C-1206 -> tronixio:CAPACITOR-1206-1N-10P-X7R; Mouser (none) -> 80-C1206C102K5R; Tolerance (none) -> 10%; Voltage (none) -> 50V
- H3: renamed from H1; value MOUNTING-HOLE-MASK-3MM -> MOUNTING-HOLE-3MM-MASK; footprint tronixio:M3-MASK -> tronixio:MOUNTING-HOLE-3MM-MASK; symbol tronixio:MOUNTING-HOLE-MASK-3MM -> tronixio:MOUNTING-HOLE-3MM-MASK
- H4: renamed from H2; value MOUNTING-HOLE-MASK-3MM -> MOUNTING-HOLE-3MM-MASK; footprint tronixio:M3-MASK -> tronixio:MOUNTING-HOLE-3MM-MASK; symbol tronixio:MOUNTING-HOLE-MASK-3MM -> tronixio:MOUNTING-HOLE-3MM-MASK
- IC1: value TTE-OPB606 -> OPB606; footprint tronixio:zzOPB-606 -> tronixio:OPB-606; Name RIGHT -> (none)
- IC2: value TTE-OPB606 -> OPB606; footprint tronixio:zzOPB-606 -> tronixio:OPB-606; Name LEFT -> (none)
- K1: value RIGHT -> Right; MOUSER 538-53254-0370 -> (none)
- K2: value LEFT -> Left; MOUSER 538-53254-0370 -> (none)
- P1: value BOURNS-TC33X-200K -> 200k; footprint tronixio:zzzTC33X -> tronixio:TC33X; Name 200K -> (none)
- R1: footprint tronixio:RESISTOR-1206 -> tronixio:RESISTOR-SMD-1206; symbol tronixio:R-1206 -> tronixio:RESISTOR-1206-220R-5P; Mouser (none) -> 660-RK73B2BTTDD221J; Tolerance (none) -> 5%
- R2: value 100K -> 100k; footprint tronixio:RESISTOR-1206 -> tronixio:RESISTOR-SMD-1206; symbol tronixio:R-1206 -> tronixio:RESISTOR-1206-100K-5P; Mouser (none) -> 660-RK73B2BTTDD104J; Tolerance (none) -> 5%
- R3: value 10K -> 10k; footprint tronixio:RESISTOR-1206 -> tronixio:RESISTOR-SMD-1206; symbol tronixio:R-1206 -> tronixio:RESISTOR-1206-10K-5P; Mouser (none) -> 660-RK73B2BTTDD103J; Tolerance (none) -> 5%
- U1: value MICROCHIP-MCP6541-SOT-23 -> MCP6541; symbol tronixio:MICROCHIP-MCP6541-SOT-23 -> tronixio:MICROCHIP-MCP6541-SOT; Name MCP6541U -> (none)
Other:
- moved on the sheet: C1, C2, U1B

Commit message: Up
Parts:
- C3: symbol tronixio:CAPACITOR-1206-1N-10P-X7R -> tronixio:CAPACITOR-1206-1N-50V-5P-X7R; Mouser 80-C1206C102K5R -> C1206C102J5R; Tolerance 10% -> 5%
- IC1, IC2: symbol tronixio:TTE-OPB606 -> tronixio:TTE-OPB606C; Mouser 828-OPB606 -> 828-OPB606C
Connections:
- net at IC1.4 (EMITTER), IC2.4 (EMITTER), R2.2: now also U1.1 (+); no longer U1.3 (-)
- net at P1.2: now also U1.3 (-); no longer U1.1 (+)
Changed lines of the file:
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@@
     )
   )
-  (symbol (lib_id "tronixio:TTE-OPB606") (at 116.84 83.82 0) (unit 1)
+  (symbol (lib_id "tronixio:TTE-OPB606C") (at 116.84 83.82 0) (unit 1)
     (in_bom yes) (on_board yes) (dnp no)
     (property "Reference" "IC1" (at 111.76 81.28 0)
@@
       (effects (font (size 1 1)) hide)
     )
-    (property "Datasheet" "https://www.ttelectronics.com/products/categories/optoelectronics/optoelectronics/opb606a/" (at 111.76 99.06 0) (do_not_autoplace)
-      (effects (font (size 1 1)) hide)
-    )
-    (property "Mouser" "828-OPB606" (at 111.76 101.6 0) (do_not_autoplace)
+    (property "Datasheet" "https://www.ttelectronics.com/Products/Sensors/Optoelectronics/Reflective-Sensors/OPB606C" (at 111.76 99.06 0) (do_not_autoplace)
+      (effects (font (size 1 1)) hide)
+    )
+    (property "Mouser" "828-OPB606C" (at 111.76 101.6 0) (do_not_autoplace)
       (effects (font (size 1 1)) hide)
     )
@@
     )
   )
-  (symbol (lib_id "tronixio:TTE-OPB606") (at 116.84 104.14 0) (unit 1)
+  (symbol (lib_id "tronixio:TTE-OPB606C") (at 116.84 104.14 0) (unit 1)
     (in_bom yes) (on_board yes) (dnp no)
     (property "Reference" "IC2" (at 111.76 101.6 0)
@@
       (effects (font (size 1 1)) hide)
     )
-    (property "Datasheet" "https://www.ttelectronics.com/products/categories/optoelectronics/optoelectronics/opb606a/" (at 111.76 119.38 0) (do_not_autoplace)
-      (effects (font (size 1 1)) hide)
-    )
-    (property "Mouser" "828-OPB606" (at 111.76 121.92 0) (do_not_autoplace)
+    (property "Datasheet" "https://www.ttelectronics.com/Products/Sensors/Optoelectronics/Reflective-Sensors/OPB606C" (at 111.76 119.38 0) (do_not_autoplace)
+      (effects (font (size 1 1)) hide)
+    )
+    (property "Mouser" "828-OPB606C" (at 111.76 121.92 0) (do_not_autoplace)
       (effects (font (size 1 1)) hide)
     )
@@
     )
   )
-  (symbol (lib_id "tronixio:CAPACITOR-1206-1N-10P-X7R") (at 175.26 106.68 0) (unit 1)
+  (symbol (lib_id "tronixio:CAPACITOR-1206-1N-50V-5P-X7R") (at 175.26 106.68 0) (unit 1)
     (in_bom yes) (on_board yes) (dnp no)
     (property "Reference" "C3" (at 175.895 104.14 0)
@@
       (effects (font (size 1.15 1.15)) (justify left) hide)
     )
-    (property "Tolerance" "10%" (at 176.26 111.76 0) (do_not_autoplace)
-      (effects (font (size 1.15 1.15)) (justify left) hide)
-    )
-    (property "Mouser" "80-C1206C102K5R" (at 175.26 119.38 0) (do_not_autoplace)
+    (property "Tolerance" "5%" (at 176.26 111.76 0) (do_not_autoplace)
+      (effects (font (size 1.15 1.15)) (justify left) hide)
+    )
+    (property "Mouser" "C1206C102J5R" (at 175.26 119.38 0) (do_not_autoplace)
       (effects (font (size 1 1)) hide)
     )
@@
     )
   )
-  (symbol (lib_id "tronixio:MICROCHIP-MCP6541-SOT") (at 165.1 93.98 0) (mirror x) (unit 1)
-    (in_bom yes) (on_board yes) (dnp no)
-    (property "Reference" "U1" (at 165.1 88.9 0)
-      (effects (font (size 1.15 1.15)))
-    )
-    (property "Value" "MCP6541" (at 165.1 100.33 0) (do_not_autoplace)
-      (effects (font (size 1.15 1.15)))
-    )
-    (property "Footprint" "tronixio:SOT-23-5" (at 165.1 83.82 0)
-      (effects (font (size 1 1)) hide)
-    )
-    (property "Datasheet" "https://www.microchip.com/en-us/product/MCP6541" (at 165.1 81.28 0) (do_not_autoplace)
-      (effects (font (size 1 1)) hide)
-    )
-    (property "Mouser" "579-MCP6541UT-E/OT" (at 165.1 78.74 0) (do_not_autoplace)
-      (effects (font (size 1 1)) hide)
-    )
+  (symbol (lib_id "tronixio:MICROCHIP-MCP6541-SOT") (at 165.1 93.98 0) (unit 1)
+    (in_bom yes) (on_board yes) (dnp no)
+    (property "Reference" "U1" (at 162.56 86.36 0) (do_not_autoplace)
+      (effects (font (size 1.15 1.15)) (justify left))
+    )
+    (property "Value" "MCP6541" (at 162.56 88.9 0) (do_not_autoplace)
+      (effects (font (size 1.15 1.15)) (justify left))
+    )
+    (property "Footprint" "tronixio:SOT-23-5" (at 165.1 104.14 0)
+      (effects (font (size 1 1)) hide)
+    )
+    (property "Datasheet" "https://www.microchip.com/en-us/product/MCP6541" (at 165.1 106.68 0) (do_not_autoplace)
+      (effects (font (size 1 1)) hide)
+    )
+    (property "Mouser" "579-MCP6541UT-E/OT" (at 165.1 109.22 0) (do_not_autoplace)
+      (effects (font (size 1 1)) hide)
+    )
