File: Kicad/mcu16/mcu.kicad_sch (KiCad schematic)
At the start: 11 parts, among them IC301 PIC24FJxxGA002-ISP, K301 MCU 1, K302 ICSP, K303 MCU 2

Commit message: Update mcu.kicad_sch
Connections:
- net RA3/LED renamed RA3/LED_DEBUG
Changed lines of the file:
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@@
     (effects (font (size 1.27 1.27)) (justify right bottom))
   )
-  (text "DRAFT" (at 132.08 119.38 0)
+  (text "DRAFT" (at 213.36 185.42 0)
     (effects (font (size 5 5)) (justify left bottom))
   )
@@
     (effects (font (size 1.27 1.27)) (justify right))
   )
-  (hierarchical_label "RA3{slash}LED" (shape output) (at 78.74 111.76 180)
+  (hierarchical_label "RA3{slash}LED_DEBUG" (shape output) (at 78.74 111.76 180)
     (effects (font (size 1.27 1.27)) (justify right))
   )

Commit message: Update
Parts:
- removed IC301: PIC24FJxxGA002-ISP, tronixio:DIP-28-W762, symbol tronixio:MICROCHIP-PIC24FJxxGA002-ISP
- added IC301: (no value), symbol tronixio:MICROCHIP-PIC24FJ64GA102-ISP
Connections:
- net +3V3: now also IC301.13 (VDD), IC301.28 (VDD)
- net GND: now also IC301.19 (DISVREG), IC301.27 (VSS), IC301.8 (VSS)
- net RA0/BATTERY_SENSE: now also IC301.2 (RA0)
- net RA1: now also IC301.3 (RA1)
- net RA2: now also IC301.9 (RA2/CLKI)
- net RA3/LED_DEBUG: now also IC301.10 (RA3/CLKO)
- net RA4: now also IC301.12 (RA4)
- net RB0: now also IC301.4 (RB0/PGD1)
- net RB1: now also IC301.5 (RB1/PGC1)
- net RB10/PGD/URX: now also IC301.21 (RB10)
- net RB11/PGC/UTX: now also IC301.22 (RB11)
- net RB12: now also IC301.23 (RB12)
- net RB13: now also IC301.24 (RB13)
- net RB14/WHEEL_L: now also IC301.25 (RB14)
- net RB15/SERVO_L: now also IC301.26 (RB15)
- net RB2: now also IC301.6 (RB2)
- net RB3: now also IC301.7 (RB3)
- net RB4: now also IC301.11 (RB4)
- net RB5: now also IC301.14 (RB5)
- net RB6/SERVO_R: now also IC301.15 (RB6)
- net RB7/EMERGENCY: now also IC301.16 (RB7)
- net RB8/WHEEL_R: now also IC301.17 (RB8)
- net RB9: now also IC301.18 (RB9)
- net ~{MCLR}: now also IC301.1 (~{MCLR})
- net at C304.1, K303.9 (Pin_9): now also IC301.20 (VCAP/VDDCORE)
