File: Kicad/mcu16/tbot-16bit.kicad_sch (KiCad schematic)
At the start: 24 parts, among them IC101 TLV1117-33-SOT, K101 Battery, T101 DMP2305U, T102 DMP2305U

Commit message: Update tbot-16bit.kicad_sch
Parts:
- removed H107, H108: MOUNTING-HOLE-3MM, tronixio:M3, symbol tronixio:MOUNTING-HOLE-3MM
- removed T101, T102: DMP2305U, tronixio:SOT-23-3, symbol tronixio:DMP2305U-NEW
- added T101, T102: DMP2305U, tronixio:SOT-23-3, symbol tronixio:DMP2305U
Connections:
- net GND: now also T101.1 (G)
- net VBAT: now also T101.3 (D)
- net VIN: now also T102.3 (D)
- net at R102.2: now also T101.2 (S), T102.2 (S)
- net at R102.1, S101.3: now also T102.1 (G)
Other:
- sheet HID ports: added RA3/LED_DEBUG; removed RA3/LED
- sheet MCU ports: added RA3/LED_DEBUG; removed RA3/LED
