File: Kicad/gp2y/gp2y.kicad_sch (KiCad schematic)
At the start: 12 parts

Commit message: Update GP2Y
Parts:
- IC1: value (none) -> MCP1755-50
- IR1: value (none) -> SHARP-GP2Y0xx1
- K1: value (none) -> GP2Y
- K2: value (none) -> MCU
- LED1: value (none) -> Power
Other:
- title: TBOT - Front SHARP-GP2Y -> TBOT - SHARP-GP2Y
Changed lines of the file:
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@@
   (paper "A4")
   (title_block
-    (title "TBOT - Front SHARP-GP2Y")
+    (title "TBOT - SHARP-GP2Y")
     (date "01/2022")
     (rev "A")
@@
       (effects (font (size 1.15 1.15)))
     )
-    (property "Value" "" (id 1) (at 208.28 88.9 0)
+    (property "Value" "MCU" (id 1) (at 208.28 88.9 0)
       (effects (font (size 1.15 1.15)))
     )
@@
       (effects (font (size 1.15 1.15)))
     )
-    (property "Value" "" (id 1) (at 261.62 171.45 0)
+    (property "Value" "SHARP-GP2Y0xx1" (id 1) (at 261.62 171.45 0)
       (effects (font (size 1 1)) hide)
     )
@@
       (effects (font (size 1.15 1.15)))
     )
-    (property "Value" "" (id 1) (at 114.3 87.63 0)
+    (property "Value" "MCP1755-50" (id 1) (at 114.3 87.63 0)
       (effects (font (size 1.15 1.15)))
     )
@@
       (effects (font (size 1.15 1.15)))
     )
-    (property "Value" "" (id 1) (at 150.495 91.44 90)
+    (property "Value" "Power" (id 1) (at 150.495 91.44 90)
       (effects (font (size 1.15 1.15)) (justify left))
     )
@@
       (effects (font (size 1.15 1.15)))
     )
-    (property "Value" "" (id 1) (at 167.64 86.36 0)
-      (effects (font (size 1.15 1.15)))
-    )
+    (property "Value" "GP2Y" (id 1) (at 167.64 86.36 0)
+      (effects (font (size 1.15 1.15)))
+    )
