File: Kicad/gp2y/gp2y.kicad_sch (KiCad schematic)
At the start: 12 parts, among them IC1 MCP1755-50, K1 GP2Y, K2 MCU

Commit message: Update
Parts:
- C1, C2: symbol tronixio:C-1206 -> tronixio:CAPACITOR-1206-1U; Mouser (none) -> C1206C105M5RACTU; Name (none) -> CAPACITOR-1206-1U; Tolerance (none) -> 20%; Voltage (none) -> 50V
- IC1: Name MCP1755-50 -> MICROCHIP-MCP1755-50-SOT23
- IR1: Name GP2Y0A21 -> SHARP-GP2Y0A21
- K1: Name (none) -> MOLEX-MICRO-LATCH-03-RIGHT-ANGLE
- K2: Name (none) -> MOLEX-MICRO-LATCH-04-RIGHT-ANGLE
- LED1: symbol tronixio:LED-1206-ORANGE -> tronixio:KINGBRIGHT-LED-1206-PURPLE; Mouser 604-APT3216LSECKJ4RV -> 604-APTR3216-VFX; Name (none) -> KINGBRIGHT-LED-1206-PURPLE
- R1: symbol tronixio:R-1206 -> tronixio:RESISTOR-1206-100K; Mouser (none) -> 660-RK73B2BTTDD104J; Name (none) -> RESISTOR-1206-100K; Tolerance (none) -> 5%
- R2: symbol tronixio:R-1206 -> tronixio:RESISTOR-1206-4K7; Mouser (none) -> 660-RK73B2BTTDD472J; Name (none) -> RESISTOR-1206-4K7; Tolerance (none) -> 5%
- R3: symbol tronixio:R-1206 -> tronixio:RESISTOR-1206-10K; Mouser (none) -> 660-RK73B2BTTDD103J; Name (none) -> RESISTOR-1206-10K; Tolerance (none) -> 5%
Other:
- moved on the sheet: C2, IC1

Commit message: Update
Parts:
- C1, C2: footprint tronixio:CAPACITOR-1206 -> tronixio:CAPACITOR-SMD-1206
- H1, H2: footprint tronixio:M3-MASK -> tronixio:MOUNTING-HOLE-3MM-MASK; symbol tronixio:MOUNTING-HOLE-MASK-3MM -> tronixio:MOUNTING-HOLE-3MM-MASK
- LED1: footprint tronixio:LED-1206 -> tronixio:LED-SMD-1206
- R1, R2, R3: footprint tronixio:RESISTOR-1206 -> tronixio:RESISTOR-SMD-1206
- renumbered IC1 to U1
Changed lines of the file:
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@@
       (effects (font (size 1.15 1.15)))
     )
-    (property "Footprint" "tronixio:RESISTOR-1206" (id 2) (at 83.82 104.14 0)
-      (effects (font (size 1 1)) hide)
-    )
-    (property "Datasheet" "https://www.koaspeer.com/pdfs/RK73B.pdf" (id 3) (at 83.82 106.68 0)
+    (property "Footprint" "tronixio:RESISTOR-SMD-1206" (id 2) (at 83.82 104.14 0)
+      (effects (font (size 1 1)) hide)
+    )
+    (property "Datasheet" "https://www.koaspeer.com/products/resistors/general-purpose/rk73b/" (id 3) (at 83.82 106.68 0)
       (effects (font (size 1 1)) hide)
     )
@@
       (effects (font (size 1.15 1.15)) (justify left))
     )
-    (property "Footprint" "tronixio:CAPACITOR-1206" (id 2) (at 129.54 101.6 0)
+    (property "Footprint" "tronixio:CAPACITOR-SMD-1206" (id 2) (at 129.54 101.6 0)
       (effects (font (size 1 1)) hide)
     )
@@
     )
     (property "Footprint" "" (id 2) (at 167.64 185.42 0)
-      (effects (font (size 1.27 1.27)) hide)
-    )
-    (property "Datasheet" "~" (id 3) (at 167.64 185.42 0)
-      (effects (font (size 1.27 1.27)) hide)
+      (effects (font (size 1 1)) hide)
+    )
+    (property "Datasheet" "" (id 3) (at 167.64 185.42 0)
+      (effects (font (size 1 1)) hide)
     )
     (pin "1")
@@
     )
   )
-  (symbol (lib_id "tronixio:MOUNTING-HOLE-MASK-3MM") (at 269.24 177.8 0) (unit 1)
+  (symbol (lib_id "tronixio:MOUNTING-HOLE-3MM-MASK") (at 269.24 177.8 0) (unit 1)
     (in_bom yes) (on_board yes)
     (property "Reference" "H1" (id 0) (at 269.24 175.26 0)
@@
       (effects (font (size 1 1)) hide)
     )
-    (property "Footprint" "tronixio:M3-MASK" (id 2) (at 269.24 182.88 0)
+    (property "Footprint" "tronixio:MOUNTING-HOLE-3MM-MASK" (id 2) (at 269.24 182.88 0)
       (effects (font (size 1 1)) hide)
     )
@@
     )
     (property "Footprint" "" (id 2) (at 175.26 190.5 0)
-      (effects (font (size 1.27 1.27)) hide)
-    )
-    (property "Datasheet" "~" (id 3) (at 175.26 190.5 0)
-      (effects (font (size 1.27 1.27)) hide)
+      (effects (font (size 1 1)) hide)
+    )
+    (property "Datasheet" "" (id 3) (at 175.26 190.5 0)
+      (effects (font (size 1 1)) hide)
     )
     (pin "1")
@@
       (effects (font (size 1.15 1.15)))
     )
-    (property "Footprint" "tronixio:RESISTOR-1206" (id 2) (at 175.26 91.44 0)
-      (effects (font (size 1 1)) hide)
-    )
-    (property "Datasheet" "https://www.koaspeer.com/pdfs/RK73B.pdf" (id 3) (at 175.26 93.98 0)
+    (property "Footprint" "tronixio:RESISTOR-SMD-1206" (id 2) (at 175.26 91.44 0)
+      (effects (font (size 1 1)) hide)
+    )
+    (property "Datasheet" "https://www.koaspeer.com/products/resistors/general-purpose/rk73b/" (id 3) (at 175.26 93.98 0)
       (effects (font (size 1 1)) hide)
     )
@@
     (pin "2")
   )
-  (symbol (lib_id "tronixio:MOUNTING-HOLE-MASK-3MM") (at 274.32 177.8 0) (unit 1)
+  (symbol (lib_id "tronixio:MOUNTING-HOLE-3MM-MASK") (at 274.32 177.8 0) (unit 1)
     (in_bom yes) (on_board yes)
     (property "Reference" "H2" (id 0) (at 274.32 175.26 0)
@@
       (effects (font (size 1 1)) hide)
     )
-    (property "Footprint" "tronixio:M3-MASK" (id 2) (at 274.32 182.88 0)
+    (property "Footprint" "tronixio:MOUNTING-HOLE-3MM-MASK" (id 2) (at 274.32 182.88 0)
       (effects (font (size 1 1)) hide)
     )
@@
       (effects (font (size 1.15 1.15)) (justify right))
     )
-    (property "Footprint" "tronixio:CAPACITOR-1206" (id 2) (at 91.44 101.6 0)
+    (property "Footprint" "tronixio:CAPACITOR-SMD-1206" (id 2) (at 91.44 101.6 0)
       (effects (font (size 1 1)) hide)
     )
@@
     (pin "1")
   )
-  (symbol (lib_id "tronixio:MICROCHIP-MCP1755-50-SOT23") (at 111.76 81.28 0) (unit 1)
-    (in_bom yes) (on_board yes)
-    (property "Reference" "IC1" (id 0) (at 111.76 74.93 0)
+  (symbol (lib_id "tronixio:MICROCHIP-MCP1755-50-SOT23") (at 104.14 78.74 0) (unit 1)
+    (in_bom yes) (on_board yes)
+    (property "Reference" "U1" (id 0) (at 111.76 74.93 0)
       (effects (font (size 1.15 1.15)))
     )
@@
       (effects (font (size 1.15 1.15)) (justify left))
     )
-    (property "Footprint" "tronixio:LED-1206" (id 2) (at 134.62 88.9 0)
+    (property "Footprint" "tronixio:LED-SMD-1206" (id 2) (at 134.62 88.9 0)
       (effects (font (size 1 1)) hide)
     )
@@
       (effects (font (size 1.15 1.15)))
     )
-    (property "Footprint" "tronixio:RESISTOR-1206" (id 2) (at 144.78 93.98 0)
-      (effects (font (size 1 1)) hide)
-    )
-    (property "Datasheet" "https://www.koaspeer.com/pdfs/RK73B.pdf" (id 3) (at 144.78 96.52 0)
+    (property "Footprint" "tronixio:RESISTOR-SMD-1206" (id 2) (at 144.78 93.98 0)
+      (effects (font (size 1 1)) hide)
+    )
+    (property "Datasheet" "https://www.koaspeer.com/products/resistors/general-purpose/rk73b/" (id 3) (at 144.78 96.52 0)
       (effects (font (size 1 1)) hide)
     )
@@
     )
     (path "/9d2a1175-bbe4-4d6a-ada6-70ba5ee6c4e9"
-      (reference "C1") (unit 1) (value "1µ") (footprint "tronixio:CAPACITOR-1206")
+      (reference "C1") (unit 1) (value "1µ") (footprint "tronixio:CAPACITOR-SMD-1206")
     )
     (path "/1501b311-7fa6-4998-ac74-8b68649a4caa"
-      (reference "C2") (unit 1) (value "1µ") (footprint "tronixio:CAPACITOR-1206")
+      (reference "C2") (unit 1) (value "1µ") (footprint "tronixio:CAPACITOR-SMD-1206")
     )
     (path "/6a78ce04-184c-400b-8ef3-0a4f2acdb633"
-      (reference "H1") (unit 1) (value "MOUNTING-HOLE-MASK-3MM") (footprint "tronixio:M3-MASK")
+      (reference "H1") (unit 1) (value "MOUNTING-HOLE-MASK-3MM") (footprint "tronixio:MOUNTING-HOLE-3MM-MASK")
     )
     (path "/7eb30e6d-4863-449a-9254-8fe71cd8cfb2"
-      (reference "H2") (unit 1) (value "MOUNTING-HOLE-MASK-3MM") (footprint "tronixio:M3-MASK")
-    )
-    (path "/b0f807f7-df5c-4c93-8b4c-5933ccbdfd3a"
-      (reference "IC1") (unit 1) (value "MCP1755-50") (footprint "tronixio:SOT-23-5")
+      (reference "H2") (unit 1) (value "MOUNTING-HOLE-MASK-3MM") (footprint "tronixio:MOUNTING-HOLE-3MM-MASK")
     )
     (path "/61de8734-825b-4a6f-8a19-c68b9be180d1"
@@
     )
     (path "/cbe63f48-fbff-446e-be37-61c1c3ae4d87"
-      (reference "LED1") (unit 1) (value "Power") (footprint "tronixio:LED-1206")
+      (reference "LED1") (unit 1) (value "Power") (footprint "tronixio:LED-SMD-1206")
     )
     (path "/083e5795-d002-42d8-ace7-9c0d49ce6d55"
-      (reference "R1") (unit 1) (value "100K") (footprint "tronixio:RESISTOR-1206")
+      (reference "R1") (unit 1) (value "100K") (footprint "tronixio:RESISTOR-SMD-1206")
     )
     (path "/e4da9f9f-2bc9-49d0-a58b-be85b4ebf131"
-      (reference "R2") (unit 1) (value "4K7") (footprint "tronixio:RESISTOR-1206")
+      (reference "R2") (unit 1) (value "4K7") (footprint "tronixio:RESISTOR-SMD-1206")
     )
     (path "/7bd40de0-7f89-4558-8bbf-b6a812e84074"
-      (reference "R3") (unit 1) (value "10K") (footprint "tronixio:RESISTOR-1206")
-    )
-  )
+      (reference "R3") (unit 1) (value "10K") (footprint "tronixio:RESISTOR-SMD-1206")
+    )
+    (path "/b0f807f7-df5c-4c93-8b4c-5933ccbdfd3a"
+      (reference "U1") (unit 1) (value "MCP1755-50") (footprint "tronixio:SOT-23-5")
+    )
+  )

Commit message: Update
Parts:
- C1, C2: symbol tronixio:CAPACITOR-1206-1U -> tronixio:CAPACITOR-1206-1U-10P-X7R; Mouser C1206C105M5RACTU -> 80-C1206C105K4R; Name CAPACITOR-1206-1U -> (none); Tolerance 20% -> 10%; Voltage 50V -> 16V
- K1: Name MOLEX-MICRO-LATCH-03-RIGHT-ANGLE -> (none)
- LED1: Name KINGBRIGHT-LED-1206-PURPLE -> (none)
- R1: value 100K -> 100k; symbol tronixio:RESISTOR-1206-100K -> tronixio:RESISTOR-1206-100K-5P; Name RESISTOR-1206-100K -> (none)
- R2: value 4K7 -> 4k7; symbol tronixio:RESISTOR-1206-4K7 -> tronixio:RESISTOR-1206-4K7-5P; Name RESISTOR-1206-4K7 -> (none)
- R3: value 10K -> 10k; symbol tronixio:RESISTOR-1206-10K -> tronixio:RESISTOR-1206-10K-5P; Name RESISTOR-1206-10K -> (none)
- U1: Name MICROCHIP-MCP1755-50-SOT23 -> (none)

Commit message: Update
Parts:
- IR1: value SHARP-GP2Y0xx1 -> GP2Y0xx1; Name SHARP-GP2Y0A21 -> (none)
- K2: Name MOLEX-MICRO-LATCH-04-RIGHT-ANGLE -> (none)
Changed lines of the file:
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@@
     (effects (font (size 1.27 1.27)) (justify left bottom))
   )
-  (text "*R3: For GP2Y0D21 or MCU Pull-Up Resistor" (at 180.34 179.07 0)
+  (text "*R3: For GP2Y0D21 or MCU Pull-Up Resistor" (at 181.61 179.07 0)
     (effects (font (size 1.27 1.27)) (justify left bottom))
   )
@@
       (effects (font (size 1 1)) hide)
     )
-    (property "Name" "MOLEX-MICRO-LATCH-04-RIGHT-ANGLE" (at 203.2 73.66 0)
-      (effects (font (size 1 1)) hide)
-    )
     (pin "1")
     (pin "2")
@@
   (symbol (lib_id "tronixio:SHARP-GP2Y0A21") (at 256.54 175.26 0) (unit 1)
     (in_bom yes) (on_board yes) (dnp no)
-    (property "Reference" "IR1" (at 256.54 171.45 0)
-      (effects (font (size 1.15 1.15)))
-    )
-    (property "Value" "SHARP-GP2Y0xx1" (at 256.54 171.45 0)
-      (effects (font (size 1 1)) hide)
+    (property "Reference" "IR1" (at 256.54 168.91 0) (do_not_autoplace)
+      (effects (font (size 1.15 1.15)))
+    )
+    (property "Value" "GP2Y0xx1" (at 256.54 171.45 0) (do_not_autoplace)
+      (effects (font (size 1 1)))
     )
     (property "Footprint" "tronixio:SHARP-GP2Y0A" (at 256.54 182.88 0)
@@
       (effects (font (size 1 1)) hide)
     )
-    (property "Name" "SHARP-GP2Y0A21" (at 256.54 180.34 0)
-      (effects (font (size 1 1)) hide)
-    )

Commit message: Up
Parts:
- added LED2: Power, tronixio:LED-SMD-1206, symbol tronixio:KINGBRIGHT-LED-1206-PURPLE
- added R3: 4k7, tronixio:RESISTOR-SMD-1206, symbol tronixio:RESISTOR-1206-4K7-5P
- renumbered R3 to R4
Connections:
- net +5V: now also R3.1
- net GND: now also LED2.1 (C)
- new net: LED2.2 (A), R3.2
Other:
- note added: "*R4: For GP2Y0D21 or use MCU Pull-Up Resistor."
- note added: "GP2Y0A21YK0F: 10cm to 80cm"
- note added: "GP2Y0D21YK0F: 24cm"
- note removed: "*R3: For GP2Y0D21 or MCU Pull-Up Resistor"
- title: TBOT - SHARP-GP2Y -> TBOT - SHARP-GP2Y0x21
- moved on the sheet: C1, C2, K1, K2, LED1, R1, R2, R4, U1

Commit message: Up
Parts:
- removed LED2: Power, tronixio:LED-SMD-1206, symbol tronixio:KINGBRIGHT-LED-1206-PURPLE
- removed R3: 4k7, tronixio:RESISTOR-SMD-1206, symbol tronixio:RESISTOR-1206-4K7-5P
- C1, C2: symbol tronixio:CAPACITOR-1206-1U-10P-X7R -> tronixio:CAPACITOR-1206-1U-16V-10P-X7R
- H1, H2: value MOUNTING-HOLE-MASK-3MM -> MOUNTING-HOLE-3MM-MASK
- IR1: value GP2Y0xx1 -> GP2Y0A21
- K1: value GP2Y -> MOLEX-MICRO-LATCH-03-RIGHT-ANGLE
- K2: value MCU -> MOLEX-MICRO-LATCH-04-RIGHT-ANGLE
- LED1: value Power -> PURPLE
- renumbered R4 to R3
Connections:
- net VIN renamed +VIN
Other:
- note added: "*R3: For GP2Y0D21 or use MCU Pull-Up Resistor."
- note removed: "*R4: For GP2Y0D21 or use MCU Pull-Up Resistor."

Commit message: Up
Parts:
- K1: value MOLEX-MICRO-LATCH-03-RIGHT-ANGLE -> GP2Y
- K2: value MOLEX-MICRO-LATCH-04-RIGHT-ANGLE -> MCU
- LED1: value PURPLE -> Power
Other:
- moved on the sheet: C1, C2, K1, K2, LED1, R1, R2, R3, U1
