File: Kicad/gp2y/gp2y.kicad_pcb (KiCad board)
At the start: 2 copper layers, 48 x 35 mm, 18 parts, among them IC1 MCP1755-50, K1 GP2Y, K2 MCU

Commit message: Update GP2Y
Other:
- board text added: "TBOT SHARP-GP2Y - Rev.A - (01/2022) - Scale 100%"
- board text added: "TBOT SHRAP-GP2Y"
- board text removed: "TBOT Front GP2Y"
- board text removed: "TBOT Front SHARP-GP2Y - Rev.A - (01/2022) - Scale 100%"
Changed lines of the file:
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@@
   (paper "A4")
   (title_block
-    (title "TBOT - Front SHARP-GP2Y")
+    (title "TBOT - SHARP-GP2Y")
     (date "01/2022")
     (rev "A")
@@
     (attr board_only exclude_from_pos_files exclude_from_bom)
     (fp_text reference "kibuzzard-6277EDE4" (at 0 -3.7592 90) (layer "F.SilkS") hide
-      (effects (font (size 0 0)))
+      (effects (font (size 0 0) (thickness 0.15)))
     )
     (fp_text value "G002" (at 0 3.7592 90) (layer "F.SilkS") hide
-      (effects (font (size 0 0)))
+      (effects (font (size 0 0) (thickness 0.15)))
     )
     (fp_poly (pts
@@
     (attr board_only exclude_from_pos_files exclude_from_bom)
     (fp_text reference "kibuzzard-6277EE50" (at 0 -3.748088 90) (layer "F.SilkS") hide
-      (effects (font (size 0 0)))
+      (effects (font (size 0 0) (thickness 0.15)))
     )
     (fp_text value "G001" (at 0 3.748088 90) (layer "F.SilkS") hide
-      (effects (font (size 0 0)))
+      (effects (font (size 0 0) (thickness 0.15)))
     )
     (fp_poly (pts
@@
     (attr board_only exclude_from_pos_files exclude_from_bom)
     (fp_text reference "kibuzzard-6277EE2E" (at 0 -3.737769 90) (layer "F.SilkS") hide
-      (effects (font (size 0 0)))
+      (effects (font (size 0 0) (thickness 0.15)))
     )
     (fp_text value "G003" (at 0 3.737769 90) (layer "F.SilkS") hide
-      (effects (font (size 0 0)))
+      (effects (font (size 0 0) (thickness 0.15)))
     )
     (fp_poly (pts
@@
     (attr board_only exclude_from_pos_files exclude_from_bom)
     (fp_text reference "kibuzzard-6277EDE4" (at 0 -3.7592 90) (layer "F.SilkS") hide
-      (effects (font (size 0 0)))
+      (effects (font (size 0 0) (thickness 0.15)))
     )
     (fp_text value "G004" (at 0 3.7592 90) (layer "F.SilkS") hide
-      (effects (font (size 0 0)))
+      (effects (font (size 0 0) (thickness 0.15)))
     )
     (fp_poly (pts
@@
     (effects (font (size 1.5 1.5) (thickness 0.2)) (justify mirror))
   )
-  (gr_text "TBOT Front GP2Y" (at 124 86.5) (layer "B.SilkS")
+  (gr_text "TBOT SHRAP-GP2Y" (at 124 86.5) (layer "B.SilkS")
     (effects (font (size 1 1) (thickness 0.2)) (justify mirror))
   )
@@
     (effects (font (size 1 1) (thickness 0.15)))
   )
-  (gr_text "TBOT Front SHARP-GP2Y - Rev.A - (01/2022) - Scale 100%" (at 100 110) (layer "Dwgs.User")
+  (gr_text "TBOT SHARP-GP2Y - Rev.A - (01/2022) - Scale 100%" (at 100 110) (layer "Dwgs.User")
     (effects (font (size 1.5 1.5) (thickness 0.2)) (justify left))
   )

Commit message: Update
Parts:
- removed kibuzzard-6277EDE4: G002, kibuzzard-6277EDE4
- removed kibuzzard-6277EDE4: G004, kibuzzard-6277EDE4
- removed kibuzzard-6277EE2E: G003, kibuzzard-6277EE2E
- removed kibuzzard-6277EE50: G001, kibuzzard-6277EE50
- added kibuzzard-627E9FD9: G***, kibuzzard-627E9FD9, F.Cu at (116.0, 67.8)
- added kibuzzard-627E9FE1: G***, kibuzzard-627E9FE1, F.Cu at (118.0, 67.8)
- added kibuzzard-627E9FE7: G***, kibuzzard-627E9FE7, F.Cu at (126.0, 67.8)
- added kibuzzard-627E9FEC: G***, kibuzzard-627E9FEC, F.Cu at (132.0, 67.8)
