File: Kicad/gp2y/gp2y.kicad_pcb (KiCad board)
At the start: 2 copper layers, 48 x 35 mm, 18 parts, among them IC1 MCP1755-50, K1 GP2Y, K2 MCU

Commit message: Update GP2Y
Other:
- board text added: "TBOT SHARP-GP2Y"
- board text removed: "TBOT SHRAP-GP2Y"
Changed lines of the file:
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@@
     (effects (font (size 1.5 1.5) (thickness 0.2)) (justify mirror))
   )
-  (gr_text "TBOT SHRAP-GP2Y" (at 124 86.5) (layer "B.SilkS")
+  (gr_text "TBOT SHARP-GP2Y" (at 124 86.5) (layer "B.SilkS")
     (effects (font (size 1 1) (thickness 0.2)) (justify mirror))
   )

Commit message: Update
Parts:
- C1, C2: footprint tronixio:CAPACITOR-1206 -> tronixio:CAPACITOR-SMD-1206
- H1, H2: footprint tronixio:M3-MASK -> tronixio:MOUNTING-HOLE-3MM-MASK
- LED1: footprint tronixio:LED-1206 -> tronixio:LED-SMD-1206
- R1, R2, R3: footprint tronixio:RESISTOR-1206 -> tronixio:RESISTOR-SMD-1206
- renumbered IC1 to U1
