File: Kicad/gp2y/gp2y.kicad_pcb (KiCad board)
At the start: 2 copper layers, 48 x 35 mm, 18 parts, among them K1 GP2Y, K2 MCU, U1 MCP1755-50

Commit message: Update
Parts:
- R1: value 100K -> 100k
- R2: value 4K7 -> 4k7
- R3: value 10K -> 10k

Commit message: Update
Changed lines of the file:
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@@
   (setup
     (stackup
-      (layer "F.SilkS" (type "Top Silk Screen") (color "White"))
+      (layer "F.SilkS" (type "Top Silk Screen") (color "White") (material "Direct Printing"))
       (layer "F.Paste" (type "Top Solder Paste"))
-      (layer "F.Mask" (type "Top Solder Mask") (color "Purple") (thickness 0.01))
+      (layer "F.Mask" (type "Top Solder Mask") (color "Purple") (thickness 0.01) (material "Liquid Ink") (epsilon_r 3.3) (loss_tangent 0))
       (layer "F.Cu" (type "copper") (thickness 0.035))
-      (layer "dielectric 1" (type "prepreg") (thickness 1.51) (material "FR4") (epsilon_r 4.5) (loss_tangent 0.02))
+      (layer "dielectric 1" (type "prepreg") (color "FR4 natural") (thickness 1.51) (material "FR4") (epsilon_r 4.5) (loss_tangent 0.02))
       (layer "B.Cu" (type "copper") (thickness 0.035))
-      (layer "B.Mask" (type "Bottom Solder Mask") (color "Purple") (thickness 0.01))
+      (layer "B.Mask" (type "Bottom Solder Mask") (color "Purple") (thickness 0.01) (material "Liquid Ink") (epsilon_r 3.3) (loss_tangent 0))
       (layer "B.Paste" (type "Bottom Solder Paste"))
-      (layer "B.SilkS" (type "Bottom Silk Screen") (color "White"))
+      (layer "B.SilkS" (type "Bottom Silk Screen") (color "White") (material "Direct Printing"))
       (copper_finish "None")
       (dielectric_constraints no)
@@
     (at 124 79)
     (property "Mouser" "852-GP2Y0A21YK0F")
-    (property "Name" "SHARP-GP2Y0A21")
     (property "Sheetfile" "gp2y.kicad_sch")
     (property "Sheetname" "")
     (property "ki_description" "Distance Measuring Sensor Unit, 10-80 cm, Analog Output")
     (attr through_hole)
-    (fp_text reference "IR1" (at 0 -5) (layer "F.Fab")
+    (fp_text reference "IR1" (at 0 -5.5) (layer "F.SilkS") hide
         (effects (font (size 1 1) (thickness 0.15)))
     )
@@
     (property "Sheetfile" "gp2y.kicad_sch")
     (property "Sheetname" "")
-    (attr exclude_from_pos_files)
-    (fp_text reference "H2" (at 0 4.2) (layer "B.Fab") hide
-        (effects (font (size 1 1) (thickness 0.15)) (justify mirror))
-    )
-    (fp_text value "MOUNTING-HOLE-MASK-3MM" (at 0 -4.2) (layer "B.Fab") hide
+    (attr exclude_from_pos_files exclude_from_bom)
+    (fp_text reference "H2" (at 0 4.5) (layer "B.Fab") hide
+        (effects (font (size 1 1) (thickness 0.15)) (justify mirror))
+    )
+    (fp_text value "MOUNTING-HOLE-MASK-3MM" (at 0 -4.5) (layer "B.Fab") hide
         (effects (font (size 1 1) (thickness 0.15)) (justify mirror))
     )
     (fp_circle (center 0 0) (end 3.2 0)
-      (stroke (width 0.15) (type solid)) (fill none) (layer "B.SilkS"))
+      (stroke (width 0.2) (type solid)) (fill none) (layer "B.SilkS"))
     (fp_circle (center 0 0) (end 3.2 0)
-      (stroke (width 0.15) (type solid)) (fill none) (layer "F.SilkS"))
+      (stroke (width 0.2) (type solid)) (fill none) (layer "F.SilkS"))
     (fp_circle (center 0 0) (end 3.2 0)
       (stroke (width 0.05) (type solid)) (fill none) (layer "B.CrtYd"))
@@
     (property "ki_description" "Unpolarized Capacitor")
     (attr smd)
-    (fp_text reference "C2" (at 0 2 90) (layer "B.Fab")
+    (fp_text reference "C2" (at 0 2 90) (layer "B.SilkS") hide
         (effects (font (size 1 1) (thickness 0.15)) (justify mirror))
     )
@@
     (zone_connect 2)
     (attr smd)
-    (fp_text reference "LED1" (at 0 2 270) (layer "B.Fab")
+    (fp_text reference "LED1" (at 0 2 270) (layer "B.SilkS") hide
         (effects (font (size 1 1) (thickness 0.15)) (justify mirror))
     )
@@
     (property "ki_description" "High-Performance LDO, 300 mA")
     (attr smd)
-    (fp_text reference "U1" (at 2.5 0 180) (layer "B.Fab")
-        (effects (font (size 1 1) (thickness 0.15)) (justify mirror))
-    )
-    (fp_text value "MCP1755-50" (at -2.5 0 180) (layer "B.Fab")
+    (fp_text reference "U1" (at 0 3 90) (layer "B.SilkS") hide
+        (effects (font (size 1 1) (thickness 0.15)) (justify mirror))
+    )
+    (fp_text value "MCP1755-50" (at 0 -3 90) (layer "B.Fab")
         (effects (font (size 1 1) (thickness 0.15)) (justify mirror))
     )
@@
     (property "ki_description" "Unpolarized Capacitor")
     (attr smd)
-    (fp_text reference "C1" (at 0 2 90) (layer "B.Fab")
+    (fp_text reference "C1" (at 0 2 90) (layer "B.SilkS") hide
         (effects (font (size 1 1) (thickness 0.15)) (justify mirror))
     )
@@
     (property "Sheetfile" "gp2y.kicad_sch")
     (property "Sheetname" "")
-    (attr exclude_from_pos_files)
-    (fp_text reference "H1" (at 0 4.2 270) (layer "B.Fab") hide
-        (effects (font (size 1 1) (thickness 0.15)) (justify mirror))
-    )
-    (fp_text value "MOUNTING-HOLE-MASK-3MM" (at 0 -4.2 270) (layer "B.Fab") hide
+    (attr exclude_from_pos_files exclude_from_bom)
+    (fp_text reference "H1" (at 0 4.5 270) (layer "B.Fab") hide
+        (effects (font (size 1 1) (thickness 0.15)) (justify mirror))
+    )
+    (fp_text value "MOUNTING-HOLE-MASK-3MM" (at 0 -4.5 270) (layer "B.Fab") hide
         (effects (font (size 1 1) (thickness 0.15)) (justify mirror))
     )
     (fp_circle (center 0 0) (end 3.2 0)
-      (stroke (width 0.15) (type solid)) (fill none) (layer "B.SilkS"))
+      (stroke (width 0.2) (type solid)) (fill none) (layer "B.SilkS"))
     (fp_circle (center 0 0) (end 3.2 0)
-      (stroke (width 0.15) (type solid)) (fill none) (layer "F.SilkS"))
+      (stroke (width 0.2) (type solid)) (fill none) (layer "F.SilkS"))
     (fp_circle (center 0 0) (end 3.2 0)
       (stroke (width 0.05) (type solid)) (fill none) (layer "B.CrtYd"))
@@
     (zone_connect 2)
     (attr smd)
-    (fp_text reference "R1" (at 0 2 90) (layer "B.Fab")
+    (fp_text reference "R1" (at 0 2 90) (layer "B.SilkS") hide
         (effects (font (size 1 1) (thickness 0.15)) (justify mirror))
     )
@@
     (zone_connect 2)
     (attr smd)
-    (fp_text reference "R2" (at 0 2 270) (layer "B.Fab")
+    (fp_text reference "R2" (at 0 2 270) (layer "B.SilkS") hide
         (effects (font (size 1 1) (thickness 0.15)) (justify mirror))
     )
@@
     (at 132 71 180)
     (property "Mouser" "538-53254-0470")
-    (property "Name" "MOLEX-MICRO-LATCH-04-RIGHT-ANGLE")
     (property "Sheetfile" "gp2y.kicad_sch")
     (property "Sheetname" "")
@@
     (property "ki_keywords" "538-51065-0400 / 538-50212-8000-CT")
     (attr through_hole)
-    (fp_text reference "K2" (at 3 -0.5) (layer "B.Fab")
-        (effects (font (size 1 1) (thickness 0.15)) (justify mirror))
-    )
-    (fp_text value "MCU" (at 3 -2.5) (layer "B.Fab")
+    (fp_text reference "K2" (at 0 7) (layer "B.SilkS") hide
+        (effects (font (size 1 1) (thickness 0.15)) (justify mirror))
+    )
+    (fp_text value "MCU" (at 3 -3) (layer "B.Fab")
         (effects (font (size 1 1) (thickness 0.15)) (justify mirror))
     )
@@
     (zone_connect 2)
     (attr smd)
-    (fp_text reference "R3" (at 0 2 270) (layer "B.Fab")
+    (fp_text reference "R3" (at 0 2 270) (layer "B.SilkS") hide
         (effects (font (size 1 1) (thickness 0.15)) (justify mirror))
     )
@@
     (property "ki_keywords" "538-51065-0300 / 538-50212-8000-CT")
     (attr through_hole)
-    (fp_text reference "K1" (at 2 -0.5) (layer "B.Fab")
-        (effects (font (size 1 1) (thickness 0.15)) (justify mirror))
-    )
-    (fp_text value "GP2Y" (at 2 -2.5) (layer "B.Fab")
-        (effects (font (size 1 1) (thickness 0.15)) (justify mirror))
-    )
+    (fp_text reference "K1" (at 0 7) (layer "B.SilkS") hide
+        (effects (font (size 1 1) (thickness 0.15)) (justify mirror))
+    )
+    (fp_text value "GP2Y" (at 2 -3) (layer "B.Fab")
+        (effects (font (size 1 1) (thickness 0.15)) (justify mirror))
+    )

Commit message: Up
Parts:
- added LED2: Power, tronixio:LED-SMD-1206, F.Cu at (156.0, 77.5)
- added R4: 10k, tronixio:RESISTOR-SMD-1206, B.Cu at (117.5, 85.0)
- IR1: value SHARP-GP2Y0xx1 -> GP2Y0xx1
- LED1: moved to F.Cu
- R3: value 10k -> 4k7
- moved kibuzzard-6288C554 59.5 mm to (141.0, 121.8)
- moved kibuzzard-6288C562 59.5 mm to (143.0, 121.8)
- moved kibuzzard-6288C567 59.5 mm to (151.0, 121.8)
- moved kibuzzard-6288C56E 59.5 mm to (157.0, 121.8)
- moved R3 35.7 mm to (156.0, 83.0)
- moved GB 30.6 mm to (110.5, 122.0)
- moved GT 30.6 mm to (110.5, 122.0)
- moved R2 25.8 mm to (92.0, 83.0)
- moved LED1 22.5 mm to (92.0, 77.5), turned to -90 degrees
- moved C1 6.71 mm to (120.5, 85.0)
- moved C2 6.71 mm to (127.5, 85.0)
- moved R1 6.71 mm to (130.5, 85.0)
- moved U1 6.71 mm to (124.0, 85.0)
- moved IR1 6.00 mm to (124.0, 85.0)
- moved K1 5.01 mm to (120.2, 76.0)
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Connections:
- R3 pad 2: GP2Y_OUT -> Net-(LED2-A)
Routing:
- net +5V: track 27.4 -> 0.00 mm, vias 1 -> 0
- net GP2Y_OUT: track 18.1 -> 0.00 mm
- net MCU_ENABLE: track 14.3 -> 0.00 mm, vias 1 -> 0
- net VIN: track 10.2 -> 0.00 mm
- net Net-(LED1-A): track 3.00 -> 0.00 mm
Other:
- board size 48 x 35 mm -> 80 x 30 mm

Commit message: Up
Parts:
- removed LED2: Power, tronixio:LED-SMD-1206
- removed R4: 10k, tronixio:RESISTOR-SMD-1206
- H1, H2: value MOUNTING-HOLE-MASK-3MM -> MOUNTING-HOLE-3MM-MASK
- IR1: value GP2Y0xx1 -> GP2Y0A21
- K1: value GP2Y -> MOLEX-MICRO-LATCH-03-RIGHT-ANGLE
- K2: value MCU -> MOLEX-MICRO-LATCH-04-RIGHT-ANGLE
- LED1: value Power -> PURPLE; moved to B.Cu
- R3: value 4k7 -> 10k
- moved kibuzzard-6288C554 59.5 mm to (116.0, 67.8)
- moved kibuzzard-6288C562 59.5 mm to (118.0, 67.8)
- moved kibuzzard-6288C567 59.5 mm to (126.0, 67.8)
- moved kibuzzard-6288C56E 59.5 mm to (132.0, 67.8)
- moved R3 35.7 mm to (120.5, 79.0)
- moved GB 30.6 mm to (124.0, 94.5)
- moved GT 30.6 mm to (124.0, 94.5)
- moved R2 25.8 mm to (117.5, 79.0)
- moved LED1 22.5 mm to (114.5, 79.0), turned to 90 degrees
- moved C1 6.71 mm to (123.5, 79.0)
- moved C2 6.71 mm to (130.5, 79.0)
- moved R1 6.71 mm to (133.5, 79.0)
- moved U1 6.71 mm to (127.0, 79.0)
- moved IR1 6.00 mm to (124.0, 79.0)
- moved K1 5.01 mm to (120.0, 71.0)
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Connections:
- net VIN renamed +VIN
- R3 pad 2: Net-(LED2-A) -> GP2Y_OUT
Routing:
- net +5V: track 0.00 -> 27.4 mm, vias 0 -> 1
- net GP2Y_OUT: track 0.00 -> 18.1 mm
- net MCU_ENABLE: track 0.00 -> 14.3 mm, vias 0 -> 1
- net +VIN: track 0.00 -> 10.2 mm
- net Net-(LED1-A): track 0.00 -> 3.00 mm
Other:
- board size 80 x 30 mm -> 48 x 35 mm

Commit message: Up
Parts:
- K1: value MOLEX-MICRO-LATCH-03-RIGHT-ANGLE -> GP2Y
- K2: value MOLEX-MICRO-LATCH-04-RIGHT-ANGLE -> MCU
- LED1: value PURPLE -> Power
Changed lines of the file:
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@@
         (effects (font (size 1 1) (thickness 0.15)) (justify mirror))
     )
-    (fp_text value "PURPLE" (at 0 -2 270) (layer "B.Fab")
+    (fp_text value "Power" (at 0 -2 270) (layer "B.Fab")
         (effects (font (size 1 1) (thickness 0.15)) (justify mirror))
     )
@@
         (effects (font (size 1 1) (thickness 0.15)) (justify mirror))
     )
-    (fp_text value "MOLEX-MICRO-LATCH-04-RIGHT-ANGLE" (at 3 -3) (layer "B.Fab")
+    (fp_text value "MCU" (at 3 -3) (layer "B.Fab")
         (effects (font (size 1 1) (thickness 0.15)) (justify mirror))
     )
@@
         (effects (font (size 1 1) (thickness 0.15)) (justify mirror))
     )
-    (fp_text value "MOLEX-MICRO-LATCH-03-RIGHT-ANGLE" (at 2 -3) (layer "B.Fab")
-        (effects (font (size 1 1) (thickness 0.15)) (justify mirror))
-    )
+    (fp_text value "GP2Y" (at 2 -3) (layer "B.Fab")
+        (effects (font (size 1 1) (thickness 0.15)) (justify mirror))
+    )
