File: Kicad/hc-sr04/hc-sr04.kicad_pcb (KiCad board)
At the start: 2 copper layers, 48 x 35 mm, 13 parts, among them IC1 MCP1755, K1 HC-SR04, K2 MCU

Commit message: Update
Parts:
- added kibuzzard-627E9F99: G***, kibuzzard-627E9F99, F.Cu at (128.0, 67.8)
- added kibuzzard-627E9FA3: G***, kibuzzard-627E9FA3, F.Cu at (120.0, 67.8)
Connections:
- HC1 pad NC: (no net) -> unconnected-(HC1-PadNC)
Other:
- board text removed: "GND"
- board text removed: "VIN"

Commit message: Update HC-SR04
Other:
- board text added: "TBOT HC-SR04"
- board text added: "TBOT HC-SR04 - Rev.A - (01/2022) - Scale 100%"
- board text removed: "TBOT Front HC-SR04"
- board text removed: "TBOT Front HC-SR04 - Rev.A - (01/2022) - Scale 100%"
Changed lines of the file:
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@@
   (paper "A4")
   (title_block
-    (title "TBOT - Front HC-SR04")
+    (title "TBOT - HC-SR04")
     (date "01/2022")
     (rev "A")
@@
     (attr board_only exclude_from_pos_files exclude_from_bom)
     (fp_text reference "kibuzzard-627E9FA3" (at 0 -3.737769 90) (layer "F.SilkS") hide
-      (effects (font (size 0 0)))
+      (effects (font (size 0 0) (thickness 0.15)))
     )
     (fp_text value "G***" (at 0 3.737769 90) (layer "F.SilkS") hide
-      (effects (font (size 0 0)))
+      (effects (font (size 0 0) (thickness 0.15)))
     )
     (fp_poly (pts
@@
     (attr board_only exclude_from_pos_files exclude_from_bom)
     (fp_text reference "kibuzzard-627E9F99" (at 0 -3.7592 90) (layer "F.SilkS") hide
-      (effects (font (size 0 0)))
+      (effects (font (size 0 0) (thickness 0.15)))
     )
     (fp_text value "G***" (at 0 3.7592 90) (layer "F.SilkS") hide
-      (effects (font (size 0 0)))
+      (effects (font (size 0 0) (thickness 0.15)))
     )
     (fp_poly (pts
@@
     (effects (font (size 1.5 1.5) (thickness 0.2)) (justify mirror))
   )
-  (gr_text "TBOT Front HC-SR04" (at 124 86.5) (layer "B.SilkS")
+  (gr_text "TBOT HC-SR04" (at 124 86.5) (layer "B.SilkS")
     (effects (font (size 1 1) (thickness 0.2)) (justify mirror))
   )
@@
     (effects (font (size 0.8 0.8) (thickness 0.15)) (justify left))
   )
-  (gr_text "TBOT Front HC-SR04" (at 124 82) (layer "F.SilkS")
+  (gr_text "TBOT HC-SR04" (at 124 82) (layer "F.SilkS")
     (effects (font (size 1 1) (thickness 0.2)))
   )
@@
     (effects (font (size 0.8 0.8) (thickness 0.15)) (justify left))
   )
-  (gr_text "TBOT Front HC-SR04 - Rev.A - (01/2022) - Scale 100%" (at 100 110) (layer "Dwgs.User")
+  (gr_text "TBOT HC-SR04 - Rev.A - (01/2022) - Scale 100%" (at 100 110) (layer "Dwgs.User")
     (effects (font (size 1.5 1.5) (thickness 0.2)) (justify left))
   )

Commit message: Update
Parts:
- removed kibuzzard-627E9F99: G***, kibuzzard-627E9F99
- removed kibuzzard-627E9FA3: G***, kibuzzard-627E9FA3
- added kibuzzard-6288C61E: G***, kibuzzard-6288C61E, F.Cu at (120.0, 67.8)
- added kibuzzard-6288C626: G***, kibuzzard-6288C626, F.Cu at (128.0, 67.8)
- moved GB 3.00 mm to (130.0, 76.0)
- moved GT 3.00 mm to (118.0, 77.0)
