File: Kicad/hc-sr04/hc-sr04.kicad_pcb (KiCad board)
At the start: 2 copper layers, 48 x 35 mm, 15 parts, among them IC1 MCP1755, K1 HC-SR04, K2 MCU

Commit message: Update
Parts:
- C1, C2: footprint tronixio:CAPACITOR-1206 -> tronixio:CAPACITOR-SMD-1206
- H1, H2: footprint tronixio:M3-MASK -> tronixio:MOUNTING-HOLE-3MM-MASK
- HC1: footprint tronixio:zzHC-SR04 -> tronixioZZ:HC-SR04
- K1: footprint tronixio:zzSAMTEC-SSW-104-02-T-S-RA -> tronixioZZ:SAMTEC-SSW-104-02-T-S-RA
- LED1: footprint tronixio:LED-1206 -> tronixio:LED-SMD-1206
- R1, R2: footprint tronixio:RESISTOR-1206 -> tronixio:RESISTOR-SMD-1206

Commit message: Update
Parts:
- HC1: footprint tronixioZZ:HC-SR04 -> tronixio:HC-SR04
- IC1: value MCP1755 -> MCP1755-50
- K1: footprint tronixioZZ:SAMTEC-SSW-104-02-T-S-RA -> tronixio:SAMTEC-SSW-104-02-T-S-RA
- R1: value 100K -> 100k
- R2: value 4K7 -> 4k7

Commit message: Up
Parts:
- H1, H2: value MOUNTING-HOLE-MASK-3MM -> MOUNTING-HOLE-3MM-MASK
Connections:
- net VIN renamed +VIN
