File: Kicad/hc-sr04/hc-sr04.kicad_sch (KiCad schematic)
At the start: 11 parts, among them K1 HC-SR04, K2 MCU

Commit message: Update
Parts:
- HC1: value (none) -> HC-SR04; footprint tronixio:HC-SR04 -> tronixio:zzHC-SR04
- IC1: value (none) -> MCP1755
- K1: footprint tronixio:SAMTEC-SSW-104-02-T-S-RA -> tronixio:zzSAMTEC-SSW-104-02-T-S-RA
- LED1: value (none) -> Power
Changed lines of the file:
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@@
     (pin "1")
+  )
+  (symbol (lib_id "tronixio:HC-SR04") (at 261.62 175.26 0) (unit 1)
+    (in_bom yes) (on_board yes)
+    (property "Reference" "HC1" (id 0) (at 261.62 167.64 0)
+      (effects (font (size 1.15 1.15)))
+    )
+    (property "Value" "HC-SR04" (id 1) (at 261.62 170.18 0)
+      (effects (font (size 1.15 1.15)))
+    )
+    (property "Footprint" "tronixio:zzHC-SR04" (id 2) (at 261.62 180.34 0)
+      (effects (font (size 1 1)) hide)
+    )
+    (property "Datasheet" "https://cdn.sparkfun.com/datasheets/Sensors/Proximity/HCSR04.pdf" (id 3) (at 261.62 182.88 0)
+      (effects (font (size 1 1)) hide)
+    )
+    (pin "NC")
   )
   (symbol (lib_id "tronixio:POWER-+5V") (at 124.46 71.12 0) (unit 1)
@@
     (pin "2")
   )
-  (symbol (lib_id "tronixio:HC-SR04") (at 261.62 175.26 0) (unit 1)
-    (in_bom yes) (on_board yes)
-    (property "Reference" "HC1" (id 0) (at 261.62 168.275 0)
-      (effects (font (size 1.15 1.15)))
-    )
-    (property "Value" "" (id 1) (at 261.62 170.18 0)
-      (effects (font (size 1.15 1.15)))
-    )
-    (property "Footprint" "tronixio:HC-SR04" (id 2) (at 261.62 180.34 0)
-      (effects (font (size 1 1)) hide)
-    )
-    (property "Datasheet" "https://cdn.sparkfun.com/datasheets/Sensors/Proximity/HCSR04.pdf" (id 3) (at 261.62 182.88 0)
-      (effects (font (size 1 1)) hide)
-    )
-    (pin "NC")
-  )
   (symbol (lib_id "tronixio:MICROCHIP-MCP1755-50-SOT23") (at 111.76 81.28 0) (unit 1)
     (in_bom yes) (on_board yes)
@@
       (effects (font (size 1.15 1.15)))
     )
-    (property "Value" "" (id 1) (at 111.76 87.63 0)
+    (property "Value" "MCP1755" (id 1) (at 111.76 87.63 0)
       (effects (font (size 1 1)) hide)
     )
@@
       (effects (font (size 1.15 1.15)) (justify left))
     )
-    (property "Value" "" (id 1) (at 145.415 91.44 90)
+    (property "Value" "Power" (id 1) (at 145.415 91.44 90)
       (effects (font (size 1.15 1.15)) (justify left))
     )
@@
       (effects (font (size 1.15 1.15)))
     )
-    (property "Footprint" "tronixio:SAMTEC-SSW-104-02-T-S-RA" (id 2) (at 167.64 91.44 0)
+    (property "Footprint" "tronixio:zzSAMTEC-SSW-104-02-T-S-RA" (id 2) (at 167.64 91.44 0)
       (effects (font (size 1 1)) hide)
     )
@@
       (reference "H2") (unit 1) (value "MOUNTING-HOLE-MASK-3MM") (footprint "tronixio:M3-MASK")
     )
-    (path "/a823e788-8dff-4043-85a6-bc16ffedb2cc"
-      (reference "HC1") (unit 1) (value "HC-SR04") (footprint "tronixio:HC-SR04")
+    (path "/5c37ed15-852f-487d-94c9-e832d372bb7a"
+      (reference "HC1") (unit 1) (value "HC-SR04") (footprint "tronixio:zzHC-SR04")
     )
     (path "/b0f807f7-df5c-4c93-8b4c-5933ccbdfd3a"
@@
     )
     (path "/ed89b481-faca-420e-bee6-8599929a6bcc"
-      (reference "K1") (unit 1) (value "HC-SR04") (footprint "tronixio:SAMTEC-SSW-104-02-T-S-RA")
+      (reference "K1") (unit 1) (value "HC-SR04") (footprint "tronixio:zzSAMTEC-SSW-104-02-T-S-RA")
     )
     (path "/3759919d-bb2c-496b-a4ee-88cd6f0e1c67"

Commit message: Update HC-SR04
Other:
- title: TBOT - Front HC-SR04 -> TBOT - HC-SR04
Changed lines of the file:
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@@
   (paper "A4")
   (title_block
-    (title "TBOT - Front HC-SR04")
+    (title "TBOT - HC-SR04")
     (date "01/2022")
     (rev "A")

Commit message: Update
Other:
- moved on the sheet: C1, C2, HC1, IC1, K1, K2, LED1, R1, R2

Commit message: Update
Parts:
- C1, C2: footprint tronixio:CAPACITOR-1206 -> tronixio:CAPACITOR-SMD-1206; symbol tronixio:C-1206 -> tronixio:CAPACITOR-1206-1U; Mouser (none) -> C1206C105M5RACTU; Name (none) -> CAPACITOR-1206-1U; Tolerance (none) -> 20%; Voltage (none) -> 50V
- H1, H2: footprint tronixio:M3-MASK -> tronixio:MOUNTING-HOLE-3MM-MASK; symbol tronixio:MOUNTING-HOLE-MASK-3MM -> tronixio:MOUNTING-HOLE-3MM-MASK
- HC1: footprint tronixio:zzHC-SR04 -> tronixioZZ:HC-SR04
- IC1: Name MCP1755-50 -> MICROCHIP-MCP1755-50-SOT23
- K1: footprint tronixio:zzSAMTEC-SSW-104-02-T-S-RA -> tronixioZZ:SAMTEC-SSW-104-02-T-S-RA; Name (none) -> SAMTEC-SSW-104-02-T-S-RA
- K2: MOUSER 538-53254-0570 -> (none); Mouser (none) -> 538-53254-0570; Name (none) -> MOLEX-MICRO-LATCH-05-RIGHT-ANGLE
- LED1: footprint tronixio:LED-1206 -> tronixio:LED-SMD-1206; symbol tronixio:LED-1206-PURPLE -> tronixio:KINGBRIGHT-LED-1206-PURPLE; Name (none) -> KINGBRIGHT-LED-1206-PURPLE
- R1: footprint tronixio:RESISTOR-1206 -> tronixio:RESISTOR-SMD-1206; symbol tronixio:R-1206 -> tronixio:RESISTOR-1206-100K; Mouser (none) -> 660-RK73B2BTTDD104J; Name (none) -> RESISTOR-1206-100K; Tolerance (none) -> 5%
- R2: footprint tronixio:RESISTOR-1206 -> tronixio:RESISTOR-SMD-1206; symbol tronixio:R-1206 -> tronixio:RESISTOR-1206-4K7; Mouser (none) -> 660-RK73B2BTTDD472J; Name (none) -> RESISTOR-1206-4K7; Tolerance (none) -> 5%

Commit message: Update
Parts:
- C1, C2: symbol tronixio:CAPACITOR-1206-1U -> tronixio:CAPACITOR-1206-1U-10P-X7R; Mouser C1206C105M5RACTU -> 80-C1206C105K4R; Name CAPACITOR-1206-1U -> (none); Tolerance 20% -> 10%; Voltage 50V -> 16V
- HC1: footprint tronixioZZ:HC-SR04 -> tronixio:HC-SR04
- IC1: value MCP1755 -> MCP1755-50; Name MICROCHIP-MCP1755-50-SOT23 -> (none)
- K1: footprint tronixioZZ:SAMTEC-SSW-104-02-T-S-RA -> tronixio:SAMTEC-SSW-104-02-T-S-RA; Name SAMTEC-SSW-104-02-T-S-RA -> (none)
- K2: Name MOLEX-MICRO-LATCH-05-RIGHT-ANGLE -> (none)
- LED1: Name KINGBRIGHT-LED-1206-PURPLE -> (none)
- R1: value 100K -> 100k; symbol tronixio:RESISTOR-1206-100K -> tronixio:RESISTOR-1206-100K-5P; Name RESISTOR-1206-100K -> (none)
- R2: value 4K7 -> 4k7; symbol tronixio:RESISTOR-1206-4K7 -> tronixio:RESISTOR-1206-4K7-5P; Name RESISTOR-1206-4K7 -> (none)
Other:
- moved on the sheet: R1

Commit message: Up
Parts:
- C1, C2: symbol tronixio:CAPACITOR-1206-1U-10P-X7R -> tronixio:CAPACITOR-1206-1U-16V-10P-X7R
- H1, H2: value MOUNTING-HOLE-MASK-3MM -> MOUNTING-HOLE-3MM-MASK
Connections:
- net VIN renamed +VIN
