File: Kicad/mcu8/mcu.kicad_sch (KiCad schematic)
At the start: 9 parts, among them IC301 PIC16F1778, K301 MCU 1, K302 ICSP, K303 MCU 2

Commit message: Update MCU 8Bit
Other:
- note added: "AN0"
- note added: "AN1"
- note added: "AN2"
- note added: "AN3"
- note added: "AN4"
- note added: "GPIO"
Changed lines of the file:
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@@
     (stroke (width 0) (type solid) (color 0 0 0 0))
   )
+  (text "AN2" (at 68.58 100.33 180)
+    (effects (font (size 1.27 1.27)) (justify right bottom))
+  )
+  (text "GPIO" (at 233.68 105.41 0)
+    (effects (font (size 1.27 1.27)) (justify left bottom))
+  )
+  (text "AN1" (at 68.58 97.79 180)
+    (effects (font (size 1.27 1.27)) (justify right bottom))
+  )
   (text "GPO" (at 68.58 113.03 180)
+    (effects (font (size 1.27 1.27)) (justify right bottom))
+  )
+  (text "GPIO" (at 68.58 123.19 180)
     (effects (font (size 1.27 1.27)) (justify right bottom))
   )
@@
     (effects (font (size 1.27 1.27)) (justify left bottom))
   )
+  (text "GPIO" (at 233.68 107.95 0)
+    (effects (font (size 1.27 1.27)) (justify left bottom))
+  )
+  (text "AN3" (at 68.58 102.87 180)
+    (effects (font (size 1.27 1.27)) (justify right bottom))
+  )
+  (text "GPIO" (at 233.68 113.03 0)
+    (effects (font (size 1.27 1.27)) (justify left bottom))
+  )
+  (text "AN4" (at 68.58 107.95 180)
+    (effects (font (size 1.27 1.27)) (justify right bottom))
+  )
   (text "PWM6" (at 233.68 118.11 0)
     (effects (font (size 1.27 1.27)) (justify left bottom))
+  )
+  (text "GPIO" (at 68.58 110.49 180)
+    (effects (font (size 1.27 1.27)) (justify right bottom))
+  )
+  (text "GPIO" (at 68.58 120.65 180)
+    (effects (font (size 1.27 1.27)) (justify right bottom))
   )
   (text "EUSART.TX" (at 233.68 95.25 0)
@@
     (effects (font (size 1.27 1.27)) (justify left bottom))
   )
+  (text "GPIO" (at 233.68 120.65 0)
+    (effects (font (size 1.27 1.27)) (justify left bottom))
+  )
+  (text "GPIO" (at 68.58 118.11 180)
+    (effects (font (size 1.27 1.27)) (justify right bottom))
+  )
   (text "GPI.PULL-UP" (at 233.68 115.57 0)
     (effects (font (size 1.27 1.27)) (justify left bottom))
+  )
+  (text "GPO" (at 68.58 105.41 180)
+    (effects (font (size 1.27 1.27)) (justify right bottom))
   )
   (text "PWM11" (at 233.68 97.79 0)
@@
     (effects (font (size 1.27 1.27)) (justify left bottom))
   )
+  (text "AN0" (at 68.58 95.25 180)
+    (effects (font (size 1.27 1.27)) (justify right bottom))
+  )
   (text "AN9" (at 233.68 102.87 0)
     (effects (font (size 1.27 1.27)) (justify left bottom))
+  )
+  (text "GPIO" (at 68.58 115.57 180)
+    (effects (font (size 1.27 1.27)) (justify right bottom))
   )
   (global_label "~{MCLR}" (shape output) (at 129.54 172.72 180)
@@
     (effects (font (size 1.27 1.27)) (justify left))
   )
-  (hierarchical_label "RA5" (shape bidirectional) (at 81.28 106.68 180)
+  (hierarchical_label "RA5" (shape input) (at 81.28 106.68 180)
     (effects (font (size 1.27 1.27)) (justify right))
   )
@@
     (effects (font (size 1.27 1.27)) (justify right))
   )
-  (hierarchical_label "RA1" (shape bidirectional) (at 81.28 96.52 180)
+  (hierarchical_label "RA1" (shape input) (at 81.28 96.52 180)
     (effects (font (size 1.27 1.27)) (justify right))
   )
-  (hierarchical_label "RA3" (shape bidirectional) (at 81.28 101.6 180)
+  (hierarchical_label "RA3" (shape input) (at 81.28 101.6 180)
     (effects (font (size 1.27 1.27)) (justify right))
   )
@@
     (effects (font (size 1.27 1.27)) (justify left))
   )
-  (hierarchical_label "RA4" (shape bidirectional) (at 81.28 104.14 180)
+  (hierarchical_label "RA4" (shape output) (at 81.28 104.14 180)
     (effects (font (size 1.27 1.27)) (justify right))
   )
-  (hierarchical_label "RA0" (shape bidirectional) (at 81.28 93.98 180)
+  (hierarchical_label "RA0" (shape input) (at 81.28 93.98 180)
     (effects (font (size 1.27 1.27)) (justify right))
   )
-  (hierarchical_label "RA2" (shape bidirectional) (at 81.28 99.06 180)
+  (hierarchical_label "RA2" (shape input) (at 81.28 99.06 180)
     (effects (font (size 1.27 1.27)) (justify right))
   )

Commit message: Update MCU 8Bit
Other:
- note added: "GPIO.NC"
Changed lines of the file:
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@@
     (effects (font (size 1.27 1.27)) (justify right bottom))
   )
-  (text "GPIO" (at 233.68 105.41 0)
+  (text "GPIO.NC" (at 233.68 105.41 0)
     (effects (font (size 1.27 1.27)) (justify left bottom))
   )
@@
     (effects (font (size 1.27 1.27)) (justify right bottom))
   )
-  (text "GPIO" (at 68.58 123.19 180)
+  (text "GPIO.NC" (at 68.58 123.19 180)
     (effects (font (size 1.27 1.27)) (justify right bottom))
   )
@@
     (effects (font (size 1.27 1.27)) (justify left bottom))
   )
-  (text "GPIO" (at 233.68 107.95 0)
+  (text "GPIO.NC" (at 233.68 107.95 0)
     (effects (font (size 1.27 1.27)) (justify left bottom))
   )
@@
     (effects (font (size 1.27 1.27)) (justify right bottom))
   )
-  (text "GPIO" (at 233.68 113.03 0)
+  (text "GPIO.NC" (at 233.68 113.03 0)
     (effects (font (size 1.27 1.27)) (justify left bottom))
   )
@@
     (effects (font (size 1.27 1.27)) (justify left bottom))
   )
-  (text "GPIO" (at 68.58 110.49 180)
+  (text "GPIO.NC" (at 68.58 110.49 180)
     (effects (font (size 1.27 1.27)) (justify right bottom))
   )
@@
     (effects (font (size 1.27 1.27)) (justify left bottom))
   )
-  (text "GPIO" (at 233.68 120.65 0)
+  (text "GPIO.NC" (at 233.68 120.65 0)
     (effects (font (size 1.27 1.27)) (justify left bottom))
   )

Commit message: Update MCU 8Bit
Parts:
- renumbered C301 to C201, C302 to C202, IC301 to IC201, K301 to K201, K302 to K202, K303 to K203, R301 to R201, R302 to R202, S301 to S201
Changed lines of the file:
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@@
   (symbol (lib_id "tronixio:ALPS-SKRPAC") (at 78.74 175.26 90) (unit 1)
     (in_bom yes) (on_board yes)
-    (property "Reference" "S301" (id 0) (at 75.565 171.45 90)
+    (property "Reference" "S201" (id 0) (at 75.565 171.45 90)
       (effects (font (size 1.15 1.15)))
     )
@@
   (symbol (lib_id "tronixio:C-1206") (at 167.64 88.9 0) (unit 1)
     (in_bom yes) (on_board yes)
-    (property "Reference" "C302" (id 0) (at 168.275 86.36 0)
+    (property "Reference" "C202" (id 0) (at 168.275 86.36 0)
       (effects (font (size 1.15 1.15)) (justify left))
     )
@@
   (symbol (lib_id "tronixio:HARWIN-254-M-1X14-VERTICAL") (at 210.82 49.53 0) (unit 1)
     (in_bom yes) (on_board yes)
-    (property "Reference" "K303" (id 0) (at 210.82 46.99 0)
+    (property "Reference" "K203" (id 0) (at 210.82 46.99 0)
       (effects (font (size 1.15 1.15)))
     )
@@
   (symbol (lib_id "tronixio:C-1206") (at 86.36 175.26 0) (unit 1)
     (in_bom yes) (on_board yes)
-    (property "Reference" "C301" (id 0) (at 86.995 172.72 0)
+    (property "Reference" "C201" (id 0) (at 86.995 172.72 0)
       (effects (font (size 1.15 1.15)) (justify left))
     )
@@
   (symbol (lib_id "tronixio:MICROCHIP-PIC16F1778-ISP") (at 144.78 66.04 0) (unit 1)
     (in_bom yes) (on_board yes)
-    (property "Reference" "IC301" (id 0) (at 132.08 45.72 0)
+    (property "Reference" "IC201" (id 0) (at 132.08 45.72 0)
       (effects (font (size 1.15 1.15)) (justify left))
     )
@@
   (symbol (lib_id "tronixio:R-1206") (at 93.98 167.64 270) (unit 1)
     (in_bom yes) (on_board yes)
-    (property "Reference" "R302" (id 0) (at 93.98 165.1 90)
+    (property "Reference" "R202" (id 0) (at 93.98 165.1 90)
       (effects (font (size 1.15 1.15)))
     )
@@
   (symbol (lib_id "tronixio:MICROCHIP-ICSP-M-2x03") (at 137.16 172.72 0) (unit 1)
     (in_bom yes) (on_board yes)
-    (property "Reference" "K302" (id 0) (at 138.43 170.18 0)
+    (property "Reference" "K202" (id 0) (at 138.43 170.18 0)
       (effects (font (size 1.15 1.15)))
     )
@@
   (symbol (lib_id "tronixio:HARWIN-254-M-1X14-VERTICAL") (at 78.74 49.53 0) (mirror y) (unit 1)
     (in_bom yes) (on_board yes)
-    (property "Reference" "K301" (id 0) (at 78.74 46.99 0)
+    (property "Reference" "K201" (id 0) (at 78.74 46.99 0)
       (effects (font (size 1.15 1.15)))
     )
@@
   (symbol (lib_id "tronixio:R-1206") (at 78.74 161.29 180) (unit 1)
     (in_bom yes) (on_board yes)
-    (property "Reference" "R301" (id 0) (at 73.66 157.48 0)
+    (property "Reference" "R201" (id 0) (at 73.66 157.48 0)
       (effects (font (size 1.15 1.15)) (justify right))
     )

Commit message: Update MCU 8Bit
Other:
- note added: "GPI"
- note removed: "GPI.PULL-UP"
Changed lines of the file:
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@@
     (effects (font (size 1.27 1.27)) (justify right bottom))
   )
-  (text "GPI.PULL-UP" (at 233.68 100.33 0)
+  (text "GPI" (at 233.68 100.33 0)
     (effects (font (size 1.27 1.27)) (justify left bottom))
   )
@@
     (effects (font (size 1.27 1.27)) (justify right bottom))
   )
-  (text "GPI.PULL-UP" (at 233.68 115.57 0)
+  (text "GPI" (at 233.68 115.57 0)
     (effects (font (size 1.27 1.27)) (justify left bottom))
   )

Commit message: Draft
Other:
- note added: "DRAFT"
Changed lines of the file:
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@@
     (effects (font (size 1.27 1.27)) (justify left bottom))
+  )
+  (text "DRAFT" (at 210.82 187.96 0)
+    (effects (font (size 5 5)) (justify left bottom))
   )
   (text "GPIO.INT0" (at 233.68 110.49 0)

Commit message: Update
Parts:
- IC201: MOUSER 579-PIC16F1778-I/SP -> (none); Mouser (none) -> 579-PIC16F1778-I/SP
- K201, K203: MOUSER 855-M20-999144 -> (none); Mouser (none) -> 855-M20-999144
- K202: MOUSER 855-M20-9980346 -> (none); Mouser (none) -> 855-M20-9980346; Name (none) -> ICSP
- S201: MOUSER 688-SKRPACE010 -> (none); Mouser (none) -> 688-SKRPACE010
Changed lines of the file:
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@@
       (effects (font (size 1 1)) hide)
     )
-    (property "MOUSER" "688-SKRPACE010" (id 4) (at 91.44 175.26 0)
+    (property "Mouser" "688-SKRPACE010" (id 4) (at 91.44 175.26 0)
       (effects (font (size 1 1)) hide)
     )
@@
       (effects (font (size 1 1)) hide)
     )
-    (property "MOUSER" "855-M20-999144" (id 4) (at 210.82 92.71 0)
+    (property "Mouser" "855-M20-999144" (id 4) (at 210.82 92.71 0)
       (effects (font (size 1 1)) hide)
     )
@@
       (effects (font (size 1 1)) hide)
     )
-    (property "MOUSER" "579-PIC16F1778-I/SP" (id 4) (at 144.78 93.98 0)
-      (effects (font (size 1 1)) hide)
-    )
     (property "Name" "PIC16F1778-ISP" (id 5) (at 157.48 45.72 0)
       (effects (font (size 1.15 1.15)) (justify right))
+    )
+    (property "Mouser" "579-PIC16F1778-I/SP" (id 6) (at 144.78 93.98 0)
+      (effects (font (size 1 1)) hide)
     )
     (pin "1")
@@
       (effects (font (size 1 1)) hide)
     )
-    (property "MOUSER" "855-M20-9980346" (id 4) (at 138.43 187.96 0)
+    (property "Name" "ICSP" (id 4) (at 138.43 180.34 0)
+      (effects (font (size 1.15 1.15)))
+    )
+    (property "Mouser" "855-M20-9980346" (id 5) (at 138.43 190.5 0)
       (effects (font (size 1 1)) hide)
     )
@@
       (effects (font (size 1 1)) hide)
     )
-    (property "MOUSER" "855-M20-999144" (id 4) (at 78.74 92.71 0)
-      (effects (font (size 1 1)) hide)
-    )
+    (property "Mouser" "855-M20-999144" (id 4) (at 78.74 92.71 0)
+      (effects (font (size 1 1)) hide)
+    )

Commit message: Update MCU
Other:
- note added: "Ajouter Connerter pour IR WHEEL"
- note added: "CCP2"
- note added: "CCP7"
- note added: "RA1 INPUT"
- note added: "RAO INPUT"
- note removed: "GPI"
Changed lines of the file:
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@@
     (effects (font (size 1.27 1.27)) (justify right bottom))
   )
-  (text "GPI" (at 233.68 100.33 0)
+  (text "CCP7" (at 233.68 100.33 0)
     (effects (font (size 1.27 1.27)) (justify left bottom))
+  )
+  (text "RAO INPUT " (at 33.02 35.56 0)
+    (effects (font (size 3 3)) (justify left bottom))
   )
   (text "GPIO.NC" (at 233.68 107.95 0)
@@
   (text "AN3" (at 68.58 102.87 180)
     (effects (font (size 1.27 1.27)) (justify right bottom))
+  )
+  (text "Ajouter Connerter pour IR WHEEL" (at 30.48 27.94 0)
+    (effects (font (size 3 3)) (justify left bottom))
   )
   (text "GPIO.NC" (at 233.68 113.03 0)
@@
     (effects (font (size 1.27 1.27)) (justify left bottom))
   )
+  (text "RA1 INPUT " (at 33.02 40.64 0)
+    (effects (font (size 3 3)) (justify left bottom))
+  )
   (text "DRAFT" (at 210.82 187.96 0)
     (effects (font (size 5 5)) (justify left bottom))
@@
     (effects (font (size 1.27 1.27)) (justify right bottom))
   )
-  (text "GPI" (at 233.68 115.57 0)
+  (text "CCP2" (at 233.68 115.57 0)
     (effects (font (size 1.27 1.27)) (justify left bottom))
   )
@@
     )
   )
-  (hierarchical_label "RB6{slash}PGC{slash}UTX" (shape bidirectional) (at 208.28 93.98 0)
+  (hierarchical_label "RB6{slash}PGC{slash}UTX" (shape output) (at 208.28 93.98 0)
     (effects (font (size 1.27 1.27)) (justify left))
   )
@@
     (effects (font (size 1.27 1.27)) (justify left))
   )
-  (hierarchical_label "RB7{slash}PGD{slash}URX" (shape bidirectional) (at 208.28 91.44 0)
+  (hierarchical_label "RB7{slash}PGD{slash}URX" (shape input) (at 208.28 91.44 0)
     (effects (font (size 1.27 1.27)) (justify left))
   )

Commit message: Update
Connections:
- net RB0/EMERGENCY renamed RB0/URGENCY
Changed lines of the file:
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@@
     (effects (font (size 1.27 1.27)) (justify right))
   )
-  (hierarchical_label "RB0{slash}EMERGENCY" (shape bidirectional) (at 208.28 109.22 0)
+  (hierarchical_label "RB0{slash}URGENCY" (shape bidirectional) (at 208.28 109.22 0)
     (effects (font (size 1.27 1.27)) (justify left))
   )
