File: Kicad/mcu8/mcu.kicad_sch (KiCad schematic)
At the start: 9 parts, among them IC201 PIC16F1778, K201 MCU 1, K202 ICSP, K203 MCU 2

Commit message: Update
Connections:
- net RB2 renamed RB2/BATTERY_SENSE
- net RB3/BATTERY_SENSE renamed RB3/WHEEL_L_EN
- net RC7 renamed RC7/WHEEL_R_EN
Other:
- note added: "AN8"
- note added: "CCP2.TIMER1"
- note added: "CCP7.TIMER1"
- note added: "GPIO.OUT"
- note removed: "AN9"
- note removed: "Ajouter Connerter pour IR WHEEL"
- note removed: "CCP2"
- note removed: "CCP7"
- note removed: "GPO"
- note removed: "RA1 INPUT"
- note removed: "RAO INPUT"
Changed lines of the file:
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@@
     (effects (font (size 1.27 1.27)) (justify right bottom))
   )
-  (text "GPIO.NC" (at 233.68 105.41 0)
+  (text "AN8" (at 233.68 105.41 0)
     (effects (font (size 1.27 1.27)) (justify left bottom))
   )
@@
     (effects (font (size 1.27 1.27)) (justify right bottom))
   )
-  (text "GPO" (at 68.58 113.03 180)
+  (text "GPIO.OUT" (at 68.58 113.03 180)
     (effects (font (size 1.27 1.27)) (justify right bottom))
   )
@@
     (effects (font (size 1.27 1.27)) (justify right bottom))
   )
-  (text "CCP7" (at 233.68 100.33 0)
+  (text "CCP7.TIMER1" (at 233.68 100.33 0)
     (effects (font (size 1.27 1.27)) (justify left bottom))
-  )
-  (text "RAO INPUT " (at 33.02 35.56 0)
-    (effects (font (size 3 3)) (justify left bottom))
   )
   (text "GPIO.NC" (at 233.68 107.95 0)
@@
     (effects (font (size 1.27 1.27)) (justify right bottom))
   )
-  (text "Ajouter Connerter pour IR WHEEL" (at 30.48 27.94 0)
-    (effects (font (size 3 3)) (justify left bottom))
-  )
-  (text "GPIO.NC" (at 233.68 113.03 0)
+  (text "GPIO.OUT" (at 233.68 113.03 0)
     (effects (font (size 1.27 1.27)) (justify left bottom))
   )
@@
     (effects (font (size 1.27 1.27)) (justify left bottom))
   )
-  (text "RA1 INPUT " (at 33.02 40.64 0)
-    (effects (font (size 3 3)) (justify left bottom))
-  )
   (text "DRAFT" (at 210.82 187.96 0)
     (effects (font (size 5 5)) (justify left bottom))
@@
     (effects (font (size 1.27 1.27)) (justify right bottom))
   )
-  (text "CCP2" (at 233.68 115.57 0)
+  (text "CCP2.TIMER1" (at 233.68 115.57 0)
     (effects (font (size 1.27 1.27)) (justify left bottom))
   )
-  (text "GPO" (at 68.58 105.41 180)
+  (text "GPIO.OUT" (at 68.58 105.41 180)
     (effects (font (size 1.27 1.27)) (justify right bottom))
   )
@@
     (effects (font (size 1.27 1.27)) (justify right bottom))
   )
-  (text "AN9" (at 233.68 102.87 0)
+  (text "GPIO.OUT" (at 233.68 102.87 0)
     (effects (font (size 1.27 1.27)) (justify left bottom))
   )
@@
     )
   )
-  (global_label "RB2" (shape bidirectional) (at 208.28 104.14 0) (fields_autoplaced)
-    (effects (font (size 1.27 1.27)) (justify left))
-    (property "Intersheet References" "${INTERSHEET_REFS}" (id 0) (at 214.6331 104.0606 0)
-      (effects (font (size 1.27 1.27)) (justify left) hide)
-    )
-  )
   (global_label "RB1" (shape bidirectional) (at 208.28 106.68 0) (fields_autoplaced)
     (effects (font (size 1.27 1.27)) (justify left))
@@
     (property "Intersheet References" "${INTERSHEET_REFS}" (id 0) (at 75.1083 109.1406 0)
       (effects (font (size 1.27 1.27)) (justify right) hide)
-    )
-  )
-  (global_label "RC7" (shape bidirectional) (at 208.28 111.76 0) (fields_autoplaced)
-    (effects (font (size 1.27 1.27)) (justify left))
-    (property "Intersheet References" "${INTERSHEET_REFS}" (id 0) (at 214.6331 111.6806 0)
-      (effects (font (size 1.27 1.27)) (justify left) hide)
     )
   )
@@
     )
   )
-  (hierarchical_label "RB6{slash}PGC{slash}UTX" (shape output) (at 208.28 93.98 0)
+  (hierarchical_label "RB6{slash}PGC{slash}UTX" (shape bidirectional) (at 208.28 93.98 0)
     (effects (font (size 1.27 1.27)) (justify left))
   )
@@
     (effects (font (size 1.27 1.27)) (justify right))
   )
-  (hierarchical_label "RB3{slash}BATTERY_SENSE" (shape input) (at 208.28 101.6 0)
+  (hierarchical_label "RB2{slash}BATTERY_SENSE" (shape input) (at 208.28 104.14 0)
+    (effects (font (size 1.27 1.27)) (justify left))
+  )
+  (hierarchical_label "RB3{slash}WHEEL_L_EN" (shape output) (at 208.28 101.6 0)
     (effects (font (size 1.27 1.27)) (justify left))
   )
   (hierarchical_label "RC2" (shape bidirectional) (at 81.28 119.38 180)
     (effects (font (size 1.27 1.27)) (justify right))
+  )
+  (hierarchical_label "RC7{slash}WHEEL_R_EN" (shape output) (at 208.28 111.76 0)
+    (effects (font (size 1.27 1.27)) (justify left))
   )
   (hierarchical_label "RC0" (shape bidirectional) (at 81.28 114.3 180)
@@
     (effects (font (size 1.27 1.27)) (justify left))
   )
-  (hierarchical_label "RB7{slash}PGD{slash}URX" (shape input) (at 208.28 91.44 0)
+  (hierarchical_label "RB7{slash}PGD{slash}URX" (shape bidirectional) (at 208.28 91.44 0)
     (effects (font (size 1.27 1.27)) (justify left))
   )

Commit message: Update
Other:
- note added: "CCP2.TIMER1/?CLC"
- note added: "CCP7.TIMER1/?CLC"
- note added: "GPIO.IN/AN14"
- note removed: "CCP2.TIMER1"
- note removed: "CCP7.TIMER1"
- note removed: "GPIO"
Changed lines of the file:
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@@
     (effects (font (size 1.27 1.27)) (justify right bottom))
   )
-  (text "CCP7.TIMER1" (at 233.68 100.33 0)
+  (text "CCP7.TIMER1/?CLC" (at 233.68 100.33 0)
     (effects (font (size 1.27 1.27)) (justify left bottom))
   )
@@
     (effects (font (size 1.27 1.27)) (justify right bottom))
   )
-  (text "GPIO" (at 68.58 120.65 180)
+  (text "GPIO.IN/AN14" (at 68.58 120.65 180)
     (effects (font (size 1.27 1.27)) (justify right bottom))
   )
@@
     (effects (font (size 1.27 1.27)) (justify left bottom))
   )
-  (text "GPIO" (at 68.58 118.11 180)
+  (text "GPIO.OUT" (at 68.58 118.11 180)
     (effects (font (size 1.27 1.27)) (justify right bottom))
   )
-  (text "CCP2.TIMER1" (at 233.68 115.57 0)
+  (text "CCP2.TIMER1/?CLC" (at 233.68 115.57 0)
     (effects (font (size 1.27 1.27)) (justify left bottom))
   )
@@
     (effects (font (size 1.27 1.27)) (justify left bottom))
   )
-  (text "GPIO" (at 68.58 115.57 180)
+  (text "GPIO.OUT" (at 68.58 115.57 180)
     (effects (font (size 1.27 1.27)) (justify right bottom))
   )
@@
     (effects (font (size 1.27 1.27)) (justify left))
   )
-  (hierarchical_label "RC2" (shape bidirectional) (at 81.28 119.38 180)
+  (hierarchical_label "RC2" (shape input) (at 81.28 119.38 180)
     (effects (font (size 1.27 1.27)) (justify right))
   )
@@
     (effects (font (size 1.27 1.27)) (justify left))
   )
-  (hierarchical_label "RC0" (shape bidirectional) (at 81.28 114.3 180)
+  (hierarchical_label "RC0" (shape output) (at 81.28 114.3 180)
     (effects (font (size 1.27 1.27)) (justify right))
   )
@@
     (effects (font (size 1.27 1.27)) (justify left))
   )
-  (hierarchical_label "RC1" (shape bidirectional) (at 81.28 116.84 180)
+  (hierarchical_label "RC1" (shape output) (at 81.28 116.84 180)
     (effects (font (size 1.27 1.27)) (justify right))
   )

Commit message: Update
Connections:
- net RB4/WHEEL_L renamed RB4
- net RC4 renamed RC4/WHEEL_R
- net RC6/WHEEL_R renamed RC6/WHEEL_L
Other:
- note added: "TIMER3.CLK.GATE"
- note added: "TIMER5.CLK.GATE"
- note removed: "CCP2.TIMER1/?CLC"
- note removed: "CCP7.TIMER1/?CLC"
Changed lines of the file:
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@@
     (effects (font (size 1.27 1.27)) (justify right bottom))
   )
-  (text "CCP7.TIMER1/?CLC" (at 233.68 100.33 0)
+  (text "GPIO.NC" (at 233.68 100.33 0)
     (effects (font (size 1.27 1.27)) (justify left bottom))
   )
@@
     (effects (font (size 1.27 1.27)) (justify left bottom))
   )
-  (text "GPIO.NC" (at 233.68 120.65 0)
+  (text "TIMER3.CLK.GATE" (at 233.68 120.65 0)
     (effects (font (size 1.27 1.27)) (justify left bottom))
   )
@@
     (effects (font (size 1.27 1.27)) (justify right bottom))
   )
-  (text "CCP2.TIMER1/?CLC" (at 233.68 115.57 0)
+  (text "TIMER5.CLK.GATE" (at 233.68 115.57 0)
     (effects (font (size 1.27 1.27)) (justify left bottom))
   )
@@
     )
   )
-  (global_label "RC4" (shape bidirectional) (at 208.28 119.38 0) (fields_autoplaced)
+  (global_label "RB4" (shape bidirectional) (at 208.28 99.06 0) (fields_autoplaced)
     (effects (font (size 1.27 1.27)) (justify left))
-    (property "Intersheet References" "${INTERSHEET_REFS}" (id 0) (at 214.6331 119.3006 0)
+    (property "Intersheet References" "${INTERSHEET_REFS}" (id 0) (at 214.6331 98.9806 0)
       (effects (font (size 1.27 1.27)) (justify left) hide)
     )
@@
     (effects (font (size 1.27 1.27)) (justify right))
   )
-  (hierarchical_label "RC6{slash}WHEEL_R" (shape input) (at 208.28 114.3 0)
+  (hierarchical_label "RC4{slash}WHEEL_R" (shape input) (at 208.28 119.38 0)
     (effects (font (size 1.27 1.27)) (justify left))
   )
@@
     (effects (font (size 1.27 1.27)) (justify left))
   )
-  (hierarchical_label "RB4{slash}WHEEL_L" (shape input) (at 208.28 99.06 0)
+  (hierarchical_label "RC6{slash}WHEEL_L" (shape input) (at 208.28 114.3 0)
     (effects (font (size 1.27 1.27)) (justify left))
   )

Commit message: Update
Parts:
- C201, C202: footprint tronixio:CAPACITOR-1206 -> tronixio:CAPACITOR-SMD-1206; symbol tronixio:C-1206 -> tronixio:CAPACITOR-1206-100N; Mouser (none) -> 80-C1206C104M5R; Name (none) -> CAPACITOR-1206-100N; Tolerance (none) -> 20%; Voltage (none) -> 50V
- K201, K203: Name (none) -> HARWIN-254-M-1X14-VERTICAL
- K202: symbol tronixio:MICROCHIP-ICSP-M-2x03 -> tronixio:MICROCHIP-ICSP-M-2X03; Name ICSP -> MICROCHIP-ICSP-M-2X03
- R201: footprint tronixio:RESISTOR-1206 -> tronixio:RESISTOR-SMD-1206; symbol tronixio:R-1206 -> tronixio:RESISTOR-1206-10K; Mouser (none) -> 660-RK73B2BTTDD103J; Name (none) -> RESISTOR-1206-10K; Tolerance (none) -> 5%
- R202: footprint tronixio:RESISTOR-1206 -> tronixio:RESISTOR-SMD-1206; symbol tronixio:R-1206 -> tronixio:RESISTOR-1206-1K; Mouser (none) -> 660-RK73B2BTTDD102J; Name (none) -> RESISTOR-1206-1K; Tolerance (none) -> 5%
- S201: Name (none) -> ALPS-SKRPAC
- U201: renamed from IC201; footprint tronixio:DIP-28-W762-SOCKET -> tronixio:DIP-28-W762; Name PIC16F1778-ISP -> MICROCHIP-PIC16F1778-ISP

Commit message: Up
Parts:
- C201, C202: symbol tronixio:CAPACITOR-1206-100N -> tronixio:CAPACITOR-1206-100N-10P-X7R; Mouser 80-C1206C104M5R -> 187-CL31B106KAHNFNE; Name CAPACITOR-1206-100N -> (none); Tolerance 20% -> 10%
- K201: value MCU 1 -> HARWIN-254-M-1X14-VERTICAL; Name HARWIN-254-M-1X14-VERTICAL -> (none)
- K202: Name MICROCHIP-ICSP-M-2X03 -> (none)
- K203: value MCU 2 -> HARWIN-254-M-1X14-VERTICAL; Name HARWIN-254-M-1X14-VERTICAL -> (none)
- R201: value 10K -> 10k; symbol tronixio:RESISTOR-1206-10K -> tronixio:RESISTOR-1206-10K-5P; Name RESISTOR-1206-10K -> (none)
- R202: value 1K -> 1k; symbol tronixio:RESISTOR-1206-1K -> tronixio:RESISTOR-1206-1K-5P; Name RESISTOR-1206-1K -> (none)
- S201: Name ALPS-SKRPAC -> (none)
- U201: value PIC16F1778 -> MICROCHIP-PIC16F1778-ISP; Name MICROCHIP-PIC16F1778-ISP -> (none)

Commit message: Up
Parts:
- C201, C202: symbol tronixio:CAPACITOR-1206-100N-10P-X7R -> tronixio:CAPACITOR-1206-100N-50V-5P-X7R; Mouser 187-CL31B106KAHNFNE -> 80-C1206C104J5R; Tolerance 10% -> 5%
- K201: value HARWIN-254-M-1X14-VERTICAL -> MCU #1
- K202: Mouser 855-M20-9980346 -> 855-M20-998034
- K203: value HARWIN-254-M-1X14-VERTICAL -> MCU #2
- U201: value MICROCHIP-PIC16F1778-ISP -> PIC16F1778-ISP; footprint tronixio:DIP-28-W762 -> tronixio:DIP-28-W762-SOCKET
Connections:
- net RA6/LED renamed RA6/LED_DEBUG
- no-connect marks 0 -> 1
Other:
- moved on the sheet: K201, K203, R201, U201

Commit message: Up
Parts:
- added TP103: Debug, tronixio:KEYSTONE-2000-3, symbol tronixio:KEYSTONE-2000-3
Connections:
- net RA6/LED_DEBUG: now also TP103.1
- no-connect marks 1 -> 0
Changed lines of the file:
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@@
   (junction (at 111.76 76.2) (diameter 0.9144) (color 0 0 0 0)
   )
-  (no_connect (at 142.24 177.8))
   (wire (pts (xy 132.08 175.26) (xy 132.08 182.88))
     (stroke (width 0) (type solid))
@@
   (wire (pts (xy 200.66 50.8) (xy 208.28 50.8))
     (stroke (width 0) (type solid))
+  )
+  (wire (pts (xy 106.68 40.64) (xy 106.68 71.12))
+    (stroke (width 0) (type default))
   )
   (wire (pts (xy 78.74 180.34) (xy 81.28 180.34))
@@
         )
       )
+    )
+  )
+  (symbol (lib_id "tronixio:KEYSTONE-2000-3") (at 106.68 40.64 0) (unit 1)
+    (in_bom yes) (on_board yes) (dnp no)
+    (property "Reference" "TP103" (at 106.68 35.56 0) (do_not_autoplace)
+      (effects (font (size 1.15 1.15)))
+    )
+    (property "Value" "Debug" (at 106.68 35.56 0) (do_not_autoplace)
+      (effects (font (size 1.15 1.15)) hide)
+    )
+    (property "Footprint" "tronixio:KEYSTONE-2000-3" (at 106.68 48.26 0) (do_not_autoplace)
+      (effects (font (size 1 1)) hide)
+    )
+    (property "Datasheet" "https://www.keyelco.com/product.cfm/product_id/3037" (at 106.68 50.8 0) (do_not_autoplace)
+      (effects (font (size 1 1)) hide)
+    )
+    (property "Mouser" "534-2000-3" (at 106.68 53.34 0) (do_not_autoplace)
+      (effects (font (size 1 1)) hide)
+    )
+    (pin "1")
+    (instances
+      (project "tbot-8bit"
+        (path "/9c91caeb-16bc-4916-868d-9f9002ce0a61"
+          (reference "TP103") (unit 1)
+        )
+        (path "/9c91caeb-16bc-4916-868d-9f9002ce0a61/6012b3a0-2f30-4458-8240-bd443182c6c0"
+          (reference "TP201") (unit 1)
+        )
+      )

Commit message: Up
Parts:
- U201: footprint tronixio:DIP-28-W762-SOCKET -> tronixio:DIP-28-W762
Connections:
- net RB2/BATTERY_SENSE: no longer K203.6 (Pin_6), U201.23 (RB2)
- net RB4: no longer K203.4 (Pin_4), U201.25 (RB4)
- net RB3/WHEEL_L_EN renamed RB3/WHEEL_EN_R
- net RB5/SERVO_L: no longer names the net of K203.3 (Pin_3), U201.26 (RB5)
- net RC4/WHEEL_R renamed RC4/SERVO_L
- net RC5/SERVO_R renamed RC5/WHEEL_L
- net RC6/WHEEL_L renamed RC6/WHEEL_R
- net RC7/WHEEL_R_EN renamed RC7/WHEEL_EN_L
- new net: K203.4 (Pin_4), U201.25 (RB4)
- new net: K203.6 (Pin_6), U201.23 (RB2)
Other:
- note added: "?? TIMER.IN?? - GPIO.NC"
- note added: "TODO - GPIO.OUT"
- note added: "TODO - PWM11"
- note added: "TODO - PWM6"
- note added: "TODO - TIMER3.CLK.GATE"
- note added: "TODO - TIMER5.CLK.GATE"
- note added: "il faudrais pour les une wheel - pwm servo - 360 input - ir wheel en - ir wheel read -> 2x4= 8pins - si necessaire possible de bougerbattery sense"
- note removed: "PWM11"
- note removed: "PWM6"
- note removed: "TIMER3.CLK.GATE"
- note removed: "TIMER5.CLK.GATE"
Changed lines of the file:
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@@
     (effects (font (size 1.27 1.27)) (justify right bottom))
   )
-  (text "GPIO.NC" (at 233.68 99.695 0)
+  (text "?? TIMER.IN?? - GPIO.NC" (at 233.68 99.695 0)
     (effects (font (size 1.27 1.27)) (justify left bottom))
   )
@@
     (effects (font (size 1.27 1.27)) (justify right bottom))
   )
-  (text "GPIO.OUT" (at 233.68 112.395 0)
+  (text "il faudrais pour les une wheel\n- pwm servo\n- 360 input\n- ir wheel en\n- ir wheel read\n-> 2x4= 8pins\n- si necessaire possible de bougerbattery sense\n"
+    (at 86.36 154.94 0)
+    (effects (font (size 5 5)) (justify left bottom))
+  )
+  (text "TODO - GPIO.OUT" (at 233.68 112.395 0)
     (effects (font (size 1.27 1.27)) (justify left bottom))
   )
@@
     (effects (font (size 1.27 1.27)) (justify right bottom))
   )
-  (text "PWM6" (at 233.68 117.475 0)
+  (text "TODO - PWM6" (at 233.68 117.475 0)
     (effects (font (size 1.27 1.27)) (justify left bottom))
   )
@@
     (effects (font (size 1.27 1.27)) (justify left bottom))
   )
-  (text "TIMER3.CLK.GATE" (at 233.68 120.015 0)
+  (text "TODO - TIMER3.CLK.GATE" (at 233.68 120.015 0)
     (effects (font (size 1.27 1.27)) (justify left bottom))
   )
@@
     (effects (font (size 1.27 1.27)) (justify right bottom))
   )
-  (text "TIMER5.CLK.GATE" (at 233.68 114.935 0)
+  (text "TODO - TIMER5.CLK.GATE" (at 233.68 114.935 0)
     (effects (font (size 1.27 1.27)) (justify left bottom))
   )
@@
     (effects (font (size 1.27 1.27)) (justify right bottom))
   )
-  (text "PWM11" (at 233.68 97.155 0)
+  (text "TODO - PWM11" (at 233.68 97.155 0)
     (effects (font (size 1.27 1.27)) (justify left bottom))
   )
@@
     (effects (font (size 1.27 1.27)) (justify right bottom))
   )
-  (text "GPIO.OUT" (at 233.68 102.235 0)
+  (text "TODO - GPIO.OUT" (at 233.68 102.235 0)
     (effects (font (size 1.27 1.27)) (justify left bottom))
   )
@@
     )
   )
-  (global_label "RB4" (shape bidirectional) (at 208.28 99.06 0) (fields_autoplaced)
-    (effects (font (size 1.27 1.27)) (justify left))
-    (property "Intersheetrefs" "${INTERSHEET_REFS}" (at 214.6331 98.9806 0)
+  (global_label "RB4" (shape bidirectional) (at 223.52 86.36 0) (fields_autoplaced)
+    (effects (font (size 1.27 1.27)) (justify left))
+    (property "Intersheetrefs" "${INTERSHEET_REFS}" (at 229.8731 86.2806 0)
       (effects (font (size 1.27 1.27)) (justify left) hide)
     )
@@
     (effects (font (size 1.27 1.27)) (justify left))
   )
-  (hierarchical_label "RC4{slash}WHEEL_R" (shape input) (at 208.28 119.38 0) (fields_autoplaced)
+  (hierarchical_label "RC4{slash}SERVO_L" (shape input) (at 208.28 119.38 0) (fields_autoplaced)
     (effects (font (size 1.27 1.27)) (justify left))
   )
@@
     (effects (font (size 1.27 1.27)) (justify right))
   )
-  (hierarchical_label "RB2{slash}BATTERY_SENSE" (shape input) (at 208.28 104.14 0) (fields_autoplaced)
-    (effects (font (size 1.27 1.27)) (justify left))
-  )
-  (hierarchical_label "RB3{slash}WHEEL_L_EN" (shape output) (at 208.28 101.6 0) (fields_autoplaced)
+  (hierarchical_label "RB2{slash}BATTERY_SENSE" (shape input) (at 226.06 71.12 0) (fields_autoplaced)
+    (effects (font (size 1.27 1.27)) (justify left))
+  )
+  (hierarchical_label "RB3{slash}WHEEL_EN_R" (shape output) (at 208.28 101.6 0) (fields_autoplaced)
     (effects (font (size 1.27 1.27)) (justify left))
   )
@@
     (effects (font (size 1.27 1.27)) (justify right))
   )
-  (hierarchical_label "RC7{slash}WHEEL_R_EN" (shape output) (at 208.28 111.76 0) (fields_autoplaced)
+  (hierarchical_label "RC7{slash}WHEEL_EN_L" (shape output) (at 208.28 111.76 0) (fields_autoplaced)
     (effects (font (size 1.27 1.27)) (justify left))
   )
@@
     (effects (font (size 1.27 1.27)) (justify right))
   )
-  (hierarchical_label "RC5{slash}SERVO_R" (shape output) (at 208.28 116.84 0) (fields_autoplaced)
+  (hierarchical_label "RC5{slash}WHEEL_L" (shape output) (at 208.28 116.84 0) (fields_autoplaced)
     (effects (font (size 1.27 1.27)) (justify left))
   )
@@
     (effects (font (size 1.27 1.27)) (justify right))
   )
-  (hierarchical_label "RB5{slash}SERVO_L" (shape output) (at 208.28 96.52 0) (fields_autoplaced)
+  (hierarchical_label "RB4{slash}SERVO_R" (shape output) (at 213.36 99.06 0) (fields_autoplaced)
     (effects (font (size 1.27 1.27)) (justify left))
   )
@@
     (effects (font (size 1.27 1.27)) (justify left))
   )
-  (hierarchical_label "RC6{slash}WHEEL_L" (shape input) (at 208.28 114.3 0) (fields_autoplaced)
+  (hierarchical_label "RC6{slash}WHEEL_R" (shape input) (at 208.28 114.3 0) (fields_autoplaced)
     (effects (font (size 1.27 1.27)) (justify left))
   )
@@
       (effects (font (size 1.15 1.15)) (justify right))
     )
-    (property "Footprint" "tronixio:DIP-28-W762-SOCKET" (at 144.78 91.44 0) (do_not_autoplace)
-      (effects (font (size 1 1)) hide)
-    )
+    (property "Footprint" "tronixio:DIP-28-W762" (at 144.78 91.44 0) (do_not_autoplace)
+      (effects (font (size 1 1)) hide)
+    )
