File: Kicad/mcu8/hid.kicad_sch (KiCad schematic)
At the start: 27 parts, among them IC301 MCP2221A, K301 FRONT #1, K302 FRONT #2, K303 VIN, K304 +5V, K305 FRONT #3, K306 SERVO LEFT, K307 USB/UART, K308 SERVO RIGHT

Commit message: Draft
Other:
- note added: "DRAFT"
Changed lines of the file:
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@@
     (effects (font (size 1.27 1.27)) (justify right bottom))
+  )
+  (text "DRAFT" (at 208.28 187.96 0)
+    (effects (font (size 5 5)) (justify left bottom))
   )
   (text "IR WHEEL" (at 220.98 120.65 180)

Commit message: Update
Parts:
- removed IC301: MCP2221A, tronixio:SOIC-SL-14, symbol tronixio:MCP2221A-ISL
- added IC301: MICROCHIP-MCP2221A-ISL, tronixio:SOIC-SL-14, symbol tronixio:MICROCHIP-MCP2221A-ISL
- BB301: MOUSER 854-BB170 -> (none); Mouser (none) -> 854-BB170
- C301, C304: MOUSER 647-UVZ1E221MPD -> (none); Mouser (none) -> 647-UVZ1E221MPD
- K303, K304: MOUSER 855-M20-999084 -> (none); Mouser (none) -> 855-M20-999084
- K306, K308: MOUSER 855-M20-999044 -> (none); Mouser (none) -> 855-M20-999044
- K307: MOUSER 649-10118193-0001LF -> (none); Mouser (none) -> 649-10118193-0001LF
- LED301, LED302, LED303: MOUSER 604-APT3216LSECKJ3RV -> (none); Mouser (none) -> 604-APTR3216-VFX
- S301: MOUSER 612-TL1240RQ1JCLR -> (none); Mouser (none) -> 612-TL1240RQ1JCLR
Connections:
- net +5V: now also IC301.1 (VDD)
- net D+: now also IC301.13 (D+)
- net D-: now also IC301.12 (D-)
- net GND: now also IC301.14 (VSS)
- net RB6/PGC/UTX: now also IC301.5 (URx)
- net RB7/PGD/URX: now also IC301.6 (UTx)
- net at R307.1: now also IC301.3 (GP1)
- net at R309.1: now also IC301.2 (GP0)
- net at C303.1: now also IC301.11 (VUSB)
- net at R306.1: now also IC301.4 (~{RESET})
Other:
- moved on the sheet: LED301, R301, R302, R303, R304, S301A, S301B

Commit message: Update MCU
Changed lines of the file:
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@@
     (effects (font (size 1.27 1.27)) (justify left))
   )
-  (hierarchical_label "RB7{slash}PGD{slash}URX" (shape bidirectional) (at 248.92 50.8 0)
+  (hierarchical_label "RB7{slash}PGD{slash}URX" (shape output) (at 248.92 50.8 0)
     (effects (font (size 1.27 1.27)) (justify left))
   )
-  (hierarchical_label "RB6{slash}PGC{slash}UTX" (shape bidirectional) (at 248.92 48.26 0)
+  (hierarchical_label "RB6{slash}PGC{slash}UTX" (shape input) (at 248.92 48.26 0)
     (effects (font (size 1.27 1.27)) (justify left))
   )
@@
     (pin "3")
     (pin "4")
+    (pin "5")
+    (pin "6")
   )
   (symbol (lib_id "tronixio:POWER-+5V") (at 134.62 101.6 0) (mirror y) (unit 1)
@@
       (effects (font (size 1 1)) hide)
     )
+    (pin "1")
+    (pin "2")
+    (pin "3")
+    (pin "4")
     (pin "5")
     (pin "6")

Commit message: Update MCU 8Bit
Parts:
- added K307: WHEEL LEFT, tronixio:zzMOLEX-532530370, symbol tronixio:MOLEX-MICRO-LATCH-03-VERTICAL
- added K310: WHEEL RIGHT, tronixio:zzMOLEX-532530370, symbol tronixio:MOLEX-MICRO-LATCH-03-VERTICAL
- renumbered K307 to K308, K308 to K309
Connections:
- net +5V: now also K307.1, K310.1
- net GND: now also K307.3, K310.3
- net RB4/WHEEL_L: now also K307.2
- net RC6/WHEEL_R: now also K310.2

Commit message: Update MCU 8Bit
Parts:
- K307: value WHEEL LEFT -> LEFT
- K310: value WHEEL RIGHT -> RIGHT
Other:
- note added: "IR WHEEL LEFT"
- note added: "IR WHEEL RIGHT"
- note added: "RA0"
- note added: "RA1"
- note added: "RA2"
- note added: "RA3"
- note added: "RA4"
- note added: "RA5"
- note added: "RC SERVO"
- note added: "WHEEL 360"
- note removed: "IR WHEEL"
- note removed: "IR-LF1"
- note removed: "IR-LF2"
- note removed: "IR-LF3"
- note removed: "IR-LF4"
- note removed: "IR-LF5"
- note removed: "IR-LFEN"
- note removed: "SERVO"
Changed lines of the file:
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@@
+    (effects (font (size 1.27 1.27)) (justify right bottom))
+  )
+  (text "GND" (at 160.02 153.67 180)
     (effects (font (size 1.27 1.27)) (justify right bottom))
   )
@@
     (effects (font (size 1.27 1.27)) (justify right bottom))
   )
+  (text "IR WHEEL RIGHT" (at 220.98 151.13 180)
+    (effects (font (size 1.27 1.27)) (justify right bottom))
+  )
   (text "VIN" (at 220.98 115.57 180)
     (effects (font (size 1.27 1.27)) (justify right bottom))
@@
     (effects (font (size 1.27 1.27)) (justify right bottom))
   )
+  (text "IR WHEEL LEFT" (at 160.02 151.13 180)
+    (effects (font (size 1.27 1.27)) (justify right bottom))
+  )
   (text "GND" (at 220.98 113.03 180)
     (effects (font (size 1.27 1.27)) (justify right bottom))
@@
     (effects (font (size 1.27 1.27)) (justify right bottom))
   )
-  (text "IR-LF1" (at 53.34 59.69 180)
+  (text "RA2" (at 53.34 59.69 180)
     (effects (font (size 1.27 1.27)) (justify right bottom))
   )
@@
     (effects (font (size 1.27 1.27)) (justify right bottom))
   )
-  (text "IR-LF4" (at 93.98 59.69 180)
+  (text "RA5" (at 93.98 59.69 180)
     (effects (font (size 1.27 1.27)) (justify right bottom))
   )
@@
     (effects (font (size 1.27 1.27)) (justify right bottom))
   )
+  (text "+5V" (at 160.02 148.59 180)
+    (effects (font (size 1.27 1.27)) (justify right bottom))
+  )
+  (text "GND" (at 220.98 153.67 180)
+    (effects (font (size 1.27 1.27)) (justify right bottom))
+  )
+  (text "+5V" (at 220.98 148.59 180)
+    (effects (font (size 1.27 1.27)) (justify right bottom))
+  )
   (text "RC1" (at 134.62 62.23 180)
     (effects (font (size 1.27 1.27)) (justify right bottom))
   )
-  (text "IR WHEEL" (at 160.02 120.65 180)
-    (effects (font (size 1.27 1.27)) (justify right bottom))
-  )
-  (text "IR-LF5" (at 93.98 64.77 180)
-    (effects (font (size 1.27 1.27)) (justify right bottom))
-  )
-  (text "SERVO" (at 160.02 118.11 180)
-    (effects (font (size 1.27 1.27)) (justify right bottom))
-  )
-  (text "IR-LFEN" (at 93.98 62.23 180)
+  (text "WHEEL 360" (at 160.02 120.65 180)
+    (effects (font (size 1.27 1.27)) (justify right bottom))
+  )
+  (text "RA3" (at 93.98 64.77 180)
+    (effects (font (size 1.27 1.27)) (justify right bottom))
+  )
+  (text "RC SERVO" (at 160.02 118.11 180)
+    (effects (font (size 1.27 1.27)) (justify right bottom))
+  )
+  (text "RA4" (at 93.98 62.23 180)
     (effects (font (size 1.27 1.27)) (justify right bottom))
   )
@@
     (effects (font (size 5 5)) (justify left bottom))
   )
-  (text "IR WHEEL" (at 220.98 120.65 180)
-    (effects (font (size 1.27 1.27)) (justify right bottom))
-  )
-  (text "IR-LF3" (at 53.34 64.77 180)
+  (text "WHEEL 360" (at 220.98 120.65 180)
+    (effects (font (size 1.27 1.27)) (justify right bottom))
+  )
+  (text "RA0" (at 53.34 64.77 180)
     (effects (font (size 1.27 1.27)) (justify right bottom))
   )
@@
     (effects (font (size 1.27 1.27)) (justify right bottom))
   )
-  (text "SERVO" (at 220.98 118.11 180)
-    (effects (font (size 1.27 1.27)) (justify right bottom))
-  )
-  (text "IR-LF2" (at 53.34 62.23 180)
+  (text "RC SERVO" (at 220.98 118.11 180)
+    (effects (font (size 1.27 1.27)) (justify right bottom))
+  )
+  (text "RA1" (at 53.34 62.23 180)
     (effects (font (size 1.27 1.27)) (justify right bottom))
   )
@@
       (effects (font (size 1.15 1.15)))
     )
-    (property "Value" "WHEEL RIGHT" (id 1) (at 223.52 154.94 0)
+    (property "Value" "RIGHT" (id 1) (at 223.52 154.94 0)
       (effects (font (size 1.15 1.15)))
     )
@@
       (effects (font (size 1.15 1.15)))
     )
-    (property "Value" "WHEEL LEFT" (id 1) (at 162.56 154.94 0)
-      (effects (font (size 1.15 1.15)))
-    )
+    (property "Value" "LEFT" (id 1) (at 162.56 154.94 0)
+      (effects (font (size 1.15 1.15)))
+    )

Commit message: Update
Parts:
- removed S301: EMERGENCY, tronixio:E-SWITCH-TL1240XQ1JXXX, symbol tronixio:E-SWITCH-TL1240RQ1JCLR
- added S301: URGENCY, tronixio:zzzOMRON-B3W9000-X1, symbol tronixio:OMRON-B3W-9000-R1R
Connections:
- net GND: now also S301.3, S301.4
- net at R302.1, R303.1: now also S301.1, S301.2
- net at R301.1, R302.2: now also S301.6 (A)
- net RB0/EMERGENCY renamed RB0/URGENCY
- net RB0/URGENCY: now also S301.5 (C)
Changed lines of the file:
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@@
     (effects (font (size 1.27 1.27)) (justify left))
   )
-  (hierarchical_label "RB0{slash}EMERGENCY" (shape bidirectional) (at 66.04 167.64 180)
+  (hierarchical_label "RB0{slash}URGENCY" (shape bidirectional) (at 66.04 167.64 180)
     (effects (font (size 1.27 1.27)) (justify right))
   )
@@
     )
     (pin "1")
+  )
+  (symbol (lib_id "tronixio:OMRON-B3W-9000-R1R") (at 88.9 172.72 270) (unit 1)
+    (in_bom yes) (on_board yes)
+    (property "Reference" "S301" (id 0) (at 91.44 169.545 90)
+      (effects (font (size 1.15 1.15)) (justify left))
+    )
+    (property "Value" "URGENCY" (id 1) (at 91.44 175.895 90)
+      (effects (font (size 1.15 1.15)) (justify left))
+    )
+    (property "Footprint" "tronixio:zzzOMRON-B3W9000-X1" (id 2) (at 81.28 172.72 0)
+      (effects (font (size 1 1)) hide)
+    )
+    (property "Datasheet" "https://components.omron.com/us-en/datasheet_pdf/A167-E1.pdf" (id 3) (at 78.74 172.72 0)
+      (effects (font (size 1 1)) hide)
+    )
+    (property "Mouser" "653-B3W-9000-R1R" (id 4) (at 76.2 172.72 0)
+      (effects (font (size 1 1)) hide)
+    )
+    (pin "1")
+    (pin "2")
+    (pin "3")
+    (pin "4")
+    (pin "5")
+    (pin "6")
   )
   (symbol (lib_id "tronixio:R-1206") (at 80.01 167.64 270) (unit 1)
@@
     (pin "2")
   )
-  (symbol (lib_id "tronixio:E-SWITCH-TL1240RQ1JCLR") (at 88.9 172.72 270) (mirror x) (unit 1)
-    (in_bom yes) (on_board yes)
-    (property "Reference" "S301" (id 0) (at 92.71 176.53 90)
-      (effects (font (size 1.15 1.15)))
-    )
-    (property "Value" "EMERGENCY" (id 1) (at 94.615 168.91 90)
-      (effects (font (size 1.15 1.15)))
-    )
-    (property "Footprint" "tronixio:E-SWITCH-TL1240XQ1JXXX" (id 2) (at 81.28 172.72 0)
-      (effects (font (size 1 1)) hide)
-    )
-    (property "Datasheet" "https://www.e-switch.com/product-catalog/tact/product-lines/tl1240-series-illuminated-tact-switches#.XnJ2Ri2ZPUI" (id 3) (at 78.74 172.72 0)
-      (effects (font (size 1 1)) hide)
-    )
-    (property "Mouser" "612-TL1240RQ1JCLR" (id 4) (at 76.2 172.72 0)
-      (effects (font (size 1 1)) hide)
-    )
-    (pin "1")
-    (pin "2")
-    (pin "3")
-    (pin "4")
-    (pin "5")
-    (pin "6")
-  )
   (symbol (lib_id "tronixio:POWER-+5V") (at 134.62 101.6 0) (mirror y) (unit 1)
     (in_bom yes) (on_board yes)
@@
     (pin "2")
   )
+  (symbol (lib_id "tronixio:OMRON-B3W-9000-R1R") (at 73.66 162.56 90) (unit 2)
+    (in_bom yes) (on_board yes)
+    (property "Reference" "S301" (id 0) (at 73.025 159.385 90)
+      (effects (font (size 1.15 1.15)) (justify left))
+    )
+    (property "Value" "URGENCY" (id 1) (at 73.025 165.1 90)
+      (effects (font (size 1.15 1.15)) (justify left))
+    )
+    (property "Footprint" "tronixio:zzzOMRON-B3W9000-X1" (id 2) (at 81.28 162.56 0)
+      (effects (font (size 1 1)) hide)
+    )
+    (property "Datasheet" "https://components.omron.com/us-en/datasheet_pdf/A167-E1.pdf" (id 3) (at 83.82 162.56 0)
+      (effects (font (size 1 1)) hide)
+    )
+    (property "Mouser" "653-B3W-9000-R1R" (id 4) (at 86.36 162.56 0)
+      (effects (font (size 1 1)) hide)
+    )
+    (pin "1")
+    (pin "2")
+    (pin "3")
+    (pin "4")
+    (pin "5")
+    (pin "6")
+  )
   (symbol (lib_id "tronixio:R-1206") (at 80.01 157.48 270) (unit 1)
     (in_bom yes) (on_board yes)
@@
     (pin "5")
   )
-  (symbol (lib_id "tronixio:E-SWITCH-TL1240RQ1JCLR") (at 73.66 162.56 90) (unit 2)
-    (in_bom yes) (on_board yes)
-    (property "Reference" "S301" (id 0) (at 67.31 159.385 90)
-      (effects (font (size 1.15 1.15)) (justify right))
-    )
-    (property "Value" "EMERGENCY" (id 1) (at 62.23 165.1 90)
-      (effects (font (size 1.15 1.15)) (justify right))
-    )
-    (property "Footprint" "tronixio:E-SWITCH-TL1240XQ1JXXX" (id 2) (at 81.28 162.56 0)
-      (effects (font (size 1 1)) hide)
-    )
-    (property "Datasheet" "https://www.e-switch.com/product-catalog/tact/product-lines/tl1240-series-illuminated-tact-switches#.XnJ2Ri2ZPUI" (id 3) (at 83.82 162.56 0)
-      (effects (font (size 1 1)) hide)
-    )
-    (property "Mouser" "612-TL1240RQ1JCLR" (id 4) (at 86.36 162.56 0)
-      (effects (font (size 1 1)) hide)
-    )
-    (pin "1")
-    (pin "2")
-    (pin "3")
-    (pin "4")
-    (pin "5")
-    (pin "6")
-  )
   (symbol (lib_id "tronixio:C-1206") (at 200.66 73.66 0) (unit 1)

Commit message: Update
Parts:
- added Q301, Q302: DIODESINC-DMP2305U-SOT-23, tronixio:SOT-23-3, symbol tronixio:DIODESINC-DMP2305U-SOT-23
Connections:
- net +5V: now also Q301.2 (S), Q302.2 (S); no longer K307.1, K310.1
- new net: K310.1, Q302.3 (D)
- new net: K307.1, Q301.3 (D)
- new net RB3/WHEEL_L_EN: Q301.1 (G)
- new net RC7/WHEEL_R_EN: Q302.1 (G)
Other:
- moved on the sheet: BB301, C301, C302, C303, C304, IC301, K301, K302, K303, K304, K305, K306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

Commit message: Update
Parts:
- K302: value FRONT #2 -> FRONT #3
- K305: value FRONT #3 -> FRONT #2
Other:
- moved on the sheet: K302, K305
