File: Kicad/mcu8/hid.kicad_sch (KiCad schematic)
At the start: 31 parts, among them IC301 MICROCHIP-MCP2221A-ISL, K301 FRONT #1, K302 FRONT #3, K303 VIN, K304 +5V, K305 FRONT #2, K306 SERVO LEFT, K307 LEFT, K308 USB/UART, K309 SERVO RIGHT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

Commit message: Update
Connections:
- net RB4/WHEEL_L renamed RC6/WHEEL_L
- net RC6/WHEEL_R renamed RC4/WHEEL_R
Changed lines of the file:
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@@
     (stroke (width 0) (type solid) (color 0 0 0 0))
+  )
+  (wire (pts (xy 167.64 142.24) (xy 167.64 144.78))
+    (stroke (width 0) (type default) (color 0 0 0 0))
   )
   (wire (pts (xy 220.98 116.84) (xy 243.84 116.84))
@@
   (wire (pts (xy 180.34 114.3) (xy 182.88 114.3))
     (stroke (width 0) (type solid) (color 0 0 0 0))
+  )
+  (wire (pts (xy 228.6 142.24) (xy 228.6 144.78))
+    (stroke (width 0) (type default) (color 0 0 0 0))
   )
   (wire (pts (xy 134.62 63.5) (xy 142.24 63.5))
@@
     (effects (font (size 1.27 1.27)) (justify left))
   )
-  (hierarchical_label "RC6{slash}WHEEL_R" (shape output) (at 236.22 160.02 0)
+  (hierarchical_label "RC4{slash}WHEEL_R" (shape output) (at 236.22 160.02 0)
     (effects (font (size 1.27 1.27)) (justify left))
   )
@@
     (effects (font (size 1.27 1.27)) (justify left))
   )
-  (hierarchical_label "RB4{slash}WHEEL_L" (shape output) (at 175.26 160.02 0)
+  (hierarchical_label "RC6{slash}WHEEL_L" (shape output) (at 175.26 160.02 0)
     (effects (font (size 1.27 1.27)) (justify left))
   )
@@
     (effects (font (size 1.27 1.27)) (justify left))
   )
-  (hierarchical_label "RC6{slash}WHEEL_R" (shape output) (at 243.84 116.84 0)
+  (hierarchical_label "RC4{slash}WHEEL_R" (shape output) (at 243.84 116.84 0)
     (effects (font (size 1.27 1.27)) (justify left))
   )
@@
     (effects (font (size 1.27 1.27)) (justify left))
   )
-  (hierarchical_label "RB4{slash}WHEEL_L" (shape output) (at 182.88 116.84 0)
+  (hierarchical_label "RC6{slash}WHEEL_L" (shape output) (at 182.88 116.84 0)
     (effects (font (size 1.27 1.27)) (justify left))
   )
@@
     (pin "8")
   )
-  (symbol (lib_id "tronixio:POWER-+5V") (at 228.6 144.78 0) (mirror y) (unit 1)
-    (in_bom yes) (on_board yes)
-    (property "Reference" "#PWR0335" (id 0) (at 223.52 142.24 0)
-      (effects (font (size 1 1)) hide)
-    )
-    (property "Value" "+5V" (id 1) (at 228.6 139.7 0)
-      (effects (font (size 1 1)) hide)
-    )
-    (property "Footprint" "" (id 2) (at 228.6 144.78 0)
-      (effects (font (size 1 1)) hide)
-    )
-    (property "Datasheet" "" (id 3) (at 228.6 144.78 0)
-      (effects (font (size 1 1)) hide)
-    )
-    (property "Name" "+5V" (id 4) (at 228.6 139.7 0)
+  (symbol (lib_id "tronixio:POWER-+5V") (at 228.6 142.24 0) (mirror y) (unit 1)
+    (in_bom yes) (on_board yes)
+    (property "Reference" "#PWR0335" (id 0) (at 223.52 139.7 0)
+      (effects (font (size 1 1)) hide)
+    )
+    (property "Value" "+5V" (id 1) (at 228.6 137.16 0)
+      (effects (font (size 1 1)) hide)
+    )
+    (property "Footprint" "" (id 2) (at 228.6 142.24 0)
+      (effects (font (size 1 1)) hide)
+    )
+    (property "Datasheet" "" (id 3) (at 228.6 142.24 0)
+      (effects (font (size 1 1)) hide)
+    )
+    (property "Name" "+5V" (id 4) (at 228.6 137.16 0)
       (effects (font (size 1.15 1.15)))
     )
@@
     (pin "1")
   )
-  (symbol (lib_id "tronixio:POWER-+5V") (at 167.64 144.78 0) (mirror y) (unit 1)
-    (in_bom yes) (on_board yes)
-    (property "Reference" "#PWR0324" (id 0) (at 162.56 142.24 0)
-      (effects (font (size 1 1)) hide)
-    )
-    (property "Value" "+5V" (id 1) (at 167.64 139.7 0)
-      (effects (font (size 1 1)) hide)
-    )
-    (property "Footprint" "" (id 2) (at 167.64 144.78 0)
-      (effects (font (size 1 1)) hide)
-    )
-    (property "Datasheet" "" (id 3) (at 167.64 144.78 0)
-      (effects (font (size 1 1)) hide)
-    )
-    (property "Name" "+5V" (id 4) (at 167.64 139.7 0)
-      (effects (font (size 1.15 1.15)))
-    )
+  (symbol (lib_id "tronixio:POWER-+5V") (at 167.64 142.24 0) (mirror y) (unit 1)
+    (in_bom yes) (on_board yes)
+    (property "Reference" "#PWR0324" (id 0) (at 162.56 139.7 0)
+      (effects (font (size 1 1)) hide)
+    )
+    (property "Value" "+5V" (id 1) (at 167.64 137.16 0)
+      (effects (font (size 1 1)) hide)
+    )
+    (property "Footprint" "" (id 2) (at 167.64 142.24 0)
+      (effects (font (size 1 1)) hide)
+    )
+    (property "Datasheet" "" (id 3) (at 167.64 142.24 0)
+      (effects (font (size 1 1)) hide)
+    )
+    (property "Name" "+5V" (id 4) (at 167.64 137.16 0)
+      (effects (font (size 1.15 1.15)))
+    )

Commit message: Update
Parts:
- C301, C304: symbol tronixio:UVZ-220U-25V -> tronixio:NICHICON-UVZ-220U-25V; Name 220µ/25V -> NICHICON-UVZ-220U-25V; Tolerance (none) -> 20%; Voltage (none) -> 25V
- C302: footprint tronixio:CAPACITOR-1206 -> tronixio:CAPACITOR-SMD-1206; symbol tronixio:C-1206 -> tronixio:CAPACITOR-1206-100N; Mouser (none) -> 80-C1206C104M5R; Name (none) -> CAPACITOR-1206-100N; Tolerance (none) -> 20%; Voltage (none) -> 50V
- C303: footprint tronixio:CAPACITOR-1206 -> tronixio:CAPACITOR-SMD-1206; symbol tronixio:C-1206 -> tronixio:CAPACITOR-1206-470N; Mouser (none) -> 80-C1206C474M5R; Name (none) -> CAPACITOR-1206-470N; Tolerance (none) -> 20%; Voltage (none) -> 50V
- K301, K302, K305: MOUSER 538-53253-0570 -> (none); Mouser (none) -> 538-53253-0570; Name (none) -> MOLEX-MICRO-LATCH-05-VERTICAL
- K303, K304: Name (none) -> HARWIN-254-F-1X06-VERTICAL
- K306, K309: Name (none) -> HARWIN-254-M-1X04-VERTICAL
- K307, K310: footprint tronixio:zzMOLEX-532530370 -> tronixioZZ:MOLEX-532530370; MOUSER 538-53253-0370 -> (none); Mouser (none) -> 538-53253-0370; Name (none) -> MOLEX-MICRO-LATCH-03-VERTICAL
- K308: Name (none) -> FCI-USB-TYPE-B-MICRO-THT
- LED301, LED302, LED303: footprint tronixio:LED-1206 -> tronixio:LED-SMD-1206; symbol tronixio:LED-1206-PURPLE -> tronixio:KINGBRIGHT-LED-1206-PURPLE; Name (none) -> KINGBRIGHT-LED-1206-PURPLE
- Q301, Q302: value DIODESINC-DMP2305U-SOT-23 -> DMP2305U; Name DMP2305U -> DIODESINC-DMP2305U-SOT-23
- R301, R305, R308: footprint tronixio:RESISTOR-1206 -> tronixio:RESISTOR-SMD-1206; symbol tronixio:R-1206 -> tronixio:RESISTOR-1206-220R; Mouser (none) -> 660-RK73B2BTTDD221J; Name (none) -> RESISTOR-1206-220R; Tolerance (none) -> 5%
- R302: footprint tronixio:RESISTOR-1206 -> tronixio:RESISTOR-SMD-1206; symbol tronixio:R-1206 -> tronixio:RESISTOR-1206-150R; Mouser (none) -> 660-RK73B2BTTDD151J; Name (none) -> RESISTOR-1206-150R; Tolerance (none) -> 5%
- R303: footprint tronixio:RESISTOR-1206 -> tronixio:RESISTOR-SMD-1206; symbol tronixio:R-1206 -> tronixio:RESISTOR-1206-330R; Mouser (none) -> 660-RK73B2BTTDD331J; Name (none) -> RESISTOR-1206-330R; Tolerance (none) -> 5%
- R304, R307, R309: footprint tronixio:RESISTOR-1206 -> tronixio:RESISTOR-SMD-1206; symbol tronixio:R-1206 -> tronixio:RESISTOR-1206-4K7; Mouser (none) -> 660-RK73B2BTTDD472J; Name (none) -> RESISTOR-1206-4K7; Tolerance (none) -> 5%
- R306: footprint tronixio:RESISTOR-1206 -> tronixio:RESISTOR-SMD-1206; symbol tronixio:R-1206 -> tronixio:RESISTOR-1206-10K; Mouser (none) -> 660-RK73B2BTTDD103J; Name (none) -> RESISTOR-1206-10K; Tolerance (none) -> 5%
- S301: footprint tronixio:zzzOMRON-B3W9000-X1 -> tronixioZZZ:OMRON-B3W9000-X1; Name (none) -> OMRON-B3W-9000-R1R
- U301: renamed from IC301; value MICROCHIP-MCP2221A-ISL -> MCP2221A; footprint tronixio:SOIC-SL-14 -> tronixio:SOIC-14; Name MCP2221A-ISL -> MICROCHIP-MCP2221A-ISL

Commit message: Up
Parts:
- C301, C304: value 220µ/25V -> 220µ; Name NICHICON-UVZ-220U-25V -> (none)
- C302: symbol tronixio:CAPACITOR-1206-100N -> tronixio:CAPACITOR-1206-100N-10P-X7R; Mouser 80-C1206C104M5R -> 187-CL31B106KAHNFNE; Name CAPACITOR-1206-100N -> (none); Tolerance 20% -> 10%
- C303: symbol tronixio:CAPACITOR-1206-470N -> tronixio:CAPACITOR-1206-470N-20P-X7R; Name CAPACITOR-1206-470N -> (none)
- K301: value FRONT #1 -> Front #1; Name MOLEX-MICRO-LATCH-05-VERTICAL -> (none)
- K302: value FRONT #3 -> Front #3; Name MOLEX-MICRO-LATCH-05-VERTICAL -> (none)
- K303, K304: Name HARWIN-254-F-1X06-VERTICAL -> (none)
- K305: value FRONT #2 -> Front #2; Name MOLEX-MICRO-LATCH-05-VERTICAL -> (none)
- K306: value SERVO LEFT -> Servo Left; Name HARWIN-254-M-1X04-VERTICAL -> (none)
- K307: value LEFT -> Left; footprint tronixioZZ:MOLEX-532530370 -> tronixio:MOLEX-532530370; Name MOLEX-MICRO-LATCH-03-VERTICAL -> (none)
- K308: value USB/UART -> USB; Name FCI-USB-TYPE-B-MICRO-THT -> (none)
- K309: value SERVO RIGHT -> Servo Right; Name HARWIN-254-M-1X04-VERTICAL -> (none)
- K310: value RIGHT -> Right; footprint tronixioZZ:MOLEX-532530370 -> tronixio:MOLEX-532530370; Name MOLEX-MICRO-LATCH-03-VERTICAL -> (none)
- LED301, LED302, LED303: Name KINGBRIGHT-LED-1206-PURPLE -> (none)
- Q301, Q302: symbol tronixio:DIODESINC-DMP2305U-SOT-23 -> tronixio:DIODES-DMP2305U-SOT; Name DIODESINC-DMP2305U-SOT-23 -> (none)
- R301, R305, R308: symbol tronixio:RESISTOR-1206-220R -> tronixio:RESISTOR-1206-220R-5P; Name RESISTOR-1206-220R -> (none)
- R302: symbol tronixio:RESISTOR-1206-150R -> tronixio:RESISTOR-1206-150R-5P; Name RESISTOR-1206-150R -> (none)
- R303: symbol tronixio:RESISTOR-1206-330R -> tronixio:RESISTOR-1206-330R-5P; Name RESISTOR-1206-330R -> (none)
- R304, R307, R309: value 4K7 -> 4k7; symbol tronixio:RESISTOR-1206-4K7 -> tronixio:RESISTOR-1206-4K7-5P; Name RESISTOR-1206-4K7 -> (none)
- R306: value 10K -> 10k; symbol tronixio:RESISTOR-1206-10K -> tronixio:RESISTOR-1206-10K-5P; Name RESISTOR-1206-10K -> (none)
- S301: value URGENCY -> Urgency; footprint tronixioZZZ:OMRON-B3W9000-X1 -> tronixio:OMRON-B3W9000-X1
- U301: Name MICROCHIP-MCP2221A-ISL -> (none)

Commit message: Up
Parts:
- added R310, R311: 100Ω, tronixio:RESISTOR-SMD-1206, symbol tronixio:RESISTOR-1206-100R-5P
- C301, C304: Life (none) -> 1000H; Serie (none) -> UVZ
- C302: symbol tronixio:CAPACITOR-1206-100N-10P-X7R -> tronixio:CAPACITOR-1206-100N-50V-5P-X7R; Mouser 187-CL31B106KAHNFNE -> 80-C1206C104J5R; Tolerance 10% -> 5%
- C303: symbol tronixio:CAPACITOR-1206-470N-20P-X7R -> tronixio:CAPACITOR-1206-470N-50V-5P-X7R; Mouser 80-C1206C474M5R -> 791-1206B474J500CT; Tolerance 20% -> 5%
- K303, K304: Mouser 855-M20-999084 -> 855-M20-782084
- K307: value Left -> Wheel Left
- K308: value USB -> USB/EUSART; footprint tronixio:FCI-USB-TYPE-B-MICRO-THT -> tronixio:USB-TYPE-B-MICRO-TH; symbol tronixio:FCI-USB-TYPE-B-MICRO-THT -> tronixio:FCI-USB-TYPE-B-MICRO-TH
- K310: value Right -> Wheel Right
- S301: Name OMRON-B3W-9000-R1R -> (none)
Connections:
- net GND: now also K308.SH (SHIELD); no longer K308.6 (SHIELD)
- net RB3/WHEEL_L_EN: now also R310.1; no longer Q301.1 (G)
- net RC7/WHEEL_R_EN: now also R311.1; no longer Q302.1 (G)
- net VIN renamed +VIN
- new net: Q301.1 (G), R310.2
- new net: Q302.1 (G), R311.2
Other:
- moved on the sheet: BB301, C302, LED303, R302, R303, R309, S301A

Commit message: Up
Parts:
- added R312, R313: 100Ω, tronixio:RESISTOR-SMD-1206, symbol tronixio:RESISTOR-1206-100R-5P
Connections:
- net RB6/PGC/UTX: now also R312.1; no longer U301.5 (URx)
- net RB7/PGD/URX: now also R313.1; no longer U301.6 (UTx)
- net RA6/LED renamed RA6/LED_DEBUG
- new net: R313.2, U301.6 (UTx)
- new net: R312.2, U301.5 (URx)
Changed lines of the file:
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@@
     (stroke (width 0) (type default))
   )
-  (wire (pts (xy 228.6 50.8) (xy 246.38 50.8))
+  (wire (pts (xy 228.6 50.8) (xy 243.84 50.8))
     (stroke (width 0) (type solid))
   )
@@
     (stroke (width 0) (type solid))
   )
-  (wire (pts (xy 228.6 48.26) (xy 246.38 48.26))
+  (wire (pts (xy 228.6 48.26) (xy 243.84 48.26))
     (stroke (width 0) (type solid))
   )
@@
     (effects (font (size 1.27 1.27)) (justify left))
   )
-  (hierarchical_label "RB7{slash}PGD{slash}URX" (shape bidirectional) (at 246.38 50.8 0) (fields_autoplaced)
+  (hierarchical_label "RB7{slash}PGD{slash}URX" (shape bidirectional) (at 254 50.8 0) (fields_autoplaced)
     (effects (font (size 1.27 1.27)) (justify left))
   )
-  (hierarchical_label "RB6{slash}PGC{slash}UTX" (shape bidirectional) (at 246.38 48.26 0) (fields_autoplaced)
+  (hierarchical_label "RB6{slash}PGC{slash}UTX" (shape bidirectional) (at 254 48.26 0) (fields_autoplaced)
     (effects (font (size 1.27 1.27)) (justify left))
   )
@@
     (effects (font (size 1.27 1.27)) (justify left))
   )
-  (hierarchical_label "RA6{slash}LED" (shape input) (at 121.92 147.32 180) (fields_autoplaced)
+  (hierarchical_label "RA6{slash}LED_DEBUG" (shape input) (at 121.92 147.32 180) (fields_autoplaced)
     (effects (font (size 1.27 1.27)) (justify right))
   )
@@
         (path "/9c91caeb-16bc-4916-868d-9f9002ce0a61/56bd3a46-de12-45e9-9566-afec966f2cad"
           (reference "K310") (unit 1)
+        )
+      )
+    )
+  )
+  (symbol (lib_id "tronixio:RESISTOR-1206-100R-5P") (at 248.92 50.8 270) (unit 1)
+    (in_bom yes) (on_board yes) (dnp no)
+    (property "Reference" "R313" (at 248.92 53.34 90) (do_not_autoplace)
+      (effects (font (size 1.15 1.15)))
+    )
+    (property "Value" "100Ω" (at 248.92 50.8 90) (do_not_autoplace)
+      (effects (font (size 1.15 1.15)))
+    )
+    (property "Footprint" "tronixio:RESISTOR-SMD-1206" (at 233.68 50.8 0) (do_not_autoplace)
+      (effects (font (size 1 1)) hide)
+    )
+    (property "Datasheet" "" (at 231.14 50.8 0)
+      (effects (font (size 1 1)) hide)
+    )
+    (property "Tolerance" "5%" (at 245.11 53.34 0) (do_not_autoplace)
+      (effects (font (size 1.15 1.15)) (justify left) hide)
+    )
+    (property "Mouser" "660-RK73B2BTTDD101J" (at 228.6 50.8 0) (do_not_autoplace)
+      (effects (font (size 1 1)) hide)
+    )
+    (pin "1")
+    (pin "2")
+    (instances
+      (project "tbot-8bit"
+        (path "/9c91caeb-16bc-4916-868d-9f9002ce0a61/56bd3a46-de12-45e9-9566-afec966f2cad"
+          (reference "R313") (unit 1)
         )
       )
@@
         )
       )
+    )
+  )
+  (symbol (lib_id "tronixio:RESISTOR-1206-100R-5P") (at 248.92 48.26 270) (unit 1)
+    (in_bom yes) (on_board yes) (dnp no)
+    (property "Reference" "R312" (at 248.92 45.72 90) (do_not_autoplace)
+      (effects (font (size 1.15 1.15)))
+    )
+    (property "Value" "100Ω" (at 248.92 48.26 90) (do_not_autoplace)
+      (effects (font (size 1.15 1.15)))
+    )
+    (property "Footprint" "tronixio:RESISTOR-SMD-1206" (at 233.68 48.26 0) (do_not_autoplace)
+      (effects (font (size 1 1)) hide)
+    )
+    (property "Datasheet" "" (at 231.14 48.26 0)
+      (effects (font (size 1 1)) hide)
+    )
+    (property "Tolerance" "5%" (at 245.11 50.8 0) (do_not_autoplace)
+      (effects (font (size 1.15 1.15)) (justify left) hide)
+    )
+    (property "Mouser" "660-RK73B2BTTDD101J" (at 228.6 48.26 0) (do_not_autoplace)
+      (effects (font (size 1 1)) hide)
+    )
+    (pin "1")
+    (pin "2")
+    (instances
+      (project "tbot-8bit"
+        (path "/9c91caeb-16bc-4916-868d-9f9002ce0a61/56bd3a46-de12-45e9-9566-afec966f2cad"
+          (reference "R312") (unit 1)
+        )
+      )

Commit message: Up
Parts:
- K306: value Servo Left -> Servo Right
- K307: value Wheel Left -> Wheel Right
- K309: value Servo Right -> Servo Left
- K310: value Wheel Right -> Wheel Left
- S301: value Urgency -> Stop
Connections:
- net RB0/URGENCY renamed RB0/STOP
- net RB3/WHEEL_L_EN renamed RB3/WHEEL_EN_R
- net RB5/SERVO_L renamed RB5/SERVO_R
- net RC4/WHEEL_R renamed RC4/SERVO_L
- net RC5/SERVO_R renamed RC5/WHEEL_L
- net RC6/WHEEL_L renamed RC6/WHEEL_R
- net RC7/WHEEL_R_EN renamed RC7/WHEEL_EN_L
Changed lines of the file:
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@@
     (effects (font (size 1.27 1.27)) (justify left))
   )
-  (hierarchical_label "RC4{slash}WHEEL_R" (shape output) (at 236.22 160.02 0) (fields_autoplaced)
+  (hierarchical_label "RC4{slash}SERVO_L" (shape output) (at 236.22 160.02 0) (fields_autoplaced)
     (effects (font (size 1.27 1.27)) (justify left))
   )
-  (hierarchical_label "RC5{slash}SERVO_R" (shape input) (at 243.84 114.3 0) (fields_autoplaced)
+  (hierarchical_label "RC5{slash}WHEEL_L" (shape input) (at 243.84 114.3 0) (fields_autoplaced)
     (effects (font (size 1.27 1.27)) (justify left))
   )
@@
     (effects (font (size 1.27 1.27)) (justify left))
   )
-  (hierarchical_label "RB5{slash}SERVO_L" (shape input) (at 182.88 114.3 0) (fields_autoplaced)
+  (hierarchical_label "RB5{slash}SERVO_R" (shape input) (at 182.88 114.3 0) (fields_autoplaced)
     (effects (font (size 1.27 1.27)) (justify left))
   )
-  (hierarchical_label "RB3{slash}WHEEL_L_EN" (shape input) (at 182.88 149.86 0) (fields_autoplaced)
+  (hierarchical_label "RB3{slash}WHEEL_EN_R" (shape input) (at 182.88 149.86 0) (fields_autoplaced)
     (effects (font (size 1.27 1.27)) (justify left))
   )
@@
     (effects (font (size 1.27 1.27)) (justify right))
   )
-  (hierarchical_label "RC7{slash}WHEEL_R_EN" (shape input) (at 243.84 149.86 0) (fields_autoplaced)
+  (hierarchical_label "RC7{slash}WHEEL_EN_L" (shape input) (at 243.84 149.86 0) (fields_autoplaced)
     (effects (font (size 1.27 1.27)) (justify left))
   )
@@
     (effects (font (size 1.27 1.27)) (justify left))
   )
-  (hierarchical_label "RC6{slash}WHEEL_L" (shape output) (at 175.26 160.02 0) (fields_autoplaced)
+  (hierarchical_label "RC6{slash}WHEEL_R" (shape output) (at 175.26 160.02 0) (fields_autoplaced)
     (effects (font (size 1.27 1.27)) (justify left))
   )
-  (hierarchical_label "RB0{slash}URGENCY" (shape bidirectional) (at 60.96 154.94 180) (fields_autoplaced)
+  (hierarchical_label "RB0{slash}STOP" (shape bidirectional) (at 60.96 154.94 180) (fields_autoplaced)
     (effects (font (size 1.27 1.27)) (justify right))
   )
@@
     (effects (font (size 1.27 1.27)) (justify left))
   )
-  (hierarchical_label "RC4{slash}WHEEL_R" (shape output) (at 243.84 116.84 0) (fields_autoplaced)
+  (hierarchical_label "RC4{slash}SERVO_L" (shape output) (at 243.84 116.84 0) (fields_autoplaced)
     (effects (font (size 1.27 1.27)) (justify left))
   )
@@
     (effects (font (size 1.27 1.27)) (justify left))
   )
-  (hierarchical_label "RC6{slash}WHEEL_L" (shape output) (at 182.88 116.84 0) (fields_autoplaced)
+  (hierarchical_label "RC6{slash}WHEEL_R" (shape output) (at 182.88 116.84 0) (fields_autoplaced)
     (effects (font (size 1.27 1.27)) (justify left))
   )
@@
       (effects (font (size 1.15 1.15)) (justify left))
     )
-    (property "Value" "Urgency" (at 88.9 163.195 90) (do_not_autoplace)
+    (property "Value" "Stop" (at 88.9 163.195 90) (do_not_autoplace)
       (effects (font (size 1.15 1.15)) (justify left))
     )
@@
       (effects (font (size 1.15 1.15)))
     )
-    (property "Value" "Wheel Right" (at 223.52 165.1 0) (do_not_autoplace)
+    (property "Value" "Wheel Left" (at 223.52 165.1 0) (do_not_autoplace)
       (effects (font (size 1.15 1.15)))
     )
@@
       (effects (font (size 1.15 1.15)) (justify left))
     )
-    (property "Value" "Urgency" (at 67.31 152.4 90) (do_not_autoplace)
+    (property "Value" "Stop" (at 67.31 152.4 90) (do_not_autoplace)
       (effects (font (size 1.15 1.15)) (justify left))
     )
@@
       (effects (font (size 1.15 1.15)))
     )
-    (property "Value" "Servo Left" (at 157.48 119.38 0) (do_not_autoplace)
+    (property "Value" "Servo Right" (at 157.48 119.38 0) (do_not_autoplace)
       (effects (font (size 1.15 1.15)))
     )
@@
       (effects (font (size 1.15 1.15)))
     )
-    (property "Value" "Wheel Left" (at 162.56 165.1 0) (do_not_autoplace)
+    (property "Value" "Wheel Right" (at 162.56 165.1 0) (do_not_autoplace)
       (effects (font (size 1.15 1.15)))
     )
@@
       (effects (font (size 1.15 1.15)))
     )
-    (property "Value" "Servo Right" (at 218.44 119.38 0) (do_not_autoplace)
-      (effects (font (size 1.15 1.15)))
-    )
+    (property "Value" "Servo Left" (at 218.44 119.38 0) (do_not_autoplace)
+      (effects (font (size 1.15 1.15)))
+    )
