File: Kicad/mcu8/tbot-8bit.kicad_sch (KiCad schematic)
At the start: 22 parts, among them IC101 TLV1117-50, K101 Battery, T101 DMP2305U, T102 DMP2305U

Commit message: Draft
Other:
- note added: "DRAFT"
Changed lines of the file:
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@@
     (effects (font (size 1.27 1.27)) (justify left bottom))
+  )
+  (text "DRAFT" (at 210.82 187.96 0)
+    (effects (font (size 5 5)) (justify left bottom))
   )
   (global_label "RB3{slash}BATTERY_SENSE" (shape output) (at 198.12 53.34 0) (fields_autoplaced)

Commit message: Update
Parts:
- removed IC101: TLV1117-50, tronixio:SOT-223-3, symbol tronixio:TLV1117-50-SOT
- removed T101, T102: DMP2305U, tronixio:SOT-23-3, symbol tronixio:DMP2305U-NEW
- added IC101: TI-TLV1117-50-SOT, tronixio:SOT-223-3, symbol tronixio:TI-TLV1117-50-SOT
- added Q101, Q102: DIODESINC-DMP2305U-SOT-23, tronixio:SOT-23-3, symbol tronixio:DIODESINC-DMP2305U-SOT-23
- LED101: MOUSER 604-APT3216LSECKJ3RV -> (none); Mouser (none) -> 604-APTR3216-VFX
- S101: MOUSER 612-200USP1T1A1M2RE -> (none); Mouser (none) -> 612-200USP1T1A1M2RE
- TP101, TP102: MOUSER 534-5006 -> (none); Mouser (none) -> 534-5006
Connections:
- net +5V: now also IC101.2 (VO)
- net GND: now also IC101.1 (GND), Q101.1 (G)
- net VBAT: now also Q101.3 (D)
- net VIN: now also IC101.3 (VI), Q102.3 (D)
- net at R101.1, S101.3: now also Q102.1 (G)
- net at R101.2: now also Q101.2 (S), Q102.2 (S)

Commit message: Update MCU
Parts:
- added TP103: (no value), symbol tronixio:KEYSTONE-2000-3
- added TP104: KEYSTONE-2000-3, tronixio:KEYSTONE-2000-3, symbol tronixio:KEYSTONE-2000-3
- TP101: value GND -> (none); footprint tronixio:KEYSTONE-5006 -> (none); Name (none) -> GND
- TP102: value GND -> KEYSTONE-5006; Name (none) -> GND
Connections:
- net GND: now also TP103.1, TP104.1

Commit message: Update MCU 8Bit
Parts:
- TP101: value (none) -> KEYSTONE-5006; footprint (none) -> tronixio:KEYSTONE-5006
- TP103: value (none) -> KEYSTONE-2000-3; footprint (none) -> tronixio:KEYSTONE-2000-3
Changed lines of the file:
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@@
       (effects (font (size 1.15 1.15)))
     )
-    (property "Value" "" (id 1) (at 185.42 93.98 0)
-      (effects (font (size 1 1)) hide)
-    )
-    (property "Footprint" "" (id 2) (at 185.42 96.52 0)
+    (property "Value" "KEYSTONE-5006" (id 1) (at 185.42 93.98 0)
+      (effects (font (size 1 1)) hide)
+    )
+    (property "Footprint" "tronixio:KEYSTONE-5006" (id 2) (at 185.42 96.52 0)
       (effects (font (size 1 1)) hide)
     )
@@
       (effects (font (size 1.15 1.15)))
     )
-    (property "Value" "" (id 1) (at 210.82 93.98 0)
-      (effects (font (size 1 1)) hide)
-    )
-    (property "Footprint" "" (id 2) (at 210.82 96.52 0)
+    (property "Value" "KEYSTONE-2000-3" (id 1) (at 210.82 93.98 0)
+      (effects (font (size 1 1)) hide)
+    )
+    (property "Footprint" "tronixio:KEYSTONE-2000-3" (id 2) (at 210.82 96.52 0)
       (effects (font (size 1 1)) hide)
     )
@@
     )
     (path "/56bd3a46-de12-45e9-9566-afec966f2cad/7f74cc8c-d98d-4d1c-b394-ca438d10566c"
-      (reference "#PWR0401") (unit 1) (value "VIN") (footprint "")
+      (reference "#PWR0310") (unit 1) (value "VIN") (footprint "")
     )
     (path "/56bd3a46-de12-45e9-9566-afec966f2cad/4ffccd63-64c1-441f-bece-4a52caa97dc3"
-      (reference "#PWR0402") (unit 1) (value "GND") (footprint "")
+      (reference "#PWR0311") (unit 1) (value "GND") (footprint "")
     )
     (path "/56bd3a46-de12-45e9-9566-afec966f2cad/56612b12-cfd0-4162-8edd-fcdfd08004b0"
-      (reference "#PWR0403") (unit 1) (value "+5V") (footprint "")
+      (reference "#PWR0312") (unit 1) (value "+5V") (footprint "")
     )
     (path "/56bd3a46-de12-45e9-9566-afec966f2cad/1c793905-c3b5-40c6-a0ca-f8237e39b201"
-      (reference "#PWR0404") (unit 1) (value "GND") (footprint "")
+      (reference "#PWR0313") (unit 1) (value "GND") (footprint "")
     )
     (path "/56bd3a46-de12-45e9-9566-afec966f2cad/aa6fe2b2-35a3-410c-a1bb-d5d9a757a6bd"
-      (reference "#PWR0405") (unit 1) (value "+5V") (footprint "")
+      (reference "#PWR0314") (unit 1) (value "+5V") (footprint "")
     )
     (path "/56bd3a46-de12-45e9-9566-afec966f2cad/0f1e4c52-dfc5-4752-b9e4-dec04ba8f789"
-      (reference "#PWR0406") (unit 1) (value "GND") (footprint "")
+      (reference "#PWR0315") (unit 1) (value "GND") (footprint "")
     )
     (path "/56bd3a46-de12-45e9-9566-afec966f2cad/5a4532cd-366c-4478-bae4-a35849616abd"
-      (reference "#PWR0407") (unit 1) (value "VIN") (footprint "")
+      (reference "#PWR0316") (unit 1) (value "VIN") (footprint "")
     )
     (path "/56bd3a46-de12-45e9-9566-afec966f2cad/c9e0aa2f-e0a9-4fcf-8e34-8c75bafefb7f"
-      (reference "#PWR0408") (unit 1) (value "GND") (footprint "")
+      (reference "#PWR0317") (unit 1) (value "GND") (footprint "")
     )
     (path "/56bd3a46-de12-45e9-9566-afec966f2cad/4adcb713-d035-4ed8-a1ef-73977ed6de6b"
-      (reference "#PWR0409") (unit 1) (value "+5V") (footprint "")
+      (reference "#PWR0318") (unit 1) (value "+5V") (footprint "")
     )
     (path "/56bd3a46-de12-45e9-9566-afec966f2cad/d68518dc-1950-4d6f-b70c-e45316ed0051"
-      (reference "#PWR0410") (unit 1) (value "GND") (footprint "")
+      (reference "#PWR0319") (unit 1) (value "GND") (footprint "")
     )
     (path "/56bd3a46-de12-45e9-9566-afec966f2cad/a58db860-0ea0-4352-a741-c8f0b1759a82"
-      (reference "#PWR0411") (unit 1) (value "GND") (footprint "")
+      (reference "#PWR0320") (unit 1) (value "GND") (footprint "")
     )
     (path "/56bd3a46-de12-45e9-9566-afec966f2cad/3c53d3a6-37b0-4380-9499-be04785608e6"
-      (reference "#PWR0412") (unit 1) (value "VIN") (footprint "")
+      (reference "#PWR0321") (unit 1) (value "VIN") (footprint "")
     )
     (path "/56bd3a46-de12-45e9-9566-afec966f2cad/ce535f19-3b21-4d52-a3aa-bcb99b1f0776"
-      (reference "#PWR0413") (unit 1) (value "GND") (footprint "")
+      (reference "#PWR0322") (unit 1) (value "GND") (footprint "")
     )
     (path "/56bd3a46-de12-45e9-9566-afec966f2cad/cbe38fcb-5c89-4d31-a3ea-3be731e1664c"
-      (reference "#PWR0414") (unit 1) (value "GND") (footprint "")
+      (reference "#PWR0323") (unit 1) (value "GND") (footprint "")
+    )
+    (path "/56bd3a46-de12-45e9-9566-afec966f2cad/5013d14b-1e51-4f6e-907a-830fb235ee75"
+      (reference "#PWR0324") (unit 1) (value "+5V") (footprint "")
+    )
+    (path "/56bd3a46-de12-45e9-9566-afec966f2cad/0391f20c-9bc4-4807-bad5-071c6a07ca06"
+      (reference "#PWR0325") (unit 1) (value "GND") (footprint "")
     )
     (path "/56bd3a46-de12-45e9-9566-afec966f2cad/87f54b42-ff89-4e77-8e8f-79828f981a45"
-      (reference "#PWR0415") (unit 1) (value "VIN") (footprint "")
+      (reference "#PWR0326") (unit 1) (value "VIN") (footprint "")
     )
     (path "/56bd3a46-de12-45e9-9566-afec966f2cad/7fa60b87-d739-4e3a-9437-956fe2ce40ae"
-      (reference "#PWR0416") (unit 1) (value "GND") (footprint "")
+      (reference "#PWR0327") (unit 1) (value "GND") (footprint "")
     )
     (path "/56bd3a46-de12-45e9-9566-afec966f2cad/5c387a9d-428a-46d4-af6f-a25dad1d16a1"
-      (reference "#PWR0418") (unit 1) (value "GND") (footprint "")
+      (reference "#PWR0328") (unit 1) (value "GND") (footprint "")
+    )
+    (path "/56bd3a46-de12-45e9-9566-afec966f2cad/305274da-bf97-4273-8986-5d004f7d7a87"
+      (reference "#PWR0329") (unit 1) (value "POWER-VUSB") (footprint "")
+    )
+    (path "/56bd3a46-de12-45e9-9566-afec966f2cad/291dcf79-34e1-4262-86e0-c05f5b84b2c4"
+      (reference "#PWR0330") (unit 1) (value "GND") (footprint "")
     )
     (path "/56bd3a46-de12-45e9-9566-afec966f2cad/41648478-6ecf-4708-9686-e8866fc24cd7"
-      (reference "#PWR0419") (unit 1) (value "POWER-VUSB") (footprint "")
+      (reference "#PWR0331") (unit 1) (value "POWER-VUSB") (footprint "")
     )
     (path "/56bd3a46-de12-45e9-9566-afec966f2cad/8fbe7bcb-9e69-4e21-8858-431f6b776c22"
-      (reference "#PWR0420") (unit 1) (value "GND") (footprint "")
-    )
-    (path "/56bd3a46-de12-45e9-9566-afec966f2cad/305274da-bf97-4273-8986-5d004f7d7a87"
-      (reference "#PWR0421") (unit 1) (value "POWER-VUSB") (footprint "")
-    )
-    (path "/56bd3a46-de12-45e9-9566-afec966f2cad/291dcf79-34e1-4262-86e0-c05f5b84b2c4"
-      (reference "#PWR0422") (unit 1) (value "GND") (footprint "")
+      (reference "#PWR0332") (unit 1) (value "GND") (footprint "")
     )
     (path "/56bd3a46-de12-45e9-9566-afec966f2cad/39eadf9b-edac-4afa-b275-77672432774b"
-      (reference "#PWR0423") (unit 1) (value "GND") (footprint "")
+      (reference "#PWR0333") (unit 1) (value "GND") (footprint "")
     )
     (path "/56bd3a46-de12-45e9-9566-afec966f2cad/3cd7e818-7266-42a0-a62f-bfabbf78a737"
-      (reference "#PWR0424") (unit 1) (value "GND") (footprint "")
+      (reference "#PWR0334") (unit 1) (value "GND") (footprint "")
+    )
+    (path "/56bd3a46-de12-45e9-9566-afec966f2cad/4f55efef-fff7-4b43-805a-bfd45e5032a5"
+      (reference "#PWR0335") (unit 1) (value "+5V") (footprint "")
+    )
+    (path "/56bd3a46-de12-45e9-9566-afec966f2cad/9f952a8a-62cc-4f22-a3ce-6bbca9514026"
+      (reference "#PWR0336") (unit 1) (value "GND") (footprint "")
     )
     (path "/56bd3a46-de12-45e9-9566-afec966f2cad/851b9daf-6fe7-4b1d-b7a9-663d7baaa29f"
-      (reference "#PWR0425") (unit 1) (value "VIN") (footprint "")
+      (reference "#PWR0337") (unit 1) (value "VIN") (footprint "")
     )
     (path "/56bd3a46-de12-45e9-9566-afec966f2cad/21bf025b-fb26-4642-b14b-be3966d08117"
-      (reference "#PWR0426") (unit 1) (value "GND") (footprint "")
+      (reference "#PWR0338") (unit 1) (value "GND") (footprint "")
     )
     (path "/56bd3a46-de12-45e9-9566-afec966f2cad/ac9cf4b1-6a77-4564-a3b6-2b4125331e2f"
-      (reference "#PWR0427") (unit 1) (value "POWER-VUSB") (footprint "")
+      (reference "#PWR0339") (unit 1) (value "POWER-VUSB") (footprint "")
     )
     (path "/56bd3a46-de12-45e9-9566-afec966f2cad/1be6d15f-b39a-4723-a701-0efea71535be"
-      (reference "#PWR0428") (unit 1) (value "POWER-VUSB") (footprint "")
+      (reference "#PWR0340") (unit 1) (value "POWER-VUSB") (footprint "")
     )
     (path "/56bd3a46-de12-45e9-9566-afec966f2cad/a672eb27-6221-4b4f-89ad-f7de60019e3a"
@@
       (reference "K306") (unit 1) (value "SERVO LEFT") (footprint "tronixio:HARWIN-M20-999044x")
     )
+    (path "/56bd3a46-de12-45e9-9566-afec966f2cad/8a09b613-7dea-4056-bb42-f02f79a8fbaf"
+      (reference "K307") (unit 1) (value "WHEEL LEFT") (footprint "tronixio:zzMOLEX-532530370")
+    )
     (path "/56bd3a46-de12-45e9-9566-afec966f2cad/1c7c49d9-8392-47f1-a07e-69a84e5dbe16"
-      (reference "K307") (unit 1) (value "USB/UART") (footprint "tronixio:FCI-USB-TYPE-B-MICRO-THT")
+      (reference "K308") (unit 1) (value "USB/UART") (footprint "tronixio:FCI-USB-TYPE-B-MICRO-THT")
     )
     (path "/56bd3a46-de12-45e9-9566-afec966f2cad/cae72a7c-5124-4b85-8f23-c2978460934d"
-      (reference "K308") (unit 1) (value "SERVO RIGHT") (footprint "tronixio:HARWIN-M20-999044x")
+      (reference "K309") (unit 1) (value "SERVO RIGHT") (footprint "tronixio:HARWIN-M20-999044x")
+    )
+    (path "/56bd3a46-de12-45e9-9566-afec966f2cad/1f59f9e5-7d85-42f5-93d4-47ba7dd44dcf"
+      (reference "K310") (unit 1) (value "WHEEL RIGHT") (footprint "tronixio:zzMOLEX-532530370")
     )
     (path "/a338f5b0-e66a-4e8e-b0aa-89183cbfedd8"

Commit message: Update
Other:
- sheet HID ports: added RB0/URGENCY; removed RB0/EMERGENCY
- sheet MCU ports: added RB0/URGENCY; removed RB0/EMERGENCY
Changed lines of the file:
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@@
       (effects (font (size 1.2 1.2)) (justify left))
     )
-    (pin "RB0{slash}EMERGENCY" bidirectional (at 111.76 157.48 180)
+    (pin "RB0{slash}URGENCY" bidirectional (at 111.76 157.48 180)
       (effects (font (size 1.27 1.27)) (justify left))
     )
@@
       (effects (font (size 1.27 1.27)) (justify right))
     )
-    (pin "RB0{slash}EMERGENCY" bidirectional (at 96.52 157.48 0)
+    (pin "RB0{slash}URGENCY" bidirectional (at 96.52 157.48 0)
       (effects (font (size 1.27 1.27)) (justify right))
     )
@@
       (reference "S201") (unit 1) (value "Reset") (footprint "tronixio:ALPS-SKRPAC")
     )
-    (path "/56bd3a46-de12-45e9-9566-afec966f2cad/4295f41d-b93c-4373-93e1-239484151cd9"
-      (reference "S301") (unit 1) (value "EMERGENCY") (footprint "tronixio:E-SWITCH-TL1240XQ1JXXX")
-    )
-    (path "/56bd3a46-de12-45e9-9566-afec966f2cad/e1af4d5e-267e-461a-b356-8583444587aa"
-      (reference "S301") (unit 2) (value "EMERGENCY") (footprint "tronixio:E-SWITCH-TL1240XQ1JXXX")
+    (path "/56bd3a46-de12-45e9-9566-afec966f2cad/08a782ca-74fd-406c-b0d6-36f65802d2f1"
+      (reference "S301") (unit 1) (value "URGENCY") (footprint "tronixio:zzzOMRON-B3W9000-X1")
+    )
+    (path "/56bd3a46-de12-45e9-9566-afec966f2cad/79bc4ded-5d45-4f04-8d3c-0fbfba5f8e42"
+      (reference "S301") (unit 2) (value "URGENCY") (footprint "tronixio:zzzOMRON-B3W9000-X1")
     )
     (path "/136a714c-88c0-45ed-96e3-6e25520a1306"

Commit message: Update
Connections:
- net RB3/BATTERY_SENSE renamed RB2/BATTERY_SENSE
Other:
- sheet HID ports: added RB3/WHEEL_L_EN, RC7/WHEEL_R_EN; removed none
- sheet MCU ports: added RB2/BATTERY_SENSE, RB3/WHEEL_L_EN, RC7/WHEEL_R_EN; removed RB3/BATTERY_SENSE
- moved on the sheet: C101, C102, C103, C104, IC101, K101, LED101, Q101, Q102, R101, R102, R103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

Commit message: Update
Changed lines of the file:
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@@
       (effects (font (size 1.2 1.2)) (justify left))
     )
-    (pin "RC0" bidirectional (at 106.68 172.72 180)
-      (effects (font (size 1.27 1.27)) (justify left))
-    )
-    (pin "RC2" bidirectional (at 106.68 177.8 180)
-      (effects (font (size 1.27 1.27)) (justify left))
-    )
-    (pin "RC1" bidirectional (at 106.68 175.26 180)
-      (effects (font (size 1.27 1.27)) (justify left))
-    )
     (pin "RC5{slash}SERVO_R" input (at 106.68 180.34 180)
       (effects (font (size 1.27 1.27)) (justify left))
@@
     )
     (pin "RB6{slash}PGC{slash}UTX" input (at 106.68 165.1 180)
+      (effects (font (size 1.27 1.27)) (justify left))
+    )
+    (pin "RC2" output (at 106.68 177.8 180)
+      (effects (font (size 1.27 1.27)) (justify left))
+    )
+    (pin "RC1" input (at 106.68 175.26 180)
+      (effects (font (size 1.27 1.27)) (justify left))
+    )
+    (pin "RC0" input (at 106.68 172.72 180)
       (effects (font (size 1.27 1.27)) (justify left))
     )
@@
       (effects (font (size 1.27 1.27)) (justify right))
     )
-    (pin "RC2" bidirectional (at 91.44 177.8 0)
-      (effects (font (size 1.27 1.27)) (justify right))
-    )
-    (pin "RC0" bidirectional (at 91.44 172.72 0)
-      (effects (font (size 1.27 1.27)) (justify right))
-    )
     (pin "RA6{slash}LED" output (at 91.44 149.86 0)
       (effects (font (size 1.27 1.27)) (justify right))
     )
-    (pin "RC1" bidirectional (at 91.44 175.26 0)
-      (effects (font (size 1.27 1.27)) (justify right))
-    )
     (pin "RA5" input (at 91.44 147.32 0)
       (effects (font (size 1.27 1.27)) (justify right))
@@
     )
     (pin "RC5{slash}SERVO_R" output (at 91.44 180.34 0)
+      (effects (font (size 1.27 1.27)) (justify right))
+    )
+    (pin "RC0" output (at 91.44 172.72 0)
+      (effects (font (size 1.27 1.27)) (justify right))
+    )
+    (pin "RC1" output (at 91.44 175.26 0)
+      (effects (font (size 1.27 1.27)) (justify right))
+    )
+    (pin "RC2" input (at 91.44 177.8 0)
       (effects (font (size 1.27 1.27)) (justify right))
     )
@@
     )
     (path "/56bd3a46-de12-45e9-9566-afec966f2cad/d9843755-8f95-4acf-8931-751b53ead8bb"
-      (reference "K302") (unit 1) (value "FRONT #2") (footprint "tronixio:MOLEX-532530570")
+      (reference "K302") (unit 1) (value "FRONT #3") (footprint "tronixio:MOLEX-532530570")
     )
     (path "/56bd3a46-de12-45e9-9566-afec966f2cad/8cecd38b-8473-46ef-8222-38986fcde78c"
@@
     )
     (path "/56bd3a46-de12-45e9-9566-afec966f2cad/38a31abc-1aaf-4a2c-9ba8-60d5554770d4"
-      (reference "K305") (unit 1) (value "FRONT #3") (footprint "tronixio:MOLEX-532530570")
+      (reference "K305") (unit 1) (value "FRONT #2") (footprint "tronixio:MOLEX-532530570")
     )
     (path "/56bd3a46-de12-45e9-9566-afec966f2cad/82639bed-d839-40ca-9086-14d46ff3c9a4"
