File: Kicad/mcu8/tbot-8bit.kicad_sch (KiCad schematic)
At the start: 24 parts, among them IC101 TI-TLV1117-50-SOT, K101 Battery, Q101 DIODESINC-DMP2305U-SOT-23, Q102 DIODESINC-DMP2305U-SOT-23

Commit message: Update
Other:
- sheet HID ports: added RC4/WHEEL_R, RC6/WHEEL_L; removed RB4/WHEEL_L, RC6/WHEEL_R
- sheet MCU ports: added RC4/WHEEL_R, RC6/WHEEL_L; removed RB4/WHEEL_L, RC6/WHEEL_R
Changed lines of the file:
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@@
     (stroke (width 0) (type default) (color 0 0 0 0))
+  )
+  (wire (pts (xy 91.44 175.26) (xy 106.68 175.26))
+    (stroke (width 0) (type default) (color 0 0 0 0))
+  )
+  (wire (pts (xy 127 96.52) (xy 127 101.6))
+    (stroke (width 0) (type solid) (color 0 0 0 0))
+  )
+  (wire (pts (xy 93.98 45.72) (xy 101.6 45.72))
+    (stroke (width 0) (type solid) (color 0 0 0 0))
+  )
+  (wire (pts (xy 91.44 144.78) (xy 106.68 144.78))
+    (stroke (width 0) (type default) (color 0 0 0 0))
+  )
+  (wire (pts (xy 218.44 86.36) (xy 218.44 111.76))
+    (stroke (width 0) (type solid) (color 0 0 0 0))
+  )
+  (wire (pts (xy 180.34 53.34) (xy 180.34 57.15))
+    (stroke (width 0) (type solid) (color 0 0 0 0))
+  )
+  (wire (pts (xy 180.34 49.53) (xy 180.34 53.34))
+    (stroke (width 0) (type solid) (color 0 0 0 0))
+  )
+  (wire (pts (xy 187.96 59.69) (xy 187.96 53.34))
+    (stroke (width 0) (type solid) (color 0 0 0 0))
   )
   (wire (pts (xy 91.44 177.8) (xy 106.68 177.8))
     (stroke (width 0) (type default) (color 0 0 0 0))
   )
-  (wire (pts (xy 127 96.52) (xy 127 101.6))
-    (stroke (width 0) (type solid) (color 0 0 0 0))
-  )
-  (wire (pts (xy 93.98 45.72) (xy 101.6 45.72))
-    (stroke (width 0) (type solid) (color 0 0 0 0))
-  )
-  (wire (pts (xy 91.44 144.78) (xy 106.68 144.78))
-    (stroke (width 0) (type default) (color 0 0 0 0))
-  )
-  (wire (pts (xy 218.44 86.36) (xy 218.44 111.76))
-    (stroke (width 0) (type solid) (color 0 0 0 0))
-  )
-  (wire (pts (xy 180.34 53.34) (xy 180.34 57.15))
-    (stroke (width 0) (type solid) (color 0 0 0 0))
-  )
-  (wire (pts (xy 180.34 49.53) (xy 180.34 53.34))
-    (stroke (width 0) (type solid) (color 0 0 0 0))
-  )
-  (wire (pts (xy 187.96 59.69) (xy 187.96 53.34))
-    (stroke (width 0) (type solid) (color 0 0 0 0))
-  )
   (wire (pts (xy 205.74 86.36) (xy 205.74 111.76))
     (stroke (width 0) (type solid) (color 0 0 0 0))
@@
     (stroke (width 0) (type solid) (color 0 0 0 0))
   )
-  (wire (pts (xy 91.44 167.64) (xy 106.68 167.64))
+  (wire (pts (xy 91.44 165.1) (xy 106.68 165.1))
     (stroke (width 0) (type default) (color 0 0 0 0))
   )
@@
     (stroke (width 0) (type default) (color 0 0 0 0))
   )
+  (wire (pts (xy 91.44 160.02) (xy 106.68 160.02))
+    (stroke (width 0) (type default) (color 0 0 0 0))
+  )
+  (wire (pts (xy 106.68 101.6) (xy 106.68 111.76))
+    (stroke (width 0) (type solid) (color 0 0 0 0))
+  )
+  (wire (pts (xy 91.44 172.72) (xy 106.68 172.72))
+    (stroke (width 0) (type default) (color 0 0 0 0))
+  )
   (wire (pts (xy 91.44 162.56) (xy 106.68 162.56))
     (stroke (width 0) (type default) (color 0 0 0 0))
   )
-  (wire (pts (xy 106.68 101.6) (xy 106.68 111.76))
-    (stroke (width 0) (type solid) (color 0 0 0 0))
-  )
-  (wire (pts (xy 91.44 175.26) (xy 106.68 175.26))
-    (stroke (width 0) (type default) (color 0 0 0 0))
-  )
-  (wire (pts (xy 91.44 165.1) (xy 106.68 165.1))
-    (stroke (width 0) (type default) (color 0 0 0 0))
-  )
   (wire (pts (xy 116.84 106.68) (xy 116.84 111.76))
     (stroke (width 0) (type solid) (color 0 0 0 0))
@@
     (stroke (width 0) (type solid) (color 0 0 0 0))
   )
-  (wire (pts (xy 91.44 172.72) (xy 106.68 172.72))
+  (wire (pts (xy 91.44 170.18) (xy 106.68 170.18))
     (stroke (width 0) (type default) (color 0 0 0 0))
   )
   (wire (pts (xy 142.24 45.72) (xy 147.32 45.72))
     (stroke (width 0) (type solid) (color 0 0 0 0))
-  )
-  (wire (pts (xy 91.44 160.02) (xy 106.68 160.02))
-    (stroke (width 0) (type default) (color 0 0 0 0))
   )
   (wire (pts (xy 91.44 147.32) (xy 106.68 147.32))
@@
       (effects (font (size 1.27 1.27)) (justify left))
     )
-    (pin "RC6{slash}WHEEL_R" output (at 106.68 182.88 180)
-      (effects (font (size 1.27 1.27)) (justify left))
-    )
     (pin "RC7{slash}WHEEL_R_EN" input (at 106.68 185.42 180)
       (effects (font (size 1.27 1.27)) (justify left))
@@
       (effects (font (size 1.27 1.27)) (justify left))
     )
-    (pin "RB5{slash}SERVO_L" input (at 106.68 162.56 180)
-      (effects (font (size 1.27 1.27)) (justify left))
-    )
-    (pin "RB4{slash}WHEEL_L" output (at 106.68 160.02 180)
+    (pin "RB5{slash}SERVO_L" input (at 106.68 160.02 180)
       (effects (font (size 1.27 1.27)) (justify left))
     )
@@
       (effects (font (size 1.27 1.27)) (justify left))
     )
-    (pin "RB7{slash}PGD{slash}URX" output (at 106.68 167.64 180)
-      (effects (font (size 1.27 1.27)) (justify left))
-    )
-    (pin "RB6{slash}PGC{slash}UTX" input (at 106.68 165.1 180)
-      (effects (font (size 1.27 1.27)) (justify left))
-    )
-    (pin "RC2" output (at 106.68 177.8 180)
-      (effects (font (size 1.27 1.27)) (justify left))
-    )
-    (pin "RC1" input (at 106.68 175.26 180)
-      (effects (font (size 1.27 1.27)) (justify left))
-    )
-    (pin "RC0" input (at 106.68 172.72 180)
+    (pin "RB7{slash}PGD{slash}URX" output (at 106.68 165.1 180)
+      (effects (font (size 1.27 1.27)) (justify left))
+    )
+    (pin "RB6{slash}PGC{slash}UTX" input (at 106.68 162.56 180)
+      (effects (font (size 1.27 1.27)) (justify left))
+    )
+    (pin "RC2" output (at 106.68 175.26 180)
+      (effects (font (size 1.27 1.27)) (justify left))
+    )
+    (pin "RC1" input (at 106.68 172.72 180)
+      (effects (font (size 1.27 1.27)) (justify left))
+    )
+    (pin "RC0" input (at 106.68 170.18 180)
+      (effects (font (size 1.27 1.27)) (justify left))
+    )
+    (pin "RC6{slash}WHEEL_L" output (at 106.68 182.88 180)
+      (effects (font (size 1.27 1.27)) (justify left))
+    )
+    (pin "RC4{slash}WHEEL_R" output (at 106.68 177.8 180)
       (effects (font (size 1.27 1.27)) (justify left))
     )
@@
       (effects (font (size 1.2 1.2)) (justify left))
     )
-    (pin "RB7{slash}PGD{slash}URX" input (at 91.44 167.64 0)
+    (pin "RB7{slash}PGD{slash}URX" input (at 91.44 165.1 0)
       (effects (font (size 1.27 1.27)) (justify right))
     )
@@
       (effects (font (size 1.27 1.27)) (justify right))
     )
-    (pin "RB5{slash}SERVO_L" output (at 91.44 162.56 0)
-      (effects (font (size 1.27 1.27)) (justify right))
-    )
-    (pin "RB6{slash}PGC{slash}UTX" output (at 91.44 165.1 0)
-      (effects (font (size 1.27 1.27)) (justify right))
-    )
-    (pin "RB4{slash}WHEEL_L" input (at 91.44 160.02 0)
+    (pin "RB5{slash}SERVO_L" output (at 91.44 160.02 0)
+      (effects (font (size 1.27 1.27)) (justify right))
+    )
+    (pin "RB6{slash}PGC{slash}UTX" output (at 91.44 162.56 0)
       (effects (font (size 1.27 1.27)) (justify right))
     )
@@
       (effects (font (size 1.27 1.27)) (justify right))
     )
-    (pin "RC6{slash}WHEEL_R" input (at 91.44 182.88 0)
-      (effects (font (size 1.27 1.27)) (justify right))
-    )
     (pin "RA6{slash}LED" output (at 91.44 149.86 0)
       (effects (font (size 1.27 1.27)) (justify right))
@@
       (effects (font (size 1.27 1.27)) (justify right))
     )
-    (pin "RC0" output (at 91.44 172.72 0)
-      (effects (font (size 1.27 1.27)) (justify right))
-    )
-    (pin "RC1" output (at 91.44 175.26 0)
-      (effects (font (size 1.27 1.27)) (justify right))
-    )
-    (pin "RC2" input (at 91.44 177.8 0)
-      (effects (font (size 1.27 1.27)) (justify right))
-    )
+    (pin "RC0" output (at 91.44 170.18 0)
+      (effects (font (size 1.27 1.27)) (justify right))
+    )
+    (pin "RC1" output (at 91.44 172.72 0)
+      (effects (font (size 1.27 1.27)) (justify right))
+    )
+    (pin "RC2" input (at 91.44 175.26 0)
+      (effects (font (size 1.27 1.27)) (justify right))
+    )
+    (pin "RC6{slash}WHEEL_L" input (at 91.44 182.88 0)
+      (effects (font (size 1.27 1.27)) (justify right))
+    )
+    (pin "RC4{slash}WHEEL_R" input (at 91.44 177.8 0)
+      (effects (font (size 1.27 1.27)) (justify right))
+    )

Commit message: Update
Parts:
- C101, C103: footprint tronixio:CAPACITOR-1206 -> tronixio:CAPACITOR-SMD-1206; symbol tronixio:C-1206 -> tronixio:CAPACITOR-1206-10U; Mouser (none) -> 80-C1206C106M3R; Name (none) -> CAPACITOR-1206-10U; Tolerance (none) -> 20%; Voltage (none) -> 25V
- C102, C104: footprint tronixio:CAPACITOR-1206 -> tronixio:CAPACITOR-SMD-1206; symbol tronixio:C-1206 -> tronixio:CAPACITOR-1206-100N; Mouser (none) -> 80-C1206C104M5R; Name (none) -> CAPACITOR-1206-100N; Tolerance (none) -> 20%; Voltage (none) -> 50V
- H101, H102, H103, H104, H105, H106: footprint tronixio:M3-MASK -> tronixio:MOUNTING-HOLE-3MM-MASK; symbol tronixio:MOUNTING-HOLE-MASK-3MM -> tronixio:MOUNTING-HOLE-3MM-MASK
- K101: MOUSER 538-22-05-7025 -> (none); Mouser (none) -> 538-22-05-7025; Name (none) -> MOLEX-MINI-SPOX-02-RIGHT-ANGLE
- LED101: footprint tronixio:LED-1206 -> tronixio:LED-SMD-1206; symbol tronixio:LED-1206-PURPLE -> tronixio:KINGBRIGHT-LED-1206-PURPLE; Name (none) -> KINGBRIGHT-LED-1206-PURPLE
- Q101, Q102: Name DMP2305U -> DIODESINC-DMP2305U-SOT-23
- R101: footprint tronixio:RESISTOR-1206 -> tronixio:RESISTOR-SMD-1206; symbol tronixio:R-1206 -> tronixio:RESISTOR-1206-1M; Mouser (none) -> 660-RK73B2BTTDD105J; Name (none) -> RESISTOR-1206-1M; Tolerance (none) -> 5%
- R102: footprint tronixio:RESISTOR-1206 -> tronixio:RESISTOR-SMD-1206; symbol tronixio:R-1206 -> tronixio:RESISTOR-1206-4K7; Mouser (none) -> 660-RK73B2BTTDD472J; Name (none) -> RESISTOR-1206-4K7; Tolerance (none) -> 5%
- R103: footprint tronixio:RESISTOR-1206 -> tronixio:RESISTOR-SMD-1206; symbol tronixio:R-1206 -> tronixio:RESISTOR-1206-7K5; Mouser (none) -> 660-RK73B2BTTD752J; Name (none) -> RESISTOR-1206-7K5; Tolerance (none) -> 5%
- R104: footprint tronixio:RESISTOR-1206 -> tronixio:RESISTOR-SMD-1206; symbol tronixio:R-1206 -> tronixio:RESISTOR-1206-10K; Mouser (none) -> 660-RK73B2BTTDD103J; Name (none) -> RESISTOR-1206-10K; Tolerance (none) -> 5%
- S101: Name (none) -> E-SWITCH-200USP1T1A1M2RE
- TP101, TP102: Name GND -> KEYSTONE-5006
- TP103, TP104: Name GND -> KEYSTONE-2000-3
- U101: renamed from IC101; value TI-TLV1117-50-SOT -> TI-TLV1117-50; symbol tronixio:TI-TLV1117-50-SOT -> tronixio:TI-TLV1117-50-SOT-223; Name TLV1117-50 -> TI-TLV1117-33-SOT-223

Commit message: Up
Parts:
- C101, C103: symbol tronixio:CAPACITOR-1206-10U -> tronixio:CAPACITOR-1206-10U-10P-X7R; Mouser 80-C1206C106M3R -> 80-C1206C106K3R; Name CAPACITOR-1206-10U -> (none); Tolerance 20% -> 10%
- C102, C104: symbol tronixio:CAPACITOR-1206-100N -> tronixio:CAPACITOR-1206-100N-10P-X7R; Mouser 80-C1206C104M5R -> 187-CL31B106KAHNFNE; Name CAPACITOR-1206-100N -> (none); Tolerance 20% -> 10%
- H101, H102, H103, H104, H105, H106: value MOUNTING-HOLE-MASK-3MM -> MOUNTING-HOLE-3MM-MASK
- K101: Name MOLEX-MINI-SPOX-02-RIGHT-ANGLE -> (none)
- LED101: Name KINGBRIGHT-LED-1206-PURPLE -> (none)
- Q101, Q102: value DIODESINC-DMP2305U-SOT-23 -> DMP2305U; symbol tronixio:DIODESINC-DMP2305U-SOT-23 -> tronixio:DIODES-DMP2305U-SOT; Name DIODESINC-DMP2305U-SOT-23 -> (none)
- R101: symbol tronixio:RESISTOR-1206-1M -> tronixio:RESISTOR-1206-1M-5P; Name RESISTOR-1206-1M -> (none)
- R102: value 4K7 -> 4k7; symbol tronixio:RESISTOR-1206-4K7 -> tronixio:RESISTOR-1206-4K7-5P; Name RESISTOR-1206-4K7 -> (none)
- R103: value 7K5 -> 7k5; symbol tronixio:RESISTOR-1206-7K5 -> tronixio:RESISTOR-1206-7K5-5P; Name RESISTOR-1206-7K5 -> (none)
- R104: value 10K -> 10k; symbol tronixio:RESISTOR-1206-10K -> tronixio:RESISTOR-1206-10K-5P; Name RESISTOR-1206-10K -> (none)
- S101: value Power -> On/Off; Name E-SWITCH-200USP1T1A1M2RE -> (none)
- TP101, TP102: Name KEYSTONE-5006 -> (none)
- TP103, TP104: Name KEYSTONE-2000-3 -> (none)
- U101: value TI-TLV1117-50 -> TLV1117-50; Name TI-TLV1117-33-SOT-223 -> (none)
Other:
- moved on the sheet: C101, C102, C103, LED101, R102, TP101, TP102, TP103, TP104, U101

Commit message: Up
Parts:
- C101, C103: symbol tronixio:CAPACITOR-1206-10U-10P-X7R -> tronixio:CAPACITOR-1206-10U-25V-5P-X7R; Mouser 80-C1206C106K3R -> 791-1206X106J250CT; Tolerance 10% -> 5%
- C102, C104: symbol tronixio:CAPACITOR-1206-100N-10P-X7R -> tronixio:CAPACITOR-1206-100N-50V-5P-X7R; Mouser 187-CL31B106KAHNFNE -> 80-C1206C104J5R; Tolerance 10% -> 5%
Connections:
- net VBAT renamed +VBAT
- net VIN renamed +VIN
Other:
- sheet HID ports: added RA6/LED_DEBUG; removed RA6/LED
- sheet MCU ports: added RA6/LED_DEBUG; removed RA6/LED
- moved on the sheet: C104, R103, R104

Commit message: Up
Parts:
- removed TP102: KEYSTONE-5006, tronixio:KEYSTONE-5006, symbol tronixio:KEYSTONE-5006
- removed TP104: KEYSTONE-2000-3, tronixio:KEYSTONE-2000-3, symbol tronixio:KEYSTONE-2000-3
- TP101: value KEYSTONE-5006 -> GND
- TP102: renamed from TP103; value KEYSTONE-2000-3 -> GND
Other:
- moved on the sheet: TP102
Changed lines of the file:
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@@
     (stroke (width 0) (type default))
-  )
-  (wire (pts (xy 218.44 91.44) (xy 218.44 111.76))
-    (stroke (width 0) (type solid))
   )
   (wire (pts (xy 180.34 53.34) (xy 180.34 55.88))
@@
   (wire (pts (xy 99.06 177.8) (xy 114.3 177.8))
     (stroke (width 0) (type default))
-  )
-  (wire (pts (xy 205.74 91.44) (xy 205.74 111.76))
-    (stroke (width 0) (type solid))
   )
   (wire (pts (xy 127 63.5) (xy 127 68.58))
@@
       (effects (font (size 1.15 1.15)))
     )
-    (property "Value" "KEYSTONE-5006" (at 180.34 83.82 0) (do_not_autoplace)
+    (property "Value" "GND" (at 180.34 83.82 0) (do_not_autoplace)
       (effects (font (size 1.15 1.15)) hide)
     )
@@
     )
   )
-  (symbol (lib_id "tronixio:POWER-GND") (at 205.74 111.76 0) (unit 1)
-    (in_bom yes) (on_board yes) (dnp no)
-    (property "Reference" "#PWR0121" (at 205.74 118.11 0)
-      (effects (font (size 1 1)) hide)
-    )
-    (property "Value" "POWER-GND" (at 205.74 121.92 0)
-      (effects (font (size 1 1)) hide)
-    )
-    (property "Footprint" "" (at 205.74 111.76 0)
-      (effects (font (size 1 1)) hide)
-    )
-    (property "Datasheet" "" (at 205.74 111.76 0)
-      (effects (font (size 1 1)) hide)
-    )
-    (pin "1")
-    (instances
-      (project "tbot-8bit"
-        (path "/9c91caeb-16bc-4916-868d-9f9002ce0a61"
-          (reference "#PWR0121") (unit 1)
-        )
-      )
-    )
-  )
   (symbol (lib_id "tronixio:POWER-GND") (at 127 68.58 0) (unit 1)
     (in_bom yes) (on_board yes) (dnp no)
@@
     )
   )
-  (symbol (lib_id "tronixio:KEYSTONE-2000-3") (at 205.74 91.44 0) (unit 1)
-    (in_bom yes) (on_board yes) (dnp no)
-    (property "Reference" "TP103" (at 205.74 86.36 0) (do_not_autoplace)
-      (effects (font (size 1.15 1.15)))
-    )
-    (property "Value" "KEYSTONE-2000-3" (at 205.74 86.36 0) (do_not_autoplace)
+  (symbol (lib_id "tronixio:KEYSTONE-2000-3") (at 193.04 91.44 0) (unit 1)
+    (in_bom yes) (on_board yes) (dnp no)
+    (property "Reference" "TP102" (at 193.04 86.36 0) (do_not_autoplace)
+      (effects (font (size 1.15 1.15)))
+    )
+    (property "Value" "GND" (at 193.04 86.36 0) (do_not_autoplace)
       (effects (font (size 1.15 1.15)) hide)
     )
-    (property "Footprint" "tronixio:KEYSTONE-2000-3" (at 205.74 99.06 0) (do_not_autoplace)
-      (effects (font (size 1 1)) hide)
-    )
-    (property "Datasheet" "https://www.keyelco.com/product.cfm/product_id/3037" (at 205.74 101.6 0) (do_not_autoplace)
-      (effects (font (size 1 1)) hide)
-    )
-    (property "Mouser" "534-2000-3" (at 205.74 104.14 0) (do_not_autoplace)
-      (effects (font (size 1 1)) hide)
-    )
-    (pin "1")
-    (instances
-      (project "tbot-8bit"
-        (path "/9c91caeb-16bc-4916-868d-9f9002ce0a61"
-          (reference "TP103") (unit 1)
+    (property "Footprint" "tronixio:KEYSTONE-2000-3" (at 193.04 99.06 0) (do_not_autoplace)
+      (effects (font (size 1 1)) hide)
+    )
+    (property "Datasheet" "https://www.keyelco.com/product.cfm/product_id/3037" (at 193.04 101.6 0) (do_not_autoplace)
+      (effects (font (size 1 1)) hide)
+    )
+    (property "Mouser" "534-2000-3" (at 193.04 104.14 0) (do_not_autoplace)
+      (effects (font (size 1 1)) hide)
+    )
+    (pin "1")
+    (instances
+      (project "tbot-8bit"
+        (path "/9c91caeb-16bc-4916-868d-9f9002ce0a61"
+          (reference "TP102") (unit 1)
         )
       )
@@
         (path "/9c91caeb-16bc-4916-868d-9f9002ce0a61"
           (reference "#PWR0101") (unit 1)
-        )
-      )
-    )
-  )
-  (symbol (lib_id "tronixio:POWER-GND") (at 218.44 111.76 0) (unit 1)
-    (in_bom yes) (on_board yes) (dnp no)
-    (property "Reference" "#PWR0122" (at 218.44 118.11 0)
-      (effects (font (size 1 1)) hide)
-    )
-    (property "Value" "POWER-GND" (at 218.44 121.92 0)
-      (effects (font (size 1 1)) hide)
-    )
-    (property "Footprint" "" (at 218.44 111.76 0)
-      (effects (font (size 1 1)) hide)
-    )
-    (property "Datasheet" "" (at 218.44 111.76 0)
-      (effects (font (size 1 1)) hide)
-    )
-    (pin "1")
-    (instances
-      (project "tbot-8bit"
-        (path "/9c91caeb-16bc-4916-868d-9f9002ce0a61"
-          (reference "#PWR0122") (unit 1)
-        )
-      )
-    )
-  )
-  (symbol (lib_id "tronixio:KEYSTONE-2000-3") (at 218.44 91.44 0) (unit 1)
-    (in_bom yes) (on_board yes) (dnp no)
-    (property "Reference" "TP104" (at 218.44 86.36 0) (do_not_autoplace)
-      (effects (font (size 1.15 1.15)))
-    )
-    (property "Value" "KEYSTONE-2000-3" (at 218.44 86.36 0) (do_not_autoplace)
-      (effects (font (size 1.15 1.15)) hide)
-    )
-    (property "Footprint" "tronixio:KEYSTONE-2000-3" (at 218.44 99.06 0) (do_not_autoplace)
-      (effects (font (size 1 1)) hide)
-    )
-    (property "Datasheet" "https://www.keyelco.com/product.cfm/product_id/3037" (at 218.44 101.6 0) (do_not_autoplace)
-      (effects (font (size 1 1)) hide)
-    )
-    (property "Mouser" "534-2000-3" (at 218.44 104.14 0) (do_not_autoplace)
-      (effects (font (size 1 1)) hide)
-    )
-    (pin "1")
-    (instances
-      (project "tbot-8bit"
-        (path "/9c91caeb-16bc-4916-868d-9f9002ce0a61"
-          (reference "TP104") (unit 1)
         )
       )
@@
         )
       )
-    )
-  )
-  (symbol (lib_id "tronixio:KEYSTONE-5006") (at 193.04 91.44 0) (unit 1)
-    (in_bom yes) (on_board yes) (dnp no)
-    (property "Reference" "TP102" (at 193.04 86.36 0) (do_not_autoplace)
-      (effects (font (size 1.15 1.15)))
-    )
-    (property "Value" "KEYSTONE-5006" (at 193.04 83.82 0) (do_not_autoplace)
-      (effects (font (size 1.15 1.15)) hide)
-    )
-    (property "Footprint" "tronixio:KEYSTONE-5006" (at 193.04 99.06 0) (do_not_autoplace)
-      (effects (font (size 1 1)) hide)
-    )
-    (property "Datasheet" "https://www.keyelco.com/product.cfm/product_id/1315" (at 193.04 101.6 0) (do_not_autoplace)
-      (effects (font (size 1 1)) hide)
-    )
-    (property "Mouser" "534-5006" (at 193.04 104.14 0) (do_not_autoplace)
-      (effects (font (size 1 1)) hide)
-    )
-    (pin "1")
-    (instances
-      (project "tbot-8bit"
-        (path "/9c91caeb-16bc-4916-868d-9f9002ce0a61"
-          (reference "TP102") (unit 1)
-        )
-      )

Commit message: Up
Parts:
- C101, C103: Mouser 791-1206X106J250CT -> 80-C1206C106J3R
Other:
- sheet HID ports: added RB0/STOP, RB3/WHEEL_EN_R, RC4/SERVO_L, RC5/WHEEL_L, RC6/WHEEL_R, RC7/WHEEL_EN_L; removed RB0/URGENCY, RB3/WHEEL_L_EN, RC4/WHEEL_R, RC5/SERVO_R, RC6/WHEEL_L, RC7/WHEEL_R_EN
- sheet MCU ports: added RB0/STOP, RB3/WHEEL_EN_R, RC4/SERVO_L, RC5/WHEEL_L, RC6/WHEEL_R, RC7/WHEEL_EN_L; removed RB0/URGENCY, RB3/WHEEL_L_EN, RC4/WHEEL_R, RC5/SERVO_R, RC6/WHEEL_L, RC7/WHEEL_R_EN
Changed lines of the file:
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@@
       (effects (font (size 1.15 1.15)) (justify left) hide)
     )
-    (property "Mouser" "791-1206X106J250CT" (at 127 124.46 0) (do_not_autoplace)
+    (property "Mouser" "80-C1206C106J3R" (at 127 124.46 0) (do_not_autoplace)
       (effects (font (size 1 1)) hide)
     )
@@
       (effects (font (size 1.15 1.15)) (justify left) hide)
     )
-    (property "Mouser" "791-1206X106J250CT" (at 93.98 124.46 0) (do_not_autoplace)
+    (property "Mouser" "80-C1206C106J3R" (at 93.98 124.46 0) (do_not_autoplace)
       (effects (font (size 1 1)) hide)
     )
@@
       (effects (font (size 1.2 1.2)) (justify left))
     )
-    (pin "RC5{slash}SERVO_R" input (at 114.3 180.34 180)
-      (effects (font (size 1.27 1.27)) (justify left))
-    )
-    (pin "RC7{slash}WHEEL_R_EN" input (at 114.3 185.42 180)
-      (effects (font (size 1.27 1.27)) (justify left))
-    )
-    (pin "RB0{slash}URGENCY" bidirectional (at 114.3 154.94 180)
+    (pin "RC5{slash}WHEEL_L" input (at 114.3 180.34 180)
+      (effects (font (size 1.27 1.27)) (justify left))
+    )
+    (pin "RC7{slash}WHEEL_EN_L" input (at 114.3 185.42 180)
+      (effects (font (size 1.27 1.27)) (justify left))
+    )
+    (pin "RB0{slash}STOP" bidirectional (at 114.3 154.94 180)
       (effects (font (size 1.27 1.27)) (justify left))
     )
@@
       (effects (font (size 1.27 1.27)) (justify left))
     )
-    (pin "RB3{slash}WHEEL_L_EN" input (at 114.3 157.48 180)
+    (pin "RB3{slash}WHEEL_EN_R" input (at 114.3 157.48 180)
       (effects (font (size 1.27 1.27)) (justify left))
     )
@@
       (effects (font (size 1.27 1.27)) (justify left))
     )
-    (pin "RC6{slash}WHEEL_L" output (at 114.3 182.88 180)
-      (effects (font (size 1.27 1.27)) (justify left))
-    )
-    (pin "RC4{slash}WHEEL_R" output (at 114.3 177.8 180)
+    (pin "RC6{slash}WHEEL_R" output (at 114.3 182.88 180)
+      (effects (font (size 1.27 1.27)) (justify left))
+    )
+    (pin "RC4{slash}SERVO_L" output (at 114.3 177.8 180)
       (effects (font (size 1.27 1.27)) (justify left))
     )
@@
       (effects (font (size 1.27 1.27)) (justify right))
     )
-    (pin "RB3{slash}WHEEL_L_EN" output (at 99.06 157.48 0)
+    (pin "RB3{slash}WHEEL_EN_R" output (at 99.06 157.48 0)
       (effects (font (size 1.27 1.27)) (justify right))
     )
@@
       (effects (font (size 1.27 1.27)) (justify right))
     )
-    (pin "RB0{slash}URGENCY" bidirectional (at 99.06 154.94 0)
-      (effects (font (size 1.27 1.27)) (justify right))
-    )
-    (pin "RC7{slash}WHEEL_R_EN" output (at 99.06 185.42 0)
+    (pin "RB0{slash}STOP" bidirectional (at 99.06 154.94 0)
+      (effects (font (size 1.27 1.27)) (justify right))
+    )
+    (pin "RC7{slash}WHEEL_EN_L" output (at 99.06 185.42 0)
       (effects (font (size 1.27 1.27)) (justify right))
     )
@@
       (effects (font (size 1.27 1.27)) (justify left))
     )
-    (pin "RC5{slash}SERVO_R" output (at 99.06 180.34 0)
+    (pin "RC5{slash}WHEEL_L" output (at 99.06 180.34 0)
       (effects (font (size 1.27 1.27)) (justify right))
     )
@@
       (effects (font (size 1.27 1.27)) (justify right))
     )
-    (pin "RC6{slash}WHEEL_L" input (at 99.06 182.88 0)
-      (effects (font (size 1.27 1.27)) (justify right))
-    )
-    (pin "RC4{slash}WHEEL_R" input (at 99.06 177.8 0)
-      (effects (font (size 1.27 1.27)) (justify right))
-    )
+    (pin "RC6{slash}WHEEL_R" input (at 99.06 182.88 0)
+      (effects (font (size 1.27 1.27)) (justify right))
+    )
+    (pin "RC4{slash}SERVO_L" input (at 99.06 177.8 0)
+      (effects (font (size 1.27 1.27)) (justify right))
+    )
