File: Kicad/mcu8/tbot-8bit.kicad_pcb (KiCad board)
At the start: 2 copper layers, 80 x 100 mm, 92 parts, among them IC101 TI-TLV1117-50-SOT, IC201 PIC16F1778, IC301 MICROCHIP-MCP2221A-ISL, K101 Battery, K201 MCU 1, K202 ICSP, K203 MCU 2, K301 FRONT #1, K302 FRONT #2, K303 VIN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

Commit message: Update
Parts:
- removed the kibuzzard-62763D72 at (158.0, 56.9)
- removed the kibuzzard-62763D9F at (144.0, 56.9)
- added kibuzzard-6294682B: G***, kibuzzard-6294682B, F.Cu at (144.0, 56.9)
- added kibuzzard-62946869: G***, kibuzzard-62946869, F.Cu at (158.0, 56.9)
- K302: value FRONT #2 -> FRONT #3
- K305: value FRONT #3 -> FRONT #2
- moved K302 14.0 mm to (150.0, 53.5)
- moved K305 14.0 mm to (136.0, 53.5)
Routing:
- net /HID/RA3: track 62.3 -> 78.1 mm, vias 0 -> 2
- net /HID/RA4: track 62.1 -> 77.5 mm, vias 0 -> 2
- net /HID/RA5: track 61.9 -> 77.0 mm, vias 0 -> 2
- net +5V: track 280.2 -> 294.0 mm, vias 11 -> 12
- net /HID/RC2: track 61.3 -> 66.5 mm
- net /HID/RC1: track 61.6 -> 66.3 mm
- net /HID/RC0: track 61.8 -> 66.1 mm
- net VIN: vias 4 -> 3

Commit message: Update
Connections:
- IC201 pad 15: RC4 -> /HID/RC4/WHEEL_R
- IC201 pad 17: /HID/RC6/WHEEL_R -> /HID/RC6/WHEEL_L
- IC201 pad 25: /HID/RB4/WHEEL_L -> RB4
- K203 pad 12: /HID/RC6/WHEEL_R -> /HID/RC6/WHEEL_L
- K203 pad 14: RC4 -> /HID/RC4/WHEEL_R
- K203 pad 4: /HID/RB4/WHEEL_L -> RB4
- K306 pad 4: /HID/RB4/WHEEL_L -> /HID/RC6/WHEEL_L
- K307 pad 2: /HID/RB4/WHEEL_L -> /HID/RC6/WHEEL_L
- K309 pad 4: /HID/RC6/WHEEL_R -> /HID/RC4/WHEEL_R
- K310 pad 2: /HID/RC6/WHEEL_R -> /HID/RC4/WHEEL_R
Routing:
- net /HID/RC6/WHEEL_L: track 0.00 -> 92.4 mm
- net /HID/RB4/WHEEL_L: track 70.9 -> 0.00 mm
- net /HID/RC6/WHEEL_R: track 68.4 -> 0.00 mm
- net /HID/RC4/WHEEL_R: track 0.00 -> 66.5 mm
- net RC4: track 4.19 -> 0.00 mm
- net RB4: track 0.00 -> 4.19 mm
- net /HID/RC5/SERVO_R: track 32.0 -> 33.4 mm

Commit message: Update
Parts:
- C101, C102, C103, C104, C201, C202, C302, C303: footprint tronixio:CAPACITOR-1206 -> tronixio:CAPACITOR-SMD-1206
- H101, H102, H103, H104, H105, H106: footprint tronixio:M3-MASK -> tronixio:MOUNTING-HOLE-3MM-MASK
- K307, K310: footprint tronixio:zzMOLEX-532530370 -> tronixioZZ:MOLEX-532530370
- LED101, LED301, LED302, LED303: footprint tronixio:LED-1206 -> tronixio:LED-SMD-1206
- Q301, Q302: value DIODESINC-DMP2305U-SOT-23 -> DMP2305U
- R101, R102, R103, R104, R201, R202, R301, R302, R303, R304, R305, R306, R307, R308, R309: footprint tronixio:RESISTOR-1206 -> tronixio:RESISTOR-SMD-1206
- S301: footprint tronixio:zzzOMRON-B3W9000-X1 -> tronixioZZZ:OMRON-B3W9000-X1
- U101: renamed from IC101; value TI-TLV1117-50-SOT -> TI-TLV1117-50
- U201: renamed from IC201; footprint tronixio:DIP-28-W762-SOCKET -> tronixio:DIP-28-W762
- U301: renamed from IC301; value MICROCHIP-MCP2221A-ISL -> MCP2221A; footprint tronixio:SOIC-SL-14 -> tronixio:SOIC-14

Commit message: Up
Parts:
- C301, C304: value 220µ/25V -> 220µ
- H101, H102, H103, H104, H105, H106: value MOUNTING-HOLE-MASK-3MM -> MOUNTING-HOLE-3MM-MASK
- K201: value MCU 1 -> HARWIN-254-M-1X14-VERTICAL
- K203: value MCU 2 -> HARWIN-254-M-1X14-VERTICAL
- K301: value FRONT #1 -> Front #1
- K302: value FRONT #3 -> Front #3
- K305: value FRONT #2 -> Front #2
- K306: value SERVO LEFT -> Servo Left
- K307: value LEFT -> Left; footprint tronixioZZ:MOLEX-532530370 -> tronixio:MOLEX-532530370
- K308: value USB/UART -> USB
- K309: value SERVO RIGHT -> Servo Right
- K310: value RIGHT -> Right; footprint tronixioZZ:MOLEX-532530370 -> tronixio:MOLEX-532530370
- Q101, Q102: value DIODESINC-DMP2305U-SOT-23 -> DMP2305U
- R102, R304, R307, R309: value 4K7 -> 4k7
- R103: value 7K5 -> 7k5
- R104, R201, R306: value 10K -> 10k
- R202: value 1K -> 1k
- S101: value Power -> On/Off
- S301: value URGENCY -> Urgency; footprint tronixioZZZ:OMRON-B3W9000-X1 -> tronixio:OMRON-B3W9000-X1
- U101: value TI-TLV1117-50 -> TLV1117-50
- U201: value PIC16F1778 -> MICROCHIP-PIC16F1778-ISP
- moved kibuzzard-62763E7E 4.24 mm to (176.0, 125.0), turned to 0 degrees
- moved Q302 0.50 mm to (168.0, 88.5)
- moved kibuzzard-62763CDA 0.10 mm to (164.0, 57.0)
- moved kibuzzard-62763CDA 0.10 mm to (136.0, 57.0)
- moved kibuzzard-62763CDA 0.10 mm to (150.0, 57.0)
- moved kibuzzard-62763CDA 0.10 mm to (112.0, 57.0)
- moved kibuzzard-62763D72 0.10 mm to (130.0, 57.0)
- moved kibuzzard-62763D9F 0.10 mm to (116.0, 57.0)
- moved kibuzzard-62763D9F 0.10 mm to (168.0, 57.0)
- moved kibuzzard-6277F9C5 0.10 mm to (122.0, 57.0)
- moved kibuzzard-6294682B 0.10 mm to (144.0, 57.0)
- moved kibuzzard-62946869 0.10 mm to (158.0, 57.0)
Routing:
- net +5V: track 294.0 -> 274.1 mm, vias 12 -> 16
- net GND: track 47.5 -> 46.0 mm, vias 10 -> 11
- net /HID/RB5/SERVO_L: track 34.5 -> 35.6 mm
- net /HID/RC7/WHEEL_R_EN: track 28.3 -> 29.2 mm
- net /HID/RB3/WHEEL_L_EN: track 32.0 -> 32.9 mm
- net /HID/RA6/LED: track 24.9 -> 25.7 mm
- net VIN: track 193.5 -> 194.2 mm

Commit message: Up
Parts:
- added R310: 100Ω, tronixio:RESISTOR-SMD-1206, F.Cu at (112.5, 92.0)
- added R311: 100Ω, tronixio:RESISTOR-SMD-1206, F.Cu at (165.0, 93.5)
- K201: value HARWIN-254-M-1X14-VERTICAL -> MCU #1
- K203: value HARWIN-254-M-1X14-VERTICAL -> MCU #2
- K307: value Left -> Wheel Left
- K308: value USB -> USB/EUSART; footprint tronixio:FCI-USB-TYPE-B-MICRO-THT -> tronixio:USB-TYPE-B-MICRO-TH
- K310: value Right -> Wheel Right
- U201: value MICROCHIP-PIC16F1778-ISP -> PIC16F1778-ISP; footprint tronixio:DIP-28-W762 -> tronixio:DIP-28-W762-SOCKET
- moved TP101 6.00 mm to (176.0, 122.0)
- moved kibuzzard-62763E7E 6.00 mm to (176.0, 119.0)
- moved Q301 0.50 mm to (112.5, 88.0)
Connections:
- net VBAT renamed +VBAT
- net VIN renamed +VIN
- Q301 pad 1: /HID/RB3/WHEEL_L_EN -> Net-(Q301-G)
- Q302 pad 1: /HID/RC7/WHEEL_R_EN -> Net-(Q302-G)
Routing:
- net /HID/RC7/WHEEL_R_EN: track 29.2 -> 24.0 mm
- net Net-(Q302-G): track 0.00 -> 4.03 mm
- net Net-(Q301-G): track 0.00 -> 3.03 mm
- net /HID/RB3/WHEEL_L_EN: track 32.9 -> 30.0 mm
- net +VIN: track 194.2 -> 196.9 mm, vias 3 -> 4
- net /HID/RB6/PGC/UTX: track 87.9 -> 88.9 mm
- net ~{MCLR}: track 26.7 -> 27.6 mm
- net /HID/RC4/WHEEL_R: track 66.2 -> 66.8 mm
- net Net-(Q301-D): track 35.2 -> 34.7 mm
- net +5V: vias 16 -> 18
Other:
- board text added: "USB/EUSART"
- board text added: "W360"
- board text removed: "+5V"
- board text removed: "DATA"
- board text removed: "GND"
- board text removed: "VIN"
- board text removed: "W"

Commit message: Up
Parts:
- removed TP103, TP104: KEYSTONE-2000-3, tronixio:KEYSTONE-2000-3
- removed the kibuzzard-62763E7E at (163.5, 100.5)
- removed the kibuzzard-62763E7E at (163.5, 111.5)
- added R312: 100Ω, tronixio:RESISTOR-SMD-1206, F.Cu at (158.0, 121.5)
- added R313: 100Ω, tronixio:RESISTOR-SMD-1206, F.Cu at (155.0, 121.5)
- added TP201: Debug, tronixio:KEYSTONE-2000-3, F.Cu at (171.5, 106.0)
- TP101: value KEYSTONE-5006 -> GND
- TP102: value KEYSTONE-5006 -> GND; footprint tronixio:KEYSTONE-5006 -> tronixio:KEYSTONE-2000-3
- moved TP101 56.8 mm to (124.5, 146.0), turned to 90 degrees
- moved kibuzzard-62763E7E 56.8 mm to (124.5, 143.0)
- moved TP102 48.9 mm to (93.0, 109.0)
- moved kibuzzard-62763E7E 48.9 mm to (93.0, 106.0)
Connections:
- net /HID/RA6/LED renamed /HID/RA6/LED_DEBUG
- K202 pad 4: /HID/RB7/PGD/URX -> RB7/PGD/URX
- K202 pad 5: /HID/RB6/PGC/UTX -> RB6/PGC/UTX
- K203 pad 1: /HID/RB7/PGD/URX -> RB7/PGD/URX
- K203 pad 2: /HID/RB6/PGC/UTX -> RB6/PGC/UTX
- U201 pad 27: /HID/RB6/PGC/UTX -> RB6/PGC/UTX
- U201 pad 28: /HID/RB7/PGD/URX -> RB7/PGD/URX
- U301 pad 5: /HID/RB6/PGC/UTX -> Net-(U301-URx)
- U301 pad 6: /HID/RB7/PGD/URX -> Net-(U301-UTx)
Routing:
- net /HID/RB6/PGC/UTX: track 88.9 -> 0.00 mm, vias 1 -> 0
- net /HID/RB7/PGD/URX: track 83.6 -> 0.00 mm, vias 2 -> 0
- net RB6/PGC/UTX: track 0.00 -> 75.6 mm, vias 0 -> 1
- net RB7/PGD/URX: track 0.00 -> 69.0 mm, vias 0 -> 2
- net Net-(U301-UTx): track 0.00 -> 12.5 mm
- net Net-(U301-URx): track 0.00 -> 11.8 mm
- net /HID/RA6/LED_DEBUG: track 25.7 -> 35.1 mm

Commit message: Up
Parts:
- removed kibuzzard-6277F94E: G***, kibuzzard-6277F94E
- removed kibuzzard-627FC6B4 (x3): G***, kibuzzard-627FC6B4
- added kibuzzard-6567BC68: G***, kibuzzard-6567BC68, F.Cu at (133.5, 122.0)
- added kibuzzard-6567BC68: G***, kibuzzard-6567BC68, F.Cu at (146.5, 122.0)
- added kibuzzard-6567BC68: G***, kibuzzard-6567BC68, F.Cu at (140.0, 128.5)
- K306: value Servo Left -> Servo Right
- K307: value Wheel Left -> Wheel Right
- K309: value Servo Right -> Servo Left
- K310: value Wheel Right -> Wheel Left
- S301: value Urgency -> Stop
- U201: footprint tronixio:DIP-28-W762-SOCKET -> tronixio:DIP-28-W762
- moved TP102 81.8 mm to (174.5, 116.0)
- moved kibuzzard-62763E7E 79.6 mm to (172.0, 116.0), turned to 90 degrees
- moved R310 8.73 mm to (116.0, 100.0), turned to 90 degrees
- moved R103 2.50 mm to (113.5, 100.0)
- moved R306 1.80 mm to (175.5, 137.5)
- moved R307 1.58 mm to (153.5, 137.5)
- moved R309 1.58 mm to (172.5, 137.5)
- moved C302 1.50 mm to (169.5, 137.5)
- moved C303 1.50 mm to (156.5, 137.5)
- moved U301 1.50 mm to (163.0, 137.5)
- moved Q301 0.50 mm to (112.5, 88.5)
- moved R301 0.50 mm to (152.0, 122.0)
- moved R302 0.50 mm to (149.0, 122.0)
- moved R303 0.50 mm to (131.0, 122.0)
- moved R312 0.50 mm to (158.0, 122.0)
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Connections:
- net /HID/RB0/URGENCY renamed /HID/RB0/STOP
- net /HID/RB3/WHEEL_L_EN renamed /HID/RB3/WHEEL_EN_R
- net /HID/RC4/WHEEL_R renamed /HID/RC4/SERVO_L
- net /HID/RC5/SERVO_R renamed /HID/RC5/WHEEL_L
- net /HID/RC6/WHEEL_L renamed /HID/RC6/WHEEL_R
- net /HID/RC7/WHEEL_R_EN renamed /HID/RC7/WHEEL_EN_L
- net RB4 renamed Net-(K203-Pin_4)
- K203 pad 3: /HID/RB5/SERVO_L -> Net-(K203-Pin_3)
- K203 pad 6: RB2/BATTERY_SENSE -> Net-(K203-Pin_6)
- R305 pad 1: /HID/RB5/SERVO_L -> /HID/RB5/SERVO_R
- U201 pad 23: RB2/BATTERY_SENSE -> Net-(K203-Pin_6)
- U201 pad 26: /HID/RB5/SERVO_L -> Net-(K203-Pin_3)
Routing:
- net /HID/RC6/WHEEL_R: track 93.0 -> 29.2 mm
- net /HID/RC4/SERVO_L: track 66.8 -> 29.2 mm
- net /HID/RB5/SERVO_L: track 35.6 -> 0.00 mm
- net /HID/RC5/WHEEL_L: track 33.7 -> 4.19 mm
- net RB2/BATTERY_SENSE: track 31.8 -> 5.50 mm
- net /HID/RB3/WHEEL_EN_R: track 30.0 -> 4.19 mm
- net /HID/RC7/WHEEL_EN_L: track 24.0 -> 4.19 mm
- net Net-(Q301-G): track 3.03 -> 10.6 mm
- net Net-(LED302-C): track 12.4 -> 7.24 mm
- net Net-(LED303-C): track 12.1 -> 7.24 mm
- net Net-(K309-Pad3): track 4.70 -> 0.00 mm
- net Net-(K203-Pin_3): track 0.00 -> 4.19 mm
- net +VIN: track 196.9 -> 194.4 mm
- net Net-(U301-VUSB): track 10.0 -> 8.16 mm
- net GND: track 46.0 -> 44.5 mm
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